File: HARDWARE/ETH1CVOLT_A/Power_Isolated.kicad_sch (KiCad schematic)
At the start: 0 parts

Commit message: Development
Other:
- sheet UCC25800_1 ports: added none; removed GND_ISO
- sheet UCC25800_2 ports: added none; removed GND_ISO
Changed lines of the file:
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@@
-			)
-		)
-		(pin "GND_ISO" passive
-			(at 110.49 36.83 0)
-			(effects
-				(font
-					(size 1.27 1.27)
-				)
-				(justify right)
 			)
 		)
@@
 			)
 		)
-		(pin "GND_ISO" passive
-			(at 111.76 100.33 0)
-			(effects
-				(font
-					(size 1.27 1.27)
-				)
-				(justify right)
-			)
-		)

Commit message: Development
Other:
- removed sheet UCC25800_1
- removed sheet UCC25800_2
- removed sheet UCC25800_3
- added sheet DC-DC Isolated (DC_DC_Isolated.kicad_sch)
Changed lines of the file:
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@@
 	(paper "A3")
 	(sheet
-		(at 34.29 30.48)
-		(size 76.2 50.8)
+		(at 69.85 85.09)
+		(size 101.6 69.85)
 		(exclude_from_sim no)
 		(in_bom yes)
@@
 			(color 255 229 191 1.0000)
 		)
-		(property "Sheetname" "UCC25800_1"
-			(at 34.29 29.7684 0)
+		(property "Sheetname" "DC-DC Isolated"
+			(at 69.85 84.3784 0)
 			(effects
 				(font
@@
 			)
 		)
-		(property "Sheetfile" "UCC25800.kicad_sch"
-			(at 34.29 81.8646 0)
+		(property "Sheetfile" "DC_DC_Isolated.kicad_sch"
+			(at 69.85 155.5246 0)
 			(effects
 				(font
@@
 			)
 		)
-		(pin "+24V_ISO" passive
-			(at 110.49 44.45 0)
-			(effects
-				(font
-					(size 1.27 1.27)
-				)
-				(justify right)
-			)
-		)
 		(instances
 			(project "ETH1CVOLT_A"
 				(path "/ca79f0b4-91f7-4537-917d-68d425c03ca3/485861e8-c90d-4c19-b473-548e94ff000e/18da2cad-962d-47df-95e7-fd94fee0a7d8/ff9439b0-b623-4d10-a906-fb4e3cb6e044"
-					(page "8")
+					(page "13")
 				)
 			)
@@
 	)
 	(sheet
-		(at 35.56 90.17)
-		(size 76.2 50.8)
-		(exclude_from_sim no)
-		(in_bom yes)
-		(on_board yes)
-		(dnp no)
-		(fields_autoplaced yes)
-		(stroke
-			(width 0.1524)
-			(type solid)
-		)
-		(fill
-			(color 255 229 191 1.0000)
-		)
-		(property "Sheetname" "UCC25800_2"
-			(at 35.56 89.4584 0)
-			(effects
-				(font
-					(size 1.27 1.27)
-				)
-				(justify left bottom)
-			)
-		)
-		(property "Sheetfile" "UCC25800.kicad_sch"
-			(at 35.56 141.5546 0)
-			(effects
-				(font
-					(size 1.27 1.27)
-				)
-				(justify left top)
-			)
-		)
-		(pin "+24V_ISO" passive
-			(at 111.76 113.03 0)
-			(effects
-				(font
-					(size 1.27 1.27)
-				)
-				(justify right)
-			)
-		)
-		(instances
-			(project "ETH1CVOLT_A"
-				(path "/ca79f0b4-91f7-4537-917d-68d425c03ca3/485861e8-c90d-4c19-b473-548e94ff000e/18da2cad-962d-47df-95e7-fd94fee0a7d8/ff9439b0-b623-4d10-a906-fb4e3cb6e044"
-					(page "9")
-				)
-			)
-		)
-	)
-	(sheet
-		(at 132.08 88.9)
+		(at 213.36 85.09)
 		(size 88.9 48.26)
 		(exclude_from_sim no)
@@
 		)
 		(property "Sheetname" "Medium Voltage"
-			(at 132.08 88.1884 0)
+			(at 213.36 84.3784 0)
 			(effects
 				(font
@@
 		)
 		(property "Sheetfile" "Medium_Voltage.kicad_sch"
-			(at 132.08 137.7446 0)
+			(at 213.36 133.9346 0)
 			(effects
 				(font
@@
 	)
 	(sheet
-		(at 132.08 29.21)
+		(at 213.36 25.4)
 		(size 88.9 52.07)
 		(exclude_from_sim no)
@@
 		)
 		(property "Sheetname" "Low Voltage"
-			(at 132.08 28.4984 0)
+			(at 213.36 24.6884 0)
 			(effects
 				(font
@@
 		)
 		(property "Sheetfile" "Low_Voltage.kicad_sch"
-			(at 132.08 81.8646 0)
+			(at 213.36 78.0546 0)
 			(effects
 				(font
@@
 	)
 	(sheet
-		(at 147.32 165.1)
+		(at 228.6 161.29)
 		(size 124.46 66.04)
 		(exclude_from_sim no)
@@
 		)
 		(property "Sheetname" "High Voltage"
-			(at 147.32 164.3884 0)
+			(at 228.6 160.5784 0)
 			(effects
 				(font
@@
 		)
 		(property "Sheetfile" "High_Voltage.kicad_sch"
-			(at 147.32 231.7246 0)
+			(at 228.6 227.9146 0)
 			(effects
 				(font
@@
 				)
 			)
-		)
-	)
-	(sheet
-		(at 35.56 151.13)
-		(size 76.2 50.8)
-		(exclude_from_sim no)
-		(in_bom yes)
-		(on_board yes)
-		(dnp no)
-		(fields_autoplaced yes)
-		(stroke
-			(width 0.1524)
-			(type solid)
-		)
-		(fill
-			(color 255 229 191 1.0000)
-		)
-		(property "Sheetname" "UCC25800_3"
-			(at 35.56 150.4184 0)
-			(effects
-				(font
-					(size 1.27 1.27)
-				)
-				(justify left bottom)
-			)
-		)
-		(property "Sheetfile" "UCC25800.kicad_sch"
-			(at 35.56 202.5146 0)
-			(effects
-				(font
-					(size 1.27 1.27)
-				)
-				(justify left top)
-			)
-		)
-		(instances
-			(project "ETH1CVOLT_A"
-				(path "/ca79f0b4-91f7-4537-917d-68d425c03ca3/485861e8-c90d-4c19-b473-548e94ff000e/18da2cad-962d-47df-95e7-fd94fee0a7d8/ff9439b0-b623-4d10-a906-fb4e3cb6e044"
-					(page "10")
-				)
-			)

Commit message: Development
Changed lines of the file:
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@@
 	(generator_version "9.0")
 	(paper "A3")
+	(polyline
+		(pts
+			(xy 158.75 15.24) (xy 158.75 76.2)
+		)
+		(stroke
+			(width 1)
+			(type dash)
+		)
+	)
+	(polyline
+		(pts
+			(xy 158.75 204.47) (xy 158.75 280.67)
+		)
+		(stroke
+			(width 1)
+			(type dash)
+		)
+	)
 	(sheet
-		(at 69.85 85.09)
-		(size 101.6 69.85)
+		(at 106.68 80.01)
+		(size 101.6 119.38)
 		(exclude_from_sim no)
 		(in_bom yes)
@@
 		)
 		(property "Sheetname" "DC-DC Isolated"
-			(at 69.85 84.3784 0)
+			(at 106.68 79.2984 0)
 			(effects
 				(font
@@
 		)
 		(property "Sheetfile" "DC_DC_Isolated.kicad_sch"
-			(at 69.85 155.5246 0)
+			(at 106.68 199.9746 0)
 			(effects
 				(font
@@
 	)
 	(sheet
-		(at 213.36 85.09)
-		(size 88.9 48.26)
+		(at 217.17 121.92)
+		(size 101.6 35.56)
 		(exclude_from_sim no)
 		(in_bom yes)
@@
 		)
 		(property "Sheetname" "Medium Voltage"
-			(at 213.36 84.3784 0)
+			(at 217.17 121.2084 0)
 			(effects
 				(font
@@
 		)
 		(property "Sheetfile" "Medium_Voltage.kicad_sch"
-			(at 213.36 133.9346 0)
+			(at 217.17 158.0646 0)
 			(effects
 				(font
@@
 	)
 	(sheet
-		(at 213.36 25.4)
-		(size 88.9 52.07)
+		(at 217.17 80.01)
+		(size 101.6 35.56)
 		(exclude_from_sim no)
 		(in_bom yes)
@@
 		)
 		(property "Sheetname" "Low Voltage"
-			(at 213.36 24.6884 0)
+			(at 217.17 79.2984 0)
 			(effects
 				(font
@@
 		)
 		(property "Sheetfile" "Low_Voltage.kicad_sch"
-			(at 213.36 78.0546 0)
+			(at 217.17 116.1546 0)
 			(effects
 				(font
@@
 	)
 	(sheet
-		(at 228.6 161.29)
-		(size 124.46 66.04)
+		(at 217.17 163.83)
+		(size 101.6 35.56)
 		(exclude_from_sim no)
 		(in_bom yes)
@@
 		)
 		(property "Sheetname" "High Voltage"
-			(at 228.6 160.5784 0)
+			(at 217.17 163.1184 0)
 			(effects
 				(font
@@
 		)
 		(property "Sheetfile" "High_Voltage.kicad_sch"
-			(at 228.6 227.9146 0)
+			(at 217.17 199.9746 0)
 			(effects
 				(font
