File: HARDWARE/ETH1CVOLT_A/Output.kicad_sch (KiCad schematic)
At the start: 1 part, among them J6 FCR7350R

Commit message: Development
Parts:
- added D22, D23: 1N4148W, Diode_SMD:D_SOD-123, symbol Diode:1N4148W
- added J10, J5: FCR7350B, ETH1CVOLT_A:S16N-PC, symbol Connector_Generic:Conn_01x01
- added J12: Conn_02x05_Odd_Even, Connector_PinSocket_2.54mm:PinSocket_2x05_P2.54mm_Vertical_SMD, symbol Connector_Generic:Conn_02x05_Odd_Even
- added J9: FCR7350R, ETH1CVOLT_A:S16N-PC, symbol Connector_Generic:Conn_01x01
- added K1, K2: EE2-3NU, Relay_SMD:Relay_DPDT_Kemet_EE2_NU, symbol Relay:EE2-3NU
- added Q4, Q5: MMBT3904, Package_TO_SOT_SMD:SOT-23, symbol Transistor_BJT:MMBT3904
- added R83, R84: 10K, Resistor_SMD:R_0603_1608Metric_Pad0.98x0.95mm_HandSolder, symbol Device:R
- J6: footprint BOOST_LT8365:S16N-PC -> ETH1CVOLT_A:S16N-PC
Connections:
- net at J6.1 (Pin_1): now also K1.5
- new net: J10.1 (Pin_1), K2.8
- new net: D22.2 (A), K1.12, Q4.3 (C)
- new net: J5.1 (Pin_1), K1.8
- new net: Q4.1 (B), R83.2
- new net: Q5.1 (B), R84.2
- new net: D23.2 (A), K2.12, Q5.3 (C)
- new net: J9.1 (Pin_1), K2.5
- new net +3.3V: D22.1 (K), D23.1 (K), K1.1, K2.1
- new net GND: Q4.2 (E), Q5.2 (E)
- new net OUTPUT+: J12.1 (Pin_1), J12.2 (Pin_2), K1.4
- new net OUTPUT-: J12.3 (Pin_3), J12.4 (Pin_4), K1.9
- new net OUTPUT_RL_CTR: R83.1
- new net SENSE+: J12.7 (Pin_7), J12.8 (Pin_8), K2.4
- new net SENSE-: J12.10 (Pin_10), J12.9 (Pin_9), K2.9
- new net SENS_RL_CTR: R84.1
- no-connect marks 0 -> 6
Other:
- note added: "OUTPUT+"
- note added: "OUTPUT-"
- note added: "SENSE+"
- note added: "SENSE-"
- moved on the sheet: J6

Commit message: Development
Other:
- moved on the sheet: D22, D23, J10, J12, J5, J6, J9, K1, K2, Q4, Q5, R83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

Commit message: Development
Parts:
- renumbered D22 to D21, D23 to D22, J12 to J6, J6 to J7, J5 to J8, R83 to R77, R84 to R78

Commit message: Development
Changed lines of the file:
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@@
 	(text "OUTPUT+"
 		(exclude_from_sim no)
-		(at 232.41 111.76 0)
+		(at 227.33 111.76 0)
 		(effects
 			(font
@@
 	(text "SENSE+"
 		(exclude_from_sim no)
-		(at 228.6 177.8 0)
+		(at 227.33 177.8 0)
 		(effects
 			(font
@@
 	(text "OUTPUT-"
 		(exclude_from_sim no)
-		(at 232.41 130.81 0)
+		(at 227.33 130.81 0)
 		(effects
 			(font

Commit message: Development
Parts:
- renumbered Q4 to Q3, Q5 to Q4, R77 to R76, R78 to R77
Changed lines of the file:
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@@
 		(dnp no)
 		(fields_autoplaced yes)
-		(property "Reference" "#PWR0141"
+		(property "Reference" "#PWR0146"
 			(at 175.26 168.91 0)
 			(effects
@@
 			(project "ETH1CVOLT_A"
 				(path "/ca79f0b4-91f7-4537-917d-68d425c03ca3/485861e8-c90d-4c19-b473-548e94ff000e/8417bd5c-73ec-4e98-b7c0-b091fea457ee"
-					(reference "#PWR0141")
+					(reference "#PWR0146")
 					(unit 1)
 				)
@@
 		(dnp no)
 		(fields_autoplaced yes)
-		(property "Reference" "Q4"
+		(property "Reference" "Q3"
 			(at 189.23 106.68 90)
 			(effects
@@
 			(project ""
 				(path "/ca79f0b4-91f7-4537-917d-68d425c03ca3/485861e8-c90d-4c19-b473-548e94ff000e/8417bd5c-73ec-4e98-b7c0-b091fea457ee"
-					(reference "Q4")
+					(reference "Q3")
 					(unit 1)
 				)
@@
 		(dnp no)
 		(fields_autoplaced yes)
-		(property "Reference" "#PWR0146"
+		(property "Reference" "#PWR0151"
 			(at 213.36 102.87 0)
 			(effects
@@
 			(project "ETH1CVOLT_A"
 				(path "/ca79f0b4-91f7-4537-917d-68d425c03ca3/485861e8-c90d-4c19-b473-548e94ff000e/8417bd5c-73ec-4e98-b7c0-b091fea457ee"
-					(reference "#PWR0146")
+					(reference "#PWR0151")
 					(unit 1)
 				)
@@
 		(dnp no)
 		(fields_autoplaced yes)
-		(property "Reference" "Q5"
+		(property "Reference" "Q4"
 			(at 189.23 172.72 90)
 			(effects
@@
 			(project "ETH1CVOLT_A"
 				(path "/ca79f0b4-91f7-4537-917d-68d425c03ca3/485861e8-c90d-4c19-b473-548e94ff000e/8417bd5c-73ec-4e98-b7c0-b091fea457ee"
-					(reference "Q5")
+					(reference "Q4")
 					(unit 1)
 				)
@@
 		(dnp no)
 		(fields_autoplaced yes)
-		(property "Reference" "#PWR0140"
+		(property "Reference" "#PWR0145"
 			(at 175.26 102.87 0)
 			(effects
@@
 			(project "ETH1CVOLT_A"
 				(path "/ca79f0b4-91f7-4537-917d-68d425c03ca3/485861e8-c90d-4c19-b473-548e94ff000e/8417bd5c-73ec-4e98-b7c0-b091fea457ee"
-					(reference "#PWR0140")
+					(reference "#PWR0145")
 					(unit 1)
 				)
@@
 		(dnp no)
 		(fields_autoplaced yes)
-		(property "Reference" "R77"
+		(property "Reference" "R76"
 			(at 191.77 88.8999 0)
 			(effects
@@
 			(project ""
 				(path "/ca79f0b4-91f7-4537-917d-68d425c03ca3/485861e8-c90d-4c19-b473-548e94ff000e/8417bd5c-73ec-4e98-b7c0-b091fea457ee"
-					(reference "R77")
+					(reference "R76")
 					(unit 1)
 				)
@@
 		(dnp no)
 		(fields_autoplaced yes)
-		(property "Reference" "#PWR0147"
+		(property "Reference" "#PWR0152"
 			(at 213.36 168.91 0)
 			(effects
@@
 			(project "ETH1CVOLT_A"
 				(path "/ca79f0b4-91f7-4537-917d-68d425c03ca3/485861e8-c90d-4c19-b473-548e94ff000e/8417bd5c-73ec-4e98-b7c0-b091fea457ee"
-					(reference "#PWR0147")
+					(reference "#PWR0152")
 					(unit 1)
 				)
@@
 		(dnp no)
 		(fields_autoplaced yes)
-		(property "Reference" "R78"
+		(property "Reference" "R77"
 			(at 191.77 154.9399 0)
 			(effects
@@
 			(project "ETH1CVOLT_A"
 				(path "/ca79f0b4-91f7-4537-917d-68d425c03ca3/485861e8-c90d-4c19-b473-548e94ff000e/8417bd5c-73ec-4e98-b7c0-b091fea457ee"
-					(reference "R78")
-					(unit 1)
-				)
+					(reference "R77")
+					(unit 1)
+				)

Commit message: Development
Parts:
- renumbered D21 to D15, D22 to D16, R76 to R60, R77 to R61
Changed lines of the file:
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@@
 		(dnp no)
 		(fields_autoplaced yes)
-		(property "Reference" "#PWR0146"
+		(property "Reference" "#PWR0137"
 			(at 175.26 168.91 0)
 			(effects
@@
 			(project "ETH1CVOLT_A"
 				(path "/ca79f0b4-91f7-4537-917d-68d425c03ca3/485861e8-c90d-4c19-b473-548e94ff000e/8417bd5c-73ec-4e98-b7c0-b091fea457ee"
-					(reference "#PWR0146")
+					(reference "#PWR0137")
 					(unit 1)
 				)
@@
 		(dnp no)
 		(fields_autoplaced yes)
-		(property "Reference" "#PWR0151"
+		(property "Reference" "#PWR0142"
 			(at 213.36 102.87 0)
 			(effects
@@
 			(project "ETH1CVOLT_A"
 				(path "/ca79f0b4-91f7-4537-917d-68d425c03ca3/485861e8-c90d-4c19-b473-548e94ff000e/8417bd5c-73ec-4e98-b7c0-b091fea457ee"
-					(reference "#PWR0151")
+					(reference "#PWR0142")
 					(unit 1)
 				)
@@
 		(dnp no)
 		(fields_autoplaced yes)
-		(property "Reference" "D22"
+		(property "Reference" "D16"
 			(at 207.01 147.32 0)
 			(effects
@@
 			(project "ETH1CVOLT_A"
 				(path "/ca79f0b4-91f7-4537-917d-68d425c03ca3/485861e8-c90d-4c19-b473-548e94ff000e/8417bd5c-73ec-4e98-b7c0-b091fea457ee"
-					(reference "D22")
+					(reference "D16")
 					(unit 1)
 				)
@@
 		(dnp no)
 		(fields_autoplaced yes)
-		(property "Reference" "D21"
+		(property "Reference" "D15"
 			(at 207.01 81.28 0)
 			(effects
@@
 			(project ""
 				(path "/ca79f0b4-91f7-4537-917d-68d425c03ca3/485861e8-c90d-4c19-b473-548e94ff000e/8417bd5c-73ec-4e98-b7c0-b091fea457ee"
-					(reference "D21")
+					(reference "D15")
 					(unit 1)
 				)
@@
 		(dnp no)
 		(fields_autoplaced yes)
-		(property "Reference" "#PWR0145"
+		(property "Reference" "#PWR0136"
 			(at 175.26 102.87 0)
 			(effects
@@
 			(project "ETH1CVOLT_A"
 				(path "/ca79f0b4-91f7-4537-917d-68d425c03ca3/485861e8-c90d-4c19-b473-548e94ff000e/8417bd5c-73ec-4e98-b7c0-b091fea457ee"
-					(reference "#PWR0145")
+					(reference "#PWR0136")
 					(unit 1)
 				)
@@
 		(dnp no)
 		(fields_autoplaced yes)
-		(property "Reference" "R76"
+		(property "Reference" "R60"
 			(at 191.77 88.8999 0)
 			(effects
@@
 			(project ""
 				(path "/ca79f0b4-91f7-4537-917d-68d425c03ca3/485861e8-c90d-4c19-b473-548e94ff000e/8417bd5c-73ec-4e98-b7c0-b091fea457ee"
-					(reference "R76")
+					(reference "R60")
 					(unit 1)
 				)
@@
 		(dnp no)
 		(fields_autoplaced yes)
-		(property "Reference" "#PWR0152"
+		(property "Reference" "#PWR0143"
 			(at 213.36 168.91 0)
 			(effects
@@
 			(project "ETH1CVOLT_A"
 				(path "/ca79f0b4-91f7-4537-917d-68d425c03ca3/485861e8-c90d-4c19-b473-548e94ff000e/8417bd5c-73ec-4e98-b7c0-b091fea457ee"
-					(reference "#PWR0152")
+					(reference "#PWR0143")
 					(unit 1)
 				)
@@
 		(dnp no)
 		(fields_autoplaced yes)
-		(property "Reference" "R77"
+		(property "Reference" "R61"
 			(at 191.77 154.9399 0)
 			(effects
@@
 			(project "ETH1CVOLT_A"
 				(path "/ca79f0b4-91f7-4537-917d-68d425c03ca3/485861e8-c90d-4c19-b473-548e94ff000e/8417bd5c-73ec-4e98-b7c0-b091fea457ee"
-					(reference "R77")
-					(unit 1)
-				)
+					(reference "R61")
+					(unit 1)
+				)

Commit message: Development
Parts:
- removed D16: 1N4148W, Diode_SMD:D_SOD-123, symbol Diode:1N4148W
- removed J10: FCR7350B, ETH1CVOLT_A:S16N-PC, symbol Connector_Generic:Conn_01x01
- removed J9: FCR7350R, ETH1CVOLT_A:S16N-PC, symbol Connector_Generic:Conn_01x01
- removed K2: EE2-3NU, Relay_SMD:Relay_DPDT_Kemet_EE2_NU, symbol Relay:EE2-3NU
- removed Q4: MMBT3904, Package_TO_SOT_SMD:SOT-23, symbol Transistor_BJT:MMBT3904
- removed R61: 10K, Resistor_SMD:R_0603_1608Metric_Pad0.98x0.95mm_HandSolder, symbol Device:R
Connections:
- no-connect marks 6 -> 4
Other:
- note removed: "SENSE+"
- note removed: "SENSE-"
- moved on the sheet: D15, J7, J8, K1, Q3, R60

Commit message: Development
Parts:
- removed J6: Conn_02x05_Odd_Even, Connector_PinSocket_2.54mm:PinSocket_2x05_P2.54mm_Vertical_SMD, symbol Connector_Generic:Conn_02x05_Odd_Even
- removed K1: EE2-3NU, Relay_SMD:Relay_DPDT_Kemet_EE2_NU, symbol Relay:EE2-3NU
- removed Q3: MMBT3904, Package_TO_SOT_SMD:SOT-23, symbol Transistor_BJT:MMBT3904
- removed R60: 10K, Resistor_SMD:R_0603_1608Metric_Pad0.98x0.95mm_HandSolder, symbol Device:R
- added J9: Conn_02x04_Odd_Even, Connector_PinSocket_2.54mm:PinSocket_2x04_P2.54mm_Vertical_SMD, symbol Connector_Generic:Conn_02x04_Odd_Even
- added K2: EE2-5NU, Relay_SMD:Relay_DPDT_Kemet_EE2_NU, symbol Relay:EE2-5NU
- added R72: 340, Resistor_SMD:R_0603_1608Metric_Pad0.98x0.95mm_HandSolder, symbol Device:R
- added U19: TCMT1103, Package_SO:SOP-4_4.4x2.6mm_P1.27mm, symbol Isolator:TCMT1103
Connections:
- net GND: now also U19.2
- net OUTPUT+: now also J9.1 (Pin_1), J9.2 (Pin_2), K2.4
- net OUTPUT-: now also J9.7 (Pin_7), J9.8 (Pin_8), K2.9
- net at D15.2 (A): now also K2.12, U19.4
- net at J7.1 (Pin_1): now also K2.5
- net at J8.1 (Pin_1): now also K2.8
- net +3.3V renamed +5VD_ISO
- net +5VD_ISO: now also K2.1
- new net: R72.2, U19.1
- new net GND_ISO: U19.3
- new net MCU_OUTPUT_RL_CTR: R72.1
- no-connect marks 4 -> 6
Other:
- moved on the sheet: D15, J7, J8
