File: HARDWARE/ETH1CVOLT_A/Output.kicad_sch (KiCad schematic)
At the start: 7 parts, among them J7 FCR7350R, J8 FCR7350B, J9 Conn_02x04_Odd_Even, K2 EE2-5NU, U19 TCMT1103

Commit message: Hardware development
Parts:
- J7: renamed from J9; value Conn_02x04_Odd_Even -> 61030821821
- renumbered D15 to D12, J7 to J6, R72 to R58, U19 to U16
Other:
- moved on the sheet: D12, J6, J7, J8, K2
