File: HARDWARE/ETH1CVOLT_A/DC_DC_Isolated.kicad_sch (KiCad schematic)
At the start: 12 parts, among them U11 THL30-2415WI

Commit message: Development
Parts:
- C63, C68, C76: value 10u/50V -> 10u/100V
- C79: value 4u7/50V -> 4u7/100V
- L3, L4, L9: footprint (none) -> ETH1CVOLT_A:744774022
Changed lines of the file:
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@@
+	(wire
+		(pts
+			(xy 190.5 120.65) (xy 190.5 121.92)
+		)
+		(stroke
+			(width 0)
+			(type default)
+		)
+	)
 	(wire
 		(pts
@@
 			(width 0)
 			(type default)
+		)
+	)
+	(rule_area
+		(polyline
+			(pts
+				(xy 13.97 17.78) (xy 213.36 17.78) (xy 213.36 283.21) (xy 13.97 282.575)
+			)
+			(stroke
+				(width 0)
+				(type dash)
+			)
+			(fill
+				(type none)
+			)
+		)
+	)
+	(rule_area
+		(polyline
+			(pts
+				(xy 220.98 17.78) (xy 220.98 283.21) (xy 298.45 283.21) (xy 298.45 251.46) (xy 406.4 251.46) (xy 406.4 17.78)
+			)
+			(stroke
+				(width 0)
+				(type dash)
+			)
+			(fill
+				(type none)
+			)
+		)
+	)
+	(netclass_flag ""
+		(length 2.54)
+		(shape round)
+		(at 13.97 17.78 0)
+		(effects
+			(font
+				(size 1.27 1.27)
+			)
+			(justify left bottom)
+		)
+		(property "Netclass" "DIR"
+			(at 15.24 15.24 0)
+			(effects
+				(font
+					(size 1.27 1.27)
+				)
+				(justify left)
+			)
+		)
+		(property "Component Class" "DIR"
+			(at -603.25 -134.62 0)
+			(effects
+				(font
+					(size 1.27 1.27)
+					(italic yes)
+				)
+			)
+		)
+	)
+	(netclass_flag ""
+		(length 2.54)
+		(shape round)
+		(at 220.98 17.78 0)
+		(effects
+			(font
+				(size 1.27 1.27)
+			)
+			(justify left bottom)
+		)
+		(property "Netclass" "ISO"
+			(at 222.25 15.24 0)
+			(effects
+				(font
+					(size 1.27 1.27)
+				)
+				(justify left)
+			)
+		)
+		(property "Component Class" "ISO"
+			(at -396.24 -134.62 0)
+			(effects
+				(font
+					(size 1.27 1.27)
+					(italic yes)
+				)
+			)
 		)
 	)
@@
 			)
 		)
-		(property "Footprint" ""
+		(property "Footprint" "ETH1CVOLT_A:744774022"
 			(at 177.8 121.92 0)
 			(effects
@@
 			)
 		)
-		(property "Value" "10u/50V"
+		(property "Value" "10u/100V"
 			(at 238.76 128.2699 0)
 			(effects
@@
 			)
 		)
-		(property "Footprint" ""
+		(property "Footprint" "ETH1CVOLT_A:744774022"
 			(at 119.38 121.92 0)
 			(effects
@@
 			)
 		)
-		(property "Value" "10u/50V"
+		(property "Value" "10u/100V"
 			(at 168.91 128.2699 0)
 			(effects
@@
 			)
 		)
-		(property "Value" "4u7/50V"
+		(property "Value" "4u7/100V"
 			(at 255.27 128.2699 0)
 			(effects
@@
 			)
 		)
-		(property "Value" "10u/50V"
+		(property "Value" "10u/100V"
 			(at 194.31 128.2699 0)
 			(effects
@@
 	)
 	(symbol
+		(lib_id "power:PWR_FLAG")
+		(at 190.5 120.65 0)
+		(unit 1)
+		(exclude_from_sim no)
+		(in_bom yes)
+		(on_board yes)
+		(dnp no)
+		(fields_autoplaced yes)
+		(property "Reference" "#FLG021"
+			(at 190.5 118.745 0)
+			(effects
+				(font
+					(size 1.27 1.27)
+				)
+				(hide yes)
+			)
+		)
+		(property "Value" "PWR_FLAG"
+			(at 190.5 115.57 0)
+			(effects
+				(font
+					(size 1.27 1.27)
+				)
+			)
+		)
+		(property "Footprint" ""
+			(at 190.5 120.65 0)
+			(effects
+				(font
+					(size 1.27 1.27)
+				)
+				(hide yes)
+			)
+		)
+		(property "Datasheet" "~"
+			(at 190.5 120.65 0)
+			(effects
+				(font
+					(size 1.27 1.27)
+				)
+				(hide yes)
+			)
+		)
+		(property "Description" "Special symbol for telling ERC where power comes from"
+			(at 190.5 120.65 0)
+			(effects
+				(font
+					(size 1.27 1.27)
+				)
+				(hide yes)
+			)
+		)
+		(pin "1"
+		)
+		(instances
+			(project ""
+				(path "/ca79f0b4-91f7-4537-917d-68d425c03ca3/485861e8-c90d-4c19-b473-548e94ff000e/18da2cad-962d-47df-95e7-fd94fee0a7d8/ff9439b0-b623-4d10-a906-fb4e3cb6e044/2ca714ab-eaa4-47e2-8e62-bcadfa00e38a"
+					(reference "#FLG021")
+					(unit 1)
+				)
+			)
+		)
+	)
+	(symbol
 		(lib_id "ETH1CVOLT_A:GND_ISO")
 		(at 251.46 133.35 0)
@@
 			)
 		)
-		(property "Footprint" ""
+		(property "Footprint" "ETH1CVOLT_A:744774022"
 			(at 119.38 132.08 0)
 			(effects

Commit message: Hardware development
Parts:
- removed C53: 220u/50V, Capacitor_SMD:CP_Elec_10x14.3, symbol Device:C_Polarized
- renumbered C116 to C63, C115 to C64, C114 to C65, C63 to C66, C68 to C67, C76 to C68, C79 to C69, L3 to L5, L9 to L6, L4 to L7, U11 to U10
Connections:
- net GND: no longer C64.2, C65.2, C66.2, C67.2, L7.2, U10.2 (-Vin)
- new net: C64.2, C65.2, C66.2, C67.2, L7.2, U10.2 (-Vin)
