File: HARDWARE/ETH1CVOLT_A/Ethernet.kicad_sch (KiCad schematic)
At the start: 25 parts, among them J2 RJ45_Wuerth_7499010121A, U3 LAN8742A, Y2 NX5032GA-25

Commit message: Development
Parts:
- Y2: footprint ETH1HMSR-SMS:NX5032GA -> ETH1CVOLT_A:NX5032GA
Changed lines of the file:
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@@
 			)
 		)
-		(property "Footprint" "ETH1HMSR-SMS:NX5032GA"
+		(property "Footprint" "ETH1CVOLT_A:NX5032GA"
 			(at 146.05 176.53 0)
 			(effects

Commit message: Development
Parts:
- renumbered RN2 to RN1, RN3 to RN2, RN4 to RN3
Changed lines of the file:
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@@
 		(on_board yes)
 		(dnp no)
-		(property "Reference" "#PWR046"
+		(property "Reference" "#PWR045"
 			(at 265.43 80.01 0)
 			(effects
@@
 			(project "ETH1HMSR-SMS"
 				(path "/ca79f0b4-91f7-4537-917d-68d425c03ca3/485861e8-c90d-4c19-b473-548e94ff000e/8418af92-873a-4080-ac55-b7f0e108f36d"
-					(reference "#PWR046")
+					(reference "#PWR045")
 					(unit 1)
 				)
@@
 		(dnp no)
 		(fields_autoplaced yes)
-		(property "Reference" "#PWR031"
+		(property "Reference" "#PWR030"
 			(at 146.05 66.04 0)
 			(effects
@@
 			(project "ETH1HMSR-SMS"
 				(path "/ca79f0b4-91f7-4537-917d-68d425c03ca3/485861e8-c90d-4c19-b473-548e94ff000e/8418af92-873a-4080-ac55-b7f0e108f36d"
-					(reference "#PWR031")
+					(reference "#PWR030")
 					(unit 1)
 				)
@@
 		(dnp no)
 		(fields_autoplaced yes)
-		(property "Reference" "#PWR036"
+		(property "Reference" "#PWR035"
 			(at 161.29 217.17 0)
 			(effects
@@
 			(project "ETH1HMSR-SMS"
 				(path "/ca79f0b4-91f7-4537-917d-68d425c03ca3/485861e8-c90d-4c19-b473-548e94ff000e/8418af92-873a-4080-ac55-b7f0e108f36d"
-					(reference "#PWR036")
+					(reference "#PWR035")
 					(unit 1)
 				)
@@
 		(on_board yes)
 		(dnp no)
-		(property "Reference" "#PWR037"
+		(property "Reference" "#PWR036"
 			(at 179.07 177.8 0)
 			(effects
@@
 			(project "ETH1HMSR-SMS"
 				(path "/ca79f0b4-91f7-4537-917d-68d425c03ca3/485861e8-c90d-4c19-b473-548e94ff000e/8418af92-873a-4080-ac55-b7f0e108f36d"
-					(reference "#PWR037")
+					(reference "#PWR036")
 					(unit 1)
 				)
@@
 		(dnp no)
 		(fields_autoplaced yes)
-		(property "Reference" "#PWR039"
+		(property "Reference" "#PWR038"
 			(at 185.42 217.17 0)
 			(effects
@@
 			(project "ETH1HMSR-SMS"
 				(path "/ca79f0b4-91f7-4537-917d-68d425c03ca3/485861e8-c90d-4c19-b473-548e94ff000e/8418af92-873a-4080-ac55-b7f0e108f36d"
-					(reference "#PWR039")
+					(reference "#PWR038")
 					(unit 1)
 				)
@@
 		(on_board yes)
 		(dnp no)
-		(property "Reference" "#PWR045"
+		(property "Reference" "#PWR044"
 			(at 223.52 80.01 0)
 			(effects
@@
 			(project "ETH1HMSR-SMS"
 				(path "/ca79f0b4-91f7-4537-917d-68d425c03ca3/485861e8-c90d-4c19-b473-548e94ff000e/8418af92-873a-4080-ac55-b7f0e108f36d"
-					(reference "#PWR045")
+					(reference "#PWR044")
 					(unit 1)
 				)
@@
 		(on_board yes)
 		(dnp no)
-		(property "Reference" "#PWR034"
+		(property "Reference" "#PWR033"
 			(at 156.21 193.04 0)
 			(effects
@@
 			(project "ETH1HMSR-SMS"
 				(path "/ca79f0b4-91f7-4537-917d-68d425c03ca3/485861e8-c90d-4c19-b473-548e94ff000e/8418af92-873a-4080-ac55-b7f0e108f36d"
-					(reference "#PWR034")
+					(reference "#PWR033")
 					(unit 1)
 				)
@@
 		(dnp no)
 		(fields_autoplaced yes)
-		(property "Reference" "#PWR050"
+		(property "Reference" "#PWR049"
 			(at 312.42 166.37 0)
 			(effects
@@
 			(project "ETH1HMSR-SMS"
 				(path "/ca79f0b4-91f7-4537-917d-68d425c03ca3/485861e8-c90d-4c19-b473-548e94ff000e/8418af92-873a-4080-ac55-b7f0e108f36d"
-					(reference "#PWR050")
+					(reference "#PWR049")
 					(unit 1)
 				)
@@
 		(dnp no)
 		(fields_autoplaced yes)
-		(property "Reference" "RN4"
+		(property "Reference" "RN3"
 			(at 247.015 71.755 0)
 			(effects
@@
 			(project "ETH1HMSR-SMS"
 				(path "/ca79f0b4-91f7-4537-917d-68d425c03ca3/485861e8-c90d-4c19-b473-548e94ff000e/8418af92-873a-4080-ac55-b7f0e108f36d"
-					(reference "RN4")
+					(reference "RN3")
 					(unit 1)
 				)
@@
 		(on_board yes)
 		(dnp no)
-		(property "Reference" "RN2"
+		(property "Reference" "RN1"
 			(at 130.556 133.35 90)
 			(effects
@@
 			(project "ETH1HMSR-SMS"
 				(path "/ca79f0b4-91f7-4537-917d-68d425c03ca3/485861e8-c90d-4c19-b473-548e94ff000e/8418af92-873a-4080-ac55-b7f0e108f36d"
-					(reference "RN2")
+					(reference "RN1")
 					(unit 1)
 				)
@@
 		(on_board yes)
 		(dnp no)
-		(property "Reference" "#PWR032"
+		(property "Reference" "#PWR031"
 			(at 146.05 80.01 0)
 			(effects
@@
 			(project "ETH1HMSR-SMS"
 				(path "/ca79f0b4-91f7-4537-917d-68d425c03ca3/485861e8-c90d-4c19-b473-548e94ff000e/8418af92-873a-4080-ac55-b7f0e108f36d"
-					(reference "#PWR032")
+					(reference "#PWR031")
 					(unit 1)
 				)
@@
 		(dnp no)
 		(fields_autoplaced yes)
-		(property "Reference" "#PWR052"
+		(property "Reference" "#PWR051"
 			(at 337.82 142.24 0)
 			(effects
@@
 			(project "ETH1HMSR-SMS"
 				(path "/ca79f0b4-91f7-4537-917d-68d425c03ca3/485861e8-c90d-4c19-b473-548e94ff000e/8418af92-873a-4080-ac55-b7f0e108f36d"
-					(reference "#PWR052")
+					(reference "#PWR051")
 					(unit 1)
 				)
@@
 		(on_board yes)
 		(dnp no)
-		(property "Reference" "#PWR030"
+		(property "Reference" "#PWR029"
 			(at 134.62 193.04 0)
 			(effects
@@
 			(project "ETH1HMSR-SMS"
 				(path "/ca79f0b4-91f7-4537-917d-68d425c03ca3/485861e8-c90d-4c19-b473-548e94ff000e/8418af92-873a-4080-ac55-b7f0e108f36d"
-					(reference "#PWR030")
+					(reference "#PWR029")
 					(unit 1)
 				)
@@
 		(dnp no)
 		(fields_autoplaced yes)
-		(property "Reference" "#PWR047"
+		(property "Reference" "#PWR046"
 			(at 276.86 66.04 0)
 			(effects
@@
 			(project "ETH1HMSR-SMS"
 				(path "/ca79f0b4-91f7-4537-917d-68d425c03ca3/485861e8-c90d-4c19-b473-548e94ff000e/8418af92-873a-4080-ac55-b7f0e108f36d"
-					(reference "#PWR047")
+					(reference "#PWR046")
 					(unit 1)
 				)
@@
 		(on_board yes)
 		(dnp no)
-		(property "Reference" "#PWR038"
+		(property "Reference" "#PWR037"
 			(at 185.42 80.01 0)
 			(effects
@@
 			(project "ETH1HMSR-SMS"
 				(path "/ca79f0b4-91f7-4537-917d-68d425c03ca3/485861e8-c90d-4c19-b473-548e94ff000e/8418af92-873a-4080-ac55-b7f0e108f36d"
-					(reference "#PWR038")
+					(reference "#PWR037")
 					(unit 1)
 				)
@@
 		(on_board yes)
 		(dnp no)
-		(property "Reference" "#PWR035"
+		(property "Reference" "#PWR034"
 			(at 157.48 80.01 0)
 			(effects
@@
 			(project "ETH1HMSR-SMS"
 				(path "/ca79f0b4-91f7-4537-917d-68d425c03ca3/485861e8-c90d-4c19-b473-548e94ff000e/8418af92-873a-4080-ac55-b7f0e108f36d"
-					(reference "#PWR035")
+					(reference "#PWR034")
 					(unit 1)
 				)
@@
 		(on_board yes)
 		(dnp no)
-		(property "Reference" "#PWR043"
+		(property "Reference" "#PWR042"
 			(at 213.36 144.78 0)
 			(effects
@@
 			(project "ETH1HMSR-SMS"
 				(path "/ca79f0b4-91f7-4537-917d-68d425c03ca3/485861e8-c90d-4c19-b473-548e94ff000e/8418af92-873a-4080-ac55-b7f0e108f36d"
-					(reference "#PWR043")
+					(reference "#PWR042")
 					(unit 1)
 				)
@@
 		(on_board yes)
 		(dnp no)
-		(property "Reference" "#PWR048"
+		(property "Reference" "#PWR047"
 			(at 276.86 165.1 0)
 			(effects
@@
 			(project "ETH1HMSR-SMS"
 				(path "/ca79f0b4-91f7-4537-917d-68d425c03ca3/485861e8-c90d-4c19-b473-548e94ff000e/8418af92-873a-4080-ac55-b7f0e108f36d"
-					(reference "#PWR048")
+					(reference "#PWR047")
 					(unit 1)
 				)
@@
 		(on_board yes)
 		(dnp no)
-		(property "Reference" "#PWR042"
+		(property "Reference" "#PWR041"
 			(at 199.39 168.91 0)
 			(effects
@@
 			(project "ETH1HMSR-SMS"
 				(path "/ca79f0b4-91f7-4537-917d-68d425c03ca3/485861e8-c90d-4c19-b473-548e94ff000e/8418af92-873a-4080-ac55-b7f0e108f36d"
-					(reference "#PWR042")
+					(reference "#PWR041")
 					(unit 1)
 				)
@@
 		(on_board yes)
 		(dnp no)
-		(property "Reference" "#PWR033"
+		(property "Reference" "#PWR032"
 			(at 147.32 111.76 0)
 			(effects
@@
 			(project "ETH1HMSR-SMS"
 				(path "/ca79f0b4-91f7-4537-917d-68d425c03ca3/485861e8-c90d-4c19-b473-548e94ff000e/8418af92-873a-4080-ac55-b7f0e108f36d"
-					(reference "#PWR033")
+					(reference "#PWR032")
 					(unit 1)
 				)
@@
 		(on_board yes)
 		(dnp no)
-		(property "Reference" "#PWR041"
+		(property "Reference" "#PWR040"
 			(at 196.85 80.01 0)
 			(effects
@@
 			(project "ETH1HMSR-SMS"
 				(path "/ca79f0b4-91f7-4537-917d-68d425c03ca3/485861e8-c90d-4c19-b473-548e94ff000e/8418af92-873a-4080-ac55-b7f0e108f36d"
-					(reference "#PWR041")
+					(reference "#PWR040")
 					(unit 1)
 				)
@@
 		(dnp no)
 		(fields_autoplaced yes)
-		(property "Reference" "#PWR049"
+		(property "Reference" "#PWR048"
 			(at 312.42 154.94 0)
 			(effects
@@
 			(project "ETH1HMSR-SMS"
 				(path "/ca79f0b4-91f7-4537-917d-68d425c03ca3/485861e8-c90d-4c19-b473-548e94ff000e/8418af92-873a-4080-ac55-b7f0e108f36d"
-					(reference "#PWR049")
+					(reference "#PWR048")
 					(unit 1)
 				)
@@
 		(on_board yes)
 		(dnp no)
-		(property "Reference" "#PWR044"
+		(property "Reference" "#PWR043"
 			(at 208.28 80.01 0)
 			(effects
@@
 			(project "ETH1HMSR-SMS"
 				(path "/ca79f0b4-91f7-4537-917d-68d425c03ca3/485861e8-c90d-4c19-b473-548e94ff000e/8418af92-873a-4080-ac55-b7f0e108f36d"
-					(reference "#PWR044")
+					(reference "#PWR043")
 					(unit 1)
 				)
@@
 		(on_board yes)
 		(dnp no)
-		(property "Reference" "#PWR040"
+		(property "Reference" "#PWR039"
 			(at 190.5 104.14 0)
 			(effects
@@
 			(project "ETH1HMSR-SMS"
 				(path "/ca79f0b4-91f7-4537-917d-68d425c03ca3/485861e8-c90d-4c19-b473-548e94ff000e/8418af92-873a-4080-ac55-b7f0e108f36d"
-					(reference "#PWR040")
+					(reference "#PWR039")
 					(unit 1)
 				)
@@
 		(dnp no)
 		(fields_autoplaced yes)
-		(property "Reference" "#PWR051"
+		(property "Reference" "#PWR050"
 			(at 337.82 132.08 0)
 			(effects
@@
 			(project "ETH1HMSR-SMS"
 				(path "/ca79f0b4-91f7-4537-917d-68d425c03ca3/485861e8-c90d-4c19-b473-548e94ff000e/8418af92-873a-4080-ac55-b7f0e108f36d"
-					(reference "#PWR051")
+					(reference "#PWR050")
 					(unit 1)
 				)
@@
 		(dnp no)
 		(fields_autoplaced yes)
-		(property "Reference" "RN3"
+		(property "Reference" "RN2"
 			(at 167.64 219.075 0)
 			(effects
@@
 			(project "ETH1HMSR-SMS"
 				(path "/ca79f0b4-91f7-4537-917d-68d425c03ca3/485861e8-c90d-4c19-b473-548e94ff000e/8418af92-873a-4080-ac55-b7f0e108f36d"
-					(reference "RN3")
+					(reference "RN2")
 					(unit 1)
 				)

Commit message: Development
Parts:
- R7: value 1k5 -> 1k4
Changed lines of the file:
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@@
+		)
+	)
+	(rule_area
+		(polyline
+			(pts
+				(xy 13.97 16.51) (xy 406.4 16.51) (xy 406.4 251.46) (xy 298.45 251.46) (xy 298.45 251.46) (xy 298.45 283.21)
+				(xy 13.97 283.21)
+			)
+			(stroke
+				(width 0)
+				(type dash)
+			)
+			(fill
+				(type none)
+			)
+		)
+	)
+	(netclass_flag ""
+		(length 2.54)
+		(shape round)
+		(at 13.97 16.51 0)
+		(effects
+			(font
+				(size 1.27 1.27)
+			)
+			(justify left bottom)
+		)
+		(property "Netclass" "DIR"
+			(at 15.24 13.97 0)
+			(effects
+				(font
+					(size 1.27 1.27)
+				)
+				(justify left)
+			)
+		)
+		(property "Component Class" "DIR"
+			(at -603.25 -135.89 0)
+			(effects
+				(font
+					(size 1.27 1.27)
+					(italic yes)
+				)
+			)
 		)
 	)
@@
 			)
 		)
-		(property "Value" "1k5"
+		(property "Value" "1k4"
 			(at 187.198 220.853 0)
 			(effects

Commit message: Hardware development
Parts:
- RN1: renamed from RN3; value EXB-38V510JV -> R_Pack04; footprint Resistor_SMD:R_Array_Concave_4x0603 -> (none)
- RN2: renamed from RN1; value EXB-V8V330JV -> R_Pack04; footprint Resistor_SMD:R_Array_Concave_4x0603 -> (none)
- RN3: renamed from RN2; value EXB-V8V103JV -> R_Pack04; footprint Resistor_SMD:R_Array_Concave_4x0603 -> (none)
- renumbered C18 to C17, C20 to C18, C21 to C19, C23 to C20, C25 to C21, C26 to C22, C27 to C23, C22 to C24, C24 to C25, C28 to C26, C17 to C27, C19 to C28, R8 to R10, R7 to R11, R10 to R7, R11 to R8
