File: HARDWARE/ETH1CVOLT_A/High_Voltage.kicad_sch (KiCad schematic)
At the start: 56 parts, among them U13 LT8365, U14 LT8365

Commit message: Development
Parts:
- added J8: Conn_02x05_Odd_Even, Connector_PinSocket_2.54mm:PinSocket_2x05_P2.54mm_Vertical_SMD, symbol Connector_Generic:Conn_02x05_Odd_Even
- C100, C101, C102, C103, C104, C105, C106, C107, C112, C113, C98, C99: footprint (none) -> Capacitor_SMD:C_0603_1608Metric_Pad1.08x0.95mm_HandSolder
- L5, L6: footprint BOOST_LT8365:74437324100 -> ETH1CVOLT_A:74437324100
- R51, R52, R53, R54, R55, R56, R57, R58, R59, R60, R61, R62, R63, R64, R65, R66, R67, R68, R69, R70: footprint (none) -> Resistor_SMD:R_0603_1608Metric_Pad0.98x0.95mm_HandSolder
- U13, U14: footprint BOOST_LT8365:05-08-1871_ADI -> ETH1CVOLT_A:05-08-1871_ADI
Connections:
- net +110V_ISO: now also J8.1 (Pin_1), J8.2 (Pin_2)
- net -110V_ISO: now also J8.10 (Pin_10), J8.9 (Pin_9)
- net GND_ISO: now also J8.5 (Pin_5), J8.6 (Pin_6)
- no-connect marks 0 -> 4

Commit message: Development
Parts:
- C102, C103, C106, C107, C112, C113: value 0.1u -> 0.1u/200V; footprint Capacitor_SMD:C_0603_1608Metric_Pad1.08x0.95mm_HandSolder -> Capacitor_SMD:C_1210_3225Metric_Pad1.33x2.70mm_HandSolder
- C108, C109, C110, C111: value 0.22u -> 0.22u/200V; footprint (none) -> Capacitor_SMD:C_1210_3225Metric_Pad1.33x2.70mm_HandSolder
- C114, C115: value 4u7 -> AEF08124R7M400R; footprint (none) -> Capacitor_SMD:CP_Elec_8x11.9
- C116, C117: value 10u -> AEK0812100M250R; footprint (none) -> Capacitor_SMD:CP_Elec_8x11.9
- C94, C95: value 4u7 -> 4u7/50V; footprint (none) -> Capacitor_SMD:C_1210_3225Metric_Pad1.33x2.70mm_HandSolder
- C96, C97: value 10u -> 10u/50V; footprint (none) -> Capacitor_SMD:C_1210_3225Metric_Pad1.33x2.70mm_HandSolder
- D19: value DFLS1150 -> DFLS1200
- R59, R60, R61, R62: value 20 -> 20/200V
- R63, R64: value 47 -> 47/200V
- R65, R66, R68, R69: value 499k -> 499k/100V
Connections:
- net -110V_ISO: now also C115.2, C117.2; no longer C115.1, C117.1
- net GND_ISO: now also C115.1, C117.1; no longer C115.2, C117.2
Other:
- moved on the sheet: C113, C114, C115, C116, C117, C94, C95, C96, C97, R62

Commit message: Development
Parts:
- added D23: 1N4148W, Diode_SMD:D_SOD-123, symbol Diode:1N4148W
- added K3: EE2-3NU, Relay_SMD:Relay_DPDT_Kemet_EE2_NU, symbol Relay:EE2-3NU
- added R85, R86: 4k7/2W, Resistor_SMD:R_2512_6332Metric_Pad1.40x3.35mm_HandSolder, symbol Device:R
- renumbered C94 to C105, C95 to C106, C96 to C107, C97 to C108, C98 to C109, C99 to C110, C100 to C111, C101 to C112, C102 to C113, C103 to C114, C104 to C115, C105 to C116, C106 to C117, C107 to C118, C108 to C119, C109 to C120, C110 to C121, C111 to C122, C112 to C123, C113 to C124, C114 to C125, C115 to C126, C116 to C127, C117 to C128, D14 to D13, D15 to D14, D16 to D15, D17 to D16, D18 to D17, D19 to D18, D20 to D19, D21 to D20, J8 to J11, R51 to R63, R52 to R64, R53 to R65, R54 to R66, R55 to R67, R56 to R68, R57 to R69, R58 to R70, R59 to R71, R60 to R72, R61 to R73, R62 to R74, R63 to R75, R64 to R76, R65 to R79, R66 to R80, R67 to R81, R68 to R82, R69 to R83, R70 to R84, U13 to U16, U14 to U17
Connections:
- net +110V_ISO: now also K3.4
- net -110V_ISO: now also K3.9
- net GND: now also D23.2 (A), K3.12
- net GND_ISO: now also R85.2, R86.2
- new net: K3.3, R85.1
- new net: K3.10, R86.1
- new net +3.3V: D23.1 (K), K3.1
- no-connect marks 4 -> 6
Other:
- note added: "Connector"
- note added: "Discharge"
- moved on the sheet: C105, C106, C107, C108, C109, C110, C111, C112, C113, C114, C115, C116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

Commit message: Development
Parts:
- R85, R86: value 4k7/2W -> 10k/2W
Changed lines of the file:
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@@
 			)
 		)
-		(property "Value" "4k7/2W"
+		(property "Value" "10k/2W"
 			(at 356.87 67.31 90)
 			(effects
@@
 			)
 		)
-		(property "Value" "4k7/2W"
+		(property "Value" "10k/2W"
 			(at 356.87 77.47 90)
 			(effects

Commit message: Development
Parts:
- renumbered C105 to C109, C106 to C110, C107 to C111, C108 to C112, C109 to C113, C110 to C114, C111 to C115, C112 to C116, C113 to C117, C114 to C118, C115 to C119, C116 to C120, C117 to C121, C118 to C122, C119 to C123, C120 to C124, C121 to C125, C122 to C126, C123 to C127, C124 to C128, C125 to C129, C126 to C130, C127 to C131, C128 to C132, L5 to L6, L6 to L7, R63 to R62, R64 to R63, R65 to R64, R66 to R65, R67 to R66, R68 to R67, R69 to R68, R70 to R69, R71 to R70, R72 to R71, R73 to R72, R74 to R73, R75 to R74, R76 to R75, R79 to R78, R80 to R79, R81 to R80, R82 to R81, R83 to R82, R84 to R83, R85 to R84, R86 to R85

Commit message: Development
Parts:
- renumbered C119 to C100, C120 to C101, C121 to C102, C122 to C103, C123 to C104, C124 to C105, C125 to C106, C126 to C107, C127 to C108, C128 to C109, C129 to C110, C130 to C111, C131 to C112, C132 to C113, C109 to C90, C110 to C91, C111 to C92, C112 to C93, C113 to C94, C114 to C95, C115 to C96, C116 to C97, C117 to C98, C118 to C99, D16 to D10, D17 to D11, D18 to D12, D19 to D13, D20 to D14, D23 to D17, D13 to D7, D14 to D8, D15 to D9, L6 to L10, L7 to L11, R62 to R46, R63 to R47, R64 to R48, R65 to R49, R66 to R50, R67 to R51, R68 to R52, R69 to R53, R70 to R54, R71 to R55, R72 to R56, R73 to R57, R74 to R58, R75 to R59, R78 to R62, R79 to R63, R80 to R64, R81 to R65, R82 to R66, R83 to R67, R84 to R68, R85 to R69, U16 to U15, U17 to U16
Connections:
- net +24V_HV_ISO renamed +24V_ISO

Commit message: Development
Parts:
- C90, C91: value 4u7/50V -> 4u7/100V
- C92, C93: value 10u/50V -> 10u/100V
- R62, R63, R65, R66: footprint Resistor_SMD:R_0603_1608Metric_Pad0.98x0.95mm_HandSolder -> Resistor_SMD:R_0805_2012Metric_Pad1.20x1.40mm_HandSolder
Other:
- moved on the sheet: C100, C101, C102, C103, C104, C105, C106, C107, C108, C109, C110, C111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

Commit message: Hardware development
Parts:
- J9: renamed from J11; value Conn_02x05_Odd_Even -> 61031021821
- renumbered C94 to C100, C100 to C101, C96 to C102, C99 to C103, C103 to C104, C91 to C105, C93 to C106, C106 to C107, C111 to C108, C113 to C109, C109 to C110, C107 to C111, C95 to C112, C101 to C113, C97 to C114, C98 to C91, C102 to C92, C90 to C93, C92 to C94, C104 to C95, C110 to C96, C112 to C97, C108 to C98, C105 to C99, D9 to D10, D7 to D11, D14 to D13, D12 to D14, D10 to D15, D8 to D16, D13 to D7, D11 to D8, D17 to D9, K3 to K1, R58 to R46, R55 to R47, R54 to R48, R62 to R49, R68 to R50, R63 to R51, R69 to R52, R46 to R53, R47 to R54, R64 to R55, R52 to R56, R50 to R57, R57 to R59, R59 to R60, R56 to R61, R65 to R62, R66 to R63, R48 to R64, R49 to R65, R53 to R66, R51 to R68, U16 to U17
