File: HARDWARE/ETH1CVOLT_A/Isolation_IO.kicad_sch (KiCad schematic)
At the start: 2 parts, among them U18 ISO7763DW, U19 ISO7763DW

Commit message: Development
Parts:
- removed U19: ISO7763DW, Package_SO:SOIC-16W_7.5x10.3mm_P1.27mm, symbol Isolator:ISO7763DW
- added J13, J4: Conn_02x04_Odd_Even, Connector_PinSocket_2.54mm:PinSocket_2x04_P2.54mm_Vertical_SMD, symbol Connector_Generic:Conn_02x04_Odd_Even
- added U20: ISO7761DW, Package_SO:SOIC-16W_7.5x10.3mm_P1.27mm, symbol Isolator:ISO7761DW
Connections:
- net +3.3V: now reaches U18.1 (Vcc1)
- net +3.3V: now also U20.1 (Vcc1)
- net DAC2_~{FAULT}_ISO: now reaches U18.10 (INF)
- net DAC1_~{FAULT}_ISO: now reaches U18.11 (INE)
- net SPI1_MISO_ISO: now reaches U18.12 (IND)
- net SPI1_~{CS}_ISO: now reaches U18.13 (OUTC)
- net SPI1_MOSI_ISO: now reaches U18.14 (OUTB)
- net SPI1_SCK_ISO: now reaches U18.15 (OUTA)
- net +3V3_ISO: now reaches U18.16 (Vcc2)
- net +3V3_ISO: now also U20.16 (Vcc2)
- net SPI1_SCK: now reaches U18.2 (INA)
- net SPI1_MOSI: now reaches U18.3 (INB)
- net SPI1_~{CS}: now reaches U18.4 (INC)
- net SPI1_MISO: now reaches U18.5 (OUTD)
- net DAC1_~{FAULT}: now reaches U18.6 (OUTE)
- net DAC2_~{FAULT}: now reaches U18.7 (OUTF)
- net GND: now reaches U18.8 (GND1)
- net GND: now also U20.8 (GND1)
- net GND_ISO: now reaches U18.9 (GND2)
- net GND_ISO: now also U20.9 (GND2)
- new net SPI2_MISO: U20.7 (OUTF)
- new net SPI2_SCK: U20.5 (IND)
- new net SPI2_~{CS}: U20.6 (INE)
Other:
- moved on the sheet: U18

Commit message: Development
Parts:
- renumbered J4 to J12, U20 to U19
Changed lines of the file:
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@@
 		(dnp no)
 		(fields_autoplaced yes)
-		(property "Reference" "#PWR0157"
+		(property "Reference" "#PWR0169"
 			(at 209.55 123.19 0)
 			(effects
@@
 			(project ""
 				(path "/ca79f0b4-91f7-4537-917d-68d425c03ca3/485861e8-c90d-4c19-b473-548e94ff000e/62dce88f-62ee-4857-96f3-986f7b276210"
-					(reference "#PWR0157")
+					(reference "#PWR0169")
 					(unit 1)
 				)
@@
 		(on_board yes)
 		(dnp no)
-		(property "Reference" "#PWR0162"
+		(property "Reference" "#PWR0170"
 			(at 209.55 143.51 0)
 			(effects
@@
 			(project "ETH1CVOLT_A"
 				(path "/ca79f0b4-91f7-4537-917d-68d425c03ca3/485861e8-c90d-4c19-b473-548e94ff000e/62dce88f-62ee-4857-96f3-986f7b276210"
-					(reference "#PWR0162")
+					(reference "#PWR0170")
 					(unit 1)
 				)
@@
 		(dnp no)
 		(fields_autoplaced yes)
-		(property "Reference" "#PWR0155"
+		(property "Reference" "#PWR0164"
 			(at 199.39 85.09 0)
 			(effects
@@
 			(project "ETH1CVOLT_A"
 				(path "/ca79f0b4-91f7-4537-917d-68d425c03ca3/485861e8-c90d-4c19-b473-548e94ff000e/62dce88f-62ee-4857-96f3-986f7b276210"
-					(reference "#PWR0155")
+					(reference "#PWR0164")
 					(unit 1)
 				)
@@
 		(dnp no)
 		(fields_autoplaced yes)
-		(property "Reference" "U20"
+		(property "Reference" "U19"
 			(at 211.6933 138.43 0)
 			(effects
@@
 			(project ""
 				(path "/ca79f0b4-91f7-4537-917d-68d425c03ca3/485861e8-c90d-4c19-b473-548e94ff000e/62dce88f-62ee-4857-96f3-986f7b276210"
-					(reference "U20")
+					(reference "U19")
 					(unit 1)
 				)
@@
 		(dnp no)
 		(fields_autoplaced yes)
-		(property "Reference" "#PWR0158"
+		(property "Reference" "#PWR0167"
 			(at 199.39 181.61 0)
 			(effects
@@
 			(project "ETH1CVOLT_A"
 				(path "/ca79f0b4-91f7-4537-917d-68d425c03ca3/485861e8-c90d-4c19-b473-548e94ff000e/62dce88f-62ee-4857-96f3-986f7b276210"
-					(reference "#PWR0158")
+					(reference "#PWR0167")
 					(unit 1)
 				)
@@
 		(dnp no)
 		(fields_autoplaced yes)
-		(property "Reference" "#PWR0161"
+		(property "Reference" "#PWR0166"
 			(at 199.39 143.51 0)
 			(effects
@@
 			(project "ETH1CVOLT_A"
 				(path "/ca79f0b4-91f7-4537-917d-68d425c03ca3/485861e8-c90d-4c19-b473-548e94ff000e/62dce88f-62ee-4857-96f3-986f7b276210"
-					(reference "#PWR0161")
+					(reference "#PWR0166")
 					(unit 1)
 				)
@@
 		(on_board yes)
 		(dnp no)
-		(property "Reference" "#PWR0160"
+		(property "Reference" "#PWR0168"
 			(at 209.55 85.09 0)
 			(effects
@@
 			(project ""
 				(path "/ca79f0b4-91f7-4537-917d-68d425c03ca3/485861e8-c90d-4c19-b473-548e94ff000e/62dce88f-62ee-4857-96f3-986f7b276210"
-					(reference "#PWR0160")
+					(reference "#PWR0168")
 					(unit 1)
 				)
@@
 		(dnp no)
 		(fields_autoplaced yes)
-		(property "Reference" "J4"
+		(property "Reference" "J12"
 			(at 270.51 87.63 0)
 			(effects
@@
 			(project "ETH1CVOLT_A"
 				(path "/ca79f0b4-91f7-4537-917d-68d425c03ca3/485861e8-c90d-4c19-b473-548e94ff000e/62dce88f-62ee-4857-96f3-986f7b276210"
-					(reference "J4")
+					(reference "J12")
 					(unit 1)
 				)
@@
 		(dnp no)
 		(fields_autoplaced yes)
-		(property "Reference" "#PWR0156"
+		(property "Reference" "#PWR0165"
 			(at 199.39 123.19 0)
 			(effects
@@
 			(project ""
 				(path "/ca79f0b4-91f7-4537-917d-68d425c03ca3/485861e8-c90d-4c19-b473-548e94ff000e/62dce88f-62ee-4857-96f3-986f7b276210"
-					(reference "#PWR0156")
+					(reference "#PWR0165")
 					(unit 1)
 				)
@@
 		(dnp no)
 		(fields_autoplaced yes)
-		(property "Reference" "#PWR0159"
+		(property "Reference" "#PWR0171"
 			(at 209.55 181.61 0)
 			(effects
@@
 			(project "ETH1CVOLT_A"
 				(path "/ca79f0b4-91f7-4537-917d-68d425c03ca3/485861e8-c90d-4c19-b473-548e94ff000e/62dce88f-62ee-4857-96f3-986f7b276210"
-					(reference "#PWR0159")
-					(unit 1)
-				)
+					(reference "#PWR0171")
+					(unit 1)
+				)

Commit message: Development
Connections:
- net DAC1_~{FAULT}_ISO: now also J12.2 (Pin_2)
- net DAC2_~{FAULT}_ISO: now also J12.4 (Pin_4)
- net SPI1_MISO_ISO: now also J12.7 (Pin_7)
- net SPI1_MOSI_ISO: now also J12.3 (Pin_3)
- net SPI1_SCK_ISO: now also J12.1 (Pin_1)
- net SPI1_~{CS}_ISO: now also J12.5 (Pin_5)
- net SPI2_MISO_ISO: now reaches U19.10 (INF)
- net SPI2_MISO_ISO: now also J13.5 (Pin_5)
- net SPI2_~{CS}_ISO: now reaches U19.11 (OUTE)
- net SPI2_~{CS}_ISO: now also J13.3 (Pin_3)
- net SPI2_SCK_ISO: now reaches U19.12 (OUTD)
- net SPI2_SCK_ISO: now also J13.1 (Pin_1)
Other:
- moved on the sheet: J12, J13

Commit message: Development
Connections:
- net +3V3_ISO renamed +5VD_ISO

Commit message: Development
Parts:
- renumbered U18 to U17, U19 to U18
Connections:
- net +5VD_ISO renamed +VD_ISO
Changed lines of the file:
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@@
 		(dnp no)
 		(fields_autoplaced yes)
-		(property "Reference" "#PWR0174"
+		(property "Reference" "#PWR0165"
 			(at 209.55 123.19 0)
 			(effects
@@
 			(project ""
 				(path "/ca79f0b4-91f7-4537-917d-68d425c03ca3/485861e8-c90d-4c19-b473-548e94ff000e/62dce88f-62ee-4857-96f3-986f7b276210"
-					(reference "#PWR0174")
-					(unit 1)
-				)
-			)
-		)
-	)
-	(symbol
-		(lib_id "ETH1CVOLT_A:+5VD_ISO")
+					(reference "#PWR0165")
+					(unit 1)
+				)
+			)
+		)
+	)
+	(symbol
+		(lib_id "ETH1CVOLT_A:+VD_ISO")
 		(at 209.55 139.7 0)
 		(unit 1)
@@
 		(dnp no)
 		(fields_autoplaced yes)
-		(property "Reference" "#PWR094"
+		(property "Reference" "#PWR0166"
 			(at 209.55 143.51 0)
 			(effects
@@
 			)
 		)
-		(property "Value" "+5VD_ISO"
+		(property "Value" "+VD_ISO"
 			(at 209.55 134.62 0)
 			(effects
@@
 			(project ""
 				(path "/ca79f0b4-91f7-4537-917d-68d425c03ca3/485861e8-c90d-4c19-b473-548e94ff000e/62dce88f-62ee-4857-96f3-986f7b276210"
-					(reference "#PWR094")
+					(reference "#PWR0166")
 					(unit 1)
 				)
@@
 		(dnp no)
 		(fields_autoplaced yes)
-		(property "Reference" "#PWR0169"
+		(property "Reference" "#PWR0160"
 			(at 199.39 85.09 0)
 			(effects
@@
 			(project "ETH1CVOLT_A"
 				(path "/ca79f0b4-91f7-4537-917d-68d425c03ca3/485861e8-c90d-4c19-b473-548e94ff000e/62dce88f-62ee-4857-96f3-986f7b276210"
-					(reference "#PWR0169")
+					(reference "#PWR0160")
 					(unit 1)
 				)
@@
 		(dnp no)
 		(fields_autoplaced yes)
-		(property "Reference" "U19"
+		(property "Reference" "U18"
 			(at 211.6933 138.43 0)
 			(effects
@@
 			(project ""
 				(path "/ca79f0b4-91f7-4537-917d-68d425c03ca3/485861e8-c90d-4c19-b473-548e94ff000e/62dce88f-62ee-4857-96f3-986f7b276210"
-					(reference "U19")
+					(reference "U18")
 					(unit 1)
 				)
@@
 		(dnp no)
 		(fields_autoplaced yes)
-		(property "Reference" "#PWR0172"
+		(property "Reference" "#PWR0163"
 			(at 199.39 181.61 0)
 			(effects
@@
 			(project "ETH1CVOLT_A"
 				(path "/ca79f0b4-91f7-4537-917d-68d425c03ca3/485861e8-c90d-4c19-b473-548e94ff000e/62dce88f-62ee-4857-96f3-986f7b276210"
-					(reference "#PWR0172")
+					(reference "#PWR0163")
 					(unit 1)
 				)
@@
 		(dnp no)
 		(fields_autoplaced yes)
-		(property "Reference" "#PWR0171"
+		(property "Reference" "#PWR0162"
 			(at 199.39 143.51 0)
 			(effects
@@
 			(project "ETH1CVOLT_A"
 				(path "/ca79f0b4-91f7-4537-917d-68d425c03ca3/485861e8-c90d-4c19-b473-548e94ff000e/62dce88f-62ee-4857-96f3-986f7b276210"
-					(reference "#PWR0171")
+					(reference "#PWR0162")
 					(unit 1)
 				)
@@
 		(dnp no)
 		(fields_autoplaced yes)
-		(property "Reference" "U18"
+		(property "Reference" "U17"
 			(at 211.6933 80.01 0)
 			(effects
@@
 			(project ""
 				(path "/ca79f0b4-91f7-4537-917d-68d425c03ca3/485861e8-c90d-4c19-b473-548e94ff000e/62dce88f-62ee-4857-96f3-986f7b276210"
-					(reference "U18")
+					(reference "U17")
 					(unit 1)
 				)
@@
 		(dnp no)
 		(fields_autoplaced yes)
-		(property "Reference" "#PWR0170"
+		(property "Reference" "#PWR0161"
 			(at 199.39 123.19 0)
 			(effects
@@
 			(project ""
 				(path "/ca79f0b4-91f7-4537-917d-68d425c03ca3/485861e8-c90d-4c19-b473-548e94ff000e/62dce88f-62ee-4857-96f3-986f7b276210"
-					(reference "#PWR0170")
-					(unit 1)
-				)
-			)
-		)
-	)
-	(symbol
-		(lib_id "ETH1CVOLT_A:+5VD_ISO")
+					(reference "#PWR0161")
+					(unit 1)
+				)
+			)
+		)
+	)
+	(symbol
+		(lib_id "ETH1CVOLT_A:+VD_ISO")
 		(at 209.55 81.28 0)
 		(unit 1)
@@
 		(dnp no)
 		(fields_autoplaced yes)
-		(property "Reference" "#PWR098"
+		(property "Reference" "#PWR0164"
 			(at 209.55 85.09 0)
 			(effects
@@
 			)
 		)
-		(property "Value" "+5VD_ISO"
+		(property "Value" "+VD_ISO"
 			(at 209.55 76.2 0)
 			(effects
@@
 			(project "ETH1CVOLT_A"
 				(path "/ca79f0b4-91f7-4537-917d-68d425c03ca3/485861e8-c90d-4c19-b473-548e94ff000e/62dce88f-62ee-4857-96f3-986f7b276210"
-					(reference "#PWR098")
+					(reference "#PWR0164")
 					(unit 1)
 				)
@@
 		(dnp no)
 		(fields_autoplaced yes)
-		(property "Reference" "#PWR0176"
+		(property "Reference" "#PWR0167"
 			(at 209.55 181.61 0)
 			(effects
@@
 			(project "ETH1CVOLT_A"
 				(path "/ca79f0b4-91f7-4537-917d-68d425c03ca3/485861e8-c90d-4c19-b473-548e94ff000e/62dce88f-62ee-4857-96f3-986f7b276210"
-					(reference "#PWR0176")
-					(unit 1)
-				)
+					(reference "#PWR0167")
+					(unit 1)
+				)

Commit message: Development
Parts:
- removed U17: ISO7763DW, Package_SO:SOIC-16W_7.5x10.3mm_P1.27mm, symbol Isolator:ISO7763DW
- added J14: Conn_02x04_Odd_Even, Connector_PinSocket_2.54mm:PinSocket_2x04_P2.54mm_Vertical_SMD, symbol Connector_Generic:Conn_02x04_Odd_Even
- added U17, U19: ISO7761FDW, Package_SO:SOIC-16W_7.5x10.3mm_P1.27mm, symbol Isolator:ISO7761FDW
- added U20, U21, U22: TCMT1103, Package_SO:SOP-4_4.4x2.6mm_P1.27mm, symbol Isolator:TCMT1103
- U18: value ISO7761DW -> ISO7761FDW; symbol Isolator:ISO7761DW -> Isolator:ISO7761FDW
Connections:
- net +3.3V: now also U17.1 (Vcc1), U19.1 (Vcc1)
- net +VD_ISO: now also U17.16 (Vcc2), U19.16 (Vcc2)
- net GND: now also U17.8 (GND1), U19.8 (GND1), U20.2, U21.2, U22.2
- net GND_ISO: now also U17.9 (GND2), U19.9 (GND2), U20.3, U21.3, U22.3
- net DAC1_~{FAULT}_ISO: no longer names the net of J12.2 (Pin_2)
- net DAC2_~{FAULT}_ISO: no longer names the net of J12.4 (Pin_4)
- net SPI1_MISO_ISO: no longer names the net of J12.7 (Pin_7)
- net SPI1_MOSI_ISO: no longer names the net of J12.3 (Pin_3)
- net SPI1_SCK_ISO: no longer names the net of J12.1 (Pin_1)
- net SPI1_~{CS}_ISO: no longer names the net of J12.5 (Pin_5)
- net SPI2_MISO: no longer names the net of U18.7 (OUTF)
- net SPI2_MISO_ISO: no longer names the net of U18.10 (INF)
- net SPI2_MISO_ISO: no longer J13.5 (Pin_5)
- net SPI2_SCK: no longer names the net of U18.5 (IND)
- net SPI2_SCK_ISO: no longer names the net of U18.12 (OUTD)
- net SPI2_SCK_ISO: no longer J13.1 (Pin_1)
- net SPI2_~{CS}: no longer names the net of U18.6 (INE)
- net SPI2_~{CS}_ISO: no longer names the net of U18.11 (OUTE)
- net SPI2_~{CS}_ISO: no longer J13.3 (Pin_3)
Other:
- moved on the sheet: J12, J13, U18

Commit message: Development
Parts:
- removed U17, U18, U19: ISO7761FDW, Package_SO:SOIC-16W_7.5x10.3mm_P1.27mm, symbol Isolator:ISO7761FDW
- added R61, R70, R71: 340, Resistor_SMD:R_0603_1608Metric_Pad0.98x0.95mm_HandSolder, symbol Device:R
- added U17, U18, U24: ISO7761FDBQ, Package_SO:SSOP-16_3.9x4.9mm_P0.635mm, symbol Isolator:ISO7761FDBQ
Connections:
- net +3.3V: now also U17.1 (Vcc1), U18.1 (Vcc1), U24.1 (Vcc1)
- net GND: now also U17.8 (GND1), U18.8 (GND1), U24.8 (GND1)
- net GND_ISO: now also U17.9 (GND2), U18.9 (GND2), U24.9 (GND2)
- net at U22.1: now also R71.2
- net HV_OUT_PMOS: now reaches U22.4
- net HV_OUT_PMOS: now also J14.8 (Pin_8)
- net at U21.1: now also R61.2
- net LV_OUT_PMOS: now reaches U21.4
- net LV_OUT_PMOS: now also J14.4 (Pin_4)
- net ADC_VOLT_SCLK: now reaches J14.1 (Pin_1)
- net ADC_VOLT_SCLK: now also U17.12 (OUTD)
- net MUX_A1: now reaches J14.2 (Pin_2)
- net MUX_A1: now also U24.14 (OUTB)
- net ADC_VOLT_~{CS}: now reaches J14.3 (Pin_3)
- net ADC_VOLT_~{CS}: now also U17.11 (OUTE)
- net ADC_VOLT_SDO: now reaches J14.5 (Pin_5)
- net ADC_VOLT_SDO: now also U17.10 (INF)
- net MV_OUT_PMOS: now reaches J14.6 (Pin_6)
- net MV_OUT_PMOS: now also U20.4
- net MUX_A0: now reaches J14.7 (Pin_7)
- net MUX_A0: now also U24.15 (OUTA)
- net ADC_CURR_SDO: now reaches J13.1 (Pin_1)
- net ADC_CURR_SDO: now also U18.10 (INF)
- net ADC_CURR_~{CS}: now reaches J13.3 (Pin_3)
- net ADC_CURR_~{CS}: now also U18.11 (OUTE)
- net ADC_CURR_SCLK: now reaches J13.5 (Pin_5)
- net ADC_CURR_SCLK: now also U18.12 (OUTD)
- net ADC_CURR_SDI: now reaches J13.7 (Pin_7)
- net ADC_CURR_SDI: now also U18.13 (OUTC)
- net DAC_SDO: now reaches J12.1 (Pin_1)
- net DAC_SDO: now also U24.10 (INF)
- net AUX_SEL: now reaches J12.2 (Pin_2)
- net AUX_SEL: now also U17.13 (OUTC)
- net DAC_SCLK: now reaches J12.3 (Pin_3)
- net DAC_SCLK: now also U24.11 (OUTE)
- net SEL_x1: now reaches J12.4 (Pin_4)
- net SEL_x1: now also U17.14 (OUTB)
- net DAC_SDIN: now reaches J12.5 (Pin_5)
- net DAC_SDIN: now also U24.12 (OUTD)
- net SEL_x10: now reaches J12.6 (Pin_6)
- net SEL_x10: now also U18.15 (OUTA)
- net DAC_~{SYNC}: now reaches J12.7 (Pin_7)
- net DAC_~{SYNC}: now also U24.13 (OUTC)
- net SEL_x100: now reaches J12.8 (Pin_8)
- net SEL_x100: now also U18.14 (OUTB)
- net at U20.1: now also R70.2
- new net +5VD_ISO: U17.16 (Vcc2), U18.16 (Vcc2), U24.16 (Vcc2)
- new net MCU_ADC_CURR_SCLK: U18.5 (IND)
- new net MCU_ADC_CURR_SDI: U18.4 (INC)
- new net MCU_ADC_CURR_SDO: U18.7 (OUTF)
- new net MCU_ADC_CURR_~{CS}: U18.6 (INE)
- new net MCU_ADC_VOLT_SCLK: U17.5 (IND)
- new net MCU_ADC_VOLT_SDO: U17.7 (OUTF)
- new net MCU_ADC_VOLT_~{CS}: U17.6 (INE)
- new net MCU_AUX_SEL: U17.4 (INC)
- new net MCU_DAC_SCLK: U24.6 (INE)
- new net MCU_DAC_SDIN: U24.5 (IND)
- new net MCU_DAC_SDO: U24.7 (OUTF)
- new net MCU_DAC_~{SYNC}: U24.4 (INC)
- new net MCU_HV_OUT_PMOS: R71.1
- new net MCU_LV_OUT_PMOS: R61.1
- new net MCU_MUX_A0: U24.2 (INA)
- new net MCU_MUX_A1: U24.3 (INB)
- new net MCU_MV_OUT_PMOS: R70.1
- new net MCU_SEL_x1: U17.3 (INB)
- new net MCU_SEL_x10: U18.2 (INA)
- new net MCU_SEL_x100: U18.3 (INB)
- no-connect marks 0 -> 6
Other:
- moved on the sheet: J13

Commit message: Hardware development
Parts:
- J10: renamed from J12; value Conn_02x04_Odd_Even -> 61030821821
- J11: renamed from J14; value Conn_02x04_Odd_Even -> 61030821821
- J12: renamed from J13; value Conn_02x04_Odd_Even -> 61030821821
- renumbered R61 to R69, U21 to U18, U20 to U19, U22 to U20, U24 to U21, U17 to U22, U18 to U23
