File: HARDWARE/ETH1CVOLT_A/Low_Voltage.kicad_sch (KiCad schematic)
At the start: 63 parts, among them J5 1715734, Q3 FZT849, U10 TSR0.5-2490, U11 LT8330_S6, U12 LT8330_S6, U15 TPS7A39, U16 ADP7142ARDZ-5.0, U17 ADP7142ARDZ-3.3

Commit message: Development
Parts:
- removed J5: 1715734, TerminalBlock_Phoenix:TerminalBlock_Phoenix_MKDS-1,5-3-5.08_1x03_P5.08mm_Horizontal, symbol Connector_Generic:Conn_01x03
- added J7: Conn_02x04_Odd_Even, Connector_PinSocket_2.54mm:PinSocket_2x04_P2.54mm_Vertical_SMD, symbol Connector_Generic:Conn_02x04_Odd_Even
- C84, C85, C86, C87, C88, C89: footprint (none) -> Capacitor_SMD:C_0603_1608Metric_Pad1.08x0.95mm_HandSolder
- L3, L4: footprint UCC25800:74489440068 -> ETH1CVOLT_A:74489440068
- R41, R42, R43, R44, R45, R46, R47, R48, R49, R50, R71, R72, R73, R74, R75, R76, R77, R80, R82: footprint (none) -> Resistor_SMD:R_0603_1608Metric_Pad0.98x0.95mm_HandSolder
Connections:
- net +21V_ISO: now also J7.2 (Pin_2)
- net +3V3_ISO: now also J7.8 (Pin_8)
- net +5V_ISO: now also J7.7 (Pin_7)
- net -21V_ISO: now also J7.1 (Pin_1)
- net GND_ISO: now also J7.3 (Pin_3), J7.4 (Pin_4), J7.6 (Pin_6)
- net VDD: now also J7.5 (Pin_5)
Other:
- moved on the sheet: C118, C119, C120, C79, C80, C81, C82, C83, C84, C85, C86, C87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

Commit message: Development
Parts:
- removed Q3: FZT849, symbol Simulation_SPICE:NPN
- added C128: C, Capacitor_SMD:C_0603_1608Metric_Pad1.08x0.95mm_HandSolder, symbol Device:C
- added Q6: FZT849, Package_TO_SOT_SMD:SOT-223-3_TabPin2, symbol Transistor_BJT:Q_NPN_BCE
- C118, C120, C124, C127, C76, C78, C82, C83, C92, C93: value 10u -> 10u/50V; footprint (none) -> Capacitor_SMD:C_1210_3225Metric_Pad1.33x2.70mm_HandSolder
- C119, C123, C126, C75, C77, C79, C80, C81, C90, C91: value 4u7 -> 4u7/50V; footprint (none) -> Capacitor_SMD:C_1210_3225Metric_Pad1.33x2.70mm_HandSolder
- C121: value 100u -> 100u/16V; footprint (none) -> Capacitor_SMD:C_1210_3225Metric_Pad1.33x2.70mm_HandSolder
- C86, C87: value 1u -> 1u/50V; footprint Capacitor_SMD:C_0603_1608Metric_Pad1.08x0.95mm_HandSolder -> Capacitor_SMD:C_0805_2012Metric_Pad1.18x1.45mm_HandSolder
- R76: value R -> 499
- U11, U12: footprint Package_TO_SOT_SMD:TSOT-23-6_HandSoldering -> Package_TO_SOT_SMD:TSOT-23-6
Connections:
- net +9V: now also Q6.2 (C)
- net GND_ISO: now also C128.2
- net VDD: now also Q6.3 (E)
- net at C121.1, R76.2, R77.1: now also Q6.1 (B)
- net at U15.3 (NR/SS): now also C128.1
Other:
- moved on the sheet: C118, C120, C77, C78

Commit message: Development
Parts:
- renumbered C119 to C100, C118 to C101, C120 to C102, C126 to C103, C127 to C104, C80 to C76, C81 to C77, C76 to C78, C82 to C79, C83 to C80, C77 to C81, C84 to C82, C85 to C83, C78 to C84, C86 to C85, C87 to C86, C121 to C87, C122 to C92, C92 to C93, C93 to C94, C128 to C95, C123 to C96, C124 to C97, C125 to C98, C79 to C99, D12 to D11, D13 to D12, J7 to J5, Q6 to Q3, R42 to R41, R43 to R42, R44 to R43, R45 to R44, R76 to R45, R77 to R46, R78 to R47, R46 to R48, R47 to R49, R48 to R50, R49 to R51, R50 to R52, R79 to R53, R80 to R54, R72 to R55, R73 to R56, R75 to R57, R41 to R58, R74 to R59, R71 to R60, R81 to R61, R82 to R62, U16 to U13, U15 to U14, U17 to U15

Commit message: Development
Parts:
- removed C87: 100u/16V, Capacitor_SMD:C_1210_3225Metric_Pad1.33x2.70mm_HandSolder, symbol Device:C_Polarized
- removed Q3: FZT849, Package_TO_SOT_SMD:SOT-223-3_TabPin2, symbol Transistor_BJT:Q_NPN_BCE
- removed R45: 499, Resistor_SMD:R_0603_1608Metric_Pad0.98x0.95mm_HandSolder, symbol Device:R
- removed R46: 499k, Resistor_SMD:R_0603_1608Metric_Pad0.98x0.95mm_HandSolder, symbol Device:R
- removed R47: 0, symbol Device:R
- removed U10: TSR0.5-2490, Converter_DCDC:Converter_DCDC_TRACO_TSR0.5-24xx_TSR0.5-24xxx_THT, symbol Converter_DCDC:TSR0.5-2490
- added C129: 1u, Capacitor_SMD:C_0603_1608Metric_Pad1.08x0.95mm_HandSolder, symbol Device:C
- added L7: 74408063470, symbol Device:L
- added R87: 68k, Resistor_SMD:R_0603_1608Metric_Pad0.98x0.95mm_HandSolder, symbol Device:R
- added R88: 10k, Resistor_SMD:R_0603_1608Metric_Pad0.98x0.95mm_HandSolder, symbol Device:R
- added U20: MAX15062C, Package_DFN_QFN:DFN-8_2x2mm_P0.5mm, symbol Regulator_Switching:MAX15062C
Connections:
- net +24V_LV_ISO: now also U20.1 (VIN), U20.2 (EN/UVLO)
- net GND_ISO: now also C129.2, R88.2, U20.7 (GND)
- net VDD: no longer U13.5 (EN), U13.7 (VIN), U13.8 (VIN)
- net +9V: no longer names the net of C81.1, C84.1
- net +9V: now also U13.5 (EN), U13.7 (VIN), U13.8 (VIN), L7.2, R87.1
- new net: C129.1, U20.3 (VCC)
- new net: R87.2, R88.1, U20.4 (FB/Vout)
- new net: L7.1, U20.8 (LX)
- no-connect marks 0 -> 2
Other:
- note added: "+7V/300mA"
- moved on the sheet: C100, C101, C102, C75, C76, C77, C78, C79, C80, C81, C82, C83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

Commit message: Development
Parts:
- removed C103, C96: 4u7/50V, Capacitor_SMD:C_1210_3225Metric_Pad1.33x2.70mm_HandSolder, symbol Device:C
- removed C104: 10u/50V, Capacitor_SMD:C_1210_3225Metric_Pad1.33x2.70mm_HandSolder, symbol Device:C
- removed C92: C, symbol Device:C
- removed R53, R61: R, symbol Device:R
- removed R54, R62: 0, Resistor_SMD:R_0603_1608Metric_Pad0.98x0.95mm_HandSolder, symbol Device:R
- removed U15: ADP7142ARDZ-3.3, Package_SO:SOIC-8-1EP_3.9x4.9mm_P1.27mm_EP2.29x3mm, symbol Regulator_Linear:ADP7142ARDZ-3.3
- added C100, C99: C, symbol Device:C
- added C101, C102, C94, C95: 4u7/50V, Capacitor_SMD:C_1210_3225Metric_Pad1.33x2.70mm_HandSolder, symbol Device:C
- added C105, C106: 10u/50V, Capacitor_SMD:C_1210_3225Metric_Pad1.33x2.70mm_HandSolder, symbol Device:C
- added R55, R56: R, symbol Device:R
- added R57, R58: 0, Resistor_SMD:R_0603_1608Metric_Pad0.98x0.95mm_HandSolder, symbol Device:R
- added U14: ADP7142ARDZ-5.0, Package_SO:SOIC-8-1EP_3.9x4.9mm_P1.27mm_EP2.29x3mm, symbol Regulator_Linear:ADP7142ARDZ-5.0
- C98: value C -> 10u/50V; footprint (none) -> Capacitor_SMD:C_1210_3225Metric_Pad1.33x2.70mm_HandSolder; now fitted
- renumbered C99 to C103, C100 to C104, C101 to C107, C102 to C108, C76 to C75, C77 to C76, C75 to C77, C129 to C81, C85 to C84, C86 to C85, C81 to C86, C84 to C87, C93 to C92, C94 to C93, C95 to C96, L7 to L5, R87 to R45, R88 to R46, R48 to R47, R49 to R48, R50 to R49, R51 to R50, R52 to R51, R55 to R52, R56 to R53, R57 to R54, R58 to R59, R59 to R60, R60 to R61, U20 to U10, U14 to U15
Connections:
- net VDD is gone; now on net +7V_ISO: J5.5 (Pin_5)
- net GND_ISO: now also C100.2, C101.2, C102.2, C105.2, C106.2, C94.2, C95.2, C99.2, R55.2, R56.2, U14.4 (GND), U14.9 (GND)
- net +7V_ISO: now reaches C86.1, C87.1, L5.2, R45.1, U13.5 (EN), U13.7 (VIN), U13.8 (VIN)
- net +7V_ISO: now also C97.1, C98.1, C94.1, C95.1, U14.5 (EN), U14.7 (VIN), U14.8 (VIN)
- net at U13.3 (SENSE/ADJ): now also R55.1, R57.1
- net at U13.6 (SS): now also C99.1
- net +3V3_ISO renamed +5VD_ISO
- net +5VD_ISO: now also C102.1, C106.1, R58.2, U14.1 (VOUT), U14.2 (VOUT)
- net +5V_ISO renamed +5VA_ISO
- net +5VA_ISO: now also C101.1, C105.1, R57.2; no longer C97.1
- new net: R56.1, R58.1, U14.3 (SENSE/ADJ)
- new net: C100.1, U14.6 (SS)
Other:
- note removed: "+3V3/200mA"
- moved on the sheet: C77, C78, C81, C86, C87, J5, L5, R45, R46, U10

Commit message: Development
Parts:
- added C48, C62: 4u7/50V, Capacitor_SMD:C_1210_3225Metric_Pad1.33x2.70mm_HandSolder, symbol Device:C
- added C50, C65: 10u/50V, Capacitor_SMD:C_1210_3225Metric_Pad1.33x2.70mm_HandSolder, symbol Device:C
- added C55: 1u, Capacitor_SMD:C_0603_1608Metric_Pad1.08x0.95mm_HandSolder, symbol Device:C
- added L8: 74408063470, symbol Device:L
- added R29: 0, Resistor_SMD:R_0603_1608Metric_Pad0.98x0.95mm_HandSolder, symbol Device:R
- added R30: 10k, Resistor_SMD:R_0603_1608Metric_Pad0.98x0.95mm_HandSolder, symbol Device:R
- added U8: MAX15062B, Package_DFN_QFN:DFN-8_2x2mm_P0.5mm, symbol Regulator_Switching:MAX15062B
- renumbered C75 to C45, C76 to C46, C77 to C47, C78 to C49, C79 to C51, C80 to C52, C81 to C54, C82 to C56, C83 to C57, C84 to C59, C85 to C60, C86 to C61, C87 to C64, C88 to C66, C89 to C67, C90 to C69, C91 to C70, C92 to C71, C93 to C72, C94 to C73, C95 to C74, C96 to C75, C97 to C77, C98 to C78, C99 to C80, C100 to C81, C103 to C82, C104 to C83, C101 to C84, C102 to C85, C107 to C86, C108 to C87, C105 to C88, C106 to C89, D11 to D5, D12 to D6, L3 to L5, L4 to L6, L5 to L7, R41 to R23, R42 to R24, R43 to R25, R44 to R26, R45 to R27, R46 to R28, R47 to R31, R48 to R32, R49 to R33, R50 to R34, R51 to R35, R52 to R36, R53 to R37, R54 to R38, R55 to R39, R56 to R40, R59 to R41, R60 to R42, R61 to R43, R57 to R44, R58 to R45, U12 to U10, U15 to U12, U10 to U7, U11 to U9
Connections:
- net +5VD_ISO: now also J5.6 (Pin_6), C62.1, C65.1, L8.2, R29.1; no longer C85.1, C89.1, J5.8 (Pin_8), R45.2, U14.1 (VOUT), U14.2 (VOUT)
- net GND_ISO: now also C48.2, C50.2, C55.2, C62.2, C65.2, R30.2, U8.7 (GND); no longer J5.3 (Pin_3), J5.6 (Pin_6)
- net +24V_LV_ISO renamed +24V_ISO
- net +24V_ISO: now also J5.3 (Pin_3), C48.1, C50.1, U8.1 (VIN), U8.2 (EN/UVLO)
- net +5VA_ISO renamed +VA_ISO
- new net: R29.2, R30.1, U8.4 (FB/Vout)
- new net: C55.1, U8.3 (VCC)
- new net: L8.1, U8.8 (LX)
- new net +VD_ISO: C85.1, C89.1, J5.8 (Pin_8), R45.2, U14.1 (VOUT), U14.2 (VOUT)
- no-connect marks 2 -> 4
Other:
- note added: "+21V/100mA"
- note added: "+22V/100mA"
- note added: "+5V/300mA"
- note added: "-21V/100mA"
- note added: "-22V/100mA"
- note removed: "+21V/50mA"
- note removed: "+22V/50mA"
- note removed: "-21V/50mA"
- note removed: "-22V/50mA"
- moved on the sheet: J5

Commit message: Development
Parts:
- C45, C46, C47, C48, C61, C62, C69, C70, C73, C74, C82, C83, C84, C85: value 4u7/50V -> 4u7/100V
- C49, C50, C51, C52, C64, C65, C71, C72, C77, C78, C86, C87, C88, C89: value 10u/50V -> 10u/100V
- C59, C60: value 1u/50V -> 1u/100V
- L7, L8: footprint (none) -> ETH1CVOLT_A:74408063470
- R31, R33: footprint Resistor_SMD:R_0603_1608Metric_Pad0.98x0.95mm_HandSolder -> Resistor_SMD:R_0805_2012Metric_Pad1.20x1.40mm_HandSolder
Other:
- moved on the sheet: C45, C46, C47, C48, C49, C50, C51, C52, C54, C55, C56, C57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

Commit message: Hardware development
Parts:
- J5: value Conn_02x04_Odd_Even -> 61030821821
- renumbered C59 to C45, C66 to C46, C45 to C47, C51 to C48, C69 to C49, C71 to C50, C56 to C51, C82 to C52, C86 to C53, C75 to C54, C60 to C55, C83 to C56, C87 to C57, C67 to C58, C46 to C59, C52 to C60, C70 to C61, C72 to C62, C57 to C70, C47 to C71, C49 to C72, C61 to C73, C64 to C74, C73 to C75, C77 to C76, C80 to C77, C84 to C78, C88 to C79, C54 to C80, C48 to C81, C50 to C82, C62 to C83, C65 to C84, C74 to C85, C78 to C86, C81 to C87, C85 to C88, C55 to C90, D6 to D5, D5 to D6, L5 to L3, L6 to L4, L7 to L8, L8 to L9, R31 to R24, R24 to R25, R32 to R26, R41 to R27, R36 to R28, R42 to R29, R37 to R30, R43 to R31, R38 to R32, R25 to R33, R33 to R34, R26 to R35, R34 to R36, R35 to R37, R44 to R38, R27 to R39, R39 to R40, R28 to R41, R45 to R42, R29 to R43, R40 to R44, R30 to R45, U13 to U11, U7 to U12, U14 to U13, U8 to U14, U9 to U7, U12 to U8, U10 to U9
