File: HARDWARE/ETH1CVOLT_A/MCU.kicad_sch (KiCad schematic)
At the start: 29 parts, among them J1 20021111-00010T4LF, U1 STM32H743VITx, U2 24LC08B-E/MS, Y1 NX5032GA-16

Commit message: Development
Parts:
- Y1: footprint ETH1HMSR-SMS:NX5032GA -> ETH1CVOLT_A:NX5032GA
Changed lines of the file:
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@@
 			)
 		)
-		(property "Footprint" "ETH1HMSR-SMS:NX5032GA"
+		(property "Footprint" "ETH1CVOLT_A:NX5032GA"
 			(at 140.97 78.74 0)
 			(effects

Commit message: Development
Parts:
- removed D1: ASMB-MTB1-0B3A2, LED_SMD:LED_Avago_PLCC4_3.2x2.8mm_CW, symbol LED:ASMB-MTB1-0A3A2
- removed RN1: EXB-V8V102JV, Resistor_SMD:R_Array_Concave_4x0603, symbol Device:R_Pack04
Connections:
- net LED_BLUE: no longer names the net of U1.63 (PC6)
- net LED_GREEN: no longer names the net of U1.65 (PC8)
- net LED_RED: no longer names the net of U1.64 (PC7)
- no-connect marks 60 -> 58

Commit message: Development
Connections:
- net +3.3VADC is gone; now on net VDDA: U1.20 (VREF+)
- net MCU_DEF: now also U1.98 (PE1); no longer U1.1 (PE2)
- net MCU_ADC_VOLT_~{CS}: now reaches U1.28 (PA4)
- net MCU_ADC_VOLT_SCLK: now reaches U1.29 (PA5)
- net MCU_ADC_CURR_~{CS}: now reaches U1.3 (PE4)
- net MCU_ADC_VOLT_SDO: now reaches U1.30 (PA6)
- net MCU_ADC_CURR_SDO: now reaches U1.4 (PE5)
- net MCU_OUTPUT_RL_CTR: now reaches U1.46 (PB10)
- net MCU_ADC_CURR_SDI: now reaches U1.5 (PE6)
- net MCU_HV_OUT_PMOS: now reaches U1.62 (PD15)
- net MCU_MV_OUT_PMOS: now reaches U1.63 (PC6)
- net MCU_LV_OUT_PMOS: now reaches U1.64 (PC7)
- net MCU_AUX_SEL: now reaches U1.65 (PC8)
- net MCU_SEL_x100: now reaches U1.66 (PC9)
- net MCU_SEL_x10: now reaches U1.67 (PA8)
- net MCU_SEL_x1: now reaches U1.68 (PA9)
- net MCU_MUX_A1: now reaches U1.69 (PA10)
- net MCU_MUX_A0: now reaches U1.70 (PA11)
- net MCU_DAC_~{SYNC}: now reaches U1.77 (PA15)
- net MCU_DAC_SCLK: now reaches U1.78 (PC10)
- net MCU_DAC_SDO: now reaches U1.79 (PC11)
- net MCU_DAC_SDIN: now reaches U1.80 (PC12)
- new net MCU_ADC_CURR_SCLK: U1.1 (PE2)
- no-connect marks 58 -> 48
Other:
- moved on the sheet: C1, C10, C11, C12, C14, C2, C3, C4, C5, C6, C7, C8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

Commit message: Hardware development
Parts:
- renumbered C9 to C1, C4 to C10, C5 to C11, C6 to C12, C7 to C13, C8 to C14, C12 to C15, C14 to C16, C10 to C2, C11 to C3, C16 to C4, C13 to C5, C15 to C6, C1 to C7, C2 to C8, C3 to C9, R4 to R3, R5 to R4, R3 to R5
Other:
- moved on the sheet: C1, C2, C3, C5, C6, R1, R2, U1, Y1
