File: HARDWARE/ETH1CVOLT_A/Medium_Voltage.kicad_sch (KiCad schematic)
At the start: 29 parts, among them J4 1715734, U8 LT8330_S6, U9 LT8330_S6

Commit message: Development
Parts:
- removed J4: 1715734, TerminalBlock_Phoenix:TerminalBlock_Phoenix_MKDS-1,5-3-5.08_1x03_P5.08mm_Horizontal, symbol Connector_Generic:Conn_01x03
- added J11: Conn_02x04_Odd_Even, Connector_PinSocket_2.54mm:PinSocket_2x04_P2.54mm_Vertical_SMD, symbol Connector_Generic:Conn_02x04_Odd_Even
- C66, C67, C68, C69, C70: footprint (none) -> Capacitor_SMD:C_0603_1608Metric_Pad1.08x0.95mm_HandSolder
- L2: footprint UCC25800:74489440068 -> ETH1CVOLT_A:74489440068
- R32, R33, R34, R35, R36, R37, R38, R39, R40: footprint (none) -> Resistor_SMD:R_0603_1608Metric_Pad0.98x0.95mm_HandSolder
Connections:
- net +44V_ISO: now also J11.1 (Pin_1), J11.2 (Pin_2)
- net -41V_ISO: now also J11.7 (Pin_7), J11.8 (Pin_8)
- net GND_ISO: now also J11.3 (Pin_3), J11.4 (Pin_4), J11.5 (Pin_5), J11.6 (Pin_6)

Commit message: Development
Parts:
- C62, C63: value 4u7 -> 4u7/50V; footprint (none) -> Capacitor_SMD:C_1210_3225Metric_Pad1.33x2.70mm_HandSolder
- C64, C65: value 10u -> 10u/50V; footprint (none) -> Capacitor_SMD:C_1210_3225Metric_Pad1.33x2.70mm_HandSolder
- C68: value 1u -> 1u/100V; footprint Capacitor_SMD:C_0603_1608Metric_Pad1.08x0.95mm_HandSolder -> Capacitor_SMD:C_0805_2012Metric_Pad1.18x1.45mm_HandSolder
- C71, C72: value 4u7 -> 4u7/100V; footprint (none) -> Capacitor_SMD:C_1210_3225Metric_Pad1.33x2.70mm_HandSolder
- C73, C74: value 10u -> 10u/100V; footprint (none) -> Capacitor_SMD:C_1210_3225Metric_Pad1.33x2.70mm_HandSolder
- L1: value 6u8 -> 74438335068
- U8, U9: footprint Package_TO_SOT_SMD:TSOT-23-6_HandSoldering -> Package_TO_SOT_SMD:TSOT-23-6
Other:
- moved on the sheet: C62, C63, C64, C65, C73, C74

Commit message: Development
Parts:
- renumbered D11 to D10, D10 to D9, J11 to J4
Changed lines of the file:
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@@
 		(dnp no)
 		(fields_autoplaced yes)
-		(property "Reference" "#PWR076"
+		(property "Reference" "#PWR078"
 			(at 250.19 62.23 0)
 			(effects
@@
 			(project ""
 				(path "/ca79f0b4-91f7-4537-917d-68d425c03ca3/485861e8-c90d-4c19-b473-548e94ff000e/18da2cad-962d-47df-95e7-fd94fee0a7d8/ff9439b0-b623-4d10-a906-fb4e3cb6e044/6d967ebd-a46f-4449-b98b-985b0576b4a9"
-					(reference "#PWR076")
+					(reference "#PWR078")
 					(unit 1)
 				)
@@
 		(dnp no)
 		(fields_autoplaced yes)
-		(property "Reference" "#PWR0137"
+		(property "Reference" "#PWR084"
 			(at 245.11 271.78 0)
 			(effects
@@
 			(project "ETH1CVOLT_A"
 				(path "/ca79f0b4-91f7-4537-917d-68d425c03ca3/485861e8-c90d-4c19-b473-548e94ff000e/18da2cad-962d-47df-95e7-fd94fee0a7d8/ff9439b0-b623-4d10-a906-fb4e3cb6e044/6d967ebd-a46f-4449-b98b-985b0576b4a9"
-					(reference "#PWR0137")
+					(reference "#PWR084")
 					(unit 1)
 				)
@@
 		(dnp no)
 		(fields_autoplaced yes)
-		(property "Reference" "#PWR073"
+		(property "Reference" "#PWR075"
 			(at 121.92 171.45 0)
 			(effects
@@
 			(project ""
 				(path "/ca79f0b4-91f7-4537-917d-68d425c03ca3/485861e8-c90d-4c19-b473-548e94ff000e/18da2cad-962d-47df-95e7-fd94fee0a7d8/ff9439b0-b623-4d10-a906-fb4e3cb6e044/6d967ebd-a46f-4449-b98b-985b0576b4a9"
-					(reference "#PWR073")
+					(reference "#PWR075")
 					(unit 1)
 				)
@@
 		(dnp no)
 		(fields_autoplaced yes)
-		(property "Reference" "#PWR078"
+		(property "Reference" "#PWR080"
 			(at 250.19 171.45 0)
 			(effects
@@
 			(project ""
 				(path "/ca79f0b4-91f7-4537-917d-68d425c03ca3/485861e8-c90d-4c19-b473-548e94ff000e/18da2cad-962d-47df-95e7-fd94fee0a7d8/ff9439b0-b623-4d10-a906-fb4e3cb6e044/6d967ebd-a46f-4449-b98b-985b0576b4a9"
-					(reference "#PWR078")
+					(reference "#PWR080")
 					(unit 1)
 				)
@@
 		(dnp no)
 		(fields_autoplaced yes)
-		(property "Reference" "#PWR082"
+		(property "Reference" "#PWR089"
 			(at 267.97 274.32 0)
 			(effects
@@
 			(project "ETH1CVOLT_A"
 				(path "/ca79f0b4-91f7-4537-917d-68d425c03ca3/485861e8-c90d-4c19-b473-548e94ff000e/18da2cad-962d-47df-95e7-fd94fee0a7d8/ff9439b0-b623-4d10-a906-fb4e3cb6e044/6d967ebd-a46f-4449-b98b-985b0576b4a9"
-					(reference "#PWR082")
+					(reference "#PWR089")
 					(unit 1)
 				)
@@
 		(dnp no)
 		(fields_autoplaced yes)
-		(property "Reference" "#PWR074"
+		(property "Reference" "#PWR076"
 			(at 121.92 213.36 0)
 			(effects
@@
 			(project "ETH1CVOLT_A"
 				(path "/ca79f0b4-91f7-4537-917d-68d425c03ca3/485861e8-c90d-4c19-b473-548e94ff000e/18da2cad-962d-47df-95e7-fd94fee0a7d8/ff9439b0-b623-4d10-a906-fb4e3cb6e044/6d967ebd-a46f-4449-b98b-985b0576b4a9"
-					(reference "#PWR074")
+					(reference "#PWR076")
 					(unit 1)
 				)
@@
 		(dnp no)
 		(fields_autoplaced yes)
-		(property "Reference" "#PWR071"
+		(property "Reference" "#PWR073"
 			(at 121.92 62.23 0)
 			(effects
@@
 			(project "ETH1CVOLT_A"
 				(path "/ca79f0b4-91f7-4537-917d-68d425c03ca3/485861e8-c90d-4c19-b473-548e94ff000e/18da2cad-962d-47df-95e7-fd94fee0a7d8/ff9439b0-b623-4d10-a906-fb4e3cb6e044/6d967ebd-a46f-4449-b98b-985b0576b4a9"
-					(reference "#PWR071")
+					(reference "#PWR073")
 					(unit 1)
 				)
@@
 		(dnp no)
 		(fields_autoplaced yes)
-		(property "Reference" "J11"
+		(property "Reference" "J4"
 			(at 261.62 260.35 0)
 			(effects
@@
 			(project ""
 				(path "/ca79f0b4-91f7-4537-917d-68d425c03ca3/485861e8-c90d-4c19-b473-548e94ff000e/18da2cad-962d-47df-95e7-fd94fee0a7d8/ff9439b0-b623-4d10-a906-fb4e3cb6e044/6d967ebd-a46f-4449-b98b-985b0576b4a9"
-					(reference "J11")
+					(reference "J4")
 					(unit 1)
 				)
@@
 		(dnp no)
 		(fields_autoplaced yes)
-		(property "Reference" "#PWR081"
+		(property "Reference" "#PWR085"
 			(at 255.27 274.32 0)
 			(effects
@@
 			(project "ETH1CVOLT_A"
 				(path "/ca79f0b4-91f7-4537-917d-68d425c03ca3/485861e8-c90d-4c19-b473-548e94ff000e/18da2cad-962d-47df-95e7-fd94fee0a7d8/ff9439b0-b623-4d10-a906-fb4e3cb6e044/6d967ebd-a46f-4449-b98b-985b0576b4a9"
-					(reference "#PWR081")
+					(reference "#PWR085")
 					(unit 1)
 				)
@@
 		(dnp no)
 		(fields_autoplaced yes)
-		(property "Reference" "#PWR077"
+		(property "Reference" "#PWR079"
 			(at 250.19 104.14 0)
 			(effects
@@
 			(project "ETH1CVOLT_A"
 				(path "/ca79f0b4-91f7-4537-917d-68d425c03ca3/485861e8-c90d-4c19-b473-548e94ff000e/18da2cad-962d-47df-95e7-fd94fee0a7d8/ff9439b0-b623-4d10-a906-fb4e3cb6e044/6d967ebd-a46f-4449-b98b-985b0576b4a9"
-					(reference "#PWR077")
+					(reference "#PWR079")
 					(unit 1)
 				)
@@
 		(dnp no)
 		(fields_autoplaced yes)
-		(property "Reference" "#PWR080"
+		(property "Reference" "#PWR086"
 			(at 267.97 266.7 0)
 			(effects
@@
 			(project "ETH1CVOLT_A"
 				(path "/ca79f0b4-91f7-4537-917d-68d425c03ca3/485861e8-c90d-4c19-b473-548e94ff000e/18da2cad-962d-47df-95e7-fd94fee0a7d8/ff9439b0-b623-4d10-a906-fb4e3cb6e044/6d967ebd-a46f-4449-b98b-985b0576b4a9"
-					(reference "#PWR080")
+					(reference "#PWR086")
 					(unit 1)
 				)
@@
 		(dnp no)
 		(fields_autoplaced yes)
-		(property "Reference" "#PWR072"
+		(property "Reference" "#PWR074"
 			(at 121.92 104.14 0)
 			(effects
@@
 			(project "ETH1CVOLT_A"
 				(path "/ca79f0b4-91f7-4537-917d-68d425c03ca3/485861e8-c90d-4c19-b473-548e94ff000e/18da2cad-962d-47df-95e7-fd94fee0a7d8/ff9439b0-b623-4d10-a906-fb4e3cb6e044/6d967ebd-a46f-4449-b98b-985b0576b4a9"
-					(reference "#PWR072")
+					(reference "#PWR074")
 					(unit 1)
 				)
@@
 		(dnp no)
 		(fields_autoplaced yes)
-		(property "Reference" "#PWR0138"
+		(property "Reference" "#PWR087"
 			(at 278.13 269.24 0)
 			(effects
@@
 			(project "ETH1CVOLT_A"
 				(path "/ca79f0b4-91f7-4537-917d-68d425c03ca3/485861e8-c90d-4c19-b473-548e94ff000e/18da2cad-962d-47df-95e7-fd94fee0a7d8/ff9439b0-b623-4d10-a906-fb4e3cb6e044/6d967ebd-a46f-4449-b98b-985b0576b4a9"
-					(reference "#PWR0138")
+					(reference "#PWR087")
 					(unit 1)
 				)
@@
 		(dnp no)
 		(fields_autoplaced yes)
-		(property "Reference" "#PWR079"
+		(property "Reference" "#PWR081"
 			(at 250.19 213.36 0)
 			(effects
@@
 			(project "ETH1CVOLT_A"
 				(path "/ca79f0b4-91f7-4537-917d-68d425c03ca3/485861e8-c90d-4c19-b473-548e94ff000e/18da2cad-962d-47df-95e7-fd94fee0a7d8/ff9439b0-b623-4d10-a906-fb4e3cb6e044/6d967ebd-a46f-4449-b98b-985b0576b4a9"
-					(reference "#PWR079")
+					(reference "#PWR081")
 					(unit 1)
 				)
@@
 		(on_board yes)
 		(dnp no)
-		(property "Reference" "D10"
+		(property "Reference" "D9"
 			(at 192.5066 174.0916 90)
 			(effects
@@
 			(project "ETH1CVOLT_A"
 				(path "/ca79f0b4-91f7-4537-917d-68d425c03ca3/485861e8-c90d-4c19-b473-548e94ff000e/18da2cad-962d-47df-95e7-fd94fee0a7d8/ff9439b0-b623-4d10-a906-fb4e3cb6e044/6d967ebd-a46f-4449-b98b-985b0576b4a9"
-					(reference "D10")
+					(reference "D9")
 					(unit 1)
 				)
@@
 		(dnp no)
 		(fields_autoplaced yes)
-		(property "Reference" "#PWR0136"
+		(property "Reference" "#PWR083"
 			(at 245.11 269.24 0)
 			(effects
@@
 			(project "ETH1CVOLT_A"
 				(path "/ca79f0b4-91f7-4537-917d-68d425c03ca3/485861e8-c90d-4c19-b473-548e94ff000e/18da2cad-962d-47df-95e7-fd94fee0a7d8/ff9439b0-b623-4d10-a906-fb4e3cb6e044/6d967ebd-a46f-4449-b98b-985b0576b4a9"
-					(reference "#PWR0136")
+					(reference "#PWR083")
 					(unit 1)
 				)
@@
 		(dnp no)
 		(fields_autoplaced yes)
-		(property "Reference" "#PWR075"
+		(property "Reference" "#PWR077"
 			(at 190.5 185.42 0)
 			(effects
@@
 			(project "ETH1CVOLT_A"
 				(path "/ca79f0b4-91f7-4537-917d-68d425c03ca3/485861e8-c90d-4c19-b473-548e94ff000e/18da2cad-962d-47df-95e7-fd94fee0a7d8/ff9439b0-b623-4d10-a906-fb4e3cb6e044/6d967ebd-a46f-4449-b98b-985b0576b4a9"
-					(reference "#PWR075")
+					(reference "#PWR077")
 					(unit 1)
 				)
@@
 		(on_board yes)
 		(dnp no)
-		(property "Reference" "D11"
+		(property "Reference" "D10"
 			(at 194.31 54.2036 0)
 			(effects
@@
 			(project "ETH1CVOLT_A"
 				(path "/ca79f0b4-91f7-4537-917d-68d425c03ca3/485861e8-c90d-4c19-b473-548e94ff000e/18da2cad-962d-47df-95e7-fd94fee0a7d8/ff9439b0-b623-4d10-a906-fb4e3cb6e044/6d967ebd-a46f-4449-b98b-985b0576b4a9"
-					(reference "D11")
+					(reference "D10")
 					(unit 1)
 				)
@@
 		(dnp no)
 		(fields_autoplaced yes)
-		(property "Reference" "#PWR0139"
+		(property "Reference" "#PWR088"
 			(at 278.13 271.78 0)
 			(effects
@@
 			(project "ETH1CVOLT_A"
 				(path "/ca79f0b4-91f7-4537-917d-68d425c03ca3/485861e8-c90d-4c19-b473-548e94ff000e/18da2cad-962d-47df-95e7-fd94fee0a7d8/ff9439b0-b623-4d10-a906-fb4e3cb6e044/6d967ebd-a46f-4449-b98b-985b0576b4a9"
-					(reference "#PWR0139")
+					(reference "#PWR088")
 					(unit 1)
 				)
@@
 		(dnp no)
 		(fields_autoplaced yes)
-		(property "Reference" "#PWR0135"
+		(property "Reference" "#PWR082"
 			(at 255.27 266.7 0)
 			(effects
@@
 			(project "ETH1CVOLT_A"
 				(path "/ca79f0b4-91f7-4537-917d-68d425c03ca3/485861e8-c90d-4c19-b473-548e94ff000e/18da2cad-962d-47df-95e7-fd94fee0a7d8/ff9439b0-b623-4d10-a906-fb4e3cb6e044/6d967ebd-a46f-4449-b98b-985b0576b4a9"
-					(reference "#PWR0135")
+					(reference "#PWR082")
 					(unit 1)
 				)

Commit message: Development
Other:
- note added: "+44V/55mA"
- note added: "-41V/55mA"
- note removed: "+44V/50mA"
- note removed: "-41V/50mA"
Changed lines of the file:
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@@
 	(generator_version "9.0")
 	(paper "A3")
-	(text "-41V/50mA"
+	(text "-41V/55mA"
 		(exclude_from_sim no)
 		(at 232.41 166.37 0)
@@
 		)
 	)
-	(text "+44V/50mA"
+	(text "+44V/55mA"
 		(exclude_from_sim no)
 		(at 232.41 57.15 0)
@@
 		(dnp no)
 		(fields_autoplaced yes)
-		(property "Reference" "#PWR078"
+		(property "Reference" "#PWR079"
 			(at 250.19 62.23 0)
 			(effects
@@
 			(project ""
 				(path "/ca79f0b4-91f7-4537-917d-68d425c03ca3/485861e8-c90d-4c19-b473-548e94ff000e/18da2cad-962d-47df-95e7-fd94fee0a7d8/ff9439b0-b623-4d10-a906-fb4e3cb6e044/6d967ebd-a46f-4449-b98b-985b0576b4a9"
-					(reference "#PWR078")
+					(reference "#PWR079")
 					(unit 1)
 				)
@@
 		(dnp no)
 		(fields_autoplaced yes)
-		(property "Reference" "#PWR084"
+		(property "Reference" "#PWR085"
 			(at 245.11 271.78 0)
 			(effects
@@
 			(project "ETH1CVOLT_A"
 				(path "/ca79f0b4-91f7-4537-917d-68d425c03ca3/485861e8-c90d-4c19-b473-548e94ff000e/18da2cad-962d-47df-95e7-fd94fee0a7d8/ff9439b0-b623-4d10-a906-fb4e3cb6e044/6d967ebd-a46f-4449-b98b-985b0576b4a9"
-					(reference "#PWR084")
+					(reference "#PWR085")
 					(unit 1)
 				)
@@
 		(dnp no)
 		(fields_autoplaced yes)
-		(property "Reference" "#PWR075"
+		(property "Reference" "#PWR076"
 			(at 121.92 171.45 0)
 			(effects
@@
 			(project ""
 				(path "/ca79f0b4-91f7-4537-917d-68d425c03ca3/485861e8-c90d-4c19-b473-548e94ff000e/18da2cad-962d-47df-95e7-fd94fee0a7d8/ff9439b0-b623-4d10-a906-fb4e3cb6e044/6d967ebd-a46f-4449-b98b-985b0576b4a9"
-					(reference "#PWR075")
+					(reference "#PWR076")
 					(unit 1)
 				)
@@
 		(dnp no)
 		(fields_autoplaced yes)
-		(property "Reference" "#PWR080"
+		(property "Reference" "#PWR081"
 			(at 250.19 171.45 0)
 			(effects
@@
 			(project ""
 				(path "/ca79f0b4-91f7-4537-917d-68d425c03ca3/485861e8-c90d-4c19-b473-548e94ff000e/18da2cad-962d-47df-95e7-fd94fee0a7d8/ff9439b0-b623-4d10-a906-fb4e3cb6e044/6d967ebd-a46f-4449-b98b-985b0576b4a9"
-					(reference "#PWR080")
+					(reference "#PWR081")
 					(unit 1)
 				)
@@
 		(dnp no)
 		(fields_autoplaced yes)
-		(property "Reference" "#PWR089"
+		(property "Reference" "#PWR090"
 			(at 267.97 274.32 0)
 			(effects
@@
 			(project "ETH1CVOLT_A"
 				(path "/ca79f0b4-91f7-4537-917d-68d425c03ca3/485861e8-c90d-4c19-b473-548e94ff000e/18da2cad-962d-47df-95e7-fd94fee0a7d8/ff9439b0-b623-4d10-a906-fb4e3cb6e044/6d967ebd-a46f-4449-b98b-985b0576b4a9"
-					(reference "#PWR089")
+					(reference "#PWR090")
 					(unit 1)
 				)
@@
 		(dnp no)
 		(fields_autoplaced yes)
-		(property "Reference" "#PWR076"
+		(property "Reference" "#PWR077"
 			(at 121.92 213.36 0)
 			(effects
@@
 			(project "ETH1CVOLT_A"
 				(path "/ca79f0b4-91f7-4537-917d-68d425c03ca3/485861e8-c90d-4c19-b473-548e94ff000e/18da2cad-962d-47df-95e7-fd94fee0a7d8/ff9439b0-b623-4d10-a906-fb4e3cb6e044/6d967ebd-a46f-4449-b98b-985b0576b4a9"
-					(reference "#PWR076")
+					(reference "#PWR077")
 					(unit 1)
 				)
@@
 		(dnp no)
 		(fields_autoplaced yes)
-		(property "Reference" "#PWR073"
+		(property "Reference" "#PWR074"
 			(at 121.92 62.23 0)
 			(effects
@@
 			(project "ETH1CVOLT_A"
 				(path "/ca79f0b4-91f7-4537-917d-68d425c03ca3/485861e8-c90d-4c19-b473-548e94ff000e/18da2cad-962d-47df-95e7-fd94fee0a7d8/ff9439b0-b623-4d10-a906-fb4e3cb6e044/6d967ebd-a46f-4449-b98b-985b0576b4a9"
-					(reference "#PWR073")
+					(reference "#PWR074")
 					(unit 1)
 				)
@@
 		(dnp no)
 		(fields_autoplaced yes)
-		(property "Reference" "#PWR085"
+		(property "Reference" "#PWR086"
 			(at 255.27 274.32 0)
 			(effects
@@
 			(project "ETH1CVOLT_A"
 				(path "/ca79f0b4-91f7-4537-917d-68d425c03ca3/485861e8-c90d-4c19-b473-548e94ff000e/18da2cad-962d-47df-95e7-fd94fee0a7d8/ff9439b0-b623-4d10-a906-fb4e3cb6e044/6d967ebd-a46f-4449-b98b-985b0576b4a9"
-					(reference "#PWR085")
+					(reference "#PWR086")
 					(unit 1)
 				)
@@
 		(dnp no)
 		(fields_autoplaced yes)
-		(property "Reference" "#PWR079"
+		(property "Reference" "#PWR080"
 			(at 250.19 104.14 0)
 			(effects
@@
 			(project "ETH1CVOLT_A"
 				(path "/ca79f0b4-91f7-4537-917d-68d425c03ca3/485861e8-c90d-4c19-b473-548e94ff000e/18da2cad-962d-47df-95e7-fd94fee0a7d8/ff9439b0-b623-4d10-a906-fb4e3cb6e044/6d967ebd-a46f-4449-b98b-985b0576b4a9"
-					(reference "#PWR079")
+					(reference "#PWR080")
 					(unit 1)
 				)
@@
 		(dnp no)
 		(fields_autoplaced yes)
-		(property "Reference" "#PWR086"
+		(property "Reference" "#PWR087"
 			(at 267.97 266.7 0)
 			(effects
@@
 			(project "ETH1CVOLT_A"
 				(path "/ca79f0b4-91f7-4537-917d-68d425c03ca3/485861e8-c90d-4c19-b473-548e94ff000e/18da2cad-962d-47df-95e7-fd94fee0a7d8/ff9439b0-b623-4d10-a906-fb4e3cb6e044/6d967ebd-a46f-4449-b98b-985b0576b4a9"
-					(reference "#PWR086")
+					(reference "#PWR087")
 					(unit 1)
 				)
@@
 		(dnp no)
 		(fields_autoplaced yes)
-		(property "Reference" "#PWR074"
+		(property "Reference" "#PWR075"
 			(at 121.92 104.14 0)
 			(effects
@@
 			(project "ETH1CVOLT_A"
 				(path "/ca79f0b4-91f7-4537-917d-68d425c03ca3/485861e8-c90d-4c19-b473-548e94ff000e/18da2cad-962d-47df-95e7-fd94fee0a7d8/ff9439b0-b623-4d10-a906-fb4e3cb6e044/6d967ebd-a46f-4449-b98b-985b0576b4a9"
-					(reference "#PWR074")
+					(reference "#PWR075")
 					(unit 1)
 				)
@@
 		(dnp no)
 		(fields_autoplaced yes)
-		(property "Reference" "#PWR087"
+		(property "Reference" "#PWR088"
 			(at 278.13 269.24 0)
 			(effects
@@
 			(project "ETH1CVOLT_A"
 				(path "/ca79f0b4-91f7-4537-917d-68d425c03ca3/485861e8-c90d-4c19-b473-548e94ff000e/18da2cad-962d-47df-95e7-fd94fee0a7d8/ff9439b0-b623-4d10-a906-fb4e3cb6e044/6d967ebd-a46f-4449-b98b-985b0576b4a9"
-					(reference "#PWR087")
+					(reference "#PWR088")
 					(unit 1)
 				)
@@
 		(dnp no)
 		(fields_autoplaced yes)
-		(property "Reference" "#PWR081"
+		(property "Reference" "#PWR082"
 			(at 250.19 213.36 0)
 			(effects
@@
 			(project "ETH1CVOLT_A"
 				(path "/ca79f0b4-91f7-4537-917d-68d425c03ca3/485861e8-c90d-4c19-b473-548e94ff000e/18da2cad-962d-47df-95e7-fd94fee0a7d8/ff9439b0-b623-4d10-a906-fb4e3cb6e044/6d967ebd-a46f-4449-b98b-985b0576b4a9"
-					(reference "#PWR081")
+					(reference "#PWR082")
 					(unit 1)
 				)
@@
 		(dnp no)
 		(fields_autoplaced yes)
-		(property "Reference" "#PWR083"
+		(property "Reference" "#PWR084"
 			(at 245.11 269.24 0)
 			(effects
@@
 			(project "ETH1CVOLT_A"
 				(path "/ca79f0b4-91f7-4537-917d-68d425c03ca3/485861e8-c90d-4c19-b473-548e94ff000e/18da2cad-962d-47df-95e7-fd94fee0a7d8/ff9439b0-b623-4d10-a906-fb4e3cb6e044/6d967ebd-a46f-4449-b98b-985b0576b4a9"
-					(reference "#PWR083")
+					(reference "#PWR084")
 					(unit 1)
 				)
@@
 		(dnp no)
 		(fields_autoplaced yes)
-		(property "Reference" "#PWR077"
+		(property "Reference" "#PWR078"
 			(at 190.5 185.42 0)
 			(effects
@@
 			(project "ETH1CVOLT_A"
 				(path "/ca79f0b4-91f7-4537-917d-68d425c03ca3/485861e8-c90d-4c19-b473-548e94ff000e/18da2cad-962d-47df-95e7-fd94fee0a7d8/ff9439b0-b623-4d10-a906-fb4e3cb6e044/6d967ebd-a46f-4449-b98b-985b0576b4a9"
-					(reference "#PWR077")
+					(reference "#PWR078")
 					(unit 1)
 				)
@@
 		(dnp no)
 		(fields_autoplaced yes)
-		(property "Reference" "#PWR088"
+		(property "Reference" "#PWR089"
 			(at 278.13 271.78 0)
 			(effects
@@
 			(project "ETH1CVOLT_A"
 				(path "/ca79f0b4-91f7-4537-917d-68d425c03ca3/485861e8-c90d-4c19-b473-548e94ff000e/18da2cad-962d-47df-95e7-fd94fee0a7d8/ff9439b0-b623-4d10-a906-fb4e3cb6e044/6d967ebd-a46f-4449-b98b-985b0576b4a9"
-					(reference "#PWR088")
+					(reference "#PWR089")
 					(unit 1)
 				)
@@
 		(dnp no)
 		(fields_autoplaced yes)
-		(property "Reference" "#PWR082"
+		(property "Reference" "#PWR083"
 			(at 255.27 266.7 0)
 			(effects
@@
 			(project "ETH1CVOLT_A"
 				(path "/ca79f0b4-91f7-4537-917d-68d425c03ca3/485861e8-c90d-4c19-b473-548e94ff000e/18da2cad-962d-47df-95e7-fd94fee0a7d8/ff9439b0-b623-4d10-a906-fb4e3cb6e044/6d967ebd-a46f-4449-b98b-985b0576b4a9"
-					(reference "#PWR082")
+					(reference "#PWR083")
 					(unit 1)
 				)

Commit message: Development
Parts:
- renumbered C62 to C32, C63 to C33, C64 to C34, C65 to C35, C66 to C36, C67 to C37, C68 to C38, C69 to C39, C70 to C40, C71 to C41, C72 to C42, C73 to C43, C74 to C44, D9 to D3, D10 to D4, R32 to R14, R33 to R15, R34 to R16, R35 to R17, R36 to R18, R37 to R19, R38 to R20, R39 to R21, R40 to R22, U8 to U5, U9 to U6
Connections:
- net +24V_MV_ISO renamed +24V_ISO

Commit message: Development
Parts:
- C32, C33: value 4u7/50V -> 4u7/100V
- C34, C35: value 10u/50V -> 10u/100V
- L1: footprint (none) -> ETH1CVOLT_A:74438335068
- R18, R21: footprint Resistor_SMD:R_0603_1608Metric_Pad0.98x0.95mm_HandSolder -> Resistor_SMD:R_0805_2012Metric_Pad1.20x1.40mm_HandSolder
Connections:
- net GND is gone; now on net GND_ISO: D3.1 (K)
Other:
- moved on the sheet: J4

Commit message: Hardware development
Parts:
- J4: value Conn_02x04_Odd_Even -> 61030821821
- renumbered C39 to C32, C32 to C33, C41 to C35, C43 to C36, C36 to C37, C40 to C39, C33 to C40, C35 to C41, C44 to C43, C37 to C44, D4 to D3, D3 to D4, R18 to R15, R15 to R16, R19 to R17, R20 to R18, R16 to R19, R21 to R20, R17 to R21
