File: HARDWARE/ETH1CVOLT_A/Power_Not_Isolated.kicad_sch (KiCad schematic)
At the start: 14 parts, among them J3 1715721, Q1 FDS9435A, Q2 MMBT3904, U4 TSR1-2433E

Commit message: Development
Parts:
- C31: footprint Capacitor_Tantalum_SMD:CP_EIA-3528-21_Kemet-B_Pad1.50x2.35mm_HandSolder -> (none)
- TP1, TP2: footprint (none) -> TestPoint:TestPoint_Pad_D2.0mm
Changed lines of the file:
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@@
 			)
 		)
-		(property "Footprint" ""
+		(property "Footprint" "TestPoint:TestPoint_Pad_D2.0mm"
 			(at 132.08 144.78 0)
 			(effects
@@
 			)
 		)
-		(property "Footprint" "Capacitor_Tantalum_SMD:CP_EIA-3528-21_Kemet-B_Pad1.50x2.35mm_HandSolder"
+		(property "Footprint" ""
 			(at 277.8252 132.08 0)
 			(effects
@@
 			)
 		)
-		(property "Footprint" ""
+		(property "Footprint" "TestPoint:TestPoint_Pad_D2.0mm"
 			(at 142.24 119.38 0)
 			(effects

Commit message: Development
Parts:
- C29, C30: footprint Capacitor_SMD:C_1206_3216Metric_Pad1.33x1.80mm_HandSolder -> Capacitor_SMD:C_1210_3225Metric_Pad1.33x2.70mm_HandSolder
- C31: value 22u -> 22u/16V; footprint (none) -> Capacitor_SMD:C_1210_3225Metric_Pad1.33x2.70mm_HandSolder
Changed lines of the file:
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@@
 			)
 		)
-		(property "Footprint" "Capacitor_SMD:C_1206_3216Metric_Pad1.33x1.80mm_HandSolder"
+		(property "Footprint" "Capacitor_SMD:C_1210_3225Metric_Pad1.33x2.70mm_HandSolder"
 			(at 229.5652 132.08 0)
 			(effects
@@
 			)
 		)
-		(property "Footprint" "Capacitor_SMD:C_1206_3216Metric_Pad1.33x1.80mm_HandSolder"
+		(property "Footprint" "Capacitor_SMD:C_1210_3225Metric_Pad1.33x2.70mm_HandSolder"
 			(at 244.8052 132.08 0)
 			(effects
@@
 			)
 		)
-		(property "Value" "22u"
+		(property "Value" "22u/16V"
 			(at 280.67 128.651 0)
 			(effects
@@
 			)
 		)
-		(property "Footprint" ""
+		(property "Footprint" "Capacitor_SMD:C_1210_3225Metric_Pad1.33x2.70mm_HandSolder"
 			(at 277.8252 132.08 0)
 			(effects

Commit message: Development
Parts:
- removed C31: 22u/16V, Capacitor_SMD:C_1210_3225Metric_Pad1.33x2.70mm_HandSolder, symbol Device:C_Polarized
- added C31: 22u/16V, Capacitor_SMD:C_1210_3225Metric_Pad1.33x2.70mm_HandSolder, symbol Device:C
- renumbered D2 to D1, D3 to D2
Connections:
- net +3.3V: now also C31.1
- net GND: now also C31.2
Other:
- moved on the sheet: D1, TP1, TP2

Commit message: Development
Parts:
- removed Q1: FDS9435A, Package_SO:SOIC-8_3.9x4.9mm_P1.27mm, symbol Transistor_FET:FDS9435A
- added Q1: SiS443DN, Package_SO:Vishay_PowerPAK_1212-8_Single, symbol Transistor_FET:SiS443DN
- F1: value 1812L075/33DR -> 3425L300/36MR; footprint Fuse:Fuse_1812_4532Metric_Pad1.30x3.40mm_HandSolder -> (none)
Connections:
- net +24V: now also Q1.1 (S), Q1.2 (S), Q1.3 (S)
- net at D1.1 (A), Q2.3 (C), R12.1: now also Q1.4 (G)
- net at F1.2: now also Q1.5 (D)
Other:
- moved on the sheet: F1
Changed lines of the file:
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@@
 	(wire
 		(pts
-			(xy 165.1 121.92) (xy 172.72 121.92)
+			(xy 162.56 121.92) (xy 172.72 121.92)
 		)
 		(stroke
@@
 	(wire
 		(pts
-			(xy 137.16 121.92) (xy 157.48 121.92)
+			(xy 137.16 121.92) (xy 154.94 121.92)
 		)
 		(stroke
@@
 	(symbol
 		(lib_id "Device:Fuse")
-		(at 161.29 121.92 90)
+		(at 158.75 121.92 90)
 		(unit 1)
 		(exclude_from_sim no)
@@
 		(dnp no)
 		(property "Reference" "F1"
-			(at 161.29 116.205 90)
-			(effects
-				(font
-					(size 1.27 1.27)
-				)
-			)
-		)
-		(property "Value" "1812L075/33DR"
-			(at 161.29 118.745 90)
-			(effects
-				(font
-					(size 1.27 1.27)
-				)
-			)
-		)
-		(property "Footprint" "Fuse:Fuse_1812_4532Metric_Pad1.30x3.40mm_HandSolder"
-			(at 161.29 123.698 90)
-			(effects
-				(font
-					(size 1.27 1.27)
-				)
-				(hide yes)
-			)
-		)
-		(property "Datasheet" "https://www.littelfuse.com/assetdocs/resettable-ptcs-1812l-datasheet?assetguid=ca5c80cb-504e-4a8a-8e74-0107520a1717"
-			(at 161.29 121.92 0)
+			(at 158.75 116.205 90)
+			(effects
+				(font
+					(size 1.27 1.27)
+				)
+			)
+		)
+		(property "Value" "3425L300/36MR"
+			(at 158.75 118.745 90)
+			(effects
+				(font
+					(size 1.27 1.27)
+				)
+			)
+		)
+		(property "Footprint" ""
+			(at 158.75 123.698 90)
+			(effects
+				(font
+					(size 1.27 1.27)
+				)
+				(hide yes)
+			)
+		)
+		(property "Datasheet" "https://www.littelfuse.com/assetdocs/littelfuse-pptc-3425l-datasheet?assetguid=2d6edd27-25e8-4c94-8797-3cc720f26270"
+			(at 158.75 121.92 0)
 			(effects
 				(font
@@
 		)
 		(property "Description" ""
-			(at 161.29 121.92 0)
+			(at 158.75 121.92 0)
 			(effects
 				(font
@@
 				(path "/ca79f0b4-91f7-4537-917d-68d425c03ca3/485861e8-c90d-4c19-b473-548e94ff000e/18da2cad-962d-47df-95e7-fd94fee0a7d8/46440f40-a1d8-4f0c-8c97-f1b8c5865235"
 					(reference "D1")
+					(unit 1)
+				)
+			)
+		)
+	)
+	(symbol
+		(lib_id "Transistor_FET:SiS443DN")
+		(at 177.8 124.46 90)
+		(unit 1)
+		(exclude_from_sim no)
+		(in_bom yes)
+		(on_board yes)
+		(dnp no)
+		(fields_autoplaced yes)
+		(property "Reference" "Q1"
+			(at 177.8 115.57 90)
+			(effects
+				(font
+					(size 1.27 1.27)
+				)
+			)
+		)
+		(property "Value" "SiS443DN"
+			(at 177.8 118.11 90)
+			(effects
+				(font
+					(size 1.27 1.27)
+				)
+			)
+		)
+		(property "Footprint" "Package_SO:Vishay_PowerPAK_1212-8_Single"
+			(at 179.705 119.38 0)
+			(effects
+				(font
+					(size 1.27 1.27)
+					(italic yes)
+				)
+				(justify left)
+				(hide yes)
+			)
+		)
+		(property "Datasheet" "https://www.vishay.com/docs/63253/sis443dn.pdf"
+			(at 181.61 119.38 0)
+			(effects
+				(font
+					(size 1.27 1.27)
+				)
+				(justify left)
+				(hide yes)
+			)
+		)
+		(property "Description" "-35A Id, -40V Vds, P-Channel MOSFET, PowerPAK 1212-8 Single"
+			(at 177.8 124.46 0)
+			(effects
+				(font
+					(size 1.27 1.27)
+				)
+				(hide yes)
+			)
+		)
+		(pin "3"
+		)
+		(pin "1"
+		)
+		(pin "4"
+		)
+		(pin "5"
+		)
+		(pin "2"
+		)
+		(instances
+			(project ""
+				(path "/ca79f0b4-91f7-4537-917d-68d425c03ca3/485861e8-c90d-4c19-b473-548e94ff000e/18da2cad-962d-47df-95e7-fd94fee0a7d8/46440f40-a1d8-4f0c-8c97-f1b8c5865235"
+					(reference "Q1")
 					(unit 1)
 				)
@@
 					(unit 1)
 				)
-			)
-		)
-	)
-	(symbol
-		(lib_id "Transistor_FET:FDS9435A")
-		(at 177.8 124.46 90)
-		(unit 1)
-		(exclude_from_sim no)
-		(in_bom yes)
-		(on_board yes)
-		(dnp no)
-		(fields_autoplaced yes)
-		(property "Reference" "Q1"
-			(at 177.8 115.57 90)
-			(effects
-				(font
-					(size 1.27 1.27)
-				)
-			)
-		)
-		(property "Value" "FDS9435A"
-			(at 177.8 118.11 90)
-			(effects
-				(font
-					(size 1.27 1.27)
-				)
-			)
-		)
-		(property "Footprint" "Package_SO:SOIC-8_3.9x4.9mm_P1.27mm"
-			(at 179.705 119.38 0)
-			(effects
-				(font
-					(size 1.27 1.27)
-					(italic yes)
-				)
-				(justify left)
-				(hide yes)
-			)
-		)
-		(property "Datasheet" "https://www.onsemi.com/pub/Collateral/FDS9435A-D.PDF"
-			(at 181.61 119.38 0)
-			(effects
-				(font
-					(size 1.27 1.27)
-				)
-				(justify left)
-				(hide yes)
-			)
-		)
-		(property "Description" "-5.3A Id, -30V Vds, P-Channel MOSFET, 50mOhm Ron, SO-8"
-			(at 177.8 124.46 0)
-			(effects
-				(font
-					(size 1.27 1.27)
-				)
-				(hide yes)
-			)
-		)
-		(pin "4"
-		)
-		(pin "7"
-		)
-		(pin "6"
-		)
-		(pin "5"
-		)
-		(pin "8"
-		)
-		(pin "3"
-		)
-		(pin "2"
-		)
-		(pin "1"
-		)
-		(instances
-			(project ""
-				(path "/ca79f0b4-91f7-4537-917d-68d425c03ca3/485861e8-c90d-4c19-b473-548e94ff000e/18da2cad-962d-47df-95e7-fd94fee0a7d8/46440f40-a1d8-4f0c-8c97-f1b8c5865235"
-					(reference "Q1")
-					(unit 1)
-				)

Commit message: Development
Parts:
- C29: value 10u/50V -> 10u/100V
- C30: value 4u7/50V -> 4u7/100V
- F1: value 3425L300/36MR -> MF-GSMF300/36X-2; footprint (none) -> ETH1CVOLT_A:MF-GSMF
- J3: value 1715721 -> CONN; footprint TerminalBlock_Phoenix:TerminalBlock_Phoenix_MKDS-1,5-2_1x02_P5.00mm_Horizontal -> Connector_Phoenix_MC:PhoenixContact_MC_1,5_2-GF-3.81_1x02_P3.81mm_Horizontal_ThreadedFlange_MountHole
- TP1, TP2: now left out of the parts list
Other:
- moved on the sheet: C30, C31, F1, J3, TP1, U4

Commit message: Hardware development
Parts:
- J3: value CONN -> 1843790; footprint Connector_Phoenix_MC:PhoenixContact_MC_1,5_2-GF-3.81_1x02_P3.81mm_Horizontal_ThreadedFlange_MountHole -> Connector_Phoenix_MC:PhoenixContact_MC_1,5_2-GF-3.5_1x02_P3.50mm_Horizontal_ThreadedFlange
- renumbered D2 to D1, D1 to D2, R13 to R12, R12 to R13
Other:
- moved on the sheet: C29, C30, C31
Changed lines of the file:
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@@
 	(wire
 		(pts
-			(xy 228.6 121.92) (xy 228.6 124.46)
+			(xy 228.6 121.92) (xy 228.6 125.73)
 		)
 		(stroke
@@
 	(wire
 		(pts
-			(xy 245.11 132.08) (xy 245.11 144.78)
+			(xy 245.11 133.35) (xy 245.11 144.78)
 		)
 		(stroke
@@
 	(wire
 		(pts
-			(xy 281.94 124.46) (xy 281.94 121.92)
+			(xy 281.94 125.73) (xy 281.94 121.92)
 		)
 		(stroke
@@
 	(wire
 		(pts
-			(xy 228.6 132.08) (xy 228.6 144.78)
-		)
-		(stroke
-			(width 0)
-			(type default)
-		)
-	)
-	(wire
-		(pts
-			(xy 245.11 121.92) (xy 245.11 124.46)
+			(xy 228.6 133.35) (xy 228.6 144.78)
+		)
+		(stroke
+			(width 0)
+			(type default)
+		)
+	)
+	(wire
+		(pts
+			(xy 245.11 121.92) (xy 245.11 125.73)
 		)
 		(stroke
@@
 	(wire
 		(pts
-			(xy 281.94 144.78) (xy 281.94 132.08)
+			(xy 281.94 144.78) (xy 281.94 133.35)
 		)
 		(stroke
@@
 			)
 		)
-		(property "Component Class" "DIR"
+		(property "Component Class" ""
 			(at -603.25 -135.89 0)
 			(effects
@@
 		(dnp no)
 		(fields_autoplaced yes)
-		(property "Reference" "#PWR053"
+		(property "Reference" "#PWR052"
 			(at 228.6 124.46 0)
 			(effects
@@
 			(project ""
 				(path "/ca79f0b4-91f7-4537-917d-68d425c03ca3/485861e8-c90d-4c19-b473-548e94ff000e/18da2cad-962d-47df-95e7-fd94fee0a7d8/46440f40-a1d8-4f0c-8c97-f1b8c5865235"
-					(reference "#PWR053")
+					(reference "#PWR052")
 					(unit 1)
 				)
@@
 	(symbol
 		(lib_id "Device:C")
-		(at 228.6 128.27 0)
+		(at 228.6 129.54 0)
 		(unit 1)
 		(exclude_from_sim no)
@@
 		(dnp no)
 		(property "Reference" "C29"
-			(at 231.775 127 0)
+			(at 231.775 128.27 0)
 			(effects
 				(font
@@
 		)
 		(property "Value" "10u/100V"
-			(at 231.775 129.54 0)
+			(at 231.775 130.81 0)
 			(effects
 				(font
@@
 		)
 		(property "Footprint" "Capacitor_SMD:C_1210_3225Metric_Pad1.33x2.70mm_HandSolder"
-			(at 229.5652 132.08 0)
+			(at 229.5652 133.35 0)
 			(effects
 				(font
@@
 		)
 		(property "Datasheet" "~"
-			(at 228.6 128.27 0)
+			(at 228.6 129.54 0)
 			(effects
 				(font
@@
 		)
 		(property "Description" ""
-			(at 228.6 128.27 0)
+			(at 228.6 129.54 0)
 			(effects
 				(font
@@
 		(dnp no)
 		(fields_autoplaced yes)
-		(property "Reference" "R12"
+		(property "Reference" "R13"
 			(at 180.34 139.7 0)
 			(effects
@@
 			(project "ETH1CVOLT_A"
 				(path "/ca79f0b4-91f7-4537-917d-68d425c03ca3/485861e8-c90d-4c19-b473-548e94ff000e/18da2cad-962d-47df-95e7-fd94fee0a7d8/46440f40-a1d8-4f0c-8c97-f1b8c5865235"
-					(reference "R12")
+					(reference "R13")
 					(unit 1)
 				)
@@
 		(on_board yes)
 		(dnp no)
-		(property "Reference" "D1"
+		(property "Reference" "D2"
 			(at 186.69 128.27 90)
 			(effects
@@
 			(project "ETH1CVOLT_A"
 				(path "/ca79f0b4-91f7-4537-917d-68d425c03ca3/485861e8-c90d-4c19-b473-548e94ff000e/18da2cad-962d-47df-95e7-fd94fee0a7d8/46440f40-a1d8-4f0c-8c97-f1b8c5865235"
-					(reference "D1")
+					(reference "D2")
 					(unit 1)
 				)
@@
 		(dnp no)
 		(fields_autoplaced yes)
-		(property "Reference" "#PWR054"
+		(property "Reference" "#PWR053"
 			(at 281.94 124.46 0)
 			(effects
@@
 			(project "ETH1CVOLT_A"
 				(path "/ca79f0b4-91f7-4537-917d-68d425c03ca3/485861e8-c90d-4c19-b473-548e94ff000e/18da2cad-962d-47df-95e7-fd94fee0a7d8/46440f40-a1d8-4f0c-8c97-f1b8c5865235"
-					(reference "#PWR054")
+					(reference "#PWR053")
 					(unit 1)
 				)
@@
 		(dnp no)
 		(fields_autoplaced yes)
-		(property "Reference" "#FLG06"
+		(property "Reference" "#FLG07"
 			(at 245.11 149.225 0)
 			(effects
@@
 			(project "ETH1CVOLT_A"
 				(path "/ca79f0b4-91f7-4537-917d-68d425c03ca3/485861e8-c90d-4c19-b473-548e94ff000e/18da2cad-962d-47df-95e7-fd94fee0a7d8/46440f40-a1d8-4f0c-8c97-f1b8c5865235"
-					(reference "#FLG06")
+					(reference "#FLG07")
 					(unit 1)
 				)
@@
 	(symbol
 		(lib_id "Device:C")
-		(at 245.11 128.27 0)
+		(at 245.11 129.54 0)
 		(unit 1)
 		(exclude_from_sim no)
@@
 		(fields_autoplaced yes)
 		(property "Reference" "C30"
-			(at 248.92 126.9999 0)
+			(at 248.92 128.2699 0)
 			(effects
 				(font
@@
 		)
 		(property "Value" "4u7/100V"
-			(at 248.92 129.5399 0)
+			(at 248.92 130.8099 0)
 			(effects
 				(font
@@
 		)
 		(property "Footprint" "Capacitor_SMD:C_1210_3225Metric_Pad1.33x2.70mm_HandSolder"
-			(at 246.0752 132.08 0)
+			(at 246.0752 133.35 0)
 			(effects
 				(font
@@
 		)
 		(property "Datasheet" "~"
-			(at 245.11 128.27 0)
+			(at 245.11 129.54 0)
 			(effects
 				(font
@@
 		)
 		(property "Description" ""
-			(at 245.11 128.27 0)
+			(at 245.11 129.54 0)
 			(effects
 				(font
@@
 		(dnp no)
 		(fields_autoplaced yes)
-		(property "Reference" "R13"
+		(property "Reference" "R12"
 			(at 213.36 134.62 0)
 			(effects
@@
 			(project "ETH1CVOLT_A"
 				(path "/ca79f0b4-91f7-4537-917d-68d425c03ca3/485861e8-c90d-4c19-b473-548e94ff000e/18da2cad-962d-47df-95e7-fd94fee0a7d8/46440f40-a1d8-4f0c-8c97-f1b8c5865235"
-					(reference "R13")
+					(reference "R12")
 					(unit 1)
 				)
@@
 			)
 		)
-		(property "Value" "CONN"
+		(property "Value" "1843790"
 			(at 121.92 125.73 0)
 			(effects
@@
 			)
 		)
-		(property "Footprint" "Connector_Phoenix_MC:PhoenixContact_MC_1,5_2-GF-3.81_1x02_P3.81mm_Horizontal_ThreadedFlange_MountHole"
+		(property "Footprint" "Connector_Phoenix_MC:PhoenixContact_MC_1,5_2-GF-3.5_1x02_P3.50mm_Horizontal_ThreadedFlange"
 			(at 121.92 129.54 0)
 			(effects
@@
 	(symbol
 		(lib_id "Device:C")
-		(at 281.94 128.27 0)
+		(at 281.94 129.54 0)
 		(unit 1)
 		(exclude_from_sim no)
@@
 		(fields_autoplaced yes)
 		(property "Reference" "C31"
-			(at 285.75 126.9999 0)
+			(at 285.75 128.2699 0)
 			(effects
 				(font
@@
 		)
 		(property "Value" "22u/16V"
-			(at 285.75 129.5399 0)
+			(at 285.75 130.8099 0)
 			(effects
 				(font
@@
 		)
 		(property "Footprint" "Capacitor_SMD:C_1210_3225Metric_Pad1.33x2.70mm_HandSolder"
-			(at 282.9052 132.08 0)
+			(at 282.9052 133.35 0)
 			(effects
 				(font
@@
 		)
 		(property "Datasheet" "~"
-			(at 281.94 128.27 0)
+			(at 281.94 129.54 0)
 			(effects
 				(font
@@
 		)
 		(property "Description" "Unpolarized capacitor"
-			(at 281.94 128.27 0)
+			(at 281.94 129.54 0)
 			(effects
 				(font
@@
 		(dnp no)
 		(fields_autoplaced yes)
-		(property "Reference" "#PWR052"
+		(property "Reference" "#PWR054"
 			(at 129.54 152.4 0)
 			(effects
@@
 			(project "ETH1CVOLT_A"
 				(path "/ca79f0b4-91f7-4537-917d-68d425c03ca3/485861e8-c90d-4c19-b473-548e94ff000e/18da2cad-962d-47df-95e7-fd94fee0a7d8/46440f40-a1d8-4f0c-8c97-f1b8c5865235"
-					(reference "#PWR052")
+					(reference "#PWR054")
 					(unit 1)
 				)
@@
 		(dnp no)
 		(fields_autoplaced yes)
-		(property "Reference" "#FLG05"
+		(property "Reference" "#FLG06"
 			(at 245.11 118.745 0)
 			(effects
@@
 			(project "ETH1CVOLT_A"
 				(path "/ca79f0b4-91f7-4537-917d-68d425c03ca3/485861e8-c90d-4c19-b473-548e94ff000e/18da2cad-962d-47df-95e7-fd94fee0a7d8/46440f40-a1d8-4f0c-8c97-f1b8c5865235"
-					(reference "#FLG05")
+					(reference "#FLG06")
 					(unit 1)
 				)
@@
 		(on_board yes)
 		(dnp no)
-		(property "Reference" "D2"
+		(property "Reference" "D1"
 			(at 213.36 124.46 90)
 			(effects
@@
 			(project "ETH1CVOLT_A"
 				(path "/ca79f0b4-91f7-4537-917d-68d425c03ca3/485861e8-c90d-4c19-b473-548e94ff000e/18da2cad-962d-47df-95e7-fd94fee0a7d8/46440f40-a1d8-4f0c-8c97-f1b8c5865235"
-					(reference "D2")
-					(unit 1)
-				)
+					(reference "D1")
+					(unit 1)
+				)
