File: HARDWARE/ETH1CVOLT_A/ETH1CVOLT_A.kicad_pcb (KiCad board)
At the start: 2 copper layers, 160 x 100 mm, 232 parts, among them J1 20021111-00010T4LF, J10 FCR7350B, J11 Conn_02x04_Odd_Even, J12 Conn_02x05_Odd_Even, J2 RJ45_Wuerth_7499010121A, J3 1715721, J5 FCR7350B, J6 FCR7350R, J7 Conn_02x04_Odd_Even, J8 Conn_02x05_Odd_Even, J9 FCR7350R, K1 EE2-3NU, K2 EE2-3NU, Q1 FDS9435A, Q2 MMBT3904, Q4 MMBT3904, Q5 MMBT3904, T1 750319331, T2 750319331, T3 750319331, U1 STM32H743VITx, U10 TSR0.5-2490, U11 LT8330_S6, U12 LT8330_S6, U13 LT8365, U14 LT8365, U15 TPS7A39, U16 ADP7142ARDZ-5.0, U17 ADP7142ARDZ-3.3, U18 ISO7763DW, U19 ISO7763DW, U2 24LC08B-E/MS, U3 LAN8742A, U4 TSR1-2433E, U5 UCC25800-Q1, U6 UCC25800-Q1, U7 UCC25800-Q1, U8 LT8330_S6, U9 LT8330_S6, Y1 NX5032GA-16, Y2 NX5032GA-25

Commit message: Development
Parts:
- removed U19: ISO7763DW, Package_SO:SOIC-16W_7.5x10.3mm_P1.27mm
- added C108: 0.22u/200V, Capacitor_SMD:C_1210_3225Metric_Pad1.33x2.70mm_HandSolder, F.Cu at (183.3, 17.9)
- added C109: 0.22u/200V, Capacitor_SMD:C_1210_3225Metric_Pad1.33x2.70mm_HandSolder, F.Cu at (183.3, 22.2)
- added C110: 0.22u/200V, Capacitor_SMD:C_1210_3225Metric_Pad1.33x2.70mm_HandSolder, F.Cu at (183.3, 26.4)
- added C111: 0.22u/200V, Capacitor_SMD:C_1210_3225Metric_Pad1.33x2.70mm_HandSolder, F.Cu at (183.3, 30.7)
- added C114: AEF08124R7M400R, Capacitor_SMD:CP_Elec_8x11.9, F.Cu at (179.6, 52.7)
- added C115: AEF08124R7M400R, Capacitor_SMD:CP_Elec_8x11.9, F.Cu at (165.4, 52.7)
- added C116: AEK0812100M250R, Capacitor_SMD:CP_Elec_8x11.9, F.Cu at (148.6, 65.5)
- added C117: AEK0812100M250R, Capacitor_SMD:CP_Elec_8x11.9, F.Cu at (148.6, 75.4)
- added C118: 10u/50V, Capacitor_SMD:C_1210_3225Metric_Pad1.33x2.70mm_HandSolder, F.Cu at (119.3, -8.86)
- added C119: 4u7/50V, Capacitor_SMD:C_1210_3225Metric_Pad1.33x2.70mm_HandSolder, F.Cu at (119.3, -4.61)
- added C120: 10u/50V, Capacitor_SMD:C_1210_3225Metric_Pad1.33x2.70mm_HandSolder, F.Cu at (125.3, -21.6)
- added C121: 100u/16V, Capacitor_SMD:C_1210_3225Metric_Pad1.33x2.70mm_HandSolder, F.Cu at (50.6, 49.8)
- added C123: 4u7/50V, Capacitor_SMD:C_1210_3225Metric_Pad1.33x2.70mm_HandSolder, F.Cu at (125.3, -17.4)
- added C124: 10u/50V, Capacitor_SMD:C_1210_3225Metric_Pad1.33x2.70mm_HandSolder, F.Cu at (125.3, -13.1)
- added C126: 4u7/50V, Capacitor_SMD:C_1210_3225Metric_Pad1.33x2.70mm_HandSolder, F.Cu at (125.3, -8.86)
- added C127: 10u/50V, Capacitor_SMD:C_1210_3225Metric_Pad1.33x2.70mm_HandSolder, F.Cu at (125.3, -4.61)
- added C128: C, Capacitor_SMD:C_0603_1608Metric_Pad1.08x0.95mm_HandSolder, F.Cu at (162.1, 130.1)
- added C31: 22u/16V, Capacitor_SMD:C_1210_3225Metric_Pad1.33x2.70mm_HandSolder, F.Cu at (50.6, 43.5)
- added C32: 4u7/50V, Capacitor_SMD:C_1210_3225Metric_Pad1.33x2.70mm_HandSolder, F.Cu at (115.3, 1.64)
- added C33: 10u/50V, Capacitor_SMD:C_1210_3225Metric_Pad1.33x2.70mm_HandSolder, F.Cu at (115.3, 5.89)
- added C35: 2u2/50V, Capacitor_SMD:C_1206_3216Metric_Pad1.33x1.80mm_HandSolder, F.Cu at (121.3, 1.19)
- added C36: 2u2/50V, Capacitor_SMD:C_1206_3216Metric_Pad1.33x1.80mm_HandSolder, F.Cu at (121.3, 4.54)
- added C37: 2u2/50V, Capacitor_SMD:C_1206_3216Metric_Pad1.33x1.80mm_HandSolder, F.Cu at (121.3, 7.89)
- added C40: 10u/50V, Capacitor_SMD:C_1210_3225Metric_Pad1.33x2.70mm_HandSolder, F.Cu at (115.3, 10.1)
- added C41: 4u7/50V, Capacitor_SMD:C_1210_3225Metric_Pad1.33x2.70mm_HandSolder, F.Cu at (115.3, 14.4)
- added C42: 4u7/50V, Capacitor_SMD:C_1210_3225Metric_Pad1.33x2.70mm_HandSolder, F.Cu at (129.3, 1.64)
- added C43: 10u/50V, Capacitor_SMD:C_1210_3225Metric_Pad1.33x2.70mm_HandSolder, F.Cu at (129.3, 5.89)
- added C45: 2u2/50V, Capacitor_SMD:C_1206_3216Metric_Pad1.33x1.80mm_HandSolder, F.Cu at (135.3, 1.19)
- added C46: 2u2/50V, Capacitor_SMD:C_1206_3216Metric_Pad1.33x1.80mm_HandSolder, F.Cu at (135.3, 4.54)
- added C47: 2u2/50V, Capacitor_SMD:C_1206_3216Metric_Pad1.33x1.80mm_HandSolder, F.Cu at (135.3, 7.89)
- added C50: 10u/50V, Capacitor_SMD:C_1210_3225Metric_Pad1.33x2.70mm_HandSolder, F.Cu at (129.3, 10.1)
- added C51: 4u7/50V, Capacitor_SMD:C_1210_3225Metric_Pad1.33x2.70mm_HandSolder, F.Cu at (129.3, 14.4)
- added C52: 4u7/50V, Capacitor_SMD:C_1210_3225Metric_Pad1.33x2.70mm_HandSolder, F.Cu at (133.3, -21.6)
- added C53: 10u/50V, Capacitor_SMD:C_1210_3225Metric_Pad1.33x2.70mm_HandSolder, F.Cu at (133.3, -17.4)
- added C55: 2u2/50V, Capacitor_SMD:C_1206_3216Metric_Pad1.33x1.80mm_HandSolder, F.Cu at (139.3, -22.1)
- added C56: 2u2/50V, Capacitor_SMD:C_1206_3216Metric_Pad1.33x1.80mm_HandSolder, F.Cu at (139.3, -18.7)
- added C57: 2u2/50V, Capacitor_SMD:C_1206_3216Metric_Pad1.33x1.80mm_HandSolder, F.Cu at (139.3, -15.4)
- added C60: 10u/50V, Capacitor_SMD:C_1210_3225Metric_Pad1.33x2.70mm_HandSolder, F.Cu at (133.3, -13.1)
- added C61: 4u7/50V, Capacitor_SMD:C_1210_3225Metric_Pad1.33x2.70mm_HandSolder, F.Cu at (133.3, -8.86)
- added C62: 4u7/50V, Capacitor_SMD:C_1210_3225Metric_Pad1.33x2.70mm_HandSolder, F.Cu at (107.3, 1.64)
- added C63: 4u7/50V, Capacitor_SMD:C_1210_3225Metric_Pad1.33x2.70mm_HandSolder, F.Cu at (107.3, 5.89)
- added C64: 10u/50V, Capacitor_SMD:C_1210_3225Metric_Pad1.33x2.70mm_HandSolder, F.Cu at (107.3, 10.1)
- added C65: 10u/50V, Capacitor_SMD:C_1210_3225Metric_Pad1.33x2.70mm_HandSolder, F.Cu at (107.3, 14.4)
- added C71: 4u7/100V, Capacitor_SMD:C_1210_3225Metric_Pad1.33x2.70mm_HandSolder, F.Cu at (107.3, 18.6)
- added C72: 4u7/100V, Capacitor_SMD:C_1210_3225Metric_Pad1.33x2.70mm_HandSolder, F.Cu at (107.3, 22.9)
- added C73: 10u/100V, Capacitor_SMD:C_1210_3225Metric_Pad1.33x2.70mm_HandSolder, F.Cu at (107.3, 27.1)
- added C74: 10u/100V, Capacitor_SMD:C_1210_3225Metric_Pad1.33x2.70mm_HandSolder, F.Cu at (107.3, 32.4)
- added C75: 4u7/50V, Capacitor_SMD:C_1210_3225Metric_Pad1.33x2.70mm_HandSolder, F.Cu at (107.3, -21.6)
- added C76: 10u/50V, Capacitor_SMD:C_1210_3225Metric_Pad1.33x2.70mm_HandSolder, F.Cu at (107.3, -17.4)
- added C77: 4u7/50V, Capacitor_SMD:C_1210_3225Metric_Pad1.33x2.70mm_HandSolder, F.Cu at (107.3, -13.1)
- added C78: 10u/50V, Capacitor_SMD:C_1210_3225Metric_Pad1.33x2.70mm_HandSolder, F.Cu at (107.3, -8.86)
- added C79: 4u7/50V, Capacitor_SMD:C_1210_3225Metric_Pad1.33x2.70mm_HandSolder, F.Cu at (107.3, -4.61)
- added C80: 4u7/50V, Capacitor_SMD:C_1210_3225Metric_Pad1.33x2.70mm_HandSolder, F.Cu at (113.3, -21.6)
- added C81: 4u7/50V, Capacitor_SMD:C_1210_3225Metric_Pad1.33x2.70mm_HandSolder, F.Cu at (113.3, -17.4)
- added C82: 10u/50V, Capacitor_SMD:C_1210_3225Metric_Pad1.33x2.70mm_HandSolder, F.Cu at (113.3, -13.1)
- added C83: 10u/50V, Capacitor_SMD:C_1210_3225Metric_Pad1.33x2.70mm_HandSolder, F.Cu at (113.3, -8.86)
- added C90: 4u7/50V, Capacitor_SMD:C_1210_3225Metric_Pad1.33x2.70mm_HandSolder, F.Cu at (113.3, -4.61)
- added C91: 4u7/50V, Capacitor_SMD:C_1210_3225Metric_Pad1.33x2.70mm_HandSolder, F.Cu at (119.3, -21.6)
- added C92: 10u/50V, Capacitor_SMD:C_1210_3225Metric_Pad1.33x2.70mm_HandSolder, F.Cu at (119.3, -17.4)
- added C93: 10u/50V, Capacitor_SMD:C_1210_3225Metric_Pad1.33x2.70mm_HandSolder, F.Cu at (119.3, -13.1)
- added C94: 4u7/50V, Capacitor_SMD:C_1210_3225Metric_Pad1.33x2.70mm_HandSolder, F.Cu at (143.3, 1.64)
- added C95: 4u7/50V, Capacitor_SMD:C_1210_3225Metric_Pad1.33x2.70mm_HandSolder, F.Cu at (143.3, 5.89)
- added C96: 10u/50V, Capacitor_SMD:C_1210_3225Metric_Pad1.33x2.70mm_HandSolder, F.Cu at (143.3, 10.1)
- added C97: 10u/50V, Capacitor_SMD:C_1210_3225Metric_Pad1.33x2.70mm_HandSolder, F.Cu at (143.3, 14.4)
- added J13: Conn_02x04_Odd_Even, Connector_PinSocket_2.54mm:PinSocket_2x04_P2.54mm_Vertical_SMD, F.Cu at (138.4, 118.7)
- added J4: Conn_02x04_Odd_Even, Connector_PinSocket_2.54mm:PinSocket_2x04_P2.54mm_Vertical_SMD, F.Cu at (138.6, 131.6)
- added Q6: FZT849, Package_TO_SOT_SMD:SOT-223-3_TabPin2, F.Cu at (97.0, 109.4)
- added U20: ISO7761DW, Package_SO:SOIC-16W_7.5x10.3mm_P1.27mm, F.Cu at (123.4, 120.4)
- C102, C103, C106, C107, C112, C113: value 0.1u -> 0.1u/200V; footprint Capacitor_SMD:C_0603_1608Metric_Pad1.08x0.95mm_HandSolder -> Capacitor_SMD:C_1210_3225Metric_Pad1.33x2.70mm_HandSolder
- C29, C30: footprint Capacitor_SMD:C_1206_3216Metric_Pad1.33x1.80mm_HandSolder -> Capacitor_SMD:C_1210_3225Metric_Pad1.33x2.70mm_HandSolder
- C38, C39, C48, C49, C58, C59: value 56n -> 56n/50V
- C68: value 1u -> 1u/100V; footprint Capacitor_SMD:C_0603_1608Metric_Pad1.08x0.95mm_HandSolder -> Capacitor_SMD:C_0805_2012Metric_Pad1.18x1.45mm_HandSolder
- C86, C87: value 1u -> 1u/50V; footprint Capacitor_SMD:C_0603_1608Metric_Pad1.08x0.95mm_HandSolder -> Capacitor_SMD:C_0805_2012Metric_Pad1.18x1.45mm_HandSolder
- D19: value DFLS1150 -> DFLS1200
- R59, R60, R61, R62: value 20 -> 20/200V
- R63, R64: value 47 -> 47/200V
- R65, R66, R68, R69: value 499k -> 499k/100V
- R76: value R -> 499
- U11, U12, U8, U9: footprint Package_TO_SOT_SMD:TSOT-23-6_HandSoldering -> Package_TO_SOT_SMD:TSOT-23-6
- moved D10 104.9 mm to (204.4, 32.9)
- moved D11 104.9 mm to (204.4, 36.9)
- moved U8 104.9 mm to (197.2, 33.2)
- moved U9 104.9 mm to (197.2, 37.8)
- moved J11 29.2 mm to (123.4, 107.1)
- moved U11 0.66 mm to (132.4, 61.5)
Connections:
- U1 pad 16: /Block Diagram/MCU/RMII_MDC -> /Block Diagram/Ethernet/RMII_MDC
- U1 pad 23: /Block Diagram/MCU/REF_CLK -> /Block Diagram/Ethernet/REF_CLK
- U1 pad 24: /Block Diagram/MCU/RMII_MDIO -> /Block Diagram/Ethernet/RMII_MDIO
- U1 pad 31: /Block Diagram/MCU/RMII_CRS_DV -> /Block Diagram/Ethernet/RMII_CRS_DV
- U1 pad 32: /Block Diagram/MCU/RMII_RXD0 -> /Block Diagram/Ethernet/RMII_RXD0
- U1 pad 33: /Block Diagram/MCU/RMII_RXD1 -> /Block Diagram/Ethernet/RMII_RXD1
- U1 pad 47: /Block Diagram/MCU/RMII_TXEN -> /Block Diagram/Ethernet/RMII_TXEN
- U1 pad 51: /Block Diagram/MCU/RMII_TXD0 -> /Block Diagram/Ethernet/RMII_TXD0
- U1 pad 52: /Block Diagram/MCU/RMII_TXD1 -> /Block Diagram/Ethernet/RMII_TXD1
- U15 pad 3: unconnected-(U15-NR/SS-Pad3) -> Net-(U15-NR/SS)
- U18 pad 1: unconnected-(U18-Vcc1-Pad1) -> +3.3V
- U18 pad 10: unconnected-(U18-INF-Pad10) -> /Block Diagram/Isolation IO/DAC2_~{FAULT}_ISO
- U18 pad 11: unconnected-(U18-INE-Pad11) -> /Block Diagram/Isolation IO/DAC1_~{FAULT}_ISO
- U18 pad 12: unconnected-(U18-IND-Pad12) -> /Block Diagram/Isolation IO/SPI1_MISO_ISO
- U18 pad 13: unconnected-(U18-OUTC-Pad13) -> /Block Diagram/Isolation IO/SPI1_~{CS}_ISO
- U18 pad 14: unconnected-(U18-OUTB-Pad14) -> /Block Diagram/Isolation IO/SPI1_MOSI_ISO
- U18 pad 15: unconnected-(U18-OUTA-Pad15) -> /Block Diagram/Isolation IO/SPI1_SCK_ISO
- U18 pad 16: unconnected-(U18-Vcc2-Pad16) -> +3V3_ISO
- U18 pad 2: unconnected-(U18-INA-Pad2) -> /Block Diagram/Isolation IO/SPI1_SCK
- U18 pad 3: unconnected-(U18-INB-Pad3) -> /Block Diagram/Isolation IO/SPI1_MOSI
- U18 pad 4: unconnected-(U18-INC-Pad4) -> /Block Diagram/Isolation IO/SPI1_~{CS}
- U18 pad 5: unconnected-(U18-OUTD-Pad5) -> /Block Diagram/Isolation IO/SPI1_MISO
- U18 pad 6: unconnected-(U18-OUTE-Pad6) -> /Block Diagram/Isolation IO/DAC1_~{FAULT}
- U18 pad 7: unconnected-(U18-OUTF-Pad7) -> /Block Diagram/Isolation IO/DAC2_~{FAULT}
- U18 pad 8: unconnected-(U18-GND1-Pad8) -> GND
- U18 pad 9: unconnected-(U18-GND2-Pad9) -> GND_ISO
- U3 pad 15: /Block Diagram/Ethernet/NRST -> /Block Diagram/MCU/NRST

Commit message: Development
Parts:
- removed the D1 at (172.4, 122.0)
- removed the RN1 at (124.3, 70.2)
- added D23: 1N4148W, Diode_SMD:D_SOD-123, F.Cu at (131.3, 24.2)
- added K3: EE2-3NU, Relay_SMD:Relay_DPDT_Kemet_EE2_NU, F.Cu at (141.8, 28.3)
- added R85: 4k7/2W, Resistor_SMD:R_2512_6332Metric_Pad1.40x3.35mm_HandSolder, F.Cu at (133.0, 30.1)
- added R86: 4k7/2W, Resistor_SMD:R_2512_6332Metric_Pad1.40x3.35mm_HandSolder, F.Cu at (150.0, 30.1)
- moved Y1 148.4 mm to (18.2, 89.3)
- moved Y2 148.4 mm to (18.2, 82.7)
- moved C72 133.2 mm to (22.6, 125.8)
- moved C73 133.2 mm to (22.6, 130.0)
- moved C74 133.2 mm to (22.6, 135.3)
- moved C100 98.9 mm to (28.4, 34.5)
- moved C101 98.9 mm to (28.4, 30.2)
- moved C76 98.9 mm to (22.4, 17.5)
- moved C77 98.9 mm to (22.4, 21.8)
- moved C79 98.9 mm to (22.4, 26.0)
- moved C80 98.9 mm to (22.4, 30.2)
- moved C90 98.9 mm to (22.4, 34.5)
- moved C91 98.9 mm to (28.4, 17.5)
- moved C93 98.9 mm to (28.4, 21.8)
- moved C94 98.9 mm to (28.4, 26.0)
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- renumbered C119 to C100, C118 to C101, C120 to C102, C126 to C103, C127 to C104, C94 to C105, C95 to C106, C96 to C107, C97 to C108, C98 to C109, C99 to C110, C100 to C111, C101 to C112, C102 to C113, C103 to C114, C104 to C115, C105 to C116, C106 to C117, C107 to C118, C108 to C119, C109 to C120, C110 to C121, C111 to C122, C112 to C123, C113 to C124, C114 to C125, C115 to C126, C116 to C127, C117 to C128, C80 to C76, C81 to C77, C76 to C78, C82 to C79, C83 to C80, C77 to C81, C84 to C82, C85 to C83, C78 to C84, C86 to C85, C87 to C86, C121 to C87, C92 to C93, C93 to C94, C128 to C95, C123 to C96, C124 to C97, C79 to C99, D2 to D1, D11 to D10, D12 to D11, D13 to D12, D14 to D13, D15 to D14, D16 to D15, D17 to D16, D18 to D17, D19 to D18, D20 to D19, D3 to D2, D21 to D20, D22 to D21, D23 to D22, D4 to D3, D5 to D4, D6 to D5, D7 to D6, D8 to D7, D9 to D8, D10 to D9, H3 to H2, H2 to H3, J8 to J11, J4 to J12, J11 to J4, J7 to J5, J12 to J6, J6 to J7, J5 to J8, Q6 to Q3, R42 to R41, R43 to R42, R44 to R43, R45 to R44, R76 to R45, R77 to R46, R46 to R48, R47 to R49, R48 to R50, R49 to R51, R50 to R52, R80 to R54, R72 to R55, R73 to R56, R75 to R57, R41 to R58, R74 to R59, R71 to R60, R82 to R62, R51 to R63, R52 to R64, R53 to R65, R54 to R66, R55 to R67, R56 to R68, R57 to R69, R58 to R70, R59 to R71, R60 to R72, R61 to R73, R62 to R74, R63 to R75, R64 to R76, R83 to R77, R84 to R78, R65 to R79, R66 to R80, R67 to R81, R68 to R82, R69 to R83, R70 to R84, RN2 to RN1, RN3 to RN2, RN4 to RN3, U16 to U13, U15 to U14, U17 to U15, U13 to U16, U14 to U17, U20 to U19
Connections:
- C39 pad 2: /Block Diagram/Power/Power Isolated/UCC25800_1/GND_ISO -> GND_ISO
- C40 pad 2: /Block Diagram/Power/Power Isolated/UCC25800_1/GND_ISO -> GND_ISO
- C41 pad 2: /Block Diagram/Power/Power Isolated/UCC25800_1/GND_ISO -> GND_ISO
- C49 pad 2: /Block Diagram/Power/Power Isolated/UCC25800_2/GND_ISO -> GND_ISO
- C50 pad 2: /Block Diagram/Power/Power Isolated/UCC25800_2/GND_ISO -> GND_ISO
- C51 pad 2: /Block Diagram/Power/Power Isolated/UCC25800_2/GND_ISO -> GND_ISO
- C59 pad 2: /Block Diagram/Power/Power Isolated/UCC25800_3/GND_ISO -> GND_ISO
- C60 pad 2: /Block Diagram/Power/Power Isolated/UCC25800_3/GND_ISO -> GND_ISO
- C61 pad 2: /Block Diagram/Power/Power Isolated/UCC25800_3/GND_ISO -> GND_ISO
- D4 pad 2: /Block Diagram/Power/Power Isolated/UCC25800_1/GND_ISO -> GND_ISO
- D6 pad 2: /Block Diagram/Power/Power Isolated/UCC25800_2/GND_ISO -> GND_ISO
- D8 pad 2: /Block Diagram/Power/Power Isolated/UCC25800_3/GND_ISO -> GND_ISO
- U1 pad 63: /Block Diagram/MCU/LED_BLUE -> unconnected-(U1-PC6-Pad63)
- U1 pad 64: /Block Diagram/MCU/LED_RED -> unconnected-(U1-PC7-Pad64)
- U1 pad 65: /Block Diagram/MCU/LED_GREEN -> unconnected-(U1-PC8-Pad65)

Commit message: Development
Parts:
- removed the C103 at (34.4, 30.2)
- removed the C104 at (34.4, 34.5)
- removed the C87 at (47.8, 104.5)
- removed the C96 at (34.4, 21.8)
- removed the Q3 at (111.0, 116.4)
- removed the R54 at (186.5, 75.7)
- removed the R62 at (186.5, 78.2)
- removed the U15 at (127.8, 73.2)
- added C101: 4u7/50V, Capacitor_SMD:C_1210_3225Metric_Pad1.33x2.70mm_HandSolder, F.Cu at (43.9, 93.9)
- added C102: 4u7/50V, Capacitor_SMD:C_1210_3225Metric_Pad1.33x2.70mm_HandSolder, F.Cu at (43.9, 98.2)
- added C105: 10u/50V, Capacitor_SMD:C_1210_3225Metric_Pad1.33x2.70mm_HandSolder, F.Cu at (43.9, 102.4)
- added C106: 10u/50V, Capacitor_SMD:C_1210_3225Metric_Pad1.33x2.70mm_HandSolder, F.Cu at (43.9, 106.7)
- added C81: 1u, Capacitor_SMD:C_0603_1608Metric_Pad1.08x0.95mm_HandSolder, F.Cu at (49.1, 89.2)
- added C94: 4u7/50V, Capacitor_SMD:C_1210_3225Metric_Pad1.33x2.70mm_HandSolder, F.Cu at (43.9, 76.9)
- added C95: 4u7/50V, Capacitor_SMD:C_1210_3225Metric_Pad1.33x2.70mm_HandSolder, F.Cu at (43.9, 81.2)
- added C98: 10u/50V, Capacitor_SMD:C_1210_3225Metric_Pad1.33x2.70mm_HandSolder, F.Cu at (43.9, 89.7)
- added R57: 0, Resistor_SMD:R_0603_1608Metric_Pad0.98x0.95mm_HandSolder, F.Cu at (49.1, 96.8)
- added R58: 0, Resistor_SMD:R_0603_1608Metric_Pad0.98x0.95mm_HandSolder, F.Cu at (49.1, 99.3)
- added U14: ADP7142ARDZ-5.0, Package_SO:SOIC-8-1EP_3.9x4.9mm_P1.27mm_EP2.29x3mm, F.Cu at (51.2, 84.7)
- R45: value 499 -> 68k
- R46: value 499k -> 10k
- R84: renamed from R85; value 4k7/2W -> 10k/2W
- R85: renamed from R86; value 4k7/2W -> 10k/2W
- U10: value TSR0.5-2490 -> MAX15062C; footprint Converter_DCDC:Converter_DCDC_TRACO_TSR0.5-24xx_TSR0.5-24xxx_THT -> Package_DFN_QFN:DFN-8_2x2mm_P0.5mm
- moved R45 138.9 mm to (49.1, 91.7)
- moved R46 138.9 mm to (49.1, 94.2)
- moved U13 85.0 mm to (51.2, 78.2)
- moved C97 60.2 mm to (43.9, 85.4)
- moved U10 49.3 mm to (49.4, 102.5), turned to 0 degrees
- moved C31 24.7 mm to (60.4, 76.9)
- renumbered C99 to C103, C100 to C104, C101 to C107, C102 to C108, C105 to C109, C106 to C110, C107 to C111, C108 to C112, C109 to C113, C110 to C114, C111 to C115, C112 to C116, C113 to C117, C114 to C118, C115 to C119, C116 to C120, C117 to C121, C118 to C122, C119 to C123, C120 to C124, C121 to C125, C122 to C126, C123 to C127, C124 to C128, C125 to C129, C126 to C130, C127 to C131, C128 to C132, C76 to C75, C77 to C76, C75 to C77, C85 to C84, C86 to C85, C81 to C86, C84 to C87, C93 to C92, C94 to C93, C95 to C96, L5 to L6, L6 to L7, Q4 to Q3, Q5 to Q4, R48 to R47, R49 to R48, R50 to R49, R51 to R50, R52 to R51, R55 to R52, R56 to R53, R57 to R54, R58 to R59, R59 to R60, R60 to R61, R63 to R62, R64 to R63, R65 to R64, R66 to R65, R67 to R66, R68 to R67, R69 to R68, R70 to R69, R71 to R70, R72 to R71, R73 to R72, R74 to R73, R75 to R74, R76 to R75, R77 to R76, R78 to R77, R79 to R78, R80 to R79, R81 to R80, R82 to R81, R83 to R82, R84 to R83, U14 to U15
Connections:
- net +3V3_ISO renamed +5VD_ISO
- C86 pad 1: +9V -> +7V_ISO
- C87 pad 1: +9V -> +7V_ISO
- C97 pad 1: +5V_ISO -> +7V_ISO
- J12 pad 1: unconnected-(J12-Pin_1-Pad1) -> /Block Diagram/Isolation IO/SPI1_SCK_ISO
- J12 pad 2: unconnected-(J12-Pin_2-Pad2) -> /Block Diagram/Isolation IO/DAC1_~{FAULT}_ISO
- J12 pad 3: unconnected-(J12-Pin_3-Pad3) -> /Block Diagram/Isolation IO/SPI1_MOSI_ISO
- J12 pad 4: unconnected-(J12-Pin_4-Pad4) -> /Block Diagram/Isolation IO/DAC2_~{FAULT}_ISO
- J12 pad 5: unconnected-(J12-Pin_5-Pad5) -> /Block Diagram/Isolation IO/SPI1_~{CS}_ISO
- J12 pad 7: unconnected-(J12-Pin_7-Pad7) -> /Block Diagram/Isolation IO/SPI1_MISO_ISO
- J13 pad 1: unconnected-(J13-Pin_1-Pad1) -> /Block Diagram/Isolation IO/SPI2_SCK_ISO
- J13 pad 3: unconnected-(J13-Pin_3-Pad3) -> /Block Diagram/Isolation IO/SPI2_~{CS}_ISO
- J13 pad 5: unconnected-(J13-Pin_5-Pad5) -> /Block Diagram/Isolation IO/SPI2_MISO_ISO
- J5 pad 5: VDD -> +7V_ISO
- J5 pad 7: +5V_ISO -> +5VA_ISO
- R45 pad 1: +9V -> +7V_ISO
- R45 pad 2: Net-(Q3-B) (its old number) -> Net-(U10-FB/Vout)
- R46 pad 1: Net-(Q3-B) (its old number) -> Net-(U10-FB/Vout)
- U10 pad 2: GND_ISO -> +24V_LV_ISO
- U10 pad 3: +9V -> Net-(U10-VCC)
- U13 pad 1: +5V_ISO -> +5VA_ISO
- U13 pad 2: +5V_ISO -> +5VA_ISO
- U13 pad 5: VDD -> +7V_ISO
- U13 pad 7: VDD -> +7V_ISO
- U13 pad 8: VDD -> +7V_ISO
- U19 pad 10: unconnected-(U19-INF-Pad10) -> /Block Diagram/Isolation IO/SPI2_MISO_ISO
- U19 pad 11: unconnected-(U19-OUTE-Pad11) -> /Block Diagram/Isolation IO/SPI2_~{CS}_ISO
- U19 pad 12: unconnected-(U19-OUTD-Pad12) -> /Block Diagram/Isolation IO/SPI2_SCK_ISO

Commit message: Development
Parts:
- removed the C32 at (64.6, 17.8)
- removed the C33 at (64.6, 22.0)
- removed the C34 at (192.8, 90.2)
- removed the C35 at (70.6, 17.3)
- removed the C36 at (70.6, 20.6)
- removed the C37 at (70.6, 24.0)
- removed the C38 at (44.8, 125.5)
- removed the C39 at (44.8, 128.0)
- removed the C40 at (64.6, 26.2)
- removed the C41 at (64.6, 30.5)
- removed the C42 at (78.6, 17.8)
- removed the C43 at (78.6, 22.0)
- removed the C44 at (199.2, 90.2)
- removed the C45 at (84.6, 17.3)
- removed the C46 at (84.6, 20.6)
- removed the C47 at (84.6, 24.0)
- removed the C49 at (38.8, 138.1)
- removed the C51 at (78.6, 30.5)
- removed the C52 at (42.5, 17.5)
- removed the C54 at (205.5, 90.2)
- removed the C56 at (48.5, 20.4)
- removed the C57 at (48.5, 23.8)
- removed C58: 56n/50V, Capacitor_SMD:C_0603_1608Metric_Pad1.08x0.95mm_HandSolder
- removed the C59 at (45.1, 138.1)
- removed the C60 at (42.5, 26.0)
- removed the C61 at (42.5, 30.2)
- removed the D3 at (160.1, 90.9)
- removed the D4 at (163.4, 90.9)
- removed the D5 at (145.0, 91.5)
- removed the D6 at (145.0, 94.9)
- removed the D7 at (152.6, 113.3)
- removed the D8 at (152.6, 116.7)
- removed the R14 at (192.8, 92.7)
- removed the R15 at (192.8, 95.2)
- removed the R16 at (165.1, 96.7)
- removed the R17 at (192.8, 97.8)
- removed the R18 at (192.8, 100.3)
- removed the R19 at (192.8, 102.8)
- removed the R20 at (199.2, 92.7)
- removed the R21 at (199.2, 95.2)
- removed the R22 at (139.2, 96.5)
- removed the R23 at (199.2, 97.8)
- removed the R24 at (199.2, 100.3)
- removed the R25 at (199.2, 102.8)
- removed the R26 at (205.5, 92.7)
- removed the R27 at (205.5, 95.2)
- removed the R28 at (146.8, 118.4)
- removed the R31 at (205.5, 102.8)
- removed T1, T2, T3: 750319331, ETH1CVOLT_A:750319331
- removed TP3, TP4, TP5, TP6, TP7, TP8: TestPoint, TestPoint:TestPoint_Pad_D2.0mm
- removed the U5 at (101.5, 106.4)
- removed the U6 at (85.2, 91.6)
- removed the U7 at (153.3, 109.4)
- added C114: 220u/50V, Capacitor_SMD:CP_Elec_10x14.3, F.Cu at (97.9, 89.7)
- added C115: 220u/50V, Capacitor_SMD:CP_Elec_10x14.3, F.Cu at (82.3, 73.0)
- added C116: 220u/50V, Capacitor_SMD:CP_Elec_10x14.3, F.Cu at (82.4, 87.7)
- added C62: 4u7/50V, Capacitor_SMD:C_1210_3225Metric_Pad1.33x2.70mm_HandSolder, F.Cu at (-7.77, 96.4)
- added C63: 10u/50V, Capacitor_SMD:C_1210_3225Metric_Pad1.33x2.70mm_HandSolder, F.Cu at (-37.7, 116.4)
- added C65: 10u/50V, Capacitor_SMD:C_1210_3225Metric_Pad1.33x2.70mm_HandSolder, F.Cu at (-7.77, 100.7)
- added C68: 10u/50V, Capacitor_SMD:C_1210_3225Metric_Pad1.33x2.70mm_HandSolder, F.Cu at (-37.7, 120.6)
- added C76: 10u/50V, Capacitor_SMD:C_1210_3225Metric_Pad1.33x2.70mm_HandSolder, F.Cu at (-37.7, 124.9)
- added C79: 4u7/50V, Capacitor_SMD:C_1210_3225Metric_Pad1.33x2.70mm_HandSolder, F.Cu at (-37.7, 129.1)
- added U11: THL30-2415WI, Converter_DCDC:Converter_DCDC_TRACO_THL30-xxxxWI_THT, F.Cu at (92.5, 71.1)
- added U8: MAX15062B, Package_DFN_QFN:DFN-8_2x2mm_P0.5mm, F.Cu at (-2.36, 95.2)
- C48: value 56n/50V -> 4u7/50V; footprint Capacitor_SMD:C_0603_1608Metric_Pad1.08x0.95mm_HandSolder -> Capacitor_SMD:C_1210_3225Metric_Pad1.33x2.70mm_HandSolder
- C53: value 10u/50V -> 220u/50V; footprint Capacitor_SMD:C_1210_3225Metric_Pad1.33x2.70mm_HandSolder -> Capacitor_SMD:CP_Elec_10x14.3
- C55: value 2u2/50V -> 1u; footprint Capacitor_SMD:C_1206_3216Metric_Pad1.33x1.80mm_HandSolder -> Capacitor_SMD:C_0603_1608Metric_Pad1.08x0.95mm_HandSolder
- F1: value 1812L075/33DR -> 3425L300/36MR
- Q1: value FDS9435A -> SiS443DN; footprint Package_SO:SOIC-8_3.9x4.9mm_P1.27mm -> Package_SO:Vishay_PowerPAK_1212-8_Single
- R29: value 49k9 -> 0
- R30: value 100k -> 10k
- moved R29 208.3 mm to (-2.59, 89.5)
- moved R30 208.3 mm to (-2.59, 92.1)
- moved D5 182.7 mm to (259.6, 110.5)
- moved D6 182.7 mm to (259.6, 114.6)
- moved D10 182.7 mm to (267.6, 110.0)
- moved D11 182.7 mm to (267.6, 113.6)
- moved D12 182.7 mm to (267.6, 117.2)
- moved D13 182.7 mm to (267.6, 120.9)
- moved D14 182.7 mm to (267.6, 124.5)
- moved D7 182.7 mm to (267.6, 99.0)
- moved D8 182.7 mm to (267.6, 102.7)
- moved D9 182.7 mm to (267.6, 106.3)
- moved Q1 122.5 mm to (-7.86, 107.2)
- moved C50 108.6 mm to (-7.77, 92.2)
- moved C53 97.3 mm to (97.9, 101.7), turned to 180 degrees
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- renumbered C119 to C100, C120 to C101, C121 to C102, C122 to C103, C123 to C104, C124 to C105, C125 to C106, C126 to C107, C127 to C108, C128 to C109, C129 to C110, C130 to C111, C131 to C112, C132 to C113, C62 to C32, C63 to C33, C64 to C34, C65 to C35, C66 to C36, C67 to C37, C68 to C38, C69 to C39, C70 to C40, C71 to C41, C72 to C42, C73 to C43, C74 to C44, C75 to C45, C76 to C46, C77 to C47, C78 to C49, C79 to C51, C80 to C52, C81 to C54, C82 to C56, C83 to C57, C84 to C59, C85 to C60, C86 to C61, C87 to C64, C88 to C66, C89 to C67, C90 to C69, C91 to C70, C92 to C71, C93 to C72, C94 to C73, C95 to C74, C96 to C75, C97 to C77, C98 to C78, C103 to C82, C104 to C83, C101 to C84, C102 to C85, C107 to C86, C108 to C87, C105 to C88, C106 to C89, C109 to C90, C110 to C91, C111 to C92, C112 to C93, C113 to C94, C114 to C95, C115 to C96, C116 to C97, C117 to C98, C118 to C99, D16 to D10, D17 to D11, D18 to D12, D19 to D13, D20 to D14, D21 to D15, D22 to D16, D23 to D17, D9 to D3, D10 to D4, D11 to D5, D12 to D6, D13 to D7, D14 to D8, D15 to D9, L6 to L10, L7 to L11, L3 to L5, L4 to L6, R32 to R14, R33 to R15, R34 to R16, R35 to R17, R36 to R18, R37 to R19, R38 to R20, R39 to R21, R40 to R22, R41 to R23, R42 to R24, R43 to R25, R44 to R26, R45 to R27, R46 to R28, R47 to R31, R48 to R32, R49 to R33, R50 to R34, R51 to R35, R52 to R36, R53 to R37, R54 to R38, R59 to R41, R60 to R42, R61 to R43, R57 to R44, R58 to R45, R62 to R46, R63 to R47, R64 to R48, R65 to R49, R66 to R50, R67 to R51, R68 to R52, R69 to R53, R70 to R54, R71 to R55, R72 to R56, R73 to R57, R74 to R58, R75 to R59, R76 to R60, R77 to R61, R78 to R62, R79 to R63, R80 to R64, R81 to R65, R82 to R66, R83 to R67, R84 to R68, R85 to R69, U12 to U10, U15 to U12, U16 to U15, U17 to U16, U18 to U17, U19 to U18, U8 to U5, U9 to U6, U10 to U7, U11 to U9
Connections:
- net +5VA_ISO renamed +VA_ISO
- C32 pad 1: +24V_MV_ISO -> +24V_ISO
- C33 pad 1: +24V_MV_ISO -> +24V_ISO
- C34 pad 1: +24V_MV_ISO -> +24V_ISO
- C35 pad 1: +24V_MV_ISO -> +24V_ISO
- C45 pad 1: +24V_LV_ISO -> +24V_ISO
- C46 pad 1: +24V_LV_ISO -> +24V_ISO
- C47 pad 1: +24V_LV_ISO -> +24V_ISO
- C48 pad 1: /Block Diagram/Power/Power Isolated/UCC25800_2/+24V_ISO -> +24V_ISO
- C48 pad 2: Net-(T2-SB) -> GND_ISO
- C49 pad 1: +24V_LV_ISO -> +24V_ISO
- C50 pad 1: /Block Diagram/Power/Power Isolated/UCC25800_2/+24V_ISO -> +24V_ISO
- C51 pad 1: +24V_LV_ISO -> +24V_ISO
- C52 pad 1: +24V_LV_ISO -> +24V_ISO
- C55 pad 1: +24V -> Net-(U8-VCC)
- C55 pad 2: GND -> GND_ISO
- C85 pad 1: +5VD_ISO -> +VD_ISO
- C89 pad 1: +5VD_ISO -> +VD_ISO
- C90 pad 1: +24V_HV_ISO -> +24V_ISO
- C91 pad 1: +24V_HV_ISO -> +24V_ISO
- C92 pad 1: +24V_HV_ISO -> +24V_ISO
- C93 pad 1: +24V_HV_ISO -> +24V_ISO
- F1 pad 2: Net-(F1-Pad2) -> Net-(Q1-D)
- J5 pad 6: GND_ISO -> +5VD_ISO
- J5 pad 8: +5VD_ISO -> +VD_ISO
- L10 pad 1: +24V_HV_ISO -> +24V_ISO
- L11 pad 1: +24V_HV_ISO -> +24V_ISO
- L2 pad 1: +24V_MV_ISO -> +24V_ISO
- L5 pad 1: +24V_LV_ISO -> +24V_ISO
- L6 pad 1: +24V_LV_ISO -> +24V_ISO
- Q1 pad 5: Net-(F1-Pad2) -> Net-(Q1-D)
- R14 pad 1: +24V_MV_ISO -> +24V_ISO
- R16 pad 1: +24V_MV_ISO -> +24V_ISO
- R23 pad 1: +24V_LV_ISO -> +24V_ISO
- R25 pad 1: +24V_LV_ISO -> +24V_ISO
- R29 pad 1: Net-(U7-RT) -> +5VD_ISO
- R29 pad 2: GND -> Net-(U8-FB/Vout)
- R30 pad 1: +24V -> Net-(U8-FB/Vout)
- R30 pad 2: Net-(T3-AB) -> GND_ISO
- R45 pad 2: +5VD_ISO -> +VD_ISO
- R46 pad 1: +24V_HV_ISO -> +24V_ISO
- R48 pad 1: +24V_HV_ISO -> +24V_ISO
- U10 pad 6: +24V_LV_ISO -> +24V_ISO
- U14 pad 1: +5VD_ISO -> +VD_ISO
- U14 pad 2: +5VD_ISO -> +VD_ISO
- U15 pad 3: +24V_HV_ISO -> +24V_ISO
- U16 pad 3: +24V_HV_ISO -> +24V_ISO
- U17 pad 16: +5VD_ISO -> +VD_ISO
- U18 pad 16: +5VD_ISO -> +VD_ISO
- U5 pad 6: +24V_MV_ISO -> +24V_ISO
- U6 pad 6: +24V_MV_ISO -> +24V_ISO
- U7 pad 1: +24V_LV_ISO -> +24V_ISO
- U7 pad 2: +24V_LV_ISO -> +24V_ISO
- U9 pad 6: +24V_LV_ISO -> +24V_ISO

Commit message: Development
Parts:
- removed D16: 1N4148W, Diode_SMD:D_SOD-123
- removed J10: FCR7350B, ETH1CVOLT_A:S16N-PC
- removed J9: FCR7350R, ETH1CVOLT_A:S16N-PC
- removed K2: EE2-3NU, Relay_SMD:Relay_DPDT_Kemet_EE2_NU
- removed Q4: MMBT3904, Package_TO_SOT_SMD:SOT-23
- removed R61: 10K, Resistor_SMD:R_0603_1608Metric_Pad0.98x0.95mm_HandSolder
- added J14: Conn_02x04_Odd_Even, Connector_PinSocket_2.54mm:PinSocket_2x04_P2.54mm_Vertical_SMD, F.Cu at (96.0, 181.1)
- added U19: ISO7761DW, Package_SO:SOIC-16W_7.5x10.3mm_P1.27mm, F.Cu at (136.1, 128.7)
- added U20: TCMT1103, Package_SO:SOP-4_4.4x2.6mm_P1.27mm, F.Cu at (136.1, 110.2)
- added U21: TCMT1103, Package_SO:SOP-4_4.4x2.6mm_P1.27mm, F.Cu at (136.1, 106.8)
- added U22: TCMT1103, Package_SO:SOP-4_4.4x2.6mm_P1.27mm, F.Cu at (136.1, 103.3)
- U17: value ISO7763DW -> ISO7761DW
- moved C23 83.3 mm to (78.3, 161.2)
- moved C29 83.3 mm to (67.2, 156.4)
- moved C30 83.3 mm to (67.2, 159.8)
- moved F1 83.3 mm to (67.9, 163.9)
- moved R13 83.3 mm to (72.4, 158.5)
- moved R7 83.3 mm to (82.7, 161.2)
- moved Q2 83.3 mm to (61.8, 161.4)
- moved R12 83.3 mm to (72.4, 156.0)
- moved D1 83.3 mm to (61.8, 156.9)
- moved U17 21.2 mm to (136.1, 117.6)
- moved J4 13.1 mm to (148.5, 107.2), turned to 180 degrees
- moved U18 12.5 mm to (136.1, 139.8)
- moved J13 5.61 mm to (148.6, 121.8)
- moved J12 0.32 mm to (149.0, 138.4)
Connections:
- J12 pad 1: /Block Diagram/Isolation IO/SPI1_SCK_ISO -> unconnected-(J12-Pin_1-Pad1)
- J12 pad 2: /Block Diagram/Isolation IO/DAC1_~{FAULT}_ISO -> unconnected-(J12-Pin_2-Pad2)
- J12 pad 3: /Block Diagram/Isolation IO/SPI1_MOSI_ISO -> unconnected-(J12-Pin_3-Pad3)
- J12 pad 4: /Block Diagram/Isolation IO/DAC2_~{FAULT}_ISO -> unconnected-(J12-Pin_4-Pad4)
- J12 pad 5: /Block Diagram/Isolation IO/SPI1_~{CS}_ISO -> unconnected-(J12-Pin_5-Pad5)
- J12 pad 7: /Block Diagram/Isolation IO/SPI1_MISO_ISO -> unconnected-(J12-Pin_7-Pad7)
- J13 pad 1: /Block Diagram/Isolation IO/SPI2_SCK_ISO -> unconnected-(J13-Pin_1-Pad1)
- J13 pad 3: /Block Diagram/Isolation IO/SPI2_~{CS}_ISO -> unconnected-(J13-Pin_3-Pad3)
- J13 pad 5: /Block Diagram/Isolation IO/SPI2_MISO_ISO -> unconnected-(J13-Pin_5-Pad5)
- J5 pad 3: GND_ISO -> +24V_ISO
- U17 pad 10: /Block Diagram/Isolation IO/DAC2_~{FAULT}_ISO -> unconnected-(U17-INF-Pad10)
- U17 pad 11: /Block Diagram/Isolation IO/DAC1_~{FAULT}_ISO -> unconnected-(U17-OUTE-Pad11)
- U17 pad 12: /Block Diagram/Isolation IO/SPI1_MISO_ISO -> unconnected-(U17-OUTD-Pad12)
- U17 pad 13: /Block Diagram/Isolation IO/SPI1_~{CS}_ISO -> unconnected-(U17-OUTC-Pad13)
- U17 pad 14: /Block Diagram/Isolation IO/SPI1_MOSI_ISO -> unconnected-(U17-OUTB-Pad14)
- U17 pad 15: /Block Diagram/Isolation IO/SPI1_SCK_ISO -> unconnected-(U17-OUTA-Pad15)
- U17 pad 2: /Block Diagram/Isolation IO/SPI1_SCK -> unconnected-(U17-INA-Pad2)
- U17 pad 3: /Block Diagram/Isolation IO/SPI1_MOSI -> unconnected-(U17-INB-Pad3)
- U17 pad 4: /Block Diagram/Isolation IO/SPI1_~{CS} -> unconnected-(U17-INC-Pad4)
- U17 pad 5: /Block Diagram/Isolation IO/SPI1_MISO -> unconnected-(U17-IND-Pad5)
- U17 pad 6: /Block Diagram/Isolation IO/DAC1_~{FAULT} -> unconnected-(U17-INE-Pad6)
- U17 pad 7: /Block Diagram/Isolation IO/DAC2_~{FAULT} -> unconnected-(U17-OUTF-Pad7)
- U18 pad 10: /Block Diagram/Isolation IO/SPI2_MISO_ISO -> unconnected-(U18-INF-Pad10)
- U18 pad 11: /Block Diagram/Isolation IO/SPI2_~{CS}_ISO -> unconnected-(U18-OUTE-Pad11)
- U18 pad 12: /Block Diagram/Isolation IO/SPI2_SCK_ISO -> unconnected-(U18-OUTD-Pad12)
- U18 pad 5: /Block Diagram/Isolation IO/SPI2_SCK -> unconnected-(U18-IND-Pad5)
- U18 pad 6: /Block Diagram/Isolation IO/SPI2_~{CS} -> unconnected-(U18-INE-Pad6)
- U18 pad 7: /Block Diagram/Isolation IO/SPI2_MISO -> unconnected-(U18-OUTF-Pad7)
