File: HARDWARE/ETH1CVOLT_A/ETH1CVOLT_A.kicad_pcb (KiCad board)
At the start: 2 copper layers, 160 x 100 mm, 254 parts, among them J1 20021111-00010T4LF, J11 Conn_02x05_Odd_Even, J12 Conn_02x04_Odd_Even, J13 Conn_02x04_Odd_Even, J14 Conn_02x04_Odd_Even, J2 RJ45_Wuerth_7499010121A, J3 1715721, J4 Conn_02x04_Odd_Even, J5 Conn_02x04_Odd_Even, J6 Conn_02x05_Odd_Even, J7 FCR7350R, J8 FCR7350B, K1 EE2-3NU, K3 EE2-3NU, Q1 SiS443DN, Q2 MMBT3904, Q3 MMBT3904, U1 STM32H743VITx, U10 LT8330_S6, U11 THL30-2415WI, U12 TPS7A39, U13 ADP7142ARDZ-5.0, U14 ADP7142ARDZ-5.0, U15 LT8365, U16 LT8365, U17 ISO7761DW, U18 ISO7761DW, U19 ISO7761DW, U2 24LC08B-E/MS, U20 TCMT1103, U21 TCMT1103, U22 TCMT1103, U3 LAN8742A, U4 TSR1-2433E, U5 LT8330_S6, U6 LT8330_S6, U7 MAX15062C, U8 MAX15062B, U9 LT8330_S6, Y1 NX5032GA-16, Y2 NX5032GA-25

Commit message: Development
Parts:
- removed J6: Conn_02x05_Odd_Even, Connector_PinSocket_2.54mm:PinSocket_2x05_P2.54mm_Vertical_SMD
- removed K1: EE2-3NU, Relay_SMD:Relay_DPDT_Kemet_EE2_NU
- removed Q3: MMBT3904, Package_TO_SOT_SMD:SOT-23
- removed R60: 10K, Resistor_SMD:R_0603_1608Metric_Pad0.98x0.95mm_HandSolder
- added J9: Conn_02x04_Odd_Even, Connector_PinSocket_2.54mm:PinSocket_2x04_P2.54mm_Vertical_SMD, F.Cu at (107.5, 85.5)
- added K2: EE2-5NU, Relay_SMD:Relay_DPDT_Kemet_EE2_NU, F.Cu at (105.8, 101.9)
- added L1: 74438335068, ETH1CVOLT_A:74438335068, F.Cu at (127.2, 184.3)
- added L3: 744774022, ETH1CVOLT_A:744774022, F.Cu at (216.0, 109.0)
- added L4: 744774022, ETH1CVOLT_A:744774022, F.Cu at (118.9, 174.7)
- added L7: 74408063470, ETH1CVOLT_A:74408063470, F.Cu at (128.6, 168.1)
- added L8: 74408063470, ETH1CVOLT_A:74408063470, F.Cu at (128.6, 175.9)
- added L9: 744774022, ETH1CVOLT_A:744774022, F.Cu at (241.4, 83.0)
- added R61: 340, Resistor_SMD:R_0603_1608Metric_Pad0.98x0.95mm_HandSolder, F.Cu at (265.2, 145.2)
- added R70: 340, Resistor_SMD:R_0603_1608Metric_Pad0.98x0.95mm_HandSolder, F.Cu at (265.2, 147.7)
- added R71: 340, Resistor_SMD:R_0603_1608Metric_Pad0.98x0.95mm_HandSolder, F.Cu at (265.2, 150.2)
- added R72: 340, Resistor_SMD:R_0603_1608Metric_Pad0.98x0.95mm_HandSolder, F.Cu at (111.6, 111.4)
- added U24: ISO7761FDBQ, Package_SO:SSOP-16_3.9x4.9mm_P0.635mm, F.Cu at (164.2, 138.5)
- F1: value 3425L300/36MR -> MF-GSMF300/36X-2; footprint Fuse:Fuse_1812_4532Metric_Pad1.30x3.40mm_HandSolder -> ETH1CVOLT_A:MF-GSMF
- J3: value 1715721 -> CONN; footprint TerminalBlock_Phoenix:TerminalBlock_Phoenix_MKDS-1,5-2_1x02_P5.00mm_Horizontal -> Connector_Phoenix_MC:PhoenixContact_MC_1,5_2-GF-3.81_1x02_P3.81mm_Horizontal_ThreadedFlange_MountHole
- U17, U18: value ISO7761DW -> ISO7761FDBQ; footprint Package_SO:SOIC-16W_7.5x10.3mm_P1.27mm -> Package_SO:SSOP-16_3.9x4.9mm_P0.635mm
- U19: value ISO7761DW -> TCMT1103; footprint Package_SO:SOIC-16W_7.5x10.3mm_P1.27mm -> Package_SO:SOP-4_4.4x2.6mm_P1.27mm
- moved C63 184.7 mm to (139.7, 167.7)
- moved C68 184.7 mm to (139.7, 171.9)
- moved C76 184.7 mm to (139.7, 176.2)
- moved C79 184.7 mm to (139.7, 180.4)
- moved F1 156.1 mm to (217.2, 118.4)
- moved J3 146.1 mm to (226.2, 118.3), turned to 90 degrees
- moved C116 144.7 mm to (227.1, 86.1), turned to 180 degrees
- moved J8 134.2 mm to (89.3, 103.3), turned to 180 degrees
- moved J7 133.1 mm to (89.3, 85.2), turned to 180 degrees
- moved C115 132.2 mm to (211.9, 98.9), turned to 0 degrees
- moved U11 129.4 mm to (221.8, 74.6), turned to 180 degrees
- moved C53 129.2 mm to (227.1, 98.9)
- moved J2 120.4 mm to (214.9, 131.4), turned to 0 degrees
- moved C114 114.1 mm to (211.9, 86.1), turned to 0 degrees
- moved U4 101.3 mm to (197.0, 114.8), turned to -90 degrees
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Connections:
- D15 pad 1: +3.3V -> +5VD_ISO
- D3 pad 1: GND -> GND_ISO
- J12 pad 1: unconnected-(J12-Pin_1-Pad1) -> /Block Diagram/Isolation IO/DAC_SDO
- J12 pad 2: unconnected-(J12-Pin_2-Pad2) -> /Block Diagram/Isolation IO/AUX_SEL
- J12 pad 3: unconnected-(J12-Pin_3-Pad3) -> /Block Diagram/Isolation IO/DAC_SCLK
- J12 pad 4: unconnected-(J12-Pin_4-Pad4) -> /Block Diagram/Isolation IO/SEL_x1
- J12 pad 5: unconnected-(J12-Pin_5-Pad5) -> /Block Diagram/Isolation IO/DAC_SDIN
- J12 pad 6: unconnected-(J12-Pin_6-Pad6) -> /Block Diagram/Isolation IO/SEL_x10
- J12 pad 7: unconnected-(J12-Pin_7-Pad7) -> /Block Diagram/Isolation IO/DAC_~{SYNC}
- J12 pad 8: unconnected-(J12-Pin_8-Pad8) -> /Block Diagram/Isolation IO/SEL_x100
- J13 pad 1: unconnected-(J13-Pin_1-Pad1) -> /Block Diagram/Isolation IO/ADC_CURR_SDO
- J13 pad 3: unconnected-(J13-Pin_3-Pad3) -> /Block Diagram/Isolation IO/ADC_CURR_~{CS}
- J13 pad 5: unconnected-(J13-Pin_5-Pad5) -> /Block Diagram/Isolation IO/ADC_CURR_SCLK
- J13 pad 7: unconnected-(J13-Pin_7-Pad7) -> /Block Diagram/Isolation IO/ADC_CURR_SDI
- J14 pad 1: unconnected-(J14-Pin_1-Pad1) -> /Block Diagram/Isolation IO/ADC_VOLT_SCLK
- J14 pad 2: unconnected-(J14-Pin_2-Pad2) -> /Block Diagram/Isolation IO/MUX_A1
- J14 pad 3: unconnected-(J14-Pin_3-Pad3) -> /Block Diagram/Isolation IO/ADC_VOLT_~{CS}
- J14 pad 4: unconnected-(J14-Pin_4-Pad4) -> /Block Diagram/Isolation IO/LV_OUT_PMOS
- J14 pad 5: unconnected-(J14-Pin_5-Pad5) -> /Block Diagram/Isolation IO/ADC_VOLT_SDO
- J14 pad 6: unconnected-(J14-Pin_6-Pad6) -> /Block Diagram/Isolation IO/MV_OUT_PMOS
- J14 pad 7: unconnected-(J14-Pin_7-Pad7) -> /Block Diagram/Isolation IO/MUX_A0
- J14 pad 8: unconnected-(J14-Pin_8-Pad8) -> /Block Diagram/Isolation IO/HV_OUT_PMOS
- U1 pad 1: /Block Diagram/MCU/MCU_DEF -> /Block Diagram/Isolation IO/MCU_ADC_CURR_SCLK
- U1 pad 20: +3.3VADC -> VDDA
- U1 pad 28: unconnected-(U1-PA4-Pad28) -> /Block Diagram/Isolation IO/MCU_ADC_VOLT_~{CS}
- U1 pad 29: unconnected-(U1-PA5-Pad29) -> /Block Diagram/Isolation IO/MCU_ADC_VOLT_SCLK
- U1 pad 3: unconnected-(U1-PE4-Pad3) -> /Block Diagram/Isolation IO/MCU_ADC_CURR_~{CS}
- U1 pad 30: unconnected-(U1-PA6-Pad30) -> /Block Diagram/Isolation IO/MCU_ADC_VOLT_SDO
- U1 pad 4: unconnected-(U1-PE5-Pad4) -> /Block Diagram/Isolation IO/MCU_ADC_CURR_SDO
- U1 pad 46: unconnected-(U1-PB10-Pad46) -> /Block Diagram/MCU/MCU_OUTPUT_RL_CTR
- U1 pad 5: unconnected-(U1-PE6-Pad5) -> /Block Diagram/Isolation IO/MCU_ADC_CURR_SDI
- U1 pad 62: unconnected-(U1-PD15-Pad62) -> /Block Diagram/Isolation IO/MCU_HV_OUT_PMOS
- U1 pad 63: unconnected-(U1-PC6-Pad63) -> /Block Diagram/Isolation IO/MCU_MV_OUT_PMOS
- U1 pad 64: unconnected-(U1-PC7-Pad64) -> /Block Diagram/Isolation IO/MCU_LV_OUT_PMOS
- U1 pad 65: unconnected-(U1-PC8-Pad65) -> /Block Diagram/Isolation IO/MCU_AUX_SEL
- U1 pad 66: unconnected-(U1-PC9-Pad66) -> /Block Diagram/Isolation IO/MCU_SEL_x100
- U1 pad 67: unconnected-(U1-PA8-Pad67) -> /Block Diagram/Isolation IO/MCU_SEL_x10
- U1 pad 68: unconnected-(U1-PA9-Pad68) -> /Block Diagram/Isolation IO/MCU_SEL_x1
- U1 pad 69: unconnected-(U1-PA10-Pad69) -> /Block Diagram/Isolation IO/MCU_MUX_A1
- U1 pad 70: unconnected-(U1-PA11-Pad70) -> /Block Diagram/Isolation IO/MCU_MUX_A0
- U1 pad 77: unconnected-(U1-PA15-Pad77) -> /Block Diagram/Isolation IO/MCU_DAC_~{SYNC}
- U1 pad 78: unconnected-(U1-PC10-Pad78) -> /Block Diagram/Isolation IO/MCU_DAC_SCLK
- U1 pad 79: unconnected-(U1-PC11-Pad79) -> /Block Diagram/Isolation IO/MCU_DAC_SDO
- U1 pad 80: unconnected-(U1-PC12-Pad80) -> /Block Diagram/Isolation IO/MCU_DAC_SDIN
- U1 pad 98: unconnected-(U1-PE1-Pad98) -> /Block Diagram/MCU/MCU_DEF
- U17 pad 10: unconnected-(U17-INF-Pad10) -> /Block Diagram/Isolation IO/ADC_VOLT_SDO
- U17 pad 11: unconnected-(U17-OUTE-Pad11) -> /Block Diagram/Isolation IO/ADC_VOLT_~{CS}
- U17 pad 12: unconnected-(U17-OUTD-Pad12) -> /Block Diagram/Isolation IO/ADC_VOLT_SCLK
- U17 pad 13: unconnected-(U17-OUTC-Pad13) -> /Block Diagram/Isolation IO/AUX_SEL
- U17 pad 14: unconnected-(U17-OUTB-Pad14) -> /Block Diagram/Isolation IO/SEL_x1
- U17 pad 16: +VD_ISO -> +5VD_ISO
- U17 pad 3: unconnected-(U17-INB-Pad3) -> /Block Diagram/Isolation IO/MCU_SEL_x1
- U17 pad 4: unconnected-(U17-INC-Pad4) -> /Block Diagram/Isolation IO/MCU_AUX_SEL
- U17 pad 5: unconnected-(U17-IND-Pad5) -> /Block Diagram/Isolation IO/MCU_ADC_VOLT_SCLK
- U17 pad 6: unconnected-(U17-INE-Pad6) -> /Block Diagram/Isolation IO/MCU_ADC_VOLT_~{CS}
- U17 pad 7: unconnected-(U17-OUTF-Pad7) -> /Block Diagram/Isolation IO/MCU_ADC_VOLT_SDO
- U18 pad 10: unconnected-(U18-INF-Pad10) -> /Block Diagram/Isolation IO/ADC_CURR_SDO
- U18 pad 11: unconnected-(U18-OUTE-Pad11) -> /Block Diagram/Isolation IO/ADC_CURR_~{CS}
- U18 pad 12: unconnected-(U18-OUTD-Pad12) -> /Block Diagram/Isolation IO/ADC_CURR_SCLK
- U18 pad 13: unconnected-(U18-OUTC-Pad13) -> /Block Diagram/Isolation IO/ADC_CURR_SDI
- U18 pad 14: unconnected-(U18-OUTB-Pad14) -> /Block Diagram/Isolation IO/SEL_x100
- U18 pad 15: unconnected-(U18-OUTA-Pad15) -> /Block Diagram/Isolation IO/SEL_x10
- U18 pad 16: +VD_ISO -> +5VD_ISO
- U18 pad 2: unconnected-(U18-INA-Pad2) -> /Block Diagram/Isolation IO/MCU_SEL_x10
- U18 pad 3: unconnected-(U18-INB-Pad3) -> /Block Diagram/Isolation IO/MCU_SEL_x100
- U18 pad 4: unconnected-(U18-INC-Pad4) -> /Block Diagram/Isolation IO/MCU_ADC_CURR_SDI
- U18 pad 5: unconnected-(U18-IND-Pad5) -> /Block Diagram/Isolation IO/MCU_ADC_CURR_SCLK
- U18 pad 6: unconnected-(U18-INE-Pad6) -> /Block Diagram/Isolation IO/MCU_ADC_CURR_~{CS}
- U18 pad 7: unconnected-(U18-OUTF-Pad7) -> /Block Diagram/Isolation IO/MCU_ADC_CURR_SDO
- U19 pad 1: +3.3V -> Net-(R72-Pad2)
- U19 pad 2: unconnected-(U19-INA-Pad2) -> GND
- U19 pad 3: unconnected-(U19-INB-Pad3) -> GND_ISO
- U19 pad 4: unconnected-(U19-INC-Pad4) -> Net-(D15-A)
- U20 pad 1: unconnected-(U20-Pad1) -> Net-(R70-Pad2)
- U20 pad 2: unconnected-(U20-Pad2) -> GND
- U20 pad 3: unconnected-(U20-Pad3) -> GND_ISO
- U20 pad 4: unconnected-(U20-Pad4) -> /Block Diagram/Isolation IO/MV_OUT_PMOS
- U21 pad 1: unconnected-(U21-Pad1) -> Net-(R61-Pad2)
- U21 pad 2: unconnected-(U21-Pad2) -> GND
- U21 pad 3: unconnected-(U21-Pad3) -> GND_ISO
- U21 pad 4: unconnected-(U21-Pad4) -> /Block Diagram/Isolation IO/LV_OUT_PMOS
- U22 pad 1: unconnected-(U22-Pad1) -> Net-(R71-Pad2)
- U22 pad 2: unconnected-(U22-Pad2) -> GND
- U22 pad 3: unconnected-(U22-Pad3) -> GND_ISO
- U22 pad 4: unconnected-(U22-Pad4) -> /Block Diagram/Isolation IO/HV_OUT_PMOS
Routing:
- net Net-(D15-A): track 0.00 -> 3.40 mm

Commit message: Hardware development
Parts:
- removed the C53 at (227.1, 98.9)
- C105: renamed from C91; value 4u7/50V -> 4u7/100V
- C106: renamed from C93; value 10u/50V -> 10u/100V
- C29, C34, C89: value 10u/50V -> 10u/100V
- C30: value 4u7/50V -> 4u7/100V
- C33: renamed from C32; value 4u7/50V -> 4u7/100V
- C40: renamed from C33; value 4u7/50V -> 4u7/100V
- C41: renamed from C35; value 10u/50V -> 10u/100V
- C45: renamed from C59; value 1u/50V -> 1u/100V
- C47: renamed from C45; value 4u7/50V -> 4u7/100V
- C48: renamed from C51; value 10u/50V -> 10u/100V
- C49: renamed from C69; value 4u7/50V -> 4u7/100V
- C50: renamed from C71; value 10u/50V -> 10u/100V
- C52: renamed from C82; value 4u7/50V -> 4u7/100V
- C53: renamed from C86; value 10u/50V -> 10u/100V
- C55: renamed from C60; value 1u/50V -> 1u/100V
- C56: renamed from C83; value 4u7/50V -> 4u7/100V
- C57: renamed from C87; value 10u/50V -> 10u/100V
- C59: renamed from C46; value 4u7/50V -> 4u7/100V
- C60: renamed from C52; value 10u/50V -> 10u/100V
- C61: renamed from C70; value 4u7/50V -> 4u7/100V
- C62: renamed from C72; value 10u/50V -> 10u/100V
- C66: renamed from C63; value 10u/50V -> 10u/100V
- C67: renamed from C68; value 10u/50V -> 10u/100V
- C68: renamed from C76; value 10u/50V -> 10u/100V
- C69: renamed from C79; value 4u7/50V -> 4u7/100V
- C71: renamed from C47; value 4u7/50V -> 4u7/100V
- C72: renamed from C49; value 10u/50V -> 10u/100V
- C73: renamed from C61; value 4u7/50V -> 4u7/100V
- C74: renamed from C64; value 10u/50V -> 10u/100V
- C75: renamed from C73; value 4u7/50V -> 4u7/100V
- C76: renamed from C77; value 10u/50V -> 10u/100V
- C78: renamed from C84; value 4u7/50V -> 4u7/100V
- C79: renamed from C88; value 10u/50V -> 10u/100V
- C81: renamed from C48; value 4u7/50V -> 4u7/100V
- C82: renamed from C50; value 10u/50V -> 10u/100V
- C83: renamed from C62; value 4u7/50V -> 4u7/100V
- C84: renamed from C65; value 10u/50V -> 10u/100V
- C85: renamed from C74; value 4u7/50V -> 4u7/100V
- C86: renamed from C78; value 10u/50V -> 10u/100V
- C88: renamed from C85; value 4u7/50V -> 4u7/100V
- C93: renamed from C90; value 4u7/50V -> 4u7/100V
- C94: renamed from C92; value 10u/50V -> 10u/100V
- J3: value CONN -> 1843790; footprint Connector_Phoenix_MC:PhoenixContact_MC_1,5_2-GF-3.81_1x02_P3.81mm_Horizontal_ThreadedFlange_MountHole -> Connector_Phoenix_MC:PhoenixContact_MC_1,5_2-GF-3.5_1x02_P3.50mm_Horizontal_ThreadedFlange
- R11: renamed from R7; value 1k5 -> 1k4
- R15: renamed from R18; footprint Resistor_SMD:R_0603_1608Metric_Pad0.98x0.95mm_HandSolder -> Resistor_SMD:R_0805_2012Metric_Pad1.20x1.40mm_HandSolder
- R20: renamed from R21; footprint Resistor_SMD:R_0603_1608Metric_Pad0.98x0.95mm_HandSolder -> Resistor_SMD:R_0805_2012Metric_Pad1.20x1.40mm_HandSolder
- R24: renamed from R31; footprint Resistor_SMD:R_0603_1608Metric_Pad0.98x0.95mm_HandSolder -> Resistor_SMD:R_0805_2012Metric_Pad1.20x1.40mm_HandSolder
- R34: renamed from R33; footprint Resistor_SMD:R_0603_1608Metric_Pad0.98x0.95mm_HandSolder -> Resistor_SMD:R_0805_2012Metric_Pad1.20x1.40mm_HandSolder
- R49: renamed from R62; footprint Resistor_SMD:R_0603_1608Metric_Pad0.98x0.95mm_HandSolder -> Resistor_SMD:R_0805_2012Metric_Pad1.20x1.40mm_HandSolder
- R51: renamed from R63; footprint Resistor_SMD:R_0603_1608Metric_Pad0.98x0.95mm_HandSolder -> Resistor_SMD:R_0805_2012Metric_Pad1.20x1.40mm_HandSolder
- R62: renamed from R65; footprint Resistor_SMD:R_0603_1608Metric_Pad0.98x0.95mm_HandSolder -> Resistor_SMD:R_0805_2012Metric_Pad1.20x1.40mm_HandSolder
- R63: renamed from R66; footprint Resistor_SMD:R_0603_1608Metric_Pad0.98x0.95mm_HandSolder -> Resistor_SMD:R_0805_2012Metric_Pad1.20x1.40mm_HandSolder
- moved Q1 186.3 mm to (215.3, 114.6), turned to 180 degrees
- moved Q2 164.8 mm to (219.8, 114.6)
- moved D2 164.6 mm to (219.8, 111.0)
- moved R13 146.2 mm to (206.7, 98.2), turned to 180 degrees
- moved C29 145.0 mm to (198.4, 94.5)
- moved C30 144.9 mm to (198.3, 98.0)
- moved C31 142.0 mm to (196.6, 117.2)
- moved C67 139.3 mm to (223.4, 60.6), turned to -90 degrees
- moved C66 138.3 mm to (227.3, 60.6), turned to -90 degrees
- moved C69 134.1 mm to (187.1, 55.0), turned to 90 degrees
- moved L7 133.0 mm to (220.6, 89.0)
- moved C68 125.3 mm to (187.1, 60.2), turned to -90 degrees
- moved D1 93.4 mm to (213.5, 108.9), turned to 90 degrees
- moved C32 74.1 mm to (223.7, 43.3)
- moved C37 74.1 mm to (223.7, 35.8)
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- renumbered C9 to C1, C4 to C10, C94 to C100, C100 to C101, C96 to C102, C99 to C103, C103 to C104, C106 to C107, C111 to C108, C113 to C109, C5 to C11, C109 to C110, C107 to C111, C95 to C112, C101 to C113, C97 to C114, C6 to C12, C7 to C13, C8 to C14, C12 to C15, C14 to C16, C18 to C17, C20 to C18, C21 to C19, C10 to C2, C23 to C20, C25 to C21, C26 to C22, C27 to C23, C22 to C24, C24 to C25, C28 to C26, C17 to C27, C19 to C28, C11 to C3, C39 to C32, C41 to C35, C43 to C36, C36 to C37, C40 to C39, C16 to C4, C44 to C43, C37 to C44, C66 to C46, C13 to C5, C56 to C51, C75 to C54, C67 to C58, C15 to C6, C116 to C63, C115 to C64, C114 to C65, C1 to C7, C57 to C70, C2 to C8, C54 to C80, C3 to C9, C55 to C90, C98 to C91, C102 to C92, C104 to C95, C110 to C96, C112 to C97, C108 to C98, C105 to C99, D2 to D1, D9 to D10, D7 to D11, D15 to D12, D14 to D13, D12 to D14, D10 to D15, D8 to D16, D1 to D2, D4 to D3, D3 to D4, D6 to D5, D5 to D6, D13 to D7, D11 to D8, D17 to D9, H3 to H2, H2 to H3, J12 to J10, J14 to J11, J13 to J12, J7 to J6, J9 to J7, J11 to J9, K3 to K1, L5 to L3, L6 to L4, L3 to L5, L9 to L6, L4 to L7, L7 to L8, L8 to L9, R8 to R10, R13 to R12, R12 to R13, R15 to R16, R19 to R17, R20 to R18, R16 to R19, R17 to R21, R24 to R25, R32 to R26, R41 to R27, R36 to R28, R42 to R29, R4 to R3, R37 to R30, R43 to R31, R38 to R32, R25 to R33, R26 to R35, R34 to R36, R35 to R37, R44 to R38, R27 to R39, R5 to R4, R28 to R41, R45 to R42, R29 to R43, R30 to R45, R58 to R46, R55 to R47, R54 to R48, R3 to R5, R68 to R50, R69 to R52, R46 to R53, R47 to R54, R64 to R55, R52 to R56, R50 to R57, R72 to R58, R57 to R59, R59 to R60, R56 to R61, R48 to R64, R49 to R65, R53 to R66, R51 to R68, R61 to R69, R10 to R7, R11 to R8, RN3 to RN1, RN1 to RN2, RN2 to RN3, U11 to U10, U13 to U11, U7 to U12, U14 to U13, U8 to U14, U19 to U16, U16 to U17, U21 to U18, U20 to U19, U22 to U20, U24 to U21, U17 to U22, U18 to U23, U9 to U7, U12 to U8, U10 to U9
Connections:
- C64 pad 2: GND -> Net-(U10--Vin)
- C65 pad 2: GND -> Net-(U10--Vin)
- C66 pad 2: GND -> Net-(U10--Vin)
- C67 pad 2: GND -> Net-(U10--Vin)
- L7 pad 2: GND -> Net-(U10--Vin)
- R58 pad 1: /Block Diagram/Output/MCU_OUTPUT_RL_CTR -> /Block Diagram/MCU/MCU_OUTPUT_RL_CTR
- U10 pad 2: GND -> Net-(U10--Vin)

Commit message: Development
Parts:
- moved C29 11.0 mm to (209.3, 93.8)
- moved C30 11.0 mm to (209.2, 97.3)
- moved U4 8.88 mm to (208.7, 103.1), turned to 0 degrees
- moved R13 7.10 mm to (200.3, 101.3)
- moved C66 5.03 mm to (232.3, 60.6)
- moved L6 4.36 mm to (226.1, 59.1)
- moved C67 3.18 mm to (220.2, 60.6)
- moved D1 2.94 mm to (216.3, 109.8)
Changed lines of the file:
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@@
 	(footprint "Capacitor_SMD:C_1210_3225Metric_Pad1.33x2.70mm_HandSolder"
 		(layer "F.Cu")
-		(at 198.3625 94.5)
+		(at 209.3 93.8)
 		(descr "Capacitor SMD 1210 (3225 Metric), square (rectangular) end terminal, IPC-7351 nominal with elongated pad for handsoldering. (Body size source: IPC-SM-782 page 76, https://www.pcb-3d.com/wordpress/wp-content/uploads/ipc-sm-782a_amendment_1_and_2.pdf), generated with kicad-footprint-generator")
 		(tags "capacitor handsolder")
@@
 	(footprint "Capacitor_SMD:C_1210_3225Metric_Pad1.33x2.70mm_HandSolder"
 		(layer "F.Cu")
-		(at 198.3 98)
+		(at 209.2375 97.3)
 		(descr "Capacitor SMD 1210 (3225 Metric), square (rectangular) end terminal, IPC-7351 nominal with elongated pad for handsoldering. (Body size source: IPC-SM-782 page 76, https://www.pcb-3d.com/wordpress/wp-content/uploads/ipc-sm-782a_amendment_1_and_2.pdf), generated with kicad-footprint-generator")
 		(tags "capacitor handsolder")
@@
 	(footprint "Capacitor_SMD:C_1210_3225Metric_Pad1.33x2.70mm_HandSolder"
 		(layer "F.Cu")
-		(at 223.375 60.6 -90)
+		(at 220.2 60.6 -90)
 		(descr "Capacitor SMD 1210 (3225 Metric), square (rectangular) end terminal, IPC-7351 nominal with elongated pad for handsoldering. (Body size source: IPC-SM-782 page 76, https://www.pcb-3d.com/wordpress/wp-content/uploads/ipc-sm-782a_amendment_1_and_2.pdf), generated with kicad-footprint-generator")
 		(tags "capacitor handsolder")
@@
 	(footprint "Resistor_SMD:R_0603_1608Metric_Pad0.98x0.95mm_HandSolder"
 		(layer "F.Cu")
-		(at 206.7 98.2 180)
+		(at 200.3125 101.3 180)
 		(descr "Resistor SMD 0603 (1608 Metric), square (rectangular) end terminal, IPC-7351 nominal with elongated pad for handsoldering. (Body size source: IPC-SM-782 page 72, https://www.pcb-3d.com/wordpress/wp-content/uploads/ipc-sm-782a_amendment_1_and_2.pdf), generated with kicad-footprint-generator")
 		(tags "resistor handsolder")
@@
 	(footprint "Capacitor_SMD:C_1210_3225Metric_Pad1.33x2.70mm_HandSolder"
 		(layer "F.Cu")
-		(at 227.275 60.6 -90)
+		(at 232.3 60.6 -90)
 		(descr "Capacitor SMD 1210 (3225 Metric), square (rectangular) end terminal, IPC-7351 nominal with elongated pad for handsoldering. (Body size source: IPC-SM-782 page 76, https://www.pcb-3d.com/wordpress/wp-content/uploads/ipc-sm-782a_amendment_1_and_2.pdf), generated with kicad-footprint-generator")
 		(tags "capacitor handsolder")
@@
 	(footprint "ETH1CVOLT_A:744774022"
 		(layer "F.Cu")
-		(at 225.375 54.8 180)
+		(at 226.1 59.1 180)
 		(descr "WE-PD2 SMT Power Inductor")
 		(tags "inductor")
@@
 	(footprint "Converter_DCDC:Converter_DCDC_TRACO_TSR1-xxxxE_THT"
 		(layer "F.Cu")
-		(at 201.04 107.5825 -90)
+		(at 208.6825 103.06)
 		(descr "DCDC-Converter, TRACO, TSR1-xxxxE, 1A, Rev. October 31. 2023, https://www.tracopower.com/products/tsr1e.pdf, generated with kicad-footprint-generator StandardBox_generator.py")
 		(tags "DCDC-Converter SWITCHING-REGULATOR STEP-DOWN TRACO TSR1E 2.54MM THT SIP-3 1A")
 		(property "Reference" "U4"
-			(at 1.7 -4.21 90)
+			(at 1.7 -4.21 0)
 			(layer "F.SilkS")
 			(effects
@@
 		)
 		(property "Value" "TSR1-2433E"
-			(at 1.7 9.29 90)
+			(at 1.7 9.29 0)
 			(layer "F.Fab")
 			(effects
@@
 		)
 		(property "Datasheet" "https://www.tracopower.com/products/tsr1e.pdf"
-			(at 0 0 90)
+			(at 0 0 0)
 			(layer "F.Fab")
 			(hide yes)
@@
 		)
 		(property "Description" "1A step-down regulator, fixed 3.3V output voltage, 6-36V input voltage, TO-220 compatible LM78xx replacement"
-			(at 0 0 90)
+			(at 0 0 0)
 			(layer "F.Fab")
 			(hide yes)
@@
 		(attr through_hole)
 		(fp_line
-			(start -2.16 8.45)
-			(end -2.16 0.296)
+			(start -2.16 -3.37)
+			(end 5.56 -3.37)
 			(stroke
 				(width 0.12)
@@
 		)
 		(fp_line
-			(start 5.56 8.45)
-			(end -2.16 8.45)
+			(start -2.16 -0.296)
+			(end -2.16 -3.37)
 			(stroke
 				(width 0.12)
@@
 		)
 		(fp_line
-			(start -2.16 -0.296)
-			(end -2.16 -3.37)
+			(start -2.16 8.45)
+			(end -2.16 0.296)
 			(stroke
 				(width 0.12)
@@
 		)
 		(fp_line
-			(start -2.16 -3.37)
-			(end 5.56 -3.37)
+			(start 5.56 -3.37)
+			(end 5.56 8.45)
 			(stroke
 				(width 0.12)
@@
 		)
 		(fp_line
-			(start 5.56 -3.37)
-			(end 5.56 8.45)
+			(start 5.56 8.45)
+			(end -2.16 8.45)
 			(stroke
 				(width 0.12)
@@
 		)
 		(fp_text user "${REFERENCE}"
-			(at 1.7 2.54 90)
+			(at 1.7 2.54 0)
 			(layer "F.Fab")
 			(effects
@@
 		)
 		(pad "1" thru_hole roundrect
-			(at 0 0 270)
+			(at 0 0)
 			(size 1.5 1.5)
 			(drill 1)
@@
 		)
 		(pad "2" thru_hole circle
-			(at 0 2.54 270)
+			(at 0 2.54)
 			(size 1.5 1.5)
 			(drill 1)
@@
 		)
 		(pad "3" thru_hole circle
-			(at 0 5.08 270)
+			(at 0 5.08)
 			(size 1.5 1.5)
 			(drill 1)
@@
 	(footprint "Diode_SMD:D_SOD-123"
 		(layer "F.Cu")
-		(at 213.5 108.9 90)
+		(at 216.3 109.8 90)
 		(descr "SOD-123")
 		(tags "SOD-123")
