File: HARDWARE/ETH1CVOLT_A/ETH1CVOLT_A.kicad_pcb (KiCad board)
At the start: 2 copper layers, 160 x 100 mm, 262 parts, among them J1 20021111-00010T4LF, J10 Conn_02x04_Odd_Even, J11 Conn_02x04_Odd_Even, J12 Conn_02x04_Odd_Even, J2 RJ45_Wuerth_7499010121A, J3 1843790, J4 Conn_02x04_Odd_Even, J5 Conn_02x04_Odd_Even, J6 FCR7350R, J7 Conn_02x04_Odd_Even, J8 FCR7350B, J9 Conn_02x05_Odd_Even, K1 EE2-3NU, K2 EE2-5NU, Q1 SiS443DN, Q2 MMBT3904, U1 STM32H743VITx, U10 THL30-2415WI, U11 ADP7142ARDZ-5.0, U12 MAX15062C, U13 ADP7142ARDZ-5.0, U14 MAX15062B, U15 LT8365, U16 TCMT1103, U17 LT8365, U18 TCMT1103, U19 TCMT1103, U2 24LC08B-E/MS, U20 TCMT1103, U21 ISO7761FDBQ, U22 ISO7761FDBQ, U23 ISO7761FDBQ, U3 LAN8742A, U4 TSR1-2433E, U5 LT8330_S6, U6 LT8330_S6, U7 LT8330_S6, U8 TPS7A39, U9 LT8330_S6, Y1 NX5032GA-16, Y2 NX5032GA-25

Commit message: Design is being simplified
Parts:
- J10, J11, J12, J4, J5, J7: value Conn_02x04_Odd_Even -> 61030821821
- J9: value Conn_02x05_Odd_Even -> 61031021821
- RN1: value EXB-38V510JV -> R_Pack04
- RN2: value EXB-V8V330JV -> R_Pack04
- RN3: value EXB-V8V103JV -> R_Pack04
Routing:
- net +3.3V: track 0.00 -> 2.77 mm
