File: HARDWARE/ETH1CVOLT_A/ETH1CVOLT_A.kicad_sch (KiCad schematic)
At the start: 0 parts

Commit message: Development
Other:
- note added: "ETH1CVOLT_A"
Changed lines of the file:
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@@
 	(generator_version "9.0")
 	(paper "A3")
+	(text "ETH1CVOLT_A"
+		(exclude_from_sim no)
+		(at 209.55 34.29 0)
+		(effects
+			(font
+				(size 12.7 12.7)
+				(thickness 2.54)
+				(bold yes)
+			)
+		)
+	)
 	(sheet
 		(at 299.72 212.09)
