File: HARDWARE/ETH1CVOLT_B/Block_Diagram.kicad_sch (KiCad schematic)
At the start: 0 parts

Commit message: Development
Other:
- removed sheet Block Diagram
- added sheet DAC (DAC.kicad_sch)
Changed lines of the file:
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@@
 	(generator "eeschema")
 	(generator_version "9.0")
-	(paper "A3")
+	(paper "A4")
 	(sheet
-		(at 299.72 212.09)
-		(size 49.53 34.29)
+		(at 66.04 50.8)
+		(size 52.07 40.64)
 		(exclude_from_sim no)
 		(in_bom yes)
@@
 			(color 255 229 191 1.0000)
 		)
-		(property "Sheetname" "Block Diagram"
-			(at 299.72 211.3784 0)
+		(property "Sheetname" "DAC"
+			(at 66.04 50.0884 0)
 			(effects
 				(font
@@
 			)
 		)
-		(property "Sheetfile" "BlockDiagram.kicad_sch"
-			(at 299.72 246.9646 0)
+		(property "Sheetfile" "DAC.kicad_sch"
+			(at 66.04 92.0246 0)
 			(effects
 				(font
@@
 		)
 		(instances
-			(project "ETH1CVOLT_A"
-				(path "/ca79f0b4-91f7-4537-917d-68d425c03ca3"
-					(page "2")
+			(project "ETH1CVOLT_B"
+				(path "/18612734-e331-4379-b1d3-176cfdcf99d5/b64e35a5-c86f-43a6-acb5-469d75a46b72"
+					(page "3")
 				)
 			)
 		)
 	)
-	(sheet_instances
-		(path "/"
-			(page "1")
-		)
-	)
-	(embedded_fonts no)
 )

Commit message: Development
Other:
- added sheet ADC (ADC.kicad_sch)
- added sheet HV Output (HV_Output.kicad_sch)
- added sheet LV Output (LV_Output.kicad_sch)
- added sheet MUX (MUX.kicad_sch)
- added sheet MV Output (MV_Output.kicad_sch)
- added sheet Voltage Reference (Voltage_Reference.kicad_sch)

Commit message: Development
Other:
- added sheet Current Measurement (Current_Measurement.kicad_sch)
- added sheet Output (Output.kicad_sch)
- sheet ADC ports: added ADC_MEAS, ADC_VOLT_SCLK, ADC_VOLT_SDO, ADC_VOLT_~{CS}, SEL_x1, SEL_x10, SEL_x100; removed none
- sheet DAC ports: added DAC_OUTPUT, DAC_SCLK, DAC_SDIN, DAC_SDO, DAC_~{SYNC}; removed none
- sheet HV Output ports: added HV_DAC, HV_MEAS, HV_OUTPUT, MUX_A0, MUX_A1; removed none
- sheet LV Output ports: added LV_DAC, LV_MEAS, LV_OUTPUT; removed none
- sheet MUX ports: added ADC_MEAS, DAC_OUTPUT, HV_DAC, HV_MEAS, LV_DAC, LV_MEAS, MUX_A0, MUX_A1, MV_DAC, MV_MEAS, VREF_TEST; removed none
- sheet MV Output ports: added MUX_A0, MV_DAC, MV_MEAS, MV_OUTPUT; removed none
- sheet Voltage Reference ports: added SEL_x1, SEL_x10, SEL_x100, VREF_TEST; removed none

Commit message: Development
Other:
- added sheet Connectors Input (Connectors_Input.kicad_sch)
- added sheet Connectors Output (Connectors_Output.kicad_sch)
- sheet ADC ports: added AUX_SEL; removed none
- sheet DAC ports: added AUX_SEL; removed none
- sheet Output ports: added HV_OUT_PMOS, LV_OUT_PMOS, MV_OUT_PMOS; removed none

Commit message: Development
Other:
- sheet Output renamed Output Selection
- sheet Connectors Output ports: added OUT+; removed none
- sheet Output Selection: file Output.kicad_sch -> Output_Selection.kicad_sch
Changed lines of the file:
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@@
+	(wire
+		(pts
+			(xy 335.28 80.01) (xy 353.06 80.01)
+		)
+		(stroke
+			(width 0)
+			(type default)
+		)
+	)
 	(wire
 		(pts
@@
 			)
 		)
+		(pin "OUT+" input
+			(at 353.06 80.01 180)
+			(effects
+				(font
+					(size 1.27 1.27)
+				)
+				(justify left)
+			)
+		)
 		(instances
 			(project "ETH1CVOLT_B"
@@
 			(color 255 229 191 1.0000)
 		)
-		(property "Sheetname" "Output"
+		(property "Sheetname" "Output Selection"
 			(at 243.84 75.4884 0)
 			(effects
@@
 			)
 		)
-		(property "Sheetfile" "Output.kicad_sch"
+		(property "Sheetfile" "Output_Selection.kicad_sch"
 			(at 243.84 156.7946 0)
 			(effects
@@
 			(project "ETH1CVOLT_B"
 				(path "/18612734-e331-4379-b1d3-176cfdcf99d5/b64e35a5-c86f-43a6-acb5-469d75a46b72"
-					(page "8")
+					(page "7")
 				)
 			)
@@
 			(project "ETH1CVOLT_B"
 				(path "/18612734-e331-4379-b1d3-176cfdcf99d5/b64e35a5-c86f-43a6-acb5-469d75a46b72"
-					(page "7")
-				)
-			)
+					(page "8")
+				)
+			)
