File: HARDWARE/ETH1CVOLT_B/Output.kicad_sch (KiCad schematic)
At the start: 3 parts, among them U20 CPC1010N, U21 CPC1010N, U22 CPC1010N

Commit message: Development
Parts:
- added R65, R66, R67: 1k/0.1%, Resistor_SMD:R_0603_1608Metric_Pad0.98x0.95mm_HandSolder, symbol Device:R
- renumbered U20 to U24, U21 to U25, U22 to U26
Connections:
- net at U24.1: now also R65.2
- net at U25.1: now also R66.2
- net at U26.1: now also R67.2
- removed net GND_ISO: U24.2, U25.2, U26.2
- new net +VD_ISO: R65.1, R66.1, R67.1
- new net HV_OUT_PMOS: U26.2
- new net LV_OUT_PMOS: U24.2
- new net MV_OUT_PMOS: U25.2
Other:
- note added: "+/-100V"
- note added: "+/-20V"
- note added: "+/-40V"

Commit message: Development
Parts:
- renumbered R65 to R52, R66 to R53, R67 to R54, U24 to U23, U25 to U24, U26 to U25
Connections:
- net +VD_ISO renamed +5VD_ISO
