File: HARDWARE/ETH1CVOLT_B/ADC.kicad_sch (KiCad schematic)
At the start: 14 parts, among them U11 LTC2400, U12 AD8475xRMZ, U7 ADA4522-1

Commit message: Development
Parts:
- added R10: 180k/0.05%, Resistor_SMD:R_0603_1608Metric_Pad0.98x0.95mm_HandSolder, symbol Device:R
- added R11: 18k/0.05%, Resistor_SMD:R_0603_1608Metric_Pad0.98x0.95mm_HandSolder, symbol Device:R
- added R12: 2k/0.05%, Resistor_SMD:R_0603_1608Metric_Pad0.98x0.95mm_HandSolder, symbol Device:R
- added R6: 100k/0.1%, Resistor_SMD:R_0603_1608Metric_Pad0.98x0.95mm_HandSolder, symbol Device:R
- added U4: DG412LEDQ, Package_SO:TSSOP-16_4.4x5mm_P0.65mm, symbol Analog_Switch:DG412xUE
- added U6: LT1077S8#TRPBF, Package_SO:SOIC-8_3.9x4.9mm_P1.27mm, symbol ETH1CVOLT_B:LT1077S8#TRPBF
- C3: renamed from C5; footprint (none) -> Capacitor_SMD:C_0603_1608Metric_Pad1.08x0.95mm_HandSolder
- C4: renamed from C6; footprint (none) -> Capacitor_SMD:C_0603_1608Metric_Pad1.08x0.95mm_HandSolder
- R13: renamed from R24; footprint (none) -> Resistor_SMD:R_0603_1608Metric_Pad0.98x0.95mm_HandSolder
- R7: renamed from R13; footprint (none) -> Resistor_SMD:R_0603_1608Metric_Pad0.98x0.95mm_HandSolder
- R8: renamed from R14; footprint (none) -> Resistor_SMD:R_0603_1608Metric_Pad0.98x0.95mm_HandSolder
- R9: renamed from R15; footprint (none) -> Resistor_SMD:R_0603_1608Metric_Pad0.98x0.95mm_HandSolder
- TP1, TP4: footprint (none) -> TestPoint:TestPoint_Pad_D1.5mm
- TP2: renamed from TP3; footprint (none) -> TestPoint:TestPoint_Pad_D1.5mm
- TP3: renamed from TP2; footprint (none) -> TestPoint:TestPoint_Pad_D1.5mm
- U8: renamed from U7; value ADA4522-1 -> ADA4522-1ARMZ; footprint (none) -> Package_SO:MSOP-8_3x3mm_P0.65mm
- renumbered D2 to D1, U11 to U5, U12 to U7
Connections:
- net GND_ISO: now also R12.2, U4.4 (V-), U4.5 (GND), U6.4 (V-)
- net at D1.3 (K), R9.2: now also R10.1, U4.3, U6.6; no longer U7.5 (+)
- net +5VA_ISO renamed +VA_ISO
- net +VA_ISO: now also U4.13 (V+), U6.7 (V+)
- net +5VD_ISO renamed +VD_ISO
- net +VD_ISO: now also R6.1, U4.12 (VL)
- net ADC_SCLK renamed ADC_VOLT_SCLK
- net ADC_SDO renamed ADC_VOLT_SDO
- net ADC_~{CS} renamed ADC_VOLT_~{CS}
- new net: R10.2, R11.1, U4.7
- new net: R11.2, R12.1, U4.11
- new net: U4.10, U4.2, U4.6, U6.2 (-)
- new net: U6.3 (+), U7.5 (+)
- new net: R6.2, U4.16
- new net: U4.14, U4.15
- new net SEL_x1: U4.1
- new net SEL_x10: U4.8
- new net SEL_x100: U4.9
- no-connect marks 2 -> 4
Other:
- moved on the sheet: C3, C4, D1, R13, R7, R8, R9, TP1, TP2, TP3, TP4, U5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

Commit message: Development
Parts:
- added C18, C20, C21, C22, C23, C24, C27, C28, C29: 0.1u/100V, symbol Device:C
- added R16: 100k/0.1%, Resistor_SMD:R_0603_1608Metric_Pad0.98x0.95mm_HandSolder, symbol Device:R
- added U6: ADG5419BRMZ-RL7, Package_SO:MSOP-8_3x3mm_P0.65mm, symbol Analog_Switch:ADG419BR
- renumbered C3 to C19, C4 to C25, D1 to D3, R6 to R10, R9 to R11, R10 to R12, R11 to R13, R12 to R14, R13 to R15, R7 to R8, R8 to R9, TP1 to TP3, TP2 to TP4, TP3 to TP5, TP4 to TP6, U7 to U10, U8 to U11, U4 to U7, U5 to U8, U6 to U9
Connections:
- net +2.5VREF_ISO: now also C28.1
- net +21V_ISO: now also C18.1, C27.1, U6.4 (V+)
- net +5VREF_ISO: now also C29.1
- net +VA_ISO: now also C21.1, C22.1, C23.1, C24.1
- net +VD_ISO: now also U6.5 (VL)
- net -21V_ISO: now also C20.1, U6.7 (V-)
- net ADC_MEAS: now also U6.2; no longer TP6.1, U11.3 (+)
- net GND_ISO: now also C18.2, C20.2, C21.2, C22.2, C23.2, C24.2, C27.2, C28.2, C29.2, R16.1, U6.3 (GND)
- new net: TP6.1, U11.3 (+), U6.1
- new net: R16.2, U6.8
- new net AUX_SEL: U6.6
Other:
- note added: "GAIN x1"
- note added: "GAIN x10"
- note added: "GAIN x100"
- moved on the sheet: C19, C25, D3, R10, R11, R12, R13, R14, R15, R8, R9, TP3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

Commit message: Development
Parts:
- added D11: SMAJ14CA, Diode_SMD:D_SMA, symbol Diode:SMAJ14CA
- added R68: 100, Resistor_SMD:R_0603_1608Metric_Pad0.98x0.95mm_HandSolder, symbol Device:R
- C18: renamed from C19; value C -> 6u8/16V; footprint Capacitor_SMD:C_0603_1608Metric_Pad1.08x0.95mm_HandSolder -> Capacitor_SMD:C_0805_2012Metric_Pad1.18x1.45mm_HandSolder
- C19: renamed from C18; footprint (none) -> Capacitor_SMD:C_0603_1608Metric_Pad1.08x0.95mm_HandSolder
- C20, C21, C22, C23, C24: footprint (none) -> Capacitor_SMD:C_0603_1608Metric_Pad1.08x0.95mm_HandSolder
- C25: value C -> 6u8/16V; footprint Capacitor_SMD:C_0603_1608Metric_Pad1.08x0.95mm_HandSolder -> Capacitor_SMD:C_0805_2012Metric_Pad1.18x1.45mm_HandSolder
- C26: renamed from C27; footprint (none) -> Capacitor_SMD:C_0603_1608Metric_Pad1.08x0.95mm_HandSolder
- C27: renamed from C28; footprint (none) -> Capacitor_SMD:C_0603_1608Metric_Pad1.08x0.95mm_HandSolder
- C28: renamed from C29; footprint (none) -> Capacitor_SMD:C_0603_1608Metric_Pad1.08x0.95mm_HandSolder
- R11, R15: value R -> 100
- TP3, TP4, TP5, TP6: now left out of the parts list
Connections:
- net GND_ISO: now also D11.1 (A1)
- net at TP5.1, U10.9 (+IN0.4x): now also D11.2 (A2), R68.1; no longer U11.2 (-), U11.6
- new net: R68.2, U11.2 (-), U11.6
Other:
- moved on the sheet: C18, C19, C20, C21, C22, C23, C24, C25, C26, C27, C28, D3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

Commit message: Development
Parts:
- added TP10, TP11: TestPoint, TestPoint:TestPoint_Pad_D1.5mm, symbol Connector:TestPoint
Connections:
- net at U10.5 (+), U9.3 (+): now also TP11.1
- net at D3.3 (K), R11.2, R12.1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: now also TP10.1
Other:
- moved on the sheet: TP6
Changed lines of the file:
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@@
 	)
 	(junction
+		(at 331.47 93.98)
+		(diameter 0)
+		(color 0 0 0 0)
+	)
+	(junction
 		(at 175.26 248.92)
 		(diameter 0)
@@
 	)
 	(junction
+		(at 238.76 104.14)
+		(diameter 0)
+		(color 0 0 0 0)
+	)
+	(junction
 		(at 194.31 259.08)
 		(diameter 0)
@@
 	)
 	(junction
+		(at 148.59 106.68)
+		(diameter 0)
+		(color 0 0 0 0)
+	)
+	(junction
 		(at 185.42 248.92)
 		(diameter 0)
@@
 	)
 	(junction
-		(at 330.2 93.98)
-		(diameter 0)
-		(color 0 0 0 0)
-	)
-	(junction
 		(at 170.18 133.35)
 		(diameter 0)
@@
 	(wire
 		(pts
-			(xy 330.2 93.98) (xy 345.44 93.98)
-		)
-		(stroke
-			(width 0)
-			(type default)
-		)
-	)
-	(wire
-		(pts
 			(xy 24.13 240.03) (xy 27.94 240.03)
 		)
@@
 	(wire
 		(pts
+			(xy 238.76 104.14) (xy 238.76 105.41)
+		)
+		(stroke
+			(width 0)
+			(type default)
+		)
+	)
+	(wire
+		(pts
 			(xy 181.61 139.7) (xy 182.88 139.7)
 		)
@@
 	(wire
 		(pts
+			(xy 238.76 104.14) (xy 255.27 104.14)
+		)
+		(stroke
+			(width 0)
+			(type default)
+		)
+	)
+	(wire
+		(pts
 			(xy 181.61 161.29) (xy 181.61 162.56)
 		)
@@
 	(wire
 		(pts
-			(xy 132.08 106.68) (xy 170.18 106.68)
+			(xy 132.08 106.68) (xy 148.59 106.68)
 		)
 		(stroke
@@
 	(wire
 		(pts
+			(xy 148.59 106.68) (xy 170.18 106.68)
+		)
+		(stroke
+			(width 0)
+			(type default)
+		)
+	)
+	(wire
+		(pts
 			(xy 255.27 91.44) (xy 262.89 91.44)
 		)
@@
 	(wire
 		(pts
-			(xy 328.93 93.98) (xy 330.2 93.98)
+			(xy 328.93 93.98) (xy 331.47 93.98)
 		)
 		(stroke
@@
 	(wire
 		(pts
-			(xy 189.23 104.14) (xy 255.27 104.14)
+			(xy 189.23 104.14) (xy 238.76 104.14)
 		)
 		(stroke
@@
 	(wire
 		(pts
-			(xy 330.2 92.71) (xy 330.2 93.98)
+			(xy 331.47 92.71) (xy 331.47 93.98)
 		)
 		(stroke
@@
 	(wire
 		(pts
+			(xy 331.47 93.98) (xy 345.44 93.98)
+		)
+		(stroke
+			(width 0)
+			(type default)
+		)
+	)
+	(wire
+		(pts
 			(xy 330.2 111.76) (xy 312.42 111.76)
 		)
@@
 	(wire
 		(pts
+			(xy 148.59 106.68) (xy 148.59 109.22)
+		)
+		(stroke
+			(width 0)
+			(type default)
+		)
+	)
+	(wire
+		(pts
 			(xy 270.51 257.81) (xy 270.51 260.35)
 		)
@@
 			)
 		)
-		(property "Component Class" "ISO"
+		(property "Component Class" ""
 			(at 14.6685 15.4305 0)
 			(effects
@@
 	)
 	(symbol
+		(lib_id "Connector:TestPoint")
+		(at 148.59 109.22 180)
+		(unit 1)
+		(exclude_from_sim no)
+		(in_bom yes)
+		(on_board yes)
+		(dnp no)
+		(fields_autoplaced yes)
+		(property "Reference" "TP10"
+			(at 151.13 111.2519 0)
+			(effects
+				(font
+					(size 1.27 1.27)
+				)
+				(justify right)
+			)
+		)
+		(property "Value" "TestPoint"
+			(at 151.13 113.7919 0)
+			(effects
+				(font
+					(size 1.27 1.27)
+				)
+				(justify right)
+			)
+		)
+		(property "Footprint" "TestPoint:TestPoint_Pad_D1.5mm"
+			(at 143.51 109.22 0)
+			(effects
+				(font
+					(size 1.27 1.27)
+				)
+				(hide yes)
+			)
+		)
+		(property "Datasheet" "~"
+			(at 143.51 109.22 0)
+			(effects
+				(font
+					(size 1.27 1.27)
+				)
+				(hide yes)
+			)
+		)
+		(property "Description" "test point"
+			(at 148.59 109.22 0)
+			(effects
+				(font
+					(size 1.27 1.27)
+				)
+				(hide yes)
+			)
+		)
+		(pin "1"
+		)
+		(instances
+			(project ""
+				(path "/18612734-e331-4379-b1d3-176cfdcf99d5/b64e35a5-c86f-43a6-acb5-469d75a46b72/491d5013-f6ed-4b41-b769-ee3854033f07"
+					(reference "TP10")
+					(unit 1)
+				)
+			)
+		)
+	)
+	(symbol
 		(lib_id "Device:C")
 		(at 194.31 254 0)
@@
 	(symbol
 		(lib_id "Connector:TestPoint")
-		(at 330.2 92.71 0)
+		(at 331.47 92.71 0)
 		(unit 1)
 		(exclude_from_sim no)
@@
 		(fields_autoplaced yes)
 		(property "Reference" "TP6"
-			(at 332.74 88.1379 0)
+			(at 334.01 88.1379 0)
 			(effects
 				(font
@@
 		)
 		(property "Value" "TestPoint"
-			(at 332.74 90.6779 0)
+			(at 334.01 90.6779 0)
 			(effects
 				(font
@@
 		)
 		(property "Footprint" "TestPoint:TestPoint_Pad_D1.5mm"
-			(at 335.28 92.71 0)
+			(at 336.55 92.71 0)
 			(effects
 				(font
@@
 		)
 		(property "Datasheet" "~"
-			(at 335.28 92.71 0)
+			(at 336.55 92.71 0)
 			(effects
 				(font
@@
 		)
 		(property "Description" "test point"
-			(at 330.2 92.71 0)
+			(at 331.47 92.71 0)
 			(effects
 				(font
@@
 					(unit 1)
 				)
+			)
+		)
+	)
+	(symbol
+		(lib_id "Connector:TestPoint")
+		(at 238.76 105.41 180)
+		(unit 1)
+		(exclude_from_sim no)
+		(in_bom yes)
+		(on_board yes)
+		(dnp no)
+		(fields_autoplaced yes)
+		(property "Reference" "TP11"
+			(at 241.3 107.4419 0)
+			(effects
+				(font
+					(size 1.27 1.27)
+				)
+				(justify right)
+			)
+		)
+		(property "Value" "TestPoint"
+			(at 241.3 109.9819 0)
+			(effects
+				(font
+					(size 1.27 1.27)
+				)
+				(justify right)
+			)
+		)
+		(property "Footprint" "TestPoint:TestPoint_Pad_D1.5mm"
+			(at 233.68 105.41 0)
+			(effects
+				(font
+					(size 1.27 1.27)
+				)
+				(hide yes)
+			)
+		)
+		(property "Datasheet" "~"
+			(at 233.68 105.41 0)
+			(effects
+				(font
+					(size 1.27 1.27)
+				)
+				(hide yes)
+			)
+		)
+		(property "Description" "test point"
+			(at 238.76 105.41 0)
+			(effects
+				(font
+					(size 1.27 1.27)
+				)
+				(hide yes)
+			)
+		)
+		(pin "1"
+		)
+		(instances
+			(project "ETH1CVOLT_B"
+				(path "/18612734-e331-4379-b1d3-176cfdcf99d5/b64e35a5-c86f-43a6-acb5-469d75a46b72/491d5013-f6ed-4b41-b769-ee3854033f07"
+					(reference "TP11")
+					(unit 1)
+				)
