File: HARDWARE/ETH1CVOLT_B/Connectors_Output.kicad_sch (KiCad schematic)
At the start: 0 parts

Commit message: Development
Parts:
- added J2: Conn_02x04_Odd_Even, Connector_PinSocket_2.54mm:PinSocket_2x04_P2.54mm_Vertical_SMD, symbol Connector_Generic:Conn_02x04_Odd_Even
Connections:
- new net GND_ISO: J2.7 (Pin_7), J2.8 (Pin_8)
- new net OUT+: J2.1 (Pin_1), J2.2 (Pin_2)
- no-connect marks 0 -> 4
