File: HARDWARE/ETH1CVOLT_B/Current_Measurement.kicad_sch (KiCad schematic)
At the start: 44 parts, among them U23 TEC3-2423UI, U24 TPS7A39, U25 MAX15062C, U27 ADS8681RUM, U28 ADP7142AUJZ-5.0, U29 AD8221ARM

Commit message: Development
Parts:
- added U12: ISO7761FDW, Package_SO:SOIC-16W_7.5x10.3mm_P1.27mm, symbol Isolator:ISO7761FDW
- R53: renamed from R51; value 2k4 -> 118k
- R54: renamed from R52; value 165k -> 107k
- renumbered C19 to C50, C20 to C51, C21 to C52, C23 to C53, C22 to C54, C24 to C55, C25 to C56, C30 to C57, C82 to C58, C83 to C59, C86 to C60, C87 to C61, C28 to C62, C29 to C63, C27 to C64, C26 to C65, C47 to C66, C49 to C67, C18 to C68, C54 to C69, C61 to C70, C64 to C71, C84 to C72, C88 to C73, L7 to L1, R49 to R52, R54 to R55, R59 to R56, R50 to R57, R55 to R58, R56 to R59, R53 to R62, R57 to R63, R58 to R64, U23 to U27, U24 to U28, U27 to U29, U25 to U30, U29 to U31, U28 to U32
Connections:
- net +5V: now also U12.16 (Vcc2)
- net ADC_CURR_SCLK: now also U12.3 (INB); no longer U29.10 (SCLK)
- net ADC_CURR_SDI: now also U12.4 (INC); no longer U29.8 (SDI)
- net ADC_CURR_SDO: now also U12.7 (OUTF); no longer U29.11 (SDO-0)
- net ADC_CURR_~{CS}: now also U12.2 (INA); no longer U29.9 (CONVST/~{CS})
- net GNDS: now also U12.9 (GND2)
- net GND_ISO: now also U12.8 (GND1)
- new net +VD_ISO: U12.1 (Vcc1)
- new net ADC_CURR_SCLK_ISO: U12.14 (OUTB), U29.10 (SCLK)
- new net ADC_CURR_SDI_ISO: U12.13 (OUTC), U29.8 (SDI)
- new net ADC_CURR_SDO_ISO: U12.10 (INF), U29.11 (SDO-0)
- new net ADC_CURR_~{CS}_ISO: U12.15 (OUTA), U29.9 (CONVST/~{CS})
- no-connect marks 5 -> 9
Other:
- note added: "CURRENT MEASUREMENT"
- note added: "GAIN x100"
- note added: "ISOLATED POWER SUPPLY"
- moved on the sheet: C57, C62, C63, C64, C65, C66, C67, C68, C69, C70, C71, C72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

Commit message: Development
Parts:
- removed C64: 10u, symbol Device:C
- removed C65: 1u, symbol Device:C
- removed U12: ISO7761FDW, Package_SO:SOIC-16W_7.5x10.3mm_P1.27mm, symbol Isolator:ISO7761FDW
- added C68: 10u/16V, Capacitor_SMD:C_0805_2012Metric_Pad1.18x1.45mm_HandSolder, symbol Device:C
- added C69: 1u/50V, Capacitor_SMD:C_0805_2012Metric_Pad1.18x1.45mm_HandSolder, symbol Device:C
- added U27: ISO7761FDBQ, Package_SO:SSOP-16_3.9x4.9mm_P0.635mm, symbol Isolator:ISO7761FDBQ
- C60: renamed from C56; value C -> C/50V; footprint (none) -> Capacitor_SMD:C_0805_2012Metric_Pad1.18x1.45mm_HandSolder
- C61: renamed from C57; value 1u -> 1u/50V; footprint (none) -> Capacitor_SMD:C_0805_2012Metric_Pad1.18x1.45mm_HandSolder
- C62: value 10u -> 10u/16V; footprint (none) -> Capacitor_SMD:C_0805_2012Metric_Pad1.18x1.45mm_HandSolder
- C65: renamed from C63; value 1u -> 1u/50V; footprint (none) -> Capacitor_SMD:C_0805_2012Metric_Pad1.18x1.45mm_HandSolder
- C71: renamed from C68; value C -> C/50V; footprint (none) -> Capacitor_SMD:C_0805_2012Metric_Pad1.18x1.45mm_HandSolder
- C73: renamed from C69; value 1u -> 1u/50V
- L1: footprint (none) -> ETH1CVOLT_A:74408063470
- R59: renamed from R56; footprint (none) -> Resistor_SMD:R_0603_1608Metric_Pad0.98x0.95mm_HandSolder
- R62: renamed from R57; footprint (none) -> Resistor_SMD:R_0603_1608Metric_Pad0.98x0.95mm_HandSolder
- R63: renamed from R60; footprint (none) -> Resistor_SMD:R_1206_3216Metric_Pad1.30x1.75mm_HandSolder
- R64: renamed from R61; footprint (none) -> Resistor_SMD:R_1206_3216Metric_Pad1.30x1.75mm_HandSolder
- R65: renamed from R62; footprint (none) -> Resistor_SMD:R_1206_3216Metric_Pad1.30x1.75mm_HandSolder
- renumbered C50 to C54, C51 to C55, C52 to C56, C53 to C57, C54 to C58, C55 to C59, C58 to C63, C59 to C64, C60 to C66, C61 to C67, C66 to C70, C67 to C72, C70 to C74, C71 to C75, C72 to C76, C73 to C77, R52 to R55, R53 to R56, R54 to R57, R55 to R58, R58 to R60, R59 to R61, R63 to R66, R64 to R67, U27 to U26
Connections:
- net +5V: now also U27.16 (Vcc2)
- net +VD_ISO: now also U27.1 (Vcc1)
- net ADC_CURR_SCLK: now also U27.3 (INB)
- net ADC_CURR_SDI: now also U27.4 (INC)
- net ADC_CURR_SDO: now also U27.7 (OUTF)
- net ADC_CURR_~{CS}: now also U27.2 (INA)
- net GNDS: now also C68.2, C69.2, U27.9 (GND2)
- net GND_ISO: now also U27.8 (GND1)
- net at U29.4 (REFCAP): now also C68.1, C69.1
- net ADC_CURR_SCLK_ISO renamed CURR_SCLK_ISO
- net CURR_SCLK_ISO: now also U27.14 (OUTB)
- net ADC_CURR_SDI_ISO renamed CURR_SDI_ISO
- net CURR_SDI_ISO: now also U27.13 (OUTC)
- net ADC_CURR_SDO_ISO renamed CURR_SDO_ISO
- net CURR_SDO_ISO: now also U27.10 (INF)
- net ADC_CURR_~{CS}_ISO renamed CURR_~{CS}_ISO
- net CURR_~{CS}_ISO: now also U27.15 (OUTA)
Other:
- note added: "+15V/100mA"
- note added: "-15V/100mA"
- moved on the sheet: C61, C62, C65

Commit message: Development
Parts:
- added TP12, TP13, TP14, TP15, TP16, TP17, TP18: TestPoint, TestPoint:TestPoint_Pad_D1.5mm, symbol Connector:TestPoint
- C71: value C/50V -> 10u/100V; footprint Capacitor_SMD:C_0805_2012Metric_Pad1.18x1.45mm_HandSolder -> Capacitor_SMD:C_1210_3225Metric_Pad1.33x2.70mm_HandSolder
- R59: value R -> 100
- R63, R64: value 0 -> 0/200V
Connections:
- net +14V: now also TP15.1
- net +15V: now also TP17.1
- net +5V: now also TP13.1
- net -14V: now also TP16.1
- net -15V: now also TP18.1
- net GNDS: now also TP14.1
- net at C71.1, R59.1, U29.5 (AIN_P): now also TP12.1
Other:
- moved on the sheet: R59
