File: HARDWARE/ETH1CVOLT_B/DAC.kicad_sch (KiCad schematic)
At the start: 6 parts, among them U1 DAC81401PWR, U2 DAC81401PWR

Commit message: Development
Parts:
- added R11, R7, R9: 10k/0.1%, symbol Device:R
- added RN1, RN2: MPMT1002AT5, Package_TO_SOT_SMD:SOT-23, symbol Device:VoltageDivider_CenterPin3
- added U10, U3, U4: ADA4522-4, symbol Amplifier_Operational:ADA4522-4
- R3: renamed from R1; now not fitted; now left out of the parts list
- renumbered R2 to R4
Connections:
- net +3V3_ISO is gone; now on net +5VD_ISO: U2.17 (IOVDD)
- net +21V_ISO: now also U4.4 (V+)
- net -21V_ISO: now also U4.11 (V-)
- net GND_ISO: now also U10.3 (+), U3.5 (+)
- net VOUT_B: now reaches C2.2, R4.1, U2.9 (VOUT)
- net VOUT_B: now also U4.10 (+)
- net at U2.10 (VSENSEP): now also U4.8, U4.9 (-)
- net DAC_SCLK: now reaches U1.14 (SCLK), U2.14 (SCLK)
- net DAC_SDIN: now reaches U2.15 (SDIN)
- net DAC_~{SYNC}: now reaches U1.16 (~{SYNC}), U2.16 (~{SYNC})
- net VOUT_A: now reaches C1.2, R3.1, U1.9 (VOUT)
- net VOUT_A: now also RN1.2, U4.12 (+)
- net at R3.2: now also R4.2, R7.1, RN1.3, U10.2 (-)
- net at U1.10 (VSENSEP): now also U4.13 (-), U4.14
- net DAC_SDO: now reaches U1.13 (SDO)
- net +5VD_ISO: now reaches U1.17 (IOVDD)
- net +5V_ISO renamed +5VA_ISO
- new net: R7.2, R9.1, RN1.1, RN2.2, U10.1
- new net: R11.1, R9.2, RN2.3, U3.6 (-)
- new net DAC_OUTPUT: R11.2, RN2.1, U3.7
Other:
- note added: "+/-20V"
- moved on the sheet: C1, C2, R4, U1, U2

Commit message: Development
Parts:
- removed U10, U3, U4: ADA4522-4, symbol Amplifier_Operational:ADA4522-4
- added U1: ADA4522-4ARUZ, Package_SO:TSSOP-14_4.4x5mm_P0.65mm, symbol Amplifier_Operational:ADA4522-4
- C1, C2: footprint (none) -> Capacitor_SMD:C_0603_1608Metric_Pad1.08x0.95mm_HandSolder
- R1: renamed from R4; footprint (none) -> Resistor_SMD:R_0603_1608Metric_Pad0.98x0.95mm_HandSolder
- R2: renamed from R3; footprint (none) -> Resistor_SMD:R_0603_1608Metric_Pad0.98x0.95mm_HandSolder
- R3: renamed from R7; footprint (none) -> Resistor_SMD:R_0603_1608Metric_Pad0.98x0.95mm_HandSolder
- R4: renamed from R9; footprint (none) -> Resistor_SMD:R_0603_1608Metric_Pad0.98x0.95mm_HandSolder
- R5: renamed from R11; footprint (none) -> Resistor_SMD:R_0603_1608Metric_Pad0.98x0.95mm_HandSolder
- renumbered U1 to U2, U2 to U3
Connections:
- net +21V_ISO: now also U1.4 (V+)
- net -21V_ISO: now also U1.11 (V-)
- net DAC_OUTPUT: now also U1.7
- net GND_ISO: now also U1.3 (+), U1.5 (+)
- net VOUT_A: now also U1.10 (+)
- net VOUT_B: now also U1.12 (+)
- net at R3.2, R4.1, RN1.1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: now also U1.1
- net at R4.2, R5.1, RN2.3: now also U1.6 (-)
- net at U2.10 (VSENSEP): now also U1.8, U1.9 (-)
- net at U3.10 (VSENSEP): now also U1.13 (-), U1.14
- net at R1.2, R2.2, R3.1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: now also U1.2 (-)
- net +5VA_ISO renamed +VA_ISO
- net +5VD_ISO renamed +VD_ISO

Commit message: Development
Parts:
- added C1, C10, C13, C14, C15, C16, C17, C2, C3, C4, C5, C6, C7, C8, C9: 0.1u/100V, symbol Device:C
- added D1: SMAJ14CA, Diode_SMD:D_SMA, symbol Diode:SMAJ14CA
- added D2: BAV199, Package_TO_SOT_SMD:SOT-23, symbol Diode:BAV99
- added J1: Conn_Coaxial, symbol Connector:Conn_Coaxial
- added R5, R7: 10k/0.1%, Resistor_SMD:R_0603_1608Metric_Pad0.98x0.95mm_HandSolder, symbol Device:R
- added RN3: MPMT1002AT5, Package_TO_SOT_SMD:SOT-23, symbol Device:VoltageDivider_CenterPin3
- added TP1, TP2: TestPoint, symbol Connector:TestPoint
- added U1: ADG5419BRMZ-RL7, Package_SO:MSOP-8_3x3mm_P0.65mm, symbol Analog_Switch:ADG419BR
- added U5: ADA4522-1ARMZ, Package_SO:MSOP-8_3x3mm_P0.65mm, symbol Amplifier_Operational:ADA4522-1
- renumbered C1 to C11, C2 to C12, R5 to R6, U1 to U2, U2 to U3, U3 to U4
Connections:
- net +21V_ISO: now also C10.1, C2.1, C4.1, C6.1, C8.1, D2.2 (A), U1.4 (V+), U5.7 (V+)
- net +VA_ISO: now also C13.1, C15.1
- net +VD_ISO: now also C14.1, C16.1, C17.1, U1.5 (VL)
- net -21V_ISO: now also C1.1, C3.1, C5.1, C7.1, C9.1, D2.1 (K), U1.7 (V-), U5.4 (V-)
- net DAC_OUTPUT: now also U1.1; no longer R6.2, RN2.1, U2.7
- net GND_ISO: now also C1.2, C10.2, C13.2, C14.2, C15.2, C16.2, C17.2, C2.2, C3.2, C4.2, C5.2, C6.2, C7.2, C8.2, C9.2, D1.1 (A1), J1.2 (Ext), U1.3 (GND)
- net at U4.12 (~{FAULT}): now also TP2.1
- net at U3.12 (~{FAULT}): now also TP1.1
- new net: R7.1, RN3.2, U1.8, U5.6
- new net: R5.1, R7.2, RN3.3
- new net: R6.2, RN2.1, U1.2, U2.7
- new net: D1.2 (A2), D2.3 (K), J1.1 (In), U5.3 (+)
- new net: R5.2, RN3.1, U5.2 (-)
- new net AUX_SEL: U1.6
Other:
- note added: "+/-10V"
- moved on the sheet: C11, C12, R1, R2, R3, R4, R6, RN1, RN2, U2A, U2B, U2C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

Commit message: Development
Parts:
- added C78, C81: 0.1u/100V, Capacitor_SMD:C_0603_1608Metric_Pad1.08x0.95mm_HandSolder, symbol Device:C
- added C79, C80: 1u/50V, Capacitor_SMD:C_0603_1608Metric_Pad1.08x0.95mm_HandSolder, symbol Device:C
- C1, C10, C13, C14, C15, C16, C17, C2, C3, C4, C5, C6, C7, C8, C9: footprint (none) -> Capacitor_SMD:C_0603_1608Metric_Pad1.08x0.95mm_HandSolder
- C11, C12: value 470p -> 470p/100V
- J1: value Conn_Coaxial -> 73251-1153; footprint (none) -> Connector_Coaxial:SMA_Molex_73251-1153_EdgeMount_Horizontal
- TP1, TP2: footprint (none) -> TestPoint:TestPoint_Pad_D1.5mm; now left out of the parts list
Connections:
- net GND_ISO: now also R5.2, RN3.1, U5.2 (-), C78.1, C79.1, C80.1, C81.1
- new net +5VREF_ISO: C78.2, C79.2, C80.2, C81.2, U3.1 (VREFIO), U4.1 (VREFIO)
Other:
- moved on the sheet: C1, C10, C11, C12, C13, C14, C15, C16, C17, C2, C3, C4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

Commit message: Development
Parts:
- added R69: 100, Resistor_SMD:R_0603_1608Metric_Pad0.98x0.95mm_HandSolder, symbol Device:R
- added TP7, TP8, TP9: TestPoint, TestPoint:TestPoint_Pad_D1.5mm, symbol Connector:TestPoint
Connections:
- net at R7.1, RN3.2, U1.8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: now also TP7.1
- net at R1.2, R2.2, R3.1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: now also TP9.1
- net at R6.2, RN2.1, U1.2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: now also TP8.1
- net at D1.2 (A2), D2.3 (K), U5.3 (+): now also R69.2; no longer J1.1 (In)
- new net: J1.1 (In), R69.1
Other:
- moved on the sheet: D1, D2, J1, R5, R7, RN3, U5
