File: HARDWARE/ETH1CVOLT_B/ETH1CVOLT_B.kicad_pcb (KiCad board)
At the start: 2 copper layers, 92 parts, among them Q1 PBHV8140Z,115, Q2 PBHV9540Z,115, U1 ADA4522-4ARUZ, U10 OPA593, U11 OPA593, U12 ADA4522-1ARMZ, U13 TMUX8109PWR, U16 74LV1T08GV, U17 DG412EUE+, U18 LT1027CCS8-5#PBF, U19 ADA4077-1xRM, U2 DAC81401PWR, U20 CPC1010N, U21 CPC1010N, U22 CPC1010N, U3 DAC81401PWR, U4 DG412LEDQ, U5 LTC2400, U6 LT1077S8#TRPBF, U7 AD8475xRMZ, U8 ADA4522-1ARMZ, U9 SN74LVC1G125DBV

Commit message: Development
Parts:
- removed the D3 at (54.7, 83.4)
- added C1: 0.1u/100V, Capacitor_SMD:C_0603_1608Metric_Pad1.08x0.95mm_HandSolder, F.Cu at (154.0, 109.9)
- added C10: 0.1u/100V, Capacitor_SMD:C_0603_1608Metric_Pad1.08x0.95mm_HandSolder, F.Cu at (158.3, 117.4)
- added C13: 0.1u/100V, Capacitor_SMD:C_0603_1608Metric_Pad1.08x0.95mm_HandSolder, F.Cu at (158.3, 119.9)
- added C14: 0.1u/100V, Capacitor_SMD:C_0603_1608Metric_Pad1.08x0.95mm_HandSolder, F.Cu at (158.3, 122.4)
- added C15: 0.1u/100V, Capacitor_SMD:C_0603_1608Metric_Pad1.08x0.95mm_HandSolder, F.Cu at (162.7, 109.9)
- added C16: 0.1u/100V, Capacitor_SMD:C_0603_1608Metric_Pad1.08x0.95mm_HandSolder, F.Cu at (162.7, 112.4)
- added C17: 0.1u/100V, Capacitor_SMD:C_0603_1608Metric_Pad1.08x0.95mm_HandSolder, F.Cu at (162.7, 114.9)
- added C19: 0.1u/100V, Capacitor_SMD:C_0603_1608Metric_Pad1.08x0.95mm_HandSolder, F.Cu at (154.0, 131.5)
- added C2: 0.1u/100V, Capacitor_SMD:C_0603_1608Metric_Pad1.08x0.95mm_HandSolder, F.Cu at (154.0, 112.4)
- added C20: 0.1u/100V, Capacitor_SMD:C_0603_1608Metric_Pad1.08x0.95mm_HandSolder, F.Cu at (154.0, 134.0)
- added C21: 0.1u/100V, Capacitor_SMD:C_0603_1608Metric_Pad1.08x0.95mm_HandSolder, F.Cu at (154.0, 136.5)
- added C22: 0.1u/100V, Capacitor_SMD:C_0603_1608Metric_Pad1.08x0.95mm_HandSolder, F.Cu at (154.0, 139.0)
- added C23: 0.1u/100V, Capacitor_SMD:C_0603_1608Metric_Pad1.08x0.95mm_HandSolder, F.Cu at (154.0, 141.5)
- added C24: 0.1u/100V, Capacitor_SMD:C_0603_1608Metric_Pad1.08x0.95mm_HandSolder, F.Cu at (154.0, 144.0)
- added C26: 0.1u/100V, Capacitor_SMD:C_0603_1608Metric_Pad1.08x0.95mm_HandSolder, F.Cu at (158.3, 131.5)
- added C27: 0.1u/100V, Capacitor_SMD:C_0603_1608Metric_Pad1.08x0.95mm_HandSolder, F.Cu at (158.3, 134.0)
- added C28: 0.1u/100V, Capacitor_SMD:C_0603_1608Metric_Pad1.08x0.95mm_HandSolder, F.Cu at (158.3, 136.5)
- added C29: 0.1u/100V, Capacitor_SMD:C_0603_1608Metric_Pad1.08x0.95mm_HandSolder, F.Cu at (156.8, 149.9)
- added C3: 0.1u/100V, Capacitor_SMD:C_0603_1608Metric_Pad1.08x0.95mm_HandSolder, F.Cu at (154.0, 114.9)
- added C30: 0.1u/100V, Capacitor_SMD:C_0603_1608Metric_Pad1.08x0.95mm_HandSolder, F.Cu at (156.8, 152.5)
- added C31: 0.1u/100V, Capacitor_SMD:C_0603_1608Metric_Pad1.08x0.95mm_HandSolder, F.Cu at (156.8, 155.0)
- added C32: 0.1u/100V, Capacitor_SMD:C_0603_1608Metric_Pad1.08x0.95mm_HandSolder, F.Cu at (156.8, 157.5)
- added C33: 0.1u/100V, Capacitor_SMD:C_0603_1608Metric_Pad1.08x0.95mm_HandSolder, F.Cu at (156.8, 160.0)
- added C34: 0.1u/100V, Capacitor_SMD:C_0603_1608Metric_Pad1.08x0.95mm_HandSolder, F.Cu at (122.6, 167.5)
- added C35: 0.1u/100V, Capacitor_SMD:C_0603_1608Metric_Pad1.08x0.95mm_HandSolder, F.Cu at (122.6, 170.0)
- added C38: 0.1u/250V, Capacitor_SMD:C_1206_3216Metric_Pad1.33x1.80mm_HandSolder, F.Cu at (143.7, 150.4)
- added C39: 0.1u/250V, Capacitor_SMD:C_1206_3216Metric_Pad1.33x1.80mm_HandSolder, F.Cu at (143.7, 153.7)
- added C4: 0.1u/100V, Capacitor_SMD:C_0603_1608Metric_Pad1.08x0.95mm_HandSolder, F.Cu at (154.0, 117.4)
- added C40: 0.1u/250V, Capacitor_SMD:C_1206_3216Metric_Pad1.33x1.80mm_HandSolder, F.Cu at (143.7, 157.1)
- added C41: 0.1u/250V, Capacitor_SMD:C_1206_3216Metric_Pad1.33x1.80mm_HandSolder, F.Cu at (143.7, 160.4)
- added C42: 0.1u/100V, Capacitor_SMD:C_0603_1608Metric_Pad1.08x0.95mm_HandSolder, F.Cu at (148.8, 166.5)
- added C43: C/250V, Capacitor_SMD:C_1206_3216Metric_Pad1.33x1.80mm_HandSolder, F.Cu at (143.7, 163.8)
- added C44: C/250V, Capacitor_SMD:C_1206_3216Metric_Pad1.33x1.80mm_HandSolder, F.Cu at (143.7, 167.1)
- added C45: C/200V, Capacitor_SMD:C_1206_3216Metric_Pad1.33x1.80mm_HandSolder, F.Cu at (143.7, 170.5)
- added C5: 0.1u/100V, Capacitor_SMD:C_0603_1608Metric_Pad1.08x0.95mm_HandSolder, F.Cu at (154.0, 119.9)
- added C54: 4u7/50V, Capacitor_SMD:C_1210_3225Metric_Pad1.33x2.70mm_HandSolder, F.Cu at (128.8, 110.8)
- added C55: 10u/50V, Capacitor_SMD:C_1210_3225Metric_Pad1.33x2.70mm_HandSolder, F.Cu at (128.8, 115.0)
- added C56: 4u7/50V, Capacitor_SMD:C_1210_3225Metric_Pad1.33x2.70mm_HandSolder, F.Cu at (128.8, 119.2)
- added C57: 4u7/50V, Capacitor_SMD:C_1210_3225Metric_Pad1.33x2.70mm_HandSolder, F.Cu at (128.8, 123.5)
- added C58: 10u/50V, Capacitor_SMD:C_1210_3225Metric_Pad1.33x2.70mm_HandSolder, F.Cu at (134.8, 110.8)
- added C59: 10u/50V, Capacitor_SMD:C_1210_3225Metric_Pad1.33x2.70mm_HandSolder, F.Cu at (134.8, 115.0)
- added C6: 0.1u/100V, Capacitor_SMD:C_0603_1608Metric_Pad1.08x0.95mm_HandSolder, F.Cu at (154.0, 122.4)
- added C60: C/50V, Capacitor_SMD:C_0805_2012Metric_Pad1.18x1.45mm_HandSolder, F.Cu at (128.2, 127.1)
- added C61: 1u/50V, Capacitor_SMD:C_0805_2012Metric_Pad1.18x1.45mm_HandSolder, F.Cu at (128.2, 130.1)
- added C62: 10u/16V, Capacitor_SMD:C_0805_2012Metric_Pad1.18x1.45mm_HandSolder, F.Cu at (128.2, 133.2)
- added C63: 4u7/50V, Capacitor_SMD:C_1210_3225Metric_Pad1.33x2.70mm_HandSolder, F.Cu at (134.8, 119.2)
- added C64: 4u7/50V, Capacitor_SMD:C_1210_3225Metric_Pad1.33x2.70mm_HandSolder, F.Cu at (134.8, 123.5)
- added C65: 1u/50V, Capacitor_SMD:C_0805_2012Metric_Pad1.18x1.45mm_HandSolder, F.Cu at (128.2, 136.2)
- added C66: 10u/50V, Capacitor_SMD:C_1210_3225Metric_Pad1.33x2.70mm_HandSolder, F.Cu at (140.8, 110.8)
- added C67: 10u/50V, Capacitor_SMD:C_1210_3225Metric_Pad1.33x2.70mm_HandSolder, F.Cu at (140.8, 115.0)
- added C68: 10u/16V, Capacitor_SMD:C_0805_2012Metric_Pad1.18x1.45mm_HandSolder, F.Cu at (128.2, 139.2)
- added C69: 1u/50V, Capacitor_SMD:C_0805_2012Metric_Pad1.18x1.45mm_HandSolder, F.Cu at (128.2, 142.2)
- added C7: 0.1u/100V, Capacitor_SMD:C_0603_1608Metric_Pad1.08x0.95mm_HandSolder, F.Cu at (158.3, 109.9)
- added C70: 4u7/50V, Capacitor_SMD:C_1210_3225Metric_Pad1.33x2.70mm_HandSolder, F.Cu at (140.8, 119.2)
- added C71: C/50V, Capacitor_SMD:C_0805_2012Metric_Pad1.18x1.45mm_HandSolder, F.Cu at (128.2, 145.2)
- added C72: 10u/50V, Capacitor_SMD:C_1210_3225Metric_Pad1.33x2.70mm_HandSolder, F.Cu at (140.8, 123.5)
- added C73: 1u/50V, Capacitor_SMD:C_0603_1608Metric_Pad1.08x0.95mm_HandSolder, F.Cu at (110.5, 109.9)
- added C74: 4u7/50V, Capacitor_SMD:C_1210_3225Metric_Pad1.33x2.70mm_HandSolder, F.Cu at (146.8, 110.8)
- added C75: 10u/50V, Capacitor_SMD:C_1210_3225Metric_Pad1.33x2.70mm_HandSolder, F.Cu at (146.8, 115.0)
- added C76: 4u7/50V, Capacitor_SMD:C_1210_3225Metric_Pad1.33x2.70mm_HandSolder, F.Cu at (146.8, 119.2)
- added C77: 10u/50V, Capacitor_SMD:C_1210_3225Metric_Pad1.33x2.70mm_HandSolder, F.Cu at (146.8, 123.5)
- added C78: 0.1u/100V, Capacitor_SMD:C_0603_1608Metric_Pad1.08x0.95mm_HandSolder, F.Cu at (66.3, 96.8)
- added C79: 1u/50V, Capacitor_SMD:C_0603_1608Metric_Pad1.08x0.95mm_HandSolder, F.Cu at (66.3, 99.3)
- added C8: 0.1u/100V, Capacitor_SMD:C_0603_1608Metric_Pad1.08x0.95mm_HandSolder, F.Cu at (158.3, 112.4)
- added C80: 1u/50V, Capacitor_SMD:C_0603_1608Metric_Pad1.08x0.95mm_HandSolder, F.Cu at (66.3, 101.8)
- added C81: 0.1u/100V, Capacitor_SMD:C_0603_1608Metric_Pad1.08x0.95mm_HandSolder, F.Cu at (66.3, 104.3)
- added C9: 0.1u/100V, Capacitor_SMD:C_0603_1608Metric_Pad1.08x0.95mm_HandSolder, F.Cu at (158.3, 114.9)
- added D1: SMAJ14CA, Diode_SMD:D_SMA, F.Cu at (155.9, 126.0)
- added D11: SMAJ14CA, Diode_SMD:D_SMA, F.Cu at (164.6, 132.5)
- added D2: BAV199, Package_TO_SOT_SMD:SOT-23, F.Cu at (167.3, 120.1)
- added D5: SMAJ43CA, Diode_SMD:D_SMA, F.Cu at (163.0, 151.0)
- added J1: 73251-1153, Connector_Coaxial:SMA_Molex_73251-1153_EdgeMount_Horizontal, F.Cu at (180.1, 89.3)
- added J2: Conn_02x04_Odd_Even, Connector_PinSocket_2.54mm:PinSocket_2x04_P2.54mm_Vertical_SMD, F.Cu at (113.4, 169.1)
- added J3: Conn_02x04_Odd_Even, Connector_PinSocket_2.54mm:PinSocket_2x04_P2.54mm_Vertical_SMD, F.Cu at (113.4, 154.8)
- added J4: Conn_02x04_Odd_Even, Connector_PinSocket_2.54mm:PinSocket_2x04_P2.54mm_Vertical_SMD, F.Cu at (123.5, 154.8)
- added J5: Conn_02x04_Odd_Even, Connector_PinSocket_2.54mm:PinSocket_2x04_P2.54mm_Vertical_SMD, F.Cu at (133.6, 154.8)
- added L1: 74408063470, ETH1CVOLT_A:74408063470, F.Cu at (99.4, 106.3)
- added R16: 100k/0.1%, Resistor_SMD:R_0603_1608Metric_Pad0.98x0.95mm_HandSolder, F.Cu at (158.3, 139.0)
- added R26: 100/2W, Resistor_SMD:R_1206_3216Metric_Pad1.30x1.75mm_HandSolder, F.Cu at (161.9, 154.9)
- added R30: 100/2W, Resistor_SMD:R_1206_3216Metric_Pad1.30x1.75mm_HandSolder, F.Cu at (123.4, 164.6)
- added R36: R/200V, Resistor_SMD:R_1206_3216Metric_Pad1.30x1.75mm_HandSolder, F.Cu at (149.7, 150.3)
- added R39: TNPW120639K2BEEN, Resistor_SMD:R_1206_3216Metric_Pad1.30x1.75mm_HandSolder, F.Cu at (90.4, 113.3)
- added R40: 0/200V, Resistor_SMD:R_1206_3216Metric_Pad1.30x1.75mm_HandSolder, F.Cu at (149.7, 153.7)
- added R41: R/200V, Resistor_SMD:R_1206_3216Metric_Pad1.30x1.75mm_HandSolder, F.Cu at (149.7, 157.0)
- added R43: 1k/250mW/200V, Resistor_SMD:R_1206_3216Metric_Pad1.30x1.75mm_HandSolder, F.Cu at (149.7, 160.3)
- added R47: 100/2W, Resistor_SMD:R_1206_3216Metric_Pad1.30x1.75mm_HandSolder, F.Cu at (149.7, 163.6)
- added R5: 10k/0.1%, Resistor_SMD:R_0603_1608Metric_Pad0.98x0.95mm_HandSolder, F.Cu at (162.7, 117.4)
- added R52: 1k/0.1%, Resistor_SMD:R_0603_1608Metric_Pad0.98x0.95mm_HandSolder, F.Cu at (130.6, 164.2)
- added R53: 1k/0.1%, Resistor_SMD:R_0603_1608Metric_Pad0.98x0.95mm_HandSolder, F.Cu at (130.6, 166.7)
- added R54: 1k/0.1%, Resistor_SMD:R_0603_1608Metric_Pad0.98x0.95mm_HandSolder, F.Cu at (130.6, 169.2)
- added R55: 10k, Resistor_SMD:R_0603_1608Metric_Pad0.98x0.95mm_HandSolder, F.Cu at (110.5, 112.4)
- added R56: 118k, Resistor_SMD:R_0603_1608Metric_Pad0.98x0.95mm_HandSolder, F.Cu at (110.5, 114.9)
- added R57: 107k, Resistor_SMD:R_0603_1608Metric_Pad0.98x0.95mm_HandSolder, F.Cu at (110.5, 117.4)
- added R58: 10k, Resistor_SMD:R_0603_1608Metric_Pad0.98x0.95mm_HandSolder, F.Cu at (110.5, 119.9)
- added R59: R, Resistor_SMD:R_0603_1608Metric_Pad0.98x0.95mm_HandSolder, F.Cu at (110.5, 122.4)
- added R60: 68k, Resistor_SMD:R_0603_1608Metric_Pad0.98x0.95mm_HandSolder, F.Cu at (110.5, 124.9)
- added R61: 10k, Resistor_SMD:R_0603_1608Metric_Pad0.98x0.95mm_HandSolder, F.Cu at (110.5, 127.5)
- added R62: 499/0.1%, Resistor_SMD:R_0603_1608Metric_Pad0.98x0.95mm_HandSolder, F.Cu at (110.5, 130.0)
- added R63: 0, Resistor_SMD:R_1206_3216Metric_Pad1.30x1.75mm_HandSolder, F.Cu at (133.6, 127.3)
- added R64: 0, Resistor_SMD:R_1206_3216Metric_Pad1.30x1.75mm_HandSolder, F.Cu at (133.6, 130.6)
- added R65: RT1206BRD071RL, Resistor_SMD:R_1206_3216Metric_Pad1.30x1.75mm_HandSolder, F.Cu at (133.6, 133.9)
- added R67: 0, Resistor_SMD:R_0603_1608Metric_Pad0.98x0.95mm_HandSolder, F.Cu at (110.5, 132.5)
- added R68: 100, Resistor_SMD:R_0603_1608Metric_Pad0.98x0.95mm_HandSolder, F.Cu at (158.3, 141.5)
- added R7: 10k/0.1%, Resistor_SMD:R_0603_1608Metric_Pad0.98x0.95mm_HandSolder, F.Cu at (162.7, 119.9)
- added RN3: MPMT1002AT5, Package_TO_SOT_SMD:SOT-23, F.Cu at (167.3, 124.5)
- added RV1: R_Potentiometer_Trim, Potentiometer_SMD:Potentiometer_Bourns_3314G_Vertical, F.Cu at (100.1, 126.3)
- added TP1: TestPoint, TestPoint:TestPoint_Pad_D1.5mm, F.Cu at (171.5, 119.6)
- added TP2: TestPoint, TestPoint:TestPoint_Pad_D1.5mm, F.Cu at (171.5, 123.2)
- added U1: ADG5419BRMZ-RL7, Package_SO:MSOP-8_3x3mm_P0.65mm, F.Cu at (168.6, 111.0)
- added U18: ADHV4702-1, ETH1CVOLT_B:CP-12-8, F.Cu at (83.7, 121.3)
- added U19: ADHV4702-1, ETH1CVOLT_B:CP-12-8, F.Cu at (83.5, 135.8)
- added U26: TEC3-2423UI, Converter_DCDC:Converter_DCDC_TRACO_TEC3-24xxUI_THT, F.Cu at (121.1, 112.2)
- added U27: ISO7761FDBQ, Package_SO:SSOP-16_3.9x4.9mm_P0.635mm, F.Cu at (140.5, 129.2)
- added U28: TPS7A39, Package_SON:Texas_S-PVSON-N10_ThermalVias, F.Cu at (145.9, 139.8)
- added U29: ADS8681RUM, Package_DFN_QFN:QFN-16-1EP_4x4mm_P0.65mm_EP2.7x2.7mm, F.Cu at (140.1, 140.3)
- added U30: MAX15062C, Package_DFN_QFN:DFN-8_2x2mm_P0.5mm, F.Cu at (145.6, 144.4)
- added U31: AD8221ARM, Package_SO:MSOP-8_3x3mm_P0.65mm, F.Cu at (140.2, 134.9)
- added U32: ADP7142AUJZ-5.0, Package_TO_SOT_SMD:TSOT-23-5, F.Cu at (147.1, 128.0)
- added U5: ADA4522-1ARMZ, Package_SO:MSOP-8_3x3mm_P0.65mm, F.Cu at (168.6, 115.6)
- added U6: ADG5419BRMZ-RL7, Package_SO:MSOP-8_3x3mm_P0.65mm, F.Cu at (164.2, 137.1)
- C11: renamed from C1; value 470p -> 470p/100V
- C12: renamed from C2; value 470p -> 470p/100V
- C18: renamed from C3; value C -> 6u8/16V; footprint Capacitor_SMD:C_0603_1608Metric_Pad1.08x0.95mm_HandSolder -> Capacitor_SMD:C_0805_2012Metric_Pad1.18x1.45mm_HandSolder
- C25: renamed from C4; value C -> 6u8/16V; footprint Capacitor_SMD:C_0603_1608Metric_Pad1.08x0.95mm_HandSolder -> Capacitor_SMD:C_0805_2012Metric_Pad1.18x1.45mm_HandSolder
- C46: renamed from C10; value 4u7/50V -> 4u7/100V
- C47: renamed from C11; value 10u/50V -> 10u/100V
- C48: renamed from C12; value 1u -> 1u/50V
- C49: renamed from C13; value 4u7/50V -> 4u7/100V
- C50: renamed from C14; value 10u/50V -> 10u/100V
- C51: renamed from C15; value 4u7/50V -> 4u7/100V
- C52: renamed from C16; value 10u/50V -> 10u/100V
- C53: renamed from C17; value 10u/50V -> 10u/100V
- R11: renamed from R9; value R -> 100
- R15: renamed from R13; value R -> 100
- R45: renamed from R42; value 5/250mW -> 5/250mW/200V
- R46: renamed from R43; value 5/250mW -> 5/250mW/200V
- moved C53 3.62 mm to (43.3, 68.4)
- renumbered C5 to C36, C6 to C37, D8 to D10, D1 to D3, D2 to D4, D4 to D6, D5 to D7, D6 to D8, D7 to D9, R6 to R10, R10 to R12, R11 to R13, R12 to R14, R14 to R17, R15 to R18, R16 to R19, R17 to R20, R18 to R21, R19 to R22, R20 to R23, R21 to R24, R22 to R25, R24 to R27, R25 to R28, R26 to R29, R28 to R31, R29 to R32, R30 to R33, R31 to R34, R32 to R35, R34 to R37, R35 to R38, R39 to R42, R41 to R44, R45 to R48, R46 to R49, R47 to R50, R48 to R51, R5 to R6, R7 to R8, R8 to R9, RN3 to RN4, RN4 to RN5, TP1 to TP3, TP2 to TP4, TP3 to TP5, TP4 to TP6, U7 to U10, U8 to U11, U9 to U12, U10 to U13, U11 to U14, U12 to U15, U13 to U16, U16 to U17, U1 to U2, U17 to U20, U18 to U21, U19 to U22, U20 to U23, U21 to U24, U22 to U25, U2 to U3, U3 to U4, U4 to U7, U5 to U8, U6 to U9
Connections:
- net /Block Diagram/ADC/ADC_SCLK renamed /Block Diagram/ADC/ADC_VOLT_SCLK
- net /Block Diagram/ADC/ADC_SDO renamed /Block Diagram/ADC/ADC_VOLT_SDO
- net /Block Diagram/ADC/ADC_~{CS} renamed /Block Diagram/ADC/ADC_VOLT_~{CS}
- net /Block Diagram/DAC/DAC_SCLK renamed /Block Diagram/Connectors Input/DAC_SCLK
- net /Block Diagram/DAC/DAC_SDIN renamed /Block Diagram/Connectors Input/DAC_SDIN
- net /Block Diagram/DAC/DAC_SDO renamed /Block Diagram/Connectors Input/DAC_SDO
- net /Block Diagram/DAC/DAC_~{SYNC} renamed /Block Diagram/Connectors Input/DAC_~{SYNC}
- net /Block Diagram/Output/OUTPUT renamed /Block Diagram/Current Measurement/CURR_P_MEAS
- R18 pad 2: /Block Diagram/MV Output/MV_DAC -> /Block Diagram/MUX/MV_DAC
- R20 pad 2: /Block Diagram/MV Output/MV_MEAS -> /Block Diagram/MUX/MV_MEAS
- R21 pad 1: /Block Diagram/MV Output/MV_MEAS -> /Block Diagram/MUX/MV_MEAS
- R27 pad 2: /Block Diagram/LV Output/MV_MEAS -> /Block Diagram/LV Output/LV_MEAS
- R28 pad 1: /Block Diagram/LV Output/MV_MEAS -> /Block Diagram/LV Output/LV_MEAS
- R6 pad 2: /Block Diagram/DAC/DAC_OUTPUT -> Net-(R6-Pad2)
- RN2 pad 1: /Block Diagram/DAC/DAC_OUTPUT -> Net-(R6-Pad2)
- TP5 pad 1: Net-(U7-+IN0.4x) -> Net-(D11-A2)
- TP6 pad 1: /Block Diagram/ADC/ADC_MEAS -> Net-(U11-+)
- U10 pad 9: Net-(U7-+IN0.4x) -> Net-(D11-A2)
- U11 pad 2: Net-(U7-+IN0.4x) -> Net-(U11--)
- U11 pad 3: /Block Diagram/ADC/ADC_MEAS -> Net-(U11-+)
- U11 pad 6: Net-(U7-+IN0.4x) -> Net-(U11--)
- U12 pad 2: /Block Diagram/MV Output/MUX_A0 -> /Block Diagram/MUX/MUX_A0
- U13 pad 4: /Block Diagram/MV Output/MV_DAC -> /Block Diagram/MUX/MV_DAC
- U16 pad 11: /Block Diagram/MUX/HV_MEAS -> /Block Diagram/HV Output/HV_MEAS
- U16 pad 13: /Block Diagram/MUX/LV_MEAS -> /Block Diagram/LV Output/LV_MEAS
- U16 pad 4: /Block Diagram/MUX/LV_DAC -> /Block Diagram/LV Output/LV_DAC
- U16 pad 7: /Block Diagram/MUX/HV_DAC -> /Block Diagram/HV Output/HV_DAC
- U16 pad 8: /Block Diagram/MUX/DAC_OUTPUT -> /Block Diagram/DAC/DAC_OUTPUT
- U16 pad 9: /Block Diagram/MUX/ADC_MEAS -> /Block Diagram/ADC/ADC_MEAS
- U17 pad 1: /Block Diagram/HV Output/MUX_A1 -> /Block Diagram/MUX/MUX_A1
- U17 pad 2: /Block Diagram/HV Output/MUX_A0 -> /Block Diagram/MUX/MUX_A0
- U2 pad 7: /Block Diagram/DAC/DAC_OUTPUT -> Net-(R6-Pad2)
- U20 pad 1: /Block Diagram/Voltage Reference/SEL_x1 -> /Block Diagram/ADC/SEL_x1
- U20 pad 11: /Block Diagram/Voltage Reference/VREF_TEST -> /Block Diagram/MUX/VREF_TEST
- U20 pad 3: /Block Diagram/Voltage Reference/VREF_TEST -> /Block Diagram/MUX/VREF_TEST
- U20 pad 7: /Block Diagram/Voltage Reference/VREF_TEST -> /Block Diagram/MUX/VREF_TEST
- U20 pad 8: /Block Diagram/Voltage Reference/SEL_x10 -> /Block Diagram/ADC/SEL_x10
- U20 pad 9: /Block Diagram/Voltage Reference/SEL_x100 -> /Block Diagram/ADC/SEL_x100
- U23 pad 1: unconnected-(U20-Pad1) -> Net-(R52-Pad2)
- U23 pad 2: GND_ISO -> /Block Diagram/Connectors Input/LV_OUT_PMOS
- U23 pad 4: /Block Diagram/Output/LV_OUTPUT -> /Block Diagram/LV Output/LV_OUTPUT
- U24 pad 1: unconnected-(U21-Pad1) -> Net-(R53-Pad2)
- U24 pad 2: GND_ISO -> /Block Diagram/Connectors Input/MV_OUT_PMOS
- U24 pad 4: /Block Diagram/Output/MV_OUTPUT -> /Block Diagram/MV Output/MV_OUTPUT
- U25 pad 1: unconnected-(U22-Pad1) -> Net-(R54-Pad2)
- U25 pad 2: GND_ISO -> /Block Diagram/Connectors Input/HV_OUT_PMOS
- U25 pad 4: /Block Diagram/Output/HV_OUTPUT -> /Block Diagram/HV Output/HV_OUTPUT
- U3 pad 1: (no net) -> +5VREF_ISO
- U3 pad 12: unconnected-(U2-~{FAULT}-Pad12) -> Net-(U3-~{FAULT})
- U4 pad 1: (no net) -> +5VREF_ISO
- U4 pad 12: unconnected-(U3-~{FAULT}-Pad12) -> Net-(U4-~{FAULT})

Commit message: Development
Parts:
- added J6: 61000821121, Connector_PinSocket_2.54mm:PinSocket_2x04_P2.54mm_Vertical_SMD, F.Cu at (45.9, 119.4)
- added J7: 61000821121, Connector_PinSocket_2.54mm:PinSocket_2x04_P2.54mm_Vertical_SMD, F.Cu at (56.0, 119.4)
- added J8: 61000821121, Connector_PinSocket_2.54mm:PinSocket_2x04_P2.54mm_Vertical_SMD, F.Cu at (66.1, 119.4)
- added R69: 100, Resistor_SMD:R_0603_1608Metric_Pad0.98x0.95mm_HandSolder, F.Cu at (46.5, 128.8)
- added TP10: TestPoint, TestPoint:TestPoint_Pad_D1.5mm, F.Cu at (192.9, 122.7)
- added TP11: TestPoint, TestPoint:TestPoint_Pad_D1.5mm, F.Cu at (192.9, 126.2)
- added TP12: TestPoint, TestPoint:TestPoint_Pad_D1.5mm, F.Cu at (183.8, 113.6)
- added TP13: TestPoint, TestPoint:TestPoint_Pad_D1.5mm, F.Cu at (183.8, 117.2)
- added TP14: TestPoint, TestPoint:TestPoint_Pad_D1.5mm, F.Cu at (183.8, 120.7)
- added TP15: TestPoint, TestPoint:TestPoint_Pad_D1.5mm, F.Cu at (183.8, 124.2)
- added TP16: TestPoint, TestPoint:TestPoint_Pad_D1.5mm, F.Cu at (187.4, 113.6)
- added TP17: TestPoint, TestPoint:TestPoint_Pad_D1.5mm, F.Cu at (187.4, 117.2)
- added TP18: TestPoint, TestPoint:TestPoint_Pad_D1.5mm, F.Cu at (187.4, 120.7)
- added TP19: TestPoint, TestPoint:TestPoint_Pad_D1.5mm, F.Cu at (192.9, 131.8)
- added TP20: TestPoint, TestPoint:TestPoint_Pad_D1.5mm, F.Cu at (192.9, 113.6)
- added TP21: TestPoint, TestPoint:TestPoint_Pad_D1.5mm, F.Cu at (198.5, 122.7)
- added TP22: TestPoint, TestPoint:TestPoint_Pad_D1.5mm, F.Cu at (198.5, 113.6)
- added TP23: TestPoint, TestPoint:TestPoint_Pad_D1.5mm, F.Cu at (192.9, 117.2)
- added TP24: TestPoint, TestPoint:TestPoint_Pad_D1.5mm, F.Cu at (198.5, 126.2)
- added TP25: TestPoint, TestPoint:TestPoint_Pad_D1.5mm, F.Cu at (198.5, 117.2)
- added TP7: TestPoint, TestPoint:TestPoint_Pad_D1.5mm, F.Cu at (42.6, 129.3)
- added TP8: TestPoint, TestPoint:TestPoint_Pad_D1.5mm, F.Cu at (42.6, 132.8)
- added TP9: TestPoint, TestPoint:TestPoint_Pad_D1.5mm, F.Cu at (198.5, 131.8)
- C71: value C/50V -> 10u/100V; footprint Capacitor_SMD:C_0805_2012Metric_Pad1.18x1.45mm_HandSolder -> Capacitor_SMD:C_1210_3225Metric_Pad1.33x2.70mm_HandSolder
- J3, J4, J5: value Conn_02x04_Odd_Even -> 61000821121
- R59: value R -> 100
- R63, R64: value 0 -> 0/200V
Connections:
- J1 pad 1: Net-(D1-A2) -> Net-(J1-In)
