File: HARDWARE/ETH1CVOLT_B/ETH1CVOLT_B.kicad_sch (KiCad schematic)
At the start: 0 parts

Commit message: Development
Other:
- sheet Block Diagram: file BlockDiagram.kicad_sch -> Block_Diagram.kicad_sch
Changed lines of the file:
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@@
 	(generator "eeschema")
 	(generator_version "9.0")
-	(paper "A3")
+	(paper "A4")
 	(sheet
-		(at 299.72 212.09)
-		(size 49.53 34.29)
+		(at 189.23 127)
+		(size 59.69 31.75)
 		(exclude_from_sim no)
 		(in_bom yes)
@@
 		)
 		(property "Sheetname" "Block Diagram"
-			(at 299.72 211.3784 0)
+			(at 189.23 126.2884 0)
 			(effects
 				(font
@@
 			)
 		)
-		(property "Sheetfile" "BlockDiagram.kicad_sch"
-			(at 299.72 246.9646 0)
+		(property "Sheetfile" "Block_Diagram.kicad_sch"
+			(at 189.23 159.3346 0)
 			(effects
 				(font
@@
 		)
 		(instances
-			(project "ETH1CVOLT_A"
-				(path "/ca79f0b4-91f7-4537-917d-68d425c03ca3"
+			(project "ETH1CVOLT_B"
+				(path "/18612734-e331-4379-b1d3-176cfdcf99d5"
 					(page "2")
 				)

Commit message: Development
Changed lines of the file:
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@@
 	(generator "eeschema")
 	(generator_version "9.0")
-	(paper "A4")
+	(paper "A3")
 	(sheet
-		(at 189.23 127)
+		(at 297.18 212.09)
 		(size 59.69 31.75)
 		(exclude_from_sim no)
@@
 		)
 		(property "Sheetname" "Block Diagram"
-			(at 189.23 126.2884 0)
+			(at 297.18 211.3784 0)
 			(effects
 				(font
@@
 		)
 		(property "Sheetfile" "Block_Diagram.kicad_sch"
-			(at 189.23 159.3346 0)
+			(at 297.18 244.4246 0)
 			(effects
 				(font

Commit message: Development
Changed lines of the file:
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@@
 	(paper "A3")
 	(sheet
-		(at 297.18 212.09)
-		(size 59.69 31.75)
+		(at 299.72 214.63)
+		(size 101.6 31.75)
 		(exclude_from_sim no)
 		(in_bom yes)
@@
 		)
 		(property "Sheetname" "Block Diagram"
-			(at 297.18 211.3784 0)
+			(at 299.72 213.9184 0)
 			(effects
 				(font
@@
 		)
 		(property "Sheetfile" "Block_Diagram.kicad_sch"
-			(at 297.18 244.4246 0)
+			(at 299.72 246.9646 0)
 			(effects
 				(font

Commit message: Development
Other:
- note added: "ETH1CVOLT_B"
Changed lines of the file:
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@@
 	(generator_version "9.0")
 	(paper "A3")
+	(text "ETH1CVOLT_B"
+		(exclude_from_sim no)
+		(at 209.55 31.75 0)
+		(effects
+			(font
+				(size 12.7 12.7)
+				(thickness 1.27)
+				(bold yes)
+			)
+		)
+	)
 	(sheet
 		(at 299.72 214.63)
