File: HARDWARE/ETH1CVOLT_B/HV_Output.kicad_sch (KiCad schematic)
At the start: 21 parts, among them Q1 PBHV8140Z,115, Q2 PBHV9540Z,115, U15 ADHV4702-1, U16 ADHV4702-1, U17 74LV1T08GV

Commit message: Development
Parts:
- added C9: C, symbol Device:C
- added D6, D7: BAV199, Package_TO_SOT_SMD:SOT-23, symbol Diode:BAV99
- added R34, R35: 0, Resistor_SMD:R_0603_1608Metric_Pad0.98x0.95mm_HandSolder, symbol Device:R
- added R37: 0/200V, symbol Device:R
- Q1, Q2: footprint (none) -> Package_TO_SOT_SMD:SOT-223-3_TabPin2
- R29: renamed from R36; footprint (none) -> Resistor_SMD:R_1206_3216Metric_Pad1.30x1.75mm_HandSolder
- R30: renamed from R37; footprint (none) -> Resistor_SMD:R_0603_1608Metric_Pad0.98x0.95mm_HandSolder
- R31: renamed from R35; footprint (none) -> Resistor_SMD:R_0603_1608Metric_Pad0.98x0.95mm_HandSolder
- R32: renamed from R30; footprint (none) -> Resistor_SMD:R_0603_1608Metric_Pad0.98x0.95mm_HandSolder
- R39: renamed from R32; footprint (none) -> Resistor_SMD:R_0603_1608Metric_Pad0.98x0.95mm_HandSolder
- R41: renamed from R33; footprint (none) -> Resistor_SMD:R_0603_1608Metric_Pad0.98x0.95mm_HandSolder
- R42: renamed from R31; footprint (none) -> Resistor_SMD:R_1206_3216Metric_Pad1.30x1.75mm_HandSolder
- R43: renamed from R28; footprint (none) -> Resistor_SMD:R_1206_3216Metric_Pad1.30x1.75mm_HandSolder
- renumbered C16 to C7, C15 to C8, D7 to D8, R34 to R33, R26 to R36, R25 to R38, R29 to R40, R27 to R44, U15 to U14, U16 to U15, U17 to U16
Connections:
- net GND_ISO: now also R34.1, R35.1
- net HV_DAC: now also D6.2 (A), D7.1 (K)
- net HV_ENABLE: now also U14.8 (~{SD}), U15.8 (~{SD})
- net at R36.2, R40.2, R42.2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: now also C9.2, R37.2; no longer U15.2 (IN+)
- net at U15.9 (RADJ): now also R35.2
- net at R32.2, R36.1, U14.12 (IN-): now also C9.1, D6.1 (K), D7.2 (A)
- net at U14.9 (RADJ): now also R34.2
- net +5VD_ISO renamed +VD_ISO
- new net: R37.1, U15.2 (IN+)
- no-connect marks 4 -> 6
Other:
- moved on the sheet: C7, C8, D8, Q1, Q2, R29, R30, R31, R32, R33, R36, R38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

Commit message: Development
Parts:
- added C74, C75, C77, C78: 0.1u/250V, symbol Device:C
- added C76: 0.1u/100V, symbol Device:C
- renumbered C7 to C39, C8 to C40, C9 to C41, D8 to D10, D6 to D8, D7 to D9, R29 to R32, R30 to R33, R31 to R34, R32 to R35, R33 to R36, R34 to R37, R35 to R38, R36 to R39, R37 to R40, R38 to R41, R39 to R42, R40 to R43, R41 to R44, R42 to R45, R43 to R46, R44 to R47, U16 to U18, U14 to U19, U15 to U20
Connections:
- net +110V_ISO: now also C74.1, C78.1
- net +VD_ISO: now also C76.1
- net -110V_ISO: now also C75.1, C77.1
- net GND_ISO: now also C74.2, C75.2, C76.2, C77.2, C78.2
Other:
- moved on the sheet: U18

Commit message: Development
Parts:
- C38: renamed from C74; footprint (none) -> Capacitor_SMD:C_1206_3216Metric_Pad1.33x1.80mm_HandSolder
- C39: renamed from C78; footprint (none) -> Capacitor_SMD:C_1206_3216Metric_Pad1.33x1.80mm_HandSolder
- C40: renamed from C75; footprint (none) -> Capacitor_SMD:C_1206_3216Metric_Pad1.33x1.80mm_HandSolder
- C41: renamed from C77; footprint (none) -> Capacitor_SMD:C_1206_3216Metric_Pad1.33x1.80mm_HandSolder
- C42: renamed from C76; footprint (none) -> Capacitor_SMD:C_0603_1608Metric_Pad1.08x0.95mm_HandSolder
- C43: renamed from C39; value C -> C/250V; footprint (none) -> Capacitor_SMD:C_1206_3216Metric_Pad1.33x1.80mm_HandSolder; now not fitted; now left out of the parts list
- C44: renamed from C40; value C -> C/250V; footprint (none) -> Capacitor_SMD:C_1206_3216Metric_Pad1.33x1.80mm_HandSolder; now not fitted; now left out of the parts list
- C45: renamed from C41; value C -> C/200V; footprint (none) -> Capacitor_SMD:C_1206_3216Metric_Pad1.33x1.80mm_HandSolder
- R36, R41: value R -> R/200V; footprint (none) -> Resistor_SMD:R_1206_3216Metric_Pad1.30x1.75mm_HandSolder; now not fitted; now left out of the parts list
- R39: value 39k2/0.1%/200V/500mW -> TNPW120639K2BEEN; footprint (none) -> Resistor_SMD:R_1206_3216Metric_Pad1.30x1.75mm_HandSolder
- R40, R47: footprint (none) -> Resistor_SMD:R_1206_3216Metric_Pad1.30x1.75mm_HandSolder
- R43: value 1k/250mW -> 1k/250mW/200V; footprint (none) -> Resistor_SMD:R_1206_3216Metric_Pad1.30x1.75mm_HandSolder
- R45, R46: value 5/250mW -> 5/250mW/200V
- U18: renamed from U19; footprint (none) -> ETH1CVOLT_B:CP-12-8
- U19: renamed from U20; footprint (none) -> ETH1CVOLT_B:CP-12-8
- renumbered U18 to U17
Other:
- moved on the sheet: C45, D10, D8, D9, Q1, Q2, R32, R33, R34, R35, R37, R38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

Commit message: Development
Parts:
- added TP21, TP24: TestPoint, TestPoint:TestPoint_Pad_D1.5mm, symbol Connector:TestPoint
Connections:
- net HV_MEAS: now also TP24.1
- net HV_OUTPUT: now also TP21.1
Changed lines of the file:
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@@
 	)
 	(junction
+		(at 97.79 194.31)
+		(diameter 0)
+		(color 0 0 0 0)
+	)
+	(junction
 		(at 78.74 269.24)
 		(diameter 0)
@@
 	)
 	(junction
+		(at 322.58 78.74)
+		(diameter 0)
+		(color 0 0 0 0)
+	)
+	(junction
 		(at 234.95 118.11)
 		(diameter 0)
@@
 	(wire
 		(pts
-			(xy 300.99 78.74) (xy 323.85 78.74)
+			(xy 300.99 78.74) (xy 322.58 78.74)
 		)
 		(stroke
@@
 	(wire
 		(pts
+			(xy 322.58 77.47) (xy 322.58 78.74)
+		)
+		(stroke
+			(width 0)
+			(type default)
+		)
+	)
+	(wire
+		(pts
 			(xy 78.74 259.08) (xy 87.63 259.08)
 		)
@@
 	(wire
 		(pts
+			(xy 97.79 194.31) (xy 133.35 194.31)
+		)
+		(stroke
+			(width 0)
+			(type default)
+		)
+	)
+	(wire
+		(pts
 			(xy 40.64 269.24) (xy 30.48 269.24)
 		)
@@
 	(wire
 		(pts
-			(xy 111.76 194.31) (xy 133.35 194.31)
+			(xy 90.17 194.31) (xy 97.79 194.31)
 		)
 		(stroke
@@
 	(wire
 		(pts
+			(xy 97.79 193.04) (xy 97.79 194.31)
+		)
+		(stroke
+			(width 0)
+			(type default)
+		)
+	)
+	(wire
+		(pts
 			(xy 214.63 105.41) (xy 203.2 105.41)
 		)
@@
 	(wire
 		(pts
+			(xy 322.58 78.74) (xy 335.28 78.74)
+		)
+		(stroke
+			(width 0)
+			(type default)
+		)
+	)
+	(wire
+		(pts
 			(xy 86.36 149.86) (xy 86.36 148.59)
 		)
@@
 	(hierarchical_label "HV_MEAS"
 		(shape output)
-		(at 111.76 194.31 180)
+		(at 90.17 194.31 180)
 		(effects
 			(font
@@
 	(hierarchical_label "HV_OUTPUT"
 		(shape output)
-		(at 323.85 78.74 0)
+		(at 335.28 78.74 0)
 		(effects
 			(font
@@
 			)
 		)
-		(property "Component Class" "ISO"
+		(property "Component Class" ""
 			(at 14.6685 15.4305 0)
 			(effects
@@
 	)
 	(symbol
+		(lib_id "Connector:TestPoint")
+		(at 97.79 193.04 0)
+		(unit 1)
+		(exclude_from_sim no)
+		(in_bom yes)
+		(on_board yes)
+		(dnp no)
+		(fields_autoplaced yes)
+		(property "Reference" "TP24"
+			(at 100.33 188.4679 0)
+			(effects
+				(font
+					(size 1.27 1.27)
+				)
+				(justify left)
+			)
+		)
+		(property "Value" "TestPoint"
+			(at 100.33 191.0079 0)
+			(effects
+				(font
+					(size 1.27 1.27)
+				)
+				(justify left)
+			)
+		)
+		(property "Footprint" "TestPoint:TestPoint_Pad_D1.5mm"
+			(at 102.87 193.04 0)
+			(effects
+				(font
+					(size 1.27 1.27)
+				)
+				(hide yes)
+			)
+		)
+		(property "Datasheet" "~"
+			(at 102.87 193.04 0)
+			(effects
+				(font
+					(size 1.27 1.27)
+				)
+				(hide yes)
+			)
+		)
+		(property "Description" "test point"
+			(at 97.79 193.04 0)
+			(effects
+				(font
+					(size 1.27 1.27)
+				)
+				(hide yes)
+			)
+		)
+		(pin "1"
+		)
+		(instances
+			(project "ETH1CVOLT_B"
+				(path "/18612734-e331-4379-b1d3-176cfdcf99d5/b64e35a5-c86f-43a6-acb5-469d75a46b72/d441a377-bbc5-43e3-9bee-7a77827b9964"
+					(reference "TP24")
+					(unit 1)
+				)
+			)
+		)
+	)
+	(symbol
 		(lib_id "Device:R")
 		(at 217.17 166.37 90)
@@
 					(unit 1)
 				)
+			)
+		)
+	)
+	(symbol
+		(lib_id "Connector:TestPoint")
+		(at 322.58 77.47 0)
+		(unit 1)
+		(exclude_from_sim no)
+		(in_bom yes)
+		(on_board yes)
+		(dnp no)
+		(fields_autoplaced yes)
+		(property "Reference" "TP21"
+			(at 325.12 72.8979 0)
+			(effects
+				(font
+					(size 1.27 1.27)
+				)
+				(justify left)
+			)
+		)
+		(property "Value" "TestPoint"
+			(at 325.12 75.4379 0)
+			(effects
+				(font
+					(size 1.27 1.27)
+				)
+				(justify left)
+			)
+		)
+		(property "Footprint" "TestPoint:TestPoint_Pad_D1.5mm"
+			(at 327.66 77.47 0)
+			(effects
+				(font
+					(size 1.27 1.27)
+				)
+				(hide yes)
+			)
+		)
+		(property "Datasheet" "~"
+			(at 327.66 77.47 0)
+			(effects
+				(font
+					(size 1.27 1.27)
+				)
+				(hide yes)
+			)
+		)
+		(property "Description" "test point"
+			(at 322.58 77.47 0)
+			(effects
+				(font
+					(size 1.27 1.27)
+				)
+				(hide yes)
+			)
+		)
+		(pin "1"
+		)
+		(instances
+			(project "ETH1CVOLT_B"
+				(path "/18612734-e331-4379-b1d3-176cfdcf99d5/b64e35a5-c86f-43a6-acb5-469d75a46b72/d441a377-bbc5-43e3-9bee-7a77827b9964"
+					(reference "TP21")
+					(unit 1)
+				)
