File: HARDWARE/ETH1CVOLT_B/MUX.kicad_sch (KiCad schematic)
At the start: 4 parts, among them U6 TMUX8109PWR

Commit message: Development
Parts:
- C5: renamed from C3; footprint (none) -> Capacitor_SMD:C_0603_1608Metric_Pad1.08x0.95mm_HandSolder
- C6: renamed from C4; footprint (none) -> Capacitor_SMD:C_0603_1608Metric_Pad1.08x0.95mm_HandSolder
- R28: renamed from R10; footprint (none) -> Resistor_SMD:R_0603_1608Metric_Pad0.98x0.95mm_HandSolder
- renumbered U6 to U13
Connections:
- net +10VREF_ISO renamed VREF_TEST
- net +5VD_ISO renamed +VD_ISO
Other:
- moved on the sheet: R28

Commit message: Development
Parts:
- renumbered C5 to C37, C6 to C38, R28 to R31, U13 to U17
Other:
- moved on the sheet: C37, C38, R31, U17

Commit message: Development
Parts:
- renumbered C37 to C36, C38 to C37, U17 to U16
Changed lines of the file:
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@@
+		)
+	)
+	(rule_area
+		(polyline
+			(pts
+				(xy 13.97 16.51) (xy 405.13 16.51) (xy 406.4 17.78) (xy 406.4 251.46) (xy 298.45 251.46) (xy 298.45 283.21)
+				(xy 13.97 283.21)
+			)
+			(stroke
+				(width 0)
+				(type dash)
+			)
+			(fill
+				(type none)
+			)
+		)
+	)
+	(netclass_flag ""
+		(length 2.54)
+		(shape round)
+		(at 13.97 16.51 0)
+		(fields_autoplaced yes)
+		(effects
+			(font
+				(size 1.27 1.27)
+			)
+			(justify left bottom)
+		)
+		(property "Netclass" "ISO"
+			(at 14.6685 13.97 0)
+			(effects
+				(font
+					(size 1.27 1.27)
+				)
+				(justify left)
+			)
+		)
+		(property "Component Class" "ISO"
+			(at 14.6685 15.4305 0)
+			(effects
+				(font
+					(size 1.27 1.27)
+					(italic yes)
+				)
+				(justify left)
+				(hide yes)
+			)
 		)
 	)
@@
 		(dnp no)
 		(fields_autoplaced yes)
-		(property "Reference" "C37"
+		(property "Reference" "C36"
 			(at 31.75 266.6999 0)
 			(effects
@@
 			(project ""
 				(path "/18612734-e331-4379-b1d3-176cfdcf99d5/b64e35a5-c86f-43a6-acb5-469d75a46b72/dab81acb-601b-4578-836c-bbc42190f256"
-					(reference "C37")
+					(reference "C36")
 					(unit 1)
 				)
@@
 		(dnp no)
 		(fields_autoplaced yes)
-		(property "Reference" "#PWR0113"
+		(property "Reference" "#PWR0110"
 			(at 48.26 267.97 0)
 			(effects
@@
 			(project ""
 				(path "/18612734-e331-4379-b1d3-176cfdcf99d5/b64e35a5-c86f-43a6-acb5-469d75a46b72/dab81acb-601b-4578-836c-bbc42190f256"
-					(reference "#PWR0113")
+					(reference "#PWR0110")
 					(unit 1)
 				)
@@
 		(dnp no)
 		(fields_autoplaced yes)
-		(property "Reference" "#PWR0112"
+		(property "Reference" "#PWR0109"
 			(at 27.94 278.13 0)
 			(effects
@@
 			(project "ETH1CVOLT_B"
 				(path "/18612734-e331-4379-b1d3-176cfdcf99d5/b64e35a5-c86f-43a6-acb5-469d75a46b72/dab81acb-601b-4578-836c-bbc42190f256"
-					(reference "#PWR0112")
+					(reference "#PWR0109")
 					(unit 1)
 				)
@@
 		(dnp no)
 		(fields_autoplaced yes)
-		(property "Reference" "#PWR0117"
+		(property "Reference" "#PWR0114"
 			(at 222.25 100.33 0)
 			(effects
@@
 			(project "ETH1CVOLT_B"
 				(path "/18612734-e331-4379-b1d3-176cfdcf99d5/b64e35a5-c86f-43a6-acb5-469d75a46b72/dab81acb-601b-4578-836c-bbc42190f256"
-					(reference "#PWR0117")
+					(reference "#PWR0114")
 					(unit 1)
 				)
@@
 		(dnp no)
 		(fields_autoplaced yes)
-		(property "Reference" "#PWR0111"
+		(property "Reference" "#PWR0108"
 			(at 27.94 267.97 0)
 			(effects
@@
 			(project ""
 				(path "/18612734-e331-4379-b1d3-176cfdcf99d5/b64e35a5-c86f-43a6-acb5-469d75a46b72/dab81acb-601b-4578-836c-bbc42190f256"
-					(reference "#PWR0111")
+					(reference "#PWR0108")
 					(unit 1)
 				)
@@
 		(dnp no)
 		(fields_autoplaced yes)
-		(property "Reference" "#PWR0115"
+		(property "Reference" "#PWR0112"
 			(at 204.47 130.81 0)
 			(effects
@@
 			(project ""
 				(path "/18612734-e331-4379-b1d3-176cfdcf99d5/b64e35a5-c86f-43a6-acb5-469d75a46b72/dab81acb-601b-4578-836c-bbc42190f256"
-					(reference "#PWR0115")
+					(reference "#PWR0112")
 					(unit 1)
 				)
@@
 		(dnp no)
 		(fields_autoplaced yes)
-		(property "Reference" "#PWR0116"
+		(property "Reference" "#PWR0113"
 			(at 209.55 146.05 0)
 			(effects
@@
 			(project "ETH1CVOLT_B"
 				(path "/18612734-e331-4379-b1d3-176cfdcf99d5/b64e35a5-c86f-43a6-acb5-469d75a46b72/dab81acb-601b-4578-836c-bbc42190f256"
-					(reference "#PWR0116")
+					(reference "#PWR0113")
 					(unit 1)
 				)
@@
 		(dnp no)
 		(fields_autoplaced yes)
-		(property "Reference" "#PWR0119"
+		(property "Reference" "#PWR0116"
 			(at 264.16 111.76 0)
 			(effects
@@
 			(project "ETH1CVOLT_B"
 				(path "/18612734-e331-4379-b1d3-176cfdcf99d5/b64e35a5-c86f-43a6-acb5-469d75a46b72/dab81acb-601b-4578-836c-bbc42190f256"
-					(reference "#PWR0119")
+					(reference "#PWR0116")
 					(unit 1)
 				)
@@
 		(on_board yes)
 		(dnp no)
-		(property "Reference" "U17"
+		(property "Reference" "U16"
 			(at 209.55 95.25 0)
 			(effects
@@
 			(project "ETH1CVOLT_B"
 				(path "/18612734-e331-4379-b1d3-176cfdcf99d5/b64e35a5-c86f-43a6-acb5-469d75a46b72/dab81acb-601b-4578-836c-bbc42190f256"
-					(reference "U17")
+					(reference "U16")
 					(unit 1)
 				)
@@
 		(dnp no)
 		(fields_autoplaced yes)
-		(property "Reference" "#PWR0118"
+		(property "Reference" "#PWR0115"
 			(at 222.25 135.89 0)
 			(effects
@@
 			(project "ETH1CVOLT_B"
 				(path "/18612734-e331-4379-b1d3-176cfdcf99d5/b64e35a5-c86f-43a6-acb5-469d75a46b72/dab81acb-601b-4578-836c-bbc42190f256"
-					(reference "#PWR0118")
+					(reference "#PWR0115")
 					(unit 1)
 				)
@@
 		(dnp no)
 		(fields_autoplaced yes)
-		(property "Reference" "#PWR0114"
+		(property "Reference" "#PWR0111"
 			(at 48.26 278.13 0)
 			(effects
@@
 			(project "ETH1CVOLT_B"
 				(path "/18612734-e331-4379-b1d3-176cfdcf99d5/b64e35a5-c86f-43a6-acb5-469d75a46b72/dab81acb-601b-4578-836c-bbc42190f256"
-					(reference "#PWR0114")
+					(reference "#PWR0111")
 					(unit 1)
 				)
@@
 		(dnp no)
 		(fields_autoplaced yes)
-		(property "Reference" "C38"
+		(property "Reference" "C37"
 			(at 52.07 266.6999 0)
 			(effects
@@
 			(project "ETH1CVOLT_B"
 				(path "/18612734-e331-4379-b1d3-176cfdcf99d5/b64e35a5-c86f-43a6-acb5-469d75a46b72/dab81acb-601b-4578-836c-bbc42190f256"
-					(reference "C38")
-					(unit 1)
-				)
+					(reference "C37")
+					(unit 1)
+				)
