File: HARDWARE/ETH1CVOLT_B/MV_Output.kicad_sch (KiCad schematic)
At the start: 15 parts, among them U18 SN74LVC1G125DBV, U8 OPA593, U9 OPA593

Commit message: Development
Parts:
- R14: renamed from R18; footprint (none) -> Resistor_SMD:R_0603_1608Metric_Pad0.98x0.95mm_HandSolder
- R15: renamed from R12; footprint (none) -> Resistor_SMD:R_0603_1608Metric_Pad0.98x0.95mm_HandSolder
- R16, R19, R20, R21, R22: footprint (none) -> Resistor_SMD:R_0603_1608Metric_Pad0.98x0.95mm_HandSolder
- R17: renamed from R5; footprint (none) -> Resistor_SMD:R_0603_1608Metric_Pad0.98x0.95mm_HandSolder
- R18: renamed from R17; footprint (none) -> Resistor_SMD:R_0603_1608Metric_Pad0.98x0.95mm_HandSolder
- renumbered D3 to D2, D4 to D3, U8 to U10, U9 to U11, U18 to U9
Connections:
- net +5VD_ISO renamed +VD_ISO
Other:
- moved on the sheet: U9

Commit message: Development
Parts:
- removed D3: SMAJ45CA, Diode_SMD:D_SMA, symbol Diode:SMAJ45CA
- added C30, C31, C32, C33, C34: 0.1u/100V, symbol Device:C
- added D5: SMAJ43CA, Diode_SMD:D_SMA, symbol Diode:SMAJ43CA
- renumbered D2 to D4, R14 to R17, R15 to R18, R16 to R19, R17 to R20, R18 to R21, R19 to R22, R20 to R23, R21 to R24, R22 to R25, R23 to R26, U9 to U13, U10 to U14, U11 to U15
Connections:
- net +44V_ISO: now also C30.1, C31.1
- net +VD_ISO: now also C34.1
- net -41V_ISO: now also C32.1, C33.1
- net GND_ISO: now also C30.2, C31.2, C32.2, C33.2, C34.2, D5.1 (A1)
- net MV_OUTPUT: now also D5.2 (A2)
Other:
- moved on the sheet: D4, R17, R18, R19, R20, R21, R22, R23, R24, R25, R26, U13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

Commit message: Development
Parts:
- C29: renamed from C30; footprint (none) -> Capacitor_SMD:C_0603_1608Metric_Pad1.08x0.95mm_HandSolder
- C30: renamed from C31; footprint (none) -> Capacitor_SMD:C_0603_1608Metric_Pad1.08x0.95mm_HandSolder
- C31: renamed from C32; footprint (none) -> Capacitor_SMD:C_0603_1608Metric_Pad1.08x0.95mm_HandSolder
- C32: renamed from C33; footprint (none) -> Capacitor_SMD:C_0603_1608Metric_Pad1.08x0.95mm_HandSolder
- C33: renamed from C34; footprint (none) -> Capacitor_SMD:C_0603_1608Metric_Pad1.08x0.95mm_HandSolder
- R26: footprint (none) -> Resistor_SMD:R_1206_3216Metric_Pad1.30x1.75mm_HandSolder
- renumbered U13 to U12, U14 to U13, U15 to U14

Commit message: Development
Parts:
- added TP22, TP25: TestPoint, TestPoint:TestPoint_Pad_D1.5mm, symbol Connector:TestPoint
Connections:
- net MV_MEAS: now also TP25.1
- net MV_OUTPUT: now also TP22.1
Other:
- note added: "+/-20V"
- moved on the sheet: U12
