File: HARDWARE/ETH1CVOLT_B/Voltage_Reference.kicad_sch (KiCad schematic)
At the start: 13 parts, among them U13 LT1027CCS8-5#PBF, U14 ADA4522-1

Commit message: Development
Parts:
- removed U14: ADA4522-1, symbol Amplifier_Operational:ADA4522-1
- added R45: 100k/0.1%, Resistor_SMD:R_0603_1608Metric_Pad0.98x0.95mm_HandSolder, symbol Device:R
- added R46: 180k/0.05%, Resistor_SMD:R_0603_1608Metric_Pad0.98x0.95mm_HandSolder, symbol Device:R
- added R47: 18k/0.05%, Resistor_SMD:R_0603_1608Metric_Pad0.98x0.95mm_HandSolder, symbol Device:R
- added R48: 2k/0.05%, Resistor_SMD:R_0603_1608Metric_Pad0.98x0.95mm_HandSolder, symbol Device:R
- added U17: DG412EUE+, Package_SO:TSSOP-16_4.4x5mm_P0.65mm, symbol Analog_Switch:DG412xUE
- added U19: ADA4077-1xRM, Package_SO:MSOP-8_3x3mm_P0.65mm, symbol Amplifier_Operational:ADA4077-1xRM
- C12: renamed from C9; footprint (none) -> Capacitor_SMD:C_0603_1608Metric_Pad1.08x0.95mm_HandSolder
- renumbered C91 to C10, C93 to C11, C10 to C13, C11 to C14, C12 to C15, C13 to C16, C14 to C17, U13 to U18
Connections:
- net +21V_ISO: now also U17.13 (V+), U19.7 (V+)
- net +5VREF_ISO: now also U19.3 (+)
- net GND_ISO: now also R48.2, U17.4 (V-), U17.5 (GND), U19.4 (V-)
- net at RN4.3: now also U19.2 (-)
- net +10VREF_ISO: no longer names the net of C17.1, RN4.1
- net +10VREF_ISO: now also R46.1, U17.2, U19.6
- new net: R46.2, R47.1, U17.6
- new net: R45.2, U17.16
- new net: R47.2, R48.1, U17.10
- new net: U17.14, U17.15
- new net +VD_ISO: R45.1, U17.12 (VL)
- new net SEL_x1: U17.1
- new net SEL_x10: U17.8
- new net SEL_x100: U17.9
- new net VREF_TEST: U17.11, U17.3, U17.7
Other:
- moved on the sheet: C10, C11, C12, C13, C14, C15, C16, C17, RN3, RN4, RV1, U18

Commit message: Development
Parts:
- renumbered C10 to C42, C11 to C43, C12 to C44, C13 to C45, C14 to C46, C15 to C47, C16 to C48, C17 to C49, R45 to R48, R46 to R49, R47 to R50, R48 to R51, RN3 to RN4, RN4 to RN5, U17 to U21, U18 to U22, U19 to U23
Other:
- note added: "0.1V"
- note added: "10V"
- note added: "1V"
- moved on the sheet: U21A, U21B, U21C

Commit message: Development
Parts:
- C46: renamed from C42; value 4u7/50V -> 4u7/100V
- C47: renamed from C43; value 10u/50V -> 10u/100V
- C48: renamed from C44; value 1u -> 1u/50V
- C49: renamed from C45; value 4u7/50V -> 4u7/100V
- C50: renamed from C46; value 10u/50V -> 10u/100V
- C51: renamed from C47; value 4u7/50V -> 4u7/100V
- C52: renamed from C48; value 10u/50V -> 10u/100V
- C53: renamed from C49; value 10u/50V -> 10u/100V
- RV1: footprint (none) -> Potentiometer_SMD:Potentiometer_Bourns_3314G_Vertical; now not fitted; now left out of the parts list
- renumbered U21 to U20, U22 to U21, U23 to U22
Other:
- moved on the sheet: C46, C50, C51, C52, R48, RN4, U20D, U20E
