File: HARDWARE/ETH1CVOLT/ETH1CVOLT.kicad_pcb (KiCad board)
At the start: 4 copper layers, 160 x 100 mm, 297 parts, among them J1 20021111-00010T4LF, J2 7499010121A, J3 TSW-102-23-G-S, J4 TSW-102-23-G-S, J6 1827868, J7 FCR7350R, J8 FCR7350B, K1 G6SK-2F DC5, Q1 CSD18501Q5A, Q2 2N7002, Q3 2N7002, U1 STM32H743VITx, U10 MAX44241AUA+, U11 ISO7761FDBQ, U12 ISO7760DBQ, U13 OPA192IDR, U14 ADA4522-1ARZ, U15 RP-2424D, U16 TMR4-2423WI, U17 TEC2-2419WI, U18 TSR0.5-2465, U19 TPS7A3901DSCR, U2 24LC08B-E/MS, U20 TPS7A3901DSCR, U21 ADP7142ARDZ-5.0, U22 ADP7142ARDZ-5.0, U23 TPS7A3901DSCR, U24 TSR0.5-2433, U25 ADA4522-2ARZ-RL, U26 74LV1T08GV, U27 74LV1T08GV, U3 LAN8742A, U4 INA159AIDGKT, U5 DG412CUE+, U6 LTC2400CS8#TRPBF, U7 OPA2192ID, U8 ADR1399KEZ, U9 MAX5719GSD+, Y1 NX5032GA-16, Y2 NX5032GA-25

Commit message: Layout
Parts:
- removed the C11 at (37.8, 144.1)
- removed the C53 at (170.8, -14.2)
- removed the C7 at (33.4, 154.1)
- removed the R2 at (42.1, 141.6)
- removed the TP41 at (193.6, 74.9)
- removed the TP44 at (183.4, 56.0)
- added C36: 10u/50V/X7R, Capacitor_SMD:C_1206_3216Metric_Pad1.33x1.80mm_HandSolder, F.Cu at (172.7, 115.0)
- added FID1: Fiducial, Fiducial:Fiducial_1.5mm_Mask3mm, F.Cu at (73.0, 134.0)
- added FID2: Fiducial, Fiducial:Fiducial_1.5mm_Mask3mm, B.Cu at (73.0, 134.0)
- added FID3: Fiducial, Fiducial:Fiducial_1.5mm_Mask3mm, F.Cu at (208.0, 47.0)
- added FID4: Fiducial, Fiducial:Fiducial_1.5mm_Mask3mm, B.Cu at (208.0, 47.0)
- added FID5: Fiducial, Fiducial:Fiducial_1.5mm_Mask3mm, F.Cu at (226.0, 123.0)
- added FID6: Fiducial, Fiducial:Fiducial_1.5mm_Mask3mm, B.Cu at (226.0, 123.0)
- added TP27: TestPoint, TestPoint:TestPoint_Pad_D1.5mm, F.Cu at (130.4, 126.4)
- added TP28: TestPoint, TestPoint:TestPoint_Pad_D1.5mm, F.Cu at (130.4, 130.8)
- C25: renamed from C27; moved to B.Cu
- C26: renamed from C28; moved to B.Cu
- R39: renamed from R40; moved to F.Cu
- R40: renamed from R41; moved to F.Cu
- R5: renamed from R6; moved to B.Cu
- RN2, RN3: moved to B.Cu
- TP10, TP11, TP12, TP15, TP16, TP20: footprint TestPoint:TestPoint_Pad_D1.5mm -> TestPoint:TestPoint_Pad_D1.0mm
- TP13: renamed from TP18; footprint TestPoint:TestPoint_Pad_D1.5mm -> TestPoint:TestPoint_Pad_D1.0mm
- TP14: renamed from TP17; footprint TestPoint:TestPoint_Pad_D1.5mm -> TestPoint:TestPoint_Pad_D1.0mm
- TP17: renamed from TP14; footprint TestPoint:TestPoint_Pad_D1.5mm -> TestPoint:TestPoint_Pad_D1.0mm
- TP18: renamed from TP21; footprint TestPoint:TestPoint_Pad_D1.5mm -> TestPoint:TestPoint_Pad_D1.0mm
- TP19: renamed from TP13; footprint TestPoint:TestPoint_Pad_D1.5mm -> TestPoint:TestPoint_Pad_D1.0mm
- TP21: renamed from TP19; footprint TestPoint:TestPoint_Pad_D1.5mm -> TestPoint:TestPoint_Pad_D1.0mm
- moved C100 203.6 mm to (86.6, 78.0), turned to -90 degrees
- moved C101 193.1 mm to (98.0, 72.4), turned to 90 degrees
- moved C52 190.8 mm to (81.0, 109.0), turned to 90 degrees
- moved C99 188.9 mm to (86.6, 72.4), turned to 90 degrees
- moved C56 187.6 mm to (83.8, 94.8), turned to 90 degrees
- moved C59 176.8 mm to (83.8, 100.4), turned to -90 degrees
- moved C102 175.8 mm to (115.9, 73.5), turned to 90 degrees
- moved Y1 170.0 mm to (124.8, 45.5), turned to 180 degrees
- moved R61 167.6 mm to (152.9, 113.3)
- moved R60 167.2 mm to (152.9, 111.5)
- moved C37 164.3 mm to (187.3, 98.9), turned to 180 degrees
- moved C62 163.0 mm to (95.0, 94.8), turned to 90 degrees
- moved C38 162.8 mm to (187.2, 96.4), turned to 180 degrees
- moved TP24 161.6 mm to (83.2, 119.6)
- moved RN1 159.5 mm to (109.8, 58.1), turned to 180 degrees
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- renumbered C102 to C100, C103 to C101, C104 to C102, C105 to C103, C106 to C104, C107 to C105, C108 to C106, C14 to C11, C15 to C13, C16 to C14, C17 to C15, C18 to C16, C19 to C17, C20 to C18, C21 to C19, C22 to C20, C23 to C21, C24 to C22, C25 to C23, C26 to C24, C29 to C27, C30 to C28, C31 to C29, C32 to C30, C33 to C31, C34 to C32, C35 to C33, C36 to C34, C37 to C35, C38 to C37, C39 to C38, C40 to C39, C41 to C40, C42 to C41, C43 to C42, C44 to C43, C45 to C44, C46 to C45, C47 to C46, C48 to C47, C49 to C48, C50 to C49, C51 to C50, C52 to C51, C54 to C52, C55 to C53, C56 to C54, C57 to C55, C58 to C56, C59 to C57, C60 to C58, C61 to C59, C62 to C60, C63 to C61, C64 to C62, C65 to C63, C66 to C64, C67 to C65, C68 to C66, C69 to C67, C70 to C68, C71 to C69, C13 to C7, C72 to C70, C73 to C71, C74 to C72, C75 to C73, C76 to C74, C78 to C75, C79 to C76, C80 to C78, C81 to C79, C82 to C80, C83 to C81, C84 to C82, C85 to C83, C86 to C84, C87 to C85, C88 to C86, C89 to C87, C90 to C88, C91 to C89, C92 to C90, C93 to C91, C94 to C92, C95 to C93, C96 to C94, C97 to C95, C98 to C96, C99 to C97, C100 to C98, C101 to C99, D9 to D10, D10 to D4, D4 to D5, D5 to D6, D6 to D7, D7 to D8, D8 to D9, R11 to R10, R12 to R11, R13 to R12, R14 to R13, R15 to R14, R16 to R15, R17 to R16, R18 to R17, R19 to R18, R20 to R19, R3 to R2, R21 to R20, R22 to R21, R23 to R22, R24 to R23, R25 to R24, R26 to R25, R27 to R26, R28 to R27, R29 to R28, R30 to R29, R4 to R3, R31 to R30, R32 to R31, R33 to R32, R34 to R33, R35 to R34, R36 to R35, R37 to R36, R38 to R37, R39 to R38, R5 to R4, R42 to R41, R43 to R42, R44 to R43, R45 to R44, R46 to R45, R47 to R46, R48 to R47, R49 to R48, R50 to R49, R51 to R50, R52 to R51, R53 to R52, R54 to R53, R55 to R54, R56 to R55, R57 to R56, R58 to R57, R59 to R58, R60 to R59, R7 to R6, R62 to R60, R63 to R61, R61 to R62, R64 to R63, R65 to R64, R66 to R65, R67 to R66, R68 to R67, R69 to R68, R70 to R69, R8 to R7, R71 to R70, R72 to R71, R73 to R72, R74 to R73, R75 to R74, R76 to R75, R9 to R8, R10 to R9, TP27 to TP29, TP28 to TP30, TP29 to TP31, TP30 to TP32, TP31 to TP33, TP32 to TP34, TP33 to TP35, TP34 to TP36, TP35 to TP37, TP36 to TP38, TP37 to TP39, TP38 to TP40, TP39 to TP41, TP40 to TP42, TP42 to TP43, TP43 to TP44
Connections:
- TP10 pad 1: /BLOCK DIAGRAM/ADC/ADC_SW1 -> /BLOCK DIAGRAM/ISO DIG/REL_SET
- TP11 pad 1: /BLOCK DIAGRAM/ADC/ADC_VOLT_SCLK -> /BLOCK DIAGRAM/ADC/ADC_SW2
- TP12 pad 1: /BLOCK DIAGRAM/DAC/DAC_~{CS} -> /BLOCK DIAGRAM/ADC/ADC_~{CS}
- TP13 pad 1: /BLOCK DIAGRAM/ADC/ADC_SW3 -> /BLOCK DIAGRAM/DAC/DAC_SCLK
- TP14 pad 1: /BLOCK DIAGRAM/ISO DIG/REL_SET -> /BLOCK DIAGRAM/ISO DIG/REL_RESET
- TP15 pad 1: /BLOCK DIAGRAM/ADC/ADC_VOLT_~{CS} -> /BLOCK DIAGRAM/ADC/ADC_SW1
- TP16 pad 1: /BLOCK DIAGRAM/DAC/DAC_DIN -> /BLOCK DIAGRAM/ADC/ADC_SCLK
- TP17 pad 1: /BLOCK DIAGRAM/ADC/ADC_SW2 -> /BLOCK DIAGRAM/DAC/DAC_~{CS}
- TP18 pad 1: /BLOCK DIAGRAM/ISO DIG/REL_RESET -> /BLOCK DIAGRAM/ADC/ADC_SW3
- TP19 pad 1: /BLOCK DIAGRAM/DAC/DAC_~{LDAC} -> /BLOCK DIAGRAM/ADC/ADC_SDO
- TP20 pad 1: /BLOCK DIAGRAM/DAC/DAC_SCLK -> /BLOCK DIAGRAM/DAC/DAC_~{LDAC}
- TP21 pad 1: /BLOCK DIAGRAM/ADC/ADC_VOLT_SDO -> /BLOCK DIAGRAM/DAC/DAC_DIN
- U1 pad 1: unconnected-(U1-PE2-Pad1) -> /BLOCK DIAGRAM/MCU/MCU_DEF
- U1 pad 28: /BLOCK DIAGRAM/MCU/ADC_VOLT_~{CS} -> /BLOCK DIAGRAM/ISO DIG/MCU_ADC_~{CS}
- U1 pad 29: /BLOCK DIAGRAM/MCU/ADC_VOLT_SCLK -> unconnected-(U1-PA5-Pad29)
- U1 pad 3: /BLOCK DIAGRAM/MCU/MCU_ADC_CURR_~{CS} -> unconnected-(U1-PE4-Pad3)
- U1 pad 30: /BLOCK DIAGRAM/MCU/ADC_VOLT_SDO -> unconnected-(U1-PA6-Pad30)
- U1 pad 4: /BLOCK DIAGRAM/MCU/MCU_ADC_CURR_SDO -> unconnected-(U1-PE5-Pad4)
- U1 pad 5: /BLOCK DIAGRAM/MCU/MCU_ADC_CURR_SDI -> unconnected-(U1-PE6-Pad5)
- U1 pad 66: unconnected-(U1-PC9-Pad66) -> /BLOCK DIAGRAM/MCU/I2C1_SDA
- U1 pad 67: unconnected-(U1-PA8-Pad67) -> /BLOCK DIAGRAM/MCU/I2C1_SCL
- U1 pad 68: unconnected-(U1-PA9-Pad68) -> /BLOCK DIAGRAM/MCU/EEPROM_nWP
- U1 pad 77: unconnected-(U1-PA15-Pad77) -> /BLOCK DIAGRAM/ISO DIG/MCU_DAC_~{CS}
- U1 pad 78: unconnected-(U1-PC10-Pad78) -> /BLOCK DIAGRAM/ISO DIG/MCU_DAC_SCLK
- U1 pad 80: unconnected-(U1-PC12-Pad80) -> /BLOCK DIAGRAM/ISO DIG/MCU_DAC_DIN
- U1 pad 81: unconnected-(U1-PD0-Pad81) -> /BLOCK DIAGRAM/ISO DIG/MCU_DAC_~{LDAC}
- U1 pad 89: unconnected-(U1-PB3-Pad89) -> /BLOCK DIAGRAM/ISO DIG/MCU_ADC_SCLK
- U1 pad 90: unconnected-(U1-PB4-Pad90) -> /BLOCK DIAGRAM/ISO DIG/MCU_ADC_SDO
- U1 pad 91: /BLOCK DIAGRAM/MCU/EEPROM_nWP -> unconnected-(U1-PB5-Pad91)
- U1 pad 92: /BLOCK DIAGRAM/MCU/I2C1_SCL -> unconnected-(U1-PB6-Pad92)
- U1 pad 93: /BLOCK DIAGRAM/MCU/I2C1_SDA -> /BLOCK DIAGRAM/ISO DIG/MCU_ADC_SW1
- U1 pad 94: Net-(U1-BOOT0) -> GND
- U1 pad 95: unconnected-(U1-PB8-Pad95) -> /BLOCK DIAGRAM/ISO DIG/MCU_ADC_SW2
- U1 pad 96: unconnected-(U1-PB9-Pad96) -> /BLOCK DIAGRAM/ISO DIG/MCU_ADC_SW3
- U1 pad 97: unconnected-(U1-PE0-Pad97) -> /BLOCK DIAGRAM/ISO DIG/MCU_REL_RESET
- U1 pad 98: /BLOCK DIAGRAM/MCU/MCU_DEF -> /BLOCK DIAGRAM/ISO DIG/MCU_REL_SET
- U11 pad 10: /BLOCK DIAGRAM/ADC/ADC_VOLT_SDO -> /BLOCK DIAGRAM/ADC/ADC_SDO
- U11 pad 11: /BLOCK DIAGRAM/ADC/ADC_VOLT_~{CS} -> /BLOCK DIAGRAM/ADC/ADC_SW1
- U11 pad 12: /BLOCK DIAGRAM/ADC/ADC_VOLT_SCLK -> /BLOCK DIAGRAM/ADC/ADC_SW2
- U11 pad 14: /BLOCK DIAGRAM/ADC/ADC_SW2 -> /BLOCK DIAGRAM/ISO DIG/REL_RESET
- U11 pad 15: /BLOCK DIAGRAM/ADC/ADC_SW1 -> /BLOCK DIAGRAM/ISO DIG/REL_SET
- U11 pad 2: /BLOCK DIAGRAM/ISO DIG/MCU_ADC_SW1 -> /BLOCK DIAGRAM/ISO DIG/MCU_REL_SET
- U11 pad 3: /BLOCK DIAGRAM/ISO DIG/MCU_ADC_SW2 -> /BLOCK DIAGRAM/ISO DIG/MCU_REL_RESET
- U11 pad 5: /BLOCK DIAGRAM/ISO DIG/MCU_ADC_VOLT_SCLK -> /BLOCK DIAGRAM/ISO DIG/MCU_ADC_SW2
- U11 pad 6: /BLOCK DIAGRAM/ISO DIG/MCU_ADC_VOLT_~{CS} -> /BLOCK DIAGRAM/ISO DIG/MCU_ADC_SW1
- U11 pad 7: /BLOCK DIAGRAM/ISO DIG/MCU_ADC_VOLT_SDO -> /BLOCK DIAGRAM/ISO DIG/MCU_ADC_SDO
- U12 pad 10: /BLOCK DIAGRAM/ISO DIG/REL_RESET -> /BLOCK DIAGRAM/DAC/DAC_DIN
- U12 pad 11: /BLOCK DIAGRAM/ISO DIG/REL_SET -> /BLOCK DIAGRAM/DAC/DAC_~{CS}
- U12 pad 12: /BLOCK DIAGRAM/DAC/DAC_~{LDAC} -> /BLOCK DIAGRAM/DAC/DAC_SCLK
- U12 pad 13: /BLOCK DIAGRAM/DAC/DAC_SCLK -> /BLOCK DIAGRAM/DAC/DAC_~{LDAC}
- U12 pad 14: /BLOCK DIAGRAM/DAC/DAC_DIN -> /BLOCK DIAGRAM/ADC/ADC_SCLK
- U12 pad 15: /BLOCK DIAGRAM/DAC/DAC_~{CS} -> /BLOCK DIAGRAM/ADC/ADC_~{CS}
- U12 pad 2: /BLOCK DIAGRAM/ISO DIG/MCU_DAC_~{CS} -> /BLOCK DIAGRAM/ISO DIG/MCU_ADC_~{CS}
- U12 pad 3: /BLOCK DIAGRAM/ISO DIG/MCU_DAC_DIN -> /BLOCK DIAGRAM/ISO DIG/MCU_ADC_SCLK
- U12 pad 4: /BLOCK DIAGRAM/ISO DIG/MCU_DAC_SCLK -> /BLOCK DIAGRAM/ISO DIG/MCU_DAC_~{LDAC}
- U12 pad 5: /BLOCK DIAGRAM/ISO DIG/MCU_DAC_~{LDAC} -> /BLOCK DIAGRAM/ISO DIG/MCU_DAC_SCLK
- U12 pad 6: /BLOCK DIAGRAM/ISO DIG/MCU_REL_SET -> /BLOCK DIAGRAM/ISO DIG/MCU_DAC_~{CS}
- U12 pad 7: /BLOCK DIAGRAM/ISO DIG/MCU_REL_RESET -> /BLOCK DIAGRAM/ISO DIG/MCU_DAC_DIN
- U6 pad 5: /BLOCK DIAGRAM/ADC/ADC_VOLT_~{CS} -> /BLOCK DIAGRAM/ADC/ADC_~{CS}
- U6 pad 6: /BLOCK DIAGRAM/ADC/ADC_VOLT_SDO -> /BLOCK DIAGRAM/ADC/ADC_SDO
- U6 pad 7: /BLOCK DIAGRAM/ADC/ADC_VOLT_SCLK -> /BLOCK DIAGRAM/ADC/ADC_SCLK
- U8 pad 1: GNDA -> GND_ISO
- U8 pad 2: GNDA -> GND_ISO
Routing:
- net /BLOCK DIAGRAM/ISO DIG/REL_SET: track 0.00 -> 102.0 mm, vias 0 -> 2
- net /BLOCK DIAGRAM/ISO DIG/REL_RESET: track 0.00 -> 53.3 mm
- net Net-(D10-A2): track 0.00 -> 49.9 mm
- net Net-(J4-Pin_1): track 0.00 -> 43.2 mm
- net /BLOCK DIAGRAM/ADC/ADC_SW3: track 0.00 -> 39.4 mm
- net /BLOCK DIAGRAM/ADC/ADC_SW2: track 0.00 -> 37.9 mm, vias 0 -> 2
- net Net-(J3-Pin_1): track 0.00 -> 37.4 mm
- net /BLOCK DIAGRAM/ADC/MEAS_OUT: track 0.00 -> 36.7 mm
- net /BLOCK DIAGRAM/OUTPUT/R20V_SIG: track 0.00 -> 35.2 mm
- net Net-(D2-K-Pad3): track 0.00 -> 32.8 mm
- net /BLOCK DIAGRAM/ADC/ADC_SW1: track 0.00 -> 31.9 mm, vias 0 -> 2
- net +5VD_ISO: track 0.00 -> 31.2 mm, vias 0 -> 10
- net +3.3V: track 0.00 -> 31.0 mm, vias 0 -> 14
- net /BLOCK DIAGRAM/MCU/NRST: track 0.00 -> 30.0 mm, vias 0 -> 1
- net Net-(U8-+REFF): track 0.00 -> 29.2 mm
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- added copper zone on In1.Cu, net GND
- added copper zone on In1.Cu, net GND_ISO
Other:
- outline, holes or cut-outs redrawn
- copper layers 4 -> 6
- board text added: "1"
- board text added: "2"
- board text added: "3"
- board text added: "4"
- board text added: "5"
- board text added: "6"

Commit message: Layout and schematic
Parts:
- removed the C39 at (191.0, 89.4)
- removed J3: TSW-102-23-G-S, Connector_PinHeader_2.54mm:PinHeader_1x02_P2.54mm_Vertical
- removed the J4 at (157.0, 88.8)
- removed JP2, JP3, JP4, JP5, JP6, JP7, JP8, JP9: SolderJumper_2_Open, Jumper:SolderJumper-2_P1.3mm_Open_Pad1.0x1.5mm
- removed the R20 at (181.7, 113.6)
- removed the R21 at (191.0, 96.9)
- removed the R22 at (179.5, 94.0)
- removed the R23 at (167.0, 86.2)
- removed the R24 at (165.2, 86.2)
- removed the R25 at (177.0, 94.0)
- removed the R26 at (167.0, 89.8)
- removed the R27 at (174.5, 94.0)
- removed the R28 at (172.0, 94.0)
- removed the R29 at (169.5, 94.0)
- removed the R30 at (167.0, 94.0)
- removed the R31 at (164.5, 94.0)
- removed the R32 at (187.0, 86.3)
- removed the R33 at (162.0, 94.0)
- removed RV1: M64Y501KB40, Potentiometer_THT:Potentiometer_Bourns_3386X_Horizontal
- removed the TP6 at (182.6, 96.9)
- removed the TP7 at (191.0, 86.4)
- removed the TP8 at (183.7, 86.3)
- added C35: 0.1u/100V/X7R, Capacitor_SMD:C_0603_1608Metric_Pad1.08x0.95mm_HandSolder, F.Cu at (162.2, 75.5)
- added C40: 1u/16V/X7R, Capacitor_SMD:C_0603_1608Metric_Pad1.08x0.95mm_HandSolder, F.Cu at (166.0, 85.8)
- added C41: 0.1u/100V/X7R, Capacitor_SMD:C_0603_1608Metric_Pad1.08x0.95mm_HandSolder, F.Cu at (150.9, 76.0)
- added C42: 1u/16V/X7R, Capacitor_SMD:C_0603_1608Metric_Pad1.08x0.95mm_HandSolder, F.Cu at (150.9, 74.4)
- C36: value 10u/50V/X7R -> 0.1u/100V/X7R; footprint Capacitor_SMD:C_1206_3216Metric_Pad1.33x1.80mm_HandSolder -> Capacitor_SMD:C_0603_1608Metric_Pad1.08x0.95mm_HandSolder
- C37: value 10u/50V/X7R -> 1u/16V/X7R; footprint Capacitor_SMD:C_1206_3216Metric_Pad1.33x1.80mm_HandSolder -> Capacitor_SMD:C_0603_1608Metric_Pad1.08x0.95mm_HandSolder
- C38: value 4u7/50V/X7R -> 10u/50V/X7R
- R19: value 0R/5%/100mW -> 100/1%/100mW
- U13: value OPA192IDR -> ADA4522-1ARZ
- U7: value OPA2192ID -> ADR4550
- U8: value ADR1399KEZ -> ADA4522-1ARZ; footprint Package_LCC:Analog_LCC-8_5x5mm_P1.27mm -> Package_SO:SOIC-8_3.9x4.9mm_P1.27mm
- moved R19 55.7 mm to (150.9, 77.6), turned to 0 degrees
- moved TP5 48.8 mm to (147.5, 78.3)
- moved R18 46.9 mm to (161.6, 78.2), turned to -90 degrees
- moved U8 43.1 mm to (156.7, 77.4), turned to 180 degrees
- moved C34 34.2 mm to (150.9, 79.2), turned to 180 degrees
- moved C39 29.5 mm to (162.4, 85.8), turned to 180 degrees
- moved C38 28.6 mm to (159.3, 90.2), turned to -90 degrees
- moved C36 24.5 mm to (162.4, 92.8), turned to 180 degrees
- moved U7 23.1 mm to (164.2, 89.3), turned to 0 degrees
- moved C37 22.1 mm to (166.0, 92.8), turned to 0 degrees
- moved TP22 6.29 mm to (91.5, 122.2)
- moved C77 2.82 mm to (141.6, 99.2)
- moved TP35 2.12 mm to (137.4, 83.3)
- moved TP36 1.89 mm to (122.8, 83.9)
- moved TP30 1.70 mm to (135.5, 134.0)
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- renumbered C97 to C100, C98 to C101, C99 to C102, C100 to C103, C101 to C104, C102 to C105, C103 to C106, C104 to C107, C105 to C108, C106 to C109, C35 to C39, C40 to C43, C41 to C44, C42 to C45, C43 to C46, C44 to C47, C45 to C48, C46 to C49, C47 to C50, C48 to C51, C49 to C52, C50 to C53, C51 to C54, C52 to C55, C53 to C56, C54 to C57, C55 to C58, C56 to C59, C57 to C60, C58 to C61, C59 to C62, C60 to C63, C61 to C64, C62 to C65, C63 to C66, C64 to C67, C65 to C68, C66 to C69, C67 to C70, C68 to C71, C69 to C72, C70 to C73, C71 to C74, C72 to C75, C73 to C76, C74 to C77, C75 to C78, C76 to C79, C77 to C80, C78 to C81, C79 to C82, C80 to C83, C81 to C84, C82 to C85, C83 to C86, C84 to C87, C85 to C88, C86 to C89, C87 to C90, C88 to C91, C89 to C92, C90 to C93, C91 to C94, C92 to C95, C93 to C96, C94 to C97, C95 to C98, C96 to C99, J6 to J4, J7 to J5, J8 to J6, R34 to R20, R35 to R21, R36 to R22, R37 to R23, R38 to R24, R39 to R25, R40 to R26, R41 to R27, R42 to R28, R43 to R29, R44 to R30, R45 to R31, R46 to R32, R47 to R33, R48 to R34, R49 to R35, R50 to R36, R51 to R37, R52 to R38, R53 to R39, R54 to R40, R55 to R41, R56 to R42, R57 to R43, R58 to R44, R59 to R45, R60 to R46, R61 to R47, R62 to R48, R63 to R49, R64 to R50, R67 to R51, R68 to R52, R65 to R53, R66 to R54, R69 to R55, R70 to R56, R71 to R57, R72 to R58, R73 to R59, R74 to R60, R75 to R61, TP13 to TP10, TP14 to TP11, TP15 to TP12, TP16 to TP13, TP17 to TP14, TP18 to TP15, TP19 to TP16, TP20 to TP17, TP21 to TP18, TP22 to TP19, TP23 to TP20, TP24 to TP21, TP25 to TP22, TP26 to TP23, TP27 to TP24, TP28 to TP25, TP29 to TP26, TP30 to TP27, TP31 to TP28, TP32 to TP29, TP33 to TP30, TP34 to TP31, TP35 to TP32, TP36 to TP33, TP37 to TP34, TP38 to TP35, TP39 to TP36, TP40 to TP37, TP41 to TP38, TP42 to TP39, TP43 to TP40, TP44 to TP41, TP9 to TP6, TP10 to TP7, TP11 to TP8, TP12 to TP9
Connections:
- C36 pad 1: +15V_ISO -> +14V_ISO
- C37 pad 1: Net-(U7A-+) -> +14V_ISO
- C38 pad 1: Net-(U7A-+) -> +14V_ISO
- C39 pad 1: -14V_ISO -> Net-(U7-OUT)
- R18 pad 1: GND_ISO -> Net-(U7-OUT)
- R18 pad 2: Net-(U8-HEATER-) -> Net-(U8--)
- R19 pad 1: -15V_ISO -> +5VREF_ISO
- R19 pad 2: Net-(U8-HEATER-) -> Net-(U8--)
- TP5 pad 1: Net-(U8-+REFF) -> +5VREF_ISO
- U7 pad 1: Net-(J3-Pin_1) -> unconnected-(U7-NC-Pad1)
- U7 pad 2: Net-(J3-Pin_1) -> +14V_ISO
- U7 pad 3: Net-(U7A-+) -> unconnected-(U7-NC-Pad3)
- U7 pad 4: -14V_ISO -> GND_ISO
- U7 pad 5: Net-(J4-Pin_1) -> unconnected-(U7-NC-Pad5)
- U7 pad 6: Net-(U7B--) -> Net-(U7-OUT)
- U7 pad 7: Net-(U7B--) -> unconnected-(U7-NC-Pad7)
- U7 pad 8: +14V_ISO -> unconnected-(U7-NC-Pad8)
- U8 pad 1: GND_ISO -> unconnected-(U8-NC-Pad1)
- U8 pad 2: GND_ISO -> Net-(U8--)
- U8 pad 3: +15V_ISO -> Net-(U7-OUT)
- U8 pad 4: unconnected-(U8-NC-Pad4) -> -14V_ISO
- U8 pad 5: Net-(U8-HEATER-) -> unconnected-(U8-NC-Pad5)
- U8 pad 6: Net-(U8-+REFF) -> Net-(U8--)
- U8 pad 7: Net-(U8-+REFF) -> +14V_ISO
Routing:
- net Net-(J4-Pin_1): track 43.2 -> 0.00 mm
- net Net-(J3-Pin_1): track 37.4 -> 0.00 mm
- net Net-(U8-+REFF): track 29.2 -> 0.00 mm
- net Net-(R22-Pad2): track 29.2 -> 0.00 mm
- net Net-(U7-OUT): track 0.00 -> 19.7 mm
- net Net-(U8-HEATER-): track 11.6 -> 0.00 mm
- net Net-(U8--): track 0.00 -> 11.1 mm
- net +14V_ISO: track 11.5 -> 22.3 mm
- net Net-(U7A-+): track 8.00 -> 0.00 mm
- net Net-(U7B--): track 6.88 -> 0.00 mm
- net Net-(U20-FBP): track 0.00 -> 4.82 mm, vias 0 -> 1
- net +15V_ISO: track 4.79 -> 0.00 mm, vias 2 -> 0
- net Net-(R44-Pad1): track 0.00 -> 3.40 mm
- net +6V5_ISO: track 0.00 -> 3.30 mm, vias 0 -> 9
- net Net-(JP9-A): track 2.54 -> 0.00 mm
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- added copper zone on F.Cu, net +14V_ISO
- added copper zone on F.Cu, net +22V_ISO
- added copper zone on F.Cu, net +24V_ISO
- added copper zone on F.Cu, net +5VA_ISO
- added copper zone on F.Cu, net +5VD_ISO
- added copper zone on F.Cu, net +6V5_ISO
- added copper zone on F.Cu, net -22V_ISO
- added copper zone on F.Cu, net -24V_ISO
- added copper zone on F.Cu, net Net-(J4-Pin_2)
Other:
- outline, holes or cut-outs redrawn
- copper layers 6 -> 4
- board text added: "${PROJECTNAME} ${REVISION}"
- board text removed: "4"
- board text removed: "5"
