File: HARDWARE/ETH1CVOLT/ETH1CVOLT.kicad_pcb (KiCad board)
At the start: 4 copper layers, 160 x 100 mm, 277 parts, among them J1 20021111-00010T4LF, J2 7499010121A, J4 1827868, J5 FCR7350R, J6 FCR7350B, J7 TSW-102-23-G-S, J8 TSW-102-23-G-S, K1 G6SK-2F DC5, Q1 CSD18501Q5A, Q2 2N7002, Q3 2N7002, U1 STM32H743VITx, U10 MAX44241AUA+, U11 ISO7761FDBQ, U12 ISO7760DBQ, U13 ADA4522-1ARZ, U14 ADA4522-1ARZ, U15 RP-2424D, U16 TMR4-2423WI, U17 TEC2-2419WI, U18 TSR0.5-2465, U19 TPS7A3901DSCR, U2 24LC08B-E/MS, U20 TPS7A3901DSCR, U21 ADP7142ARDZ-5.0, U22 ADP7142ARDZ-5.0, U23 TPS7A3901DSCR, U24 TSR0.5-2433, U25 ADA4522-2ARZ-RL, U26 74LV1T08GV, U27 74LV1T08GV, U3 LAN8742A, U4 INA159AIDGKT, U5 DG412CUE+, U6 LTC2400CS8#TRPBF, U7 ADR4550CRZ, U8 ADA4522-1ARZ, U9 MAX5719GSD+, Y1 NX5032GA-16, Y2 NX5032GA-25

Commit message: Verification
Parts:
- added C29: 10u/35V/X7R, Capacitor_SMD:C_1206_3216Metric_Pad1.33x1.80mm_HandSolder, F.Cu at (156.3, 60.6)
- added R62: 100/1%/100mW, Resistor_SMD:R_0603_1608Metric_Pad0.98x0.95mm_HandSolder, F.Cu at (172.9, 55.2)
- added TP42: TestPoint, TestPoint:TestPoint_Pad_D1.5mm, F.Cu at (125.6, 98.6)
- added TP43: TestPoint, TestPoint:TestPoint_Pad_D1.5mm, F.Cu at (145.2, 98.8)
- C100: renamed from C101; value 10u/50V/X7R -> 10u/35V/X7R
- C101: renamed from C98; value 10u/50V/X7R -> 10u/35V/X7R
- C102: renamed from C99; value 10u/50V/X7R -> 10u/35V/X7R
- C103: renamed from C102; value 10u/50V/X7R -> 10u/35V/X7R
- C106: renamed from C105; value 10u/50V/X7R -> 10u/35V/X7R
- C34: renamed from C33; value 10u/50V/X7R -> 10u/35V/X7R
- C39: renamed from C38; value 10u/50V/X7R -> 10u/35V/X7R
- C56: renamed from C55; value 10u/50V/X7R -> 10u/35V/X7R
- C58: renamed from C57; value 10u/50V/X7R -> 10u/35V/X7R
- C59: renamed from C58; value 10u/50V/X7R -> 10u/35V/X7R
- C60: renamed from C59; value 10u/50V/X7R -> 10u/35V/X7R
- C61: renamed from C60; value 10u/50V/X7R -> 10u/35V/X7R
- C67: renamed from C66; value 10u/50V/X7R -> 10u/35V/X7R
- C68: renamed from C67; value 10u/50V/X7R -> 10u/35V/X7R
- C69: renamed from C68; value 10u/50V/X7R -> 10u/35V/X7R
- C70: renamed from C69; value 10u/50V/X7R -> 10u/35V/X7R
- C71: renamed from C70; value 10u/50V/X7R -> 10u/35V/X7R
- C82: renamed from C81; value 10u/50V/X7R -> 10u/35V/X7R
- C83: renamed from C82; value 10u/50V/X7R -> 10u/35V/X7R
- C87: renamed from C86; value 10u/50V/X7R -> 10u/35V/X7R
- C88: renamed from C87; value 10u/50V/X7R -> 10u/35V/X7R
- C97: renamed from C96; value 10u/50V/X7R -> 10u/35V/X7R
- C98: renamed from C97; value 10u/50V/X7R -> 10u/35V/X7R
- C99: renamed from C100; value 10u/50V/X7R -> 10u/35V/X7R
- R49: value R -> 10k/1%/100mW
- R53: value 0R/5%/100mW -> 560/1%/100mW
- U10: value MAX44241AUA+ -> ADA4522-1ARZ; footprint Package_SO:VSSOP-8_3x3mm_P0.65mm -> Package_SO:SOIC-8_3.9x4.9mm_P1.27mm
- moved R24 1.65 mm to (164.3, 70.9)
- moved R20 1.65 mm to (164.3, 72.5)
- moved R27 1.60 mm to (161.3, 71.7)
- moved TP6 1.50 mm to (167.2, 73.0)
- moved U10 0.89 mm to (164.3, 67.4)
- moved TP24 0.80 mm to (129.6, 126.4)
- moved C71 0.70 mm to (123.1, 102.6)
- moved C76 0.70 mm to (123.1, 97.2)
- moved C31 0.40 mm to (175.4, 58.0)
- moved C54 0.10 mm to (177.0, 71.4)
- renumbered C103 to C104, C104 to C105, C106 to C107, C107 to C108, C108 to C109, C109 to C110, C29 to C30, C30 to C31, C31 to C32, C32 to C33, C34 to C35, C35 to C36, C36 to C37, C37 to C38, C39 to C40, C40 to C41, C41 to C42, C42 to C43, C43 to C44, C44 to C45, C45 to C46, C46 to C47, C47 to C48, C48 to C49, C49 to C50, C50 to C51, C51 to C52, C52 to C53, C53 to C54, C54 to C55, C56 to C57, C61 to C62, C62 to C63, C63 to C64, C64 to C65, C65 to C66, C71 to C72, C72 to C73, C73 to C74, C74 to C75, C75 to C76, C76 to C77, C77 to C78, C78 to C79, C79 to C80, C80 to C81, C83 to C84, C84 to C85, C85 to C86, C88 to C89, C89 to C90, C90 to C91, C91 to C92, C92 to C93, C93 to C94, C94 to C95, C95 to C96, J8 to J3, J7 to J4, J4 to J6, J5 to J7, J6 to J8, U23 to U21, U21 to U22, U22 to U23
Connections:
- R14 pad 1: Net-(U4-OUT) -> Net-(R14-Pad1)
- U5 pad 2: Net-(U4-OUT) -> Net-(R14-Pad1)
Routing:
- net Net-(U4-OUT): track 26.3 -> 14.4 mm
- net Net-(R14-Pad1): track 0.00 -> 10.5 mm
- net /BLOCK DIAGRAM/DAC/DAC_SIG: track 19.1 -> 16.0 mm
- net +5VD_ISO: track 32.0 -> 34.3 mm
- net +7V_ISO: track 62.7 -> 61.4 mm
- net Net-(U10--): track 7.01 -> 8.18 mm
- net Net-(U10-V+): track 8.03 -> 9.00 mm
- net -22V_ISO: track 196.9 -> 196.0 mm
- net +3.3V: track 37.2 -> 38.0 mm, vias 27 -> 26
- net Net-(U10-+): track 13.3 -> 13.9 mm
- net GND: vias 99 -> 102
Other:
- board text added: "${PROJECTNAME} ${REVISION} 01"
- board text removed: "${PROJECTNAME} ${REVISION}"

Commit message: Verfication
Parts:
- moved FID1 31.5 mm to (104.5, 135.2)
- moved FID2 31.5 mm to (104.5, 135.2)
Routing:
- net GND: vias 102 -> 101
Changed lines of the file:
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@@
 	(footprint "Fiducial:Fiducial_1.5mm_Mask3mm"
 		(layer "F.Cu")
-		(at 73 134)
+		(at 104.5 135.2)
 		(descr "Fiducial, circular marking, 1.5mm bare copper, 3mm soldermask opening")
 		(tags "fiducial")
@@
 	(footprint "Fiducial:Fiducial_1.5mm_Mask3mm"
 		(layer "B.Cu")
-		(at 73 134 180)
+		(at 104.5 135.2 180)
 		(descr "Fiducial, circular marking, 1.5mm bare copper, 3mm soldermask opening")
 		(tags "fiducial")
@@
 	)
 	(gr_line
+		(start 72.95 108.95)
+		(end 75.05 108.95)
+		(stroke
+			(width 0.5)
+			(type default)
+		)
+		(layer "F.SilkS")
+	)
+	(gr_line
+		(start 74 107.9)
+		(end 74 110)
+		(stroke
+			(width 0.5)
+			(type default)
+		)
+		(layer "F.SilkS")
+	)
+	(gr_line
+		(start 74.1 130.95)
+		(end 74.1 133.05)
+		(stroke
+			(width 0.5)
+			(type default)
+		)
+		(layer "F.SilkS")
+	)
+	(gr_line
 		(start 160.4 62.2)
 		(end 160.7 62)
@@
 	)
 	(via
-		(at 95.8 60.4)
-		(size 0.65)
-		(drill 0.25)
-		(layers "F.Cu" "B.Cu")
-		(free yes)
-		(net "GND")
-	)
-	(via
 		(at 83.8 104.85)
 		(size 0.65)
@@
 	)
 	(via
-		(at 122.5 82.4)
+		(at 125.75 82.4)
 		(size 0.65)
 		(drill 0.25)
@@
 	)
 	(via
-		(at 125.75 82.4)
+		(at 122.2 86.5)
 		(size 0.65)
 		(drill 0.25)
 		(layers "F.Cu" "B.Cu")
 		(free yes)
-		(teardrops
-			(best_length_ratio 0.5)
-			(max_length 1)
-			(best_width_ratio 1)
-			(max_width 2)
-			(curved_edges no)
-			(filter_ratio 0.9)
-			(enabled yes)
-			(allow_two_segments yes)
-			(prefer_zone_connections yes)
-		)
 		(net "+5VD_ISO")
 	)
@@
 			(thermal_bridge_width 0.3)
 			(smoothing chamfer)
-			(radius 0.4)
+			(radius 0.2)
 			(island_removal_mode 0)
 		)
 		(polygon
 			(pts
-				(xy 127.1 90.4) (xy 127.1 81.9) (xy 121.6 81.9) (xy 121.6 88.45) (xy 124.75 88.45) (xy 124.75 90.4)
+				(xy 127.1 90.4) (xy 124.75 90.4) (xy 124.75 88.45) (xy 121.6 88.45) (xy 121.6 83.8) (xy 123.5 81.9)
+				(xy 127.1 81.9)
 			)
 		)
@@
 	)
 	(zone
+		(net "/BLOCK DIAGRAM/MCU/NRST")
+		(layer "F.Cu")
+		(hatch none 0.1)
+		(priority 30053)
+		(attr
+			(teardrop
+				(type padvia)
+			)
+		)
+		(connect_pads yes
+			(clearance 0)
+		)
+		(min_thickness 0.0254)
+		(fill yes
+			(island_removal_mode 1)
+		)
+		(polygon
+			(pts
+				(xy 102.75 56.501193) (xy 102.95 56.501193) (xy 103.1 56.136564) (xy 102.85 55.850193) (xy 102.6 55.862703)
+			)
+		)
+	)
+	(zone
 		(layer "F.Cu")
 		(hatch edge 0.5)
@@
 		(polygon
 			(pts
-				(xy 79.8 55.8) (xy 79.8 65.1) (xy 94.2 65.1) (xy 94.2 59.9) (xy 100.3 59.9) (xy 100.3 55.8)
+				(xy 79.8 55.8) (xy 79.8 65.1) (xy 94.2 65.1) (xy 94.2 60.1) (xy 100.3 60.1) (xy 100.3 55.8)
 			)
 		)
