File: HARDWARE/ETH1CVOLT/ETH1CVOLT.kicad_pcb (KiCad board)
At the start: 4 copper layers, 160 x 100 mm, 281 parts, among them J1 20021111-00010T4LF, J2 7499010121A, J3 TSW-102-23-G-S, J4 TSW-102-23-G-S, J6 1827868, J7 FCR7350R, J8 FCR7350B, K1 G6SK-2F DC5, Q1 CSD18501Q5A, Q2 2N7002, Q3 2N7002, U1 STM32H743VITx, U10 ADA4522-1ARZ, U11 ISO7761FDBQ, U12 ISO7760DBQ, U13 ADA4522-1ARZ, U14 ADA4522-1ARZ, U15 RP-2424D, U16 TMR4-2423WI, U17 TEC2-2419WI, U18 TSR0.5-2465, U19 TPS7A3901DSCR, U2 24LC08B-E/MS, U20 TPS7A3901DSCR, U21 TPS7A3901DSCR, U22 ADP7142ARDZ-5.0, U23 ADP7142ARDZ-5.0, U24 TSR0.5-2433, U25 ADA4522-2ARZ-RL, U26 74LV1T08GV, U27 74LV1T08GV, U3 LAN8742A, U4 INA159AIDGKT, U5 DG412CUE+, U6 LTC2400CS8#TRPBF, U7 ADR4550CRZ, U8 ADA4522-1ARZ, U9 MAX5719GSD+, Y1 NX5032GA-16, Y2 NX5032GA-25

Commit message: Modifications
Parts:
- added C111: 0.1u/100V/X7R, Capacitor_SMD:C_0603_1608Metric_Pad1.08x0.95mm_HandSolder, F.Cu at (185.4, 86.5)
- added D11: APFA3010LSEEZGKQBKC, LED_SMD:LED_Kingbright_APFA3010_3x1.5mm_Horizontal, F.Cu at (227.0, 119.1)
- added R63: 4k7/1%/100mW, Resistor_SMD:R_0603_1608Metric_Pad0.98x0.95mm_HandSolder, F.Cu at (151.3, 60.9)
- added R64: 1k/1%/100mW, Resistor_SMD:R_0603_1608Metric_Pad0.98x0.95mm_HandSolder, F.Cu at (183.7, 84.7)
- added R65: 1k/1%/100mW, Resistor_SMD:R_0603_1608Metric_Pad0.98x0.95mm_HandSolder, F.Cu at (183.7, 83.1)
- added R66: 560/1%/100mW, Resistor_SMD:R_0603_1608Metric_Pad0.98x0.95mm_HandSolder, F.Cu at (224.0, 120.6)
- added U28: 74LVC2G74DP, Package_SO:TSSOP-8_3x3mm_P0.65mm, F.Cu at (188.4, 83.9)
- D6: value SML-A12UTT86 -> APFA3010LSEEZGKQBKC; footprint LED_SMD:LED_0603_1608Metric_Pad1.05x0.95mm_HandSolder -> LED_SMD:LED_Kingbright_APFA3010_3x1.5mm_Horizontal
- U11: value ISO7761FDBQ -> ISO7761DBQR
- moved FID5 7.00 mm to (226.0, 130.0)
- moved FID6 7.00 mm to (226.0, 130.0)
- moved D6 0.71 mm to (73.8, 96.9)
- moved Y2 0.50 mm to (103.1, 67.5)
- moved R55 0.20 mm to (191.6, 78.2)
- moved U24 0.06 mm to (104.4, 76.4)
Connections:
- net /BLOCK DIAGRAM/MCU/I2C1_SCL renamed /BLOCK DIAGRAM/MCU/I2C3_SCL
- net /BLOCK DIAGRAM/MCU/I2C1_SDA renamed /BLOCK DIAGRAM/MCU/I2C3_SDA
Routing:
- net Net-(D11-R): track 0.00 -> 77.6 mm
- net Net-(D11-B): track 0.00 -> 67.5 mm
- net +5VD_ISO: track 34.3 -> 100.6 mm, vias 13 -> 15
- net Net-(U27-Y): track 2.15 -> 39.7 mm, vias 0 -> 2
- net GND: track 1.49 -> 27.2 mm, vias 101 -> 123
- net Net-(U26-Y): track 2.92 -> 15.3 mm
- net Net-(D11-A): track 0.00 -> 2.09 mm
- net /BLOCK DIAGRAM/OUTPUT/STAT_RESET: track 0.00 -> 1.93 mm
- net /BLOCK DIAGRAM/OUTPUT/STAT_SET: track 0.00 -> 1.75 mm
- net /BLOCK DIAGRAM/DAC/DAC_~{LDAC}: track 15.9 -> 17.2 mm
- net -14V_ISO: track 183.0 -> 182.1 mm
- net -7V_ISO: track 53.6 -> 52.9 mm
- net Net-(U25B--): track 7.30 -> 6.78 mm
- net /BLOCK DIAGRAM/OUTPUT/MEAS_R10V: track 21.5 -> 21.0 mm
- net GND_ISO: vias 190 -> 225

Commit message: HW design done
Parts:
- added R67: 1k/1%/100mW, Resistor_SMD:R_0603_1608Metric_Pad0.98x0.95mm_HandSolder, F.Cu at (172.1, 59.3)
- added R68: 4k7/1%/100mW, Resistor_SMD:R_0603_1608Metric_Pad0.98x0.95mm_HandSolder, B.Cu at (127.9, 55.8)
- added R69: 4k7/1%/100mW, Resistor_SMD:R_0603_1608Metric_Pad0.98x0.95mm_HandSolder, B.Cu at (127.9, 57.5)
- added R70: 4k7/1%/100mW, Resistor_SMD:R_0603_1608Metric_Pad0.98x0.95mm_HandSolder, B.Cu at (127.9, 59.2)
- added R71: 4k7/1%/100mW, Resistor_SMD:R_0603_1608Metric_Pad0.98x0.95mm_HandSolder, B.Cu at (127.9, 52.4)
- added R72: 4k7/1%/100mW, Resistor_SMD:R_0603_1608Metric_Pad0.98x0.95mm_HandSolder, B.Cu at (127.9, 54.1)
- added R73: 4k7/1%/100mW, Resistor_SMD:R_0603_1608Metric_Pad0.98x0.95mm_HandSolder, B.Cu at (132.3, 62.6)
- added R74: 4k7/1%/100mW, Resistor_SMD:R_0603_1608Metric_Pad0.98x0.95mm_HandSolder, B.Cu at (138.1, 65.5)
- added R75: 4k7/1%/100mW, Resistor_SMD:R_0603_1608Metric_Pad0.98x0.95mm_HandSolder, B.Cu at (134.9, 62.6)
- R50: value R -> 10k/1%/100mW
- R54: value 0R/5%/100mW -> 560/1%/100mW
Connections:
- U5 pad 6: +5VREF_ISO -> Net-(R67-Pad1)
Routing:
- net +3.3V: track 38.0 -> 46.0 mm
- net +5VREF_ISO: track 61.1 -> 68.7 mm
- net /BLOCK DIAGRAM/ISO DIG/MCU_REL_RESET: track 6.31 -> 13.1 mm, vias 0 -> 1
- net /BLOCK DIAGRAM/ISO DIG/MCU_ADC_SW1: track 6.35 -> 10.7 mm, vias 0 -> 1
- net /BLOCK DIAGRAM/ISO DIG/MCU_REL_SET: track 6.37 -> 10.4 mm, vias 0 -> 1
- net /BLOCK DIAGRAM/ISO DIG/MCU_ADC_SW2: track 6.20 -> 10.1 mm, vias 0 -> 1
- net GND: track 27.2 -> 30.9 mm
- net /BLOCK DIAGRAM/ISO DIG/MCU_ADC_SW3: track 6.26 -> 9.89 mm, vias 0 -> 1
- net /BLOCK DIAGRAM/ISO DIG/MCU_DAC_~{LDAC}: track 6.74 -> 10.3 mm, vias 0 -> 1
- net Net-(R67-Pad1): track 0.00 -> 3.34 mm
- net /BLOCK DIAGRAM/ISO DIG/MCU_DAC_~{CS}: track 6.44 -> 7.85 mm, vias 0 -> 1
- net /BLOCK DIAGRAM/MCU/NRST: track 55.6 -> 56.8 mm
- net -14V_ISO: track 182.1 -> 182.6 mm
- net GND_ISO: vias 225 -> 224
Other:
- outline, holes or cut-outs redrawn
- board text added: "${PROJECTNAME}01"
- board text removed: "${PROJECTNAME} ${REVISION} 01"
