File: HARDWARE/ETH1CVOLT/Voltage_Reference.kicad_sch (KiCad schematic)
At the start: 33 parts, among them J4 Conn_01x02, J5 Conn_01x02, U14 ADR1399KEZ, U25 OPA2196xD

Commit message: Development
Parts:
- removed C52: 1u/50V/X7R, Capacitor_SMD:C_0603_1608Metric, symbol Device:C
- removed R41: 5R1/5%/100mW, Resistor_SMD:R_0603_1608Metric, symbol Device:R
- added C36, C37: 0.1u/100V/X7R, Capacitor_SMD:C_0603_1608Metric_Pad1.08x0.95mm_HandSolder, symbol Device:C
- added R22: 100/1%/100mW, Resistor_SMD:R_0603_1608Metric_Pad0.98x0.95mm_HandSolder, symbol Device:R
- C38: renamed from C35; value 10u/35V/X7R -> 10u/50V/X7R; footprint Capacitor_SMD:C_0805_2012Metric_Pad1.18x1.45mm_HandSolder -> Capacitor_SMD:C_1210_3225Metric_Pad1.33x2.70mm_HandSolder
- C39: renamed from C40; value 4u7/35V/X7R -> 4u7/50V/X7R; footprint Capacitor_SMD:C_0805_2012Metric_Pad1.18x1.45mm_HandSolder -> Capacitor_SMD:C_1210_3225Metric_Pad1.33x2.70mm_HandSolder
- C40: renamed from C53; footprint Capacitor_SMD:C_0603_1608Metric -> Capacitor_SMD:C_0603_1608Metric_Pad1.08x0.95mm_HandSolder
- J3: renamed from J4; value Conn_01x02 -> TSW-102-23-G-S; footprint Package_TO_SOT_SMD:SOT-23 -> Connector_PinHeader_2.54mm:PinHeader_1x02_P2.54mm_Vertical
- J4: renamed from J5; value Conn_01x02 -> TSW-102-23-G-S; footprint Package_TO_SOT_SMD:SOT-23 -> Connector_PinHeader_2.54mm:PinHeader_1x02_P2.54mm_Vertical
- R19: renamed from R38; value 0 -> 0R/5%/100mW; footprint Resistor_SMD:R_0603_1608Metric -> Resistor_SMD:R_0603_1608Metric_Pad0.98x0.95mm_HandSolder
- R20: renamed from R39; value 0 -> 0R/5%/100mW; footprint Resistor_SMD:R_0603_1608Metric -> Resistor_SMD:R_0603_1608Metric_Pad0.98x0.95mm_HandSolder
- R21: renamed from R40; footprint Resistor_SMD:R_0805_2012Metric -> Resistor_SMD:R_0805_2012Metric_Pad1.20x1.40mm_HandSolder
- R23: renamed from R42; footprint Resistor_SMD:R_0603_1608Metric -> Resistor_SMD:R_0603_1608Metric_Pad0.98x0.95mm_HandSolder
- R24: renamed from R43; value 20k/0.01%/100mW -> 20k/0.1%/100mW; footprint Resistor_SMD:R_0603_1608Metric -> Resistor_SMD:R_0603_1608Metric_Pad0.98x0.95mm_HandSolder
- R25: renamed from R44; footprint Resistor_SMD:R_0603_1608Metric -> Resistor_SMD:R_0603_1608Metric_Pad0.98x0.95mm_HandSolder
- R26: renamed from R53; footprint Resistor_SMD:R_0603_1608Metric -> Resistor_SMD:R_0603_1608Metric_Pad0.98x0.95mm_HandSolder; now left out of the parts list
- R27: renamed from R45; footprint Resistor_SMD:R_0603_1608Metric -> Resistor_SMD:R_0603_1608Metric_Pad0.98x0.95mm_HandSolder
- R28: renamed from R54; footprint Resistor_SMD:R_0603_1608Metric -> Resistor_SMD:R_0603_1608Metric_Pad0.98x0.95mm_HandSolder; now left out of the parts list
- R29: renamed from R50; footprint Resistor_SMD:R_0603_1608Metric -> Resistor_SMD:R_0603_1608Metric_Pad0.98x0.95mm_HandSolder
- R30: renamed from R55; footprint Resistor_SMD:R_0603_1608Metric -> Resistor_SMD:R_0603_1608Metric_Pad0.98x0.95mm_HandSolder; now left out of the parts list
- R31: renamed from R51; footprint Resistor_SMD:R_0603_1608Metric -> Resistor_SMD:R_0603_1608Metric_Pad0.98x0.95mm_HandSolder
- R32: renamed from R52; value 198k/0.05%/100mW -> 198k/0.1%/100mW; footprint Resistor_SMD:R_0603_1608Metric -> Resistor_SMD:R_0603_1608Metric_Pad0.98x0.95mm_HandSolder
- R33: renamed from R49; footprint Resistor_SMD:R_0603_1608Metric -> Resistor_SMD:R_0603_1608Metric_Pad0.98x0.95mm_HandSolder
- TP3: now left out of the parts list
- TP4: renamed from TP2; now left out of the parts list
- TP5: renamed from TP6; now left out of the parts list
- TP6: renamed from TP4; now left out of the parts list
- renumbered JP8 to JP2, JP9 to JP3, JP10 to JP4, JP11 to JP5, JP12 to JP6, JP13 to JP7, U25 to U7, U14 to U8
Connections:
- net GND_ISO: now also C36.2, C37.2
- net -14V_ISO: now reaches U7.4 (V-)
- net -14V_ISO: now also C37.1
- net +14V_ISO: now reaches U7.8 (V+)
- net +14V_ISO: now also C36.1
- net at R21.2, TP3.1, U8.6 (+REFF)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: now also R22.2; no longer C38.1, C39.1, U7.3 (+)
- net +15V_ISO: now reaches R21.1, U8.3 (HEATER+)
- net -15V_ISO: now reaches R20.1
- new net: C38.1, C39.1, R22.1, U7.3 (+)
Other:
- moved on the sheet: R19, R20, R21, TP3, U8

Commit message: Development
Parts:
- JP2, JP3, JP4, JP5, JP6, JP7: footprint Package_SO:SOIC-8_3.9x4.9mm_P1.27mm -> Jumper:SolderJumper-2_P1.3mm_Open_Pad1.0x1.5mm
Changed lines of the file:
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@@
 			)
 		)
-		(property "Footprint" "Package_SO:SOIC-8_3.9x4.9mm_P1.27mm"
+		(property "Footprint" "Jumper:SolderJumper-2_P1.3mm_Open_Pad1.0x1.5mm"
 			(at 191.77 116.84 0)
 			(hide yes)
@@
 			)
 		)
-		(property "Footprint" "Package_SO:SOIC-8_3.9x4.9mm_P1.27mm"
+		(property "Footprint" "Jumper:SolderJumper-2_P1.3mm_Open_Pad1.0x1.5mm"
 			(at 167.64 116.84 0)
 			(hide yes)
@@
 			)
 		)
-		(property "Footprint" "Package_SO:SOIC-8_3.9x4.9mm_P1.27mm"
+		(property "Footprint" "Jumper:SolderJumper-2_P1.3mm_Open_Pad1.0x1.5mm"
 			(at 264.16 116.84 0)
 			(hide yes)
@@
 			)
 		)
-		(property "Footprint" "Package_SO:SOIC-8_3.9x4.9mm_P1.27mm"
+		(property "Footprint" "Jumper:SolderJumper-2_P1.3mm_Open_Pad1.0x1.5mm"
 			(at 217.17 116.84 0)
 			(hide yes)
@@
 			)
 		)
-		(property "Footprint" "Package_SO:SOIC-8_3.9x4.9mm_P1.27mm"
+		(property "Footprint" "Jumper:SolderJumper-2_P1.3mm_Open_Pad1.0x1.5mm"
 			(at 241.3 116.84 0)
 			(hide yes)
@@
 			)
 		)
-		(property "Footprint" "Package_SO:SOIC-8_3.9x4.9mm_P1.27mm"
+		(property "Footprint" "Jumper:SolderJumper-2_P1.3mm_Open_Pad1.0x1.5mm"
 			(at 288.29 116.84 0)
 			(hide yes)

Commit message: Development
Parts:
- removed R28, R30: OPT, Resistor_SMD:R_0603_1608Metric_Pad0.98x0.95mm_HandSolder, symbol Device:R
- added JP8, JP9: SolderJumper_2_Open, Jumper:SolderJumper-2_P1.3mm_Open_Pad1.0x1.5mm, symbol Jumper:SolderJumper_2_Open
- added R31: 49k9/0.1%/100mW, Resistor_SMD:R_0603_1608Metric_Pad0.98x0.95mm_HandSolder, symbol Device:R
- added R33: 1Meg/0.1%/100mW, Resistor_SMD:R_0603_1608Metric_Pad0.98x0.95mm_HandSolder, symbol Device:R
- added RV1: M64Y501KB40, Potentiometer_THT:Potentiometer_Bourns_3386X_Horizontal, symbol Device:R_Potentiometer_Trim
- R19: now not fitted
- R23: value 8k2/0.1%/100mW -> 7k15/0.1%/100mW
- R25: value 9k65/0.1%/100mW -> 7k5/0.1%/100mW
- R26: value OPT -> 0R/5%/100mW; now in the parts list
- R27: value 40k2/0.1%/100mW -> 8k25/0.1%/100mW
- R28: renamed from R29; value 68k/0.1%/100mW -> 8k66/0.1%/100mW
- R29: renamed from R31; value 110k/0.1%/100mW -> 9k09/0.1%/100mW
- R30: renamed from R32; value 198k/0.1%/100mW -> 9k31/0.1%/100mW
- renumbered R33 to R32, TP3 to TP5, TP4 to TP6, TP5 to TP7, TP6 to TP8
Connections:
- net GND_ISO: no longer R26.2
- net at J3.1 (Pin_1), JP2.2 (B), JP3.2 (B)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: now also JP8.2 (B), JP9.2 (B)
- net at R23.2, R25.2, R26.1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: now also R31.2, R33.2, RV1.1, RV1.2; no longer C40.1, J4.1 (Pin_1), R24.1, TP7.1, U7.5 (+)
- new net: JP8.1 (A), R31.1
- new net: C40.1, J4.1 (Pin_1), R24.1, R26.2, RV1.3, TP7.1, U7.5 (+)
- new net: JP9.1 (A), R33.1
Other:
- moved on the sheet: C38, C39, C40, J3, J4, JP2, JP3, JP4, JP5, JP6, JP7, R20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

Commit message: Development
Parts:
- added R25: 10k/0.01%/100mW, Resistor_SMD:R_0603_1608Metric_Pad0.98x0.95mm_HandSolder, symbol Device:R
- C38, C39: footprint Capacitor_SMD:C_1210_3225Metric_Pad1.33x2.70mm_HandSolder -> Capacitor_SMD:C_1206_3216Metric_Pad1.33x1.80mm_HandSolder
- C40: value 100p/100V/X7R -> 0.1u/100V/X7R
- R24: value 20k/0.1%/100mW -> 10k/0.01%/100mW
- U7: value OPA2196xD -> OPA2192ID
- renumbered R25 to R26, R26 to R27, R27 to R28, R28 to R29, R29 to R30, R30 to R31, R31 to R32, R32 to R33, R33 to R34
Connections:
- net GND_ISO: now also R25.2; no longer R24.2
- new net: R24.2, R25.1
Other:
- moved on the sheet: R33, TP8

Commit message: Layout
Parts:
- added C36: 10u/50V/X7R, Capacitor_SMD:C_1206_3216Metric_Pad1.33x1.80mm_HandSolder, symbol Device:C
- renumbered C36 to C34, C37 to C35, C38 to C37, C39 to C38, C40 to C39, R19 to R18, R20 to R19, R21 to R20, R22 to R21, R23 to R22, R24 to R23, R25 to R24, R26 to R25, R27 to R26, R28 to R27, R29 to R28, R30 to R29, R31 to R30, R32 to R31, R33 to R32, R34 to R33
Connections:
- net GNDA is gone; now on net GND_ISO: U8.1 (-REFS), U8.2 (-REFF)
- net +15V_ISO: now also C36.1
- net GND_ISO: now also C36.2

Commit message: Layout and schematic
Parts:
- removed C39: 0.1u/100V/X7R, Capacitor_SMD:C_0603_1608Metric_Pad1.08x0.95mm_HandSolder, symbol Device:C
- removed J3, J4: TSW-102-23-G-S, Connector_PinHeader_2.54mm:PinHeader_1x02_P2.54mm_Vertical, symbol Connector_Generic:Conn_01x02
- removed JP2, JP3, JP4, JP5, JP6, JP7, JP8, JP9: SolderJumper_2_Open, Jumper:SolderJumper-2_P1.3mm_Open_Pad1.0x1.5mm, symbol Jumper:SolderJumper_2_Open
- removed R20: 2k67/1%/250mW, Resistor_SMD:R_0805_2012Metric_Pad1.20x1.40mm_HandSolder, symbol Device:R
- removed R21, R32: 100/1%/100mW, Resistor_SMD:R_0603_1608Metric_Pad0.98x0.95mm_HandSolder, symbol Device:R
- removed R22: 7k15/0.1%/100mW, Resistor_SMD:R_0603_1608Metric_Pad0.98x0.95mm_HandSolder, symbol Device:R
- removed R23, R24: 10k/0.01%/100mW, Resistor_SMD:R_0603_1608Metric_Pad0.98x0.95mm_HandSolder, symbol Device:R
- removed R25: 7k5/0.1%/100mW, Resistor_SMD:R_0603_1608Metric_Pad0.98x0.95mm_HandSolder, symbol Device:R
- removed R26: 0R/5%/100mW, Resistor_SMD:R_0603_1608Metric_Pad0.98x0.95mm_HandSolder, symbol Device:R
- removed R27: 8k25/0.1%/100mW, Resistor_SMD:R_0603_1608Metric_Pad0.98x0.95mm_HandSolder, symbol Device:R
- removed R28: 8k66/0.1%/100mW, Resistor_SMD:R_0603_1608Metric_Pad0.98x0.95mm_HandSolder, symbol Device:R
- removed R29: 9k09/0.1%/100mW, Resistor_SMD:R_0603_1608Metric_Pad0.98x0.95mm_HandSolder, symbol Device:R
- removed R30: 9k31/0.1%/100mW, Resistor_SMD:R_0603_1608Metric_Pad0.98x0.95mm_HandSolder, symbol Device:R
- removed R31: 49k9/0.1%/100mW, Resistor_SMD:R_0603_1608Metric_Pad0.98x0.95mm_HandSolder, symbol Device:R
- removed R33: 1Meg/0.1%/100mW, Resistor_SMD:R_0603_1608Metric_Pad0.98x0.95mm_HandSolder, symbol Device:R
- removed RV1: M64Y501KB40, Potentiometer_THT:Potentiometer_Bourns_3386X_Horizontal, symbol Device:R_Potentiometer_Trim
- removed TP6, TP7, TP8: TestPoint, TestPoint:TestPoint_Pad_D1.5mm, symbol Connector:TestPoint
- removed U7: OPA2192ID, Package_SO:SOIC-8_3.9x4.9mm_P1.27mm, symbol Amplifier_Operational:OPA2196xD
- removed U8: ADR1399KEZ, Package_LCC:Analog_LCC-8_5x5mm_P1.27mm, symbol Reference_Voltage:ADR1399KEZ
- added C35, C41: 0.1u/100V/X7R, Capacitor_SMD:C_0603_1608Metric_Pad1.08x0.95mm_HandSolder, symbol Device:C
- added C40, C42: 1u/16V/X7R, Capacitor_SMD:C_0603_1608Metric_Pad1.08x0.95mm_HandSolder, symbol Device:C
- added U7: ADR4550, Package_SO:SOIC-8_3.9x4.9mm_P1.27mm, symbol Reference_Voltage:ADR4550
- added U8: ADA4522-1ARZ, Package_SO:SOIC-8_3.9x4.9mm_P1.27mm, symbol Amplifier_Operational:ADA4522-1
- C36: value 10u/50V/X7R -> 0.1u/100V/X7R; footprint Capacitor_SMD:C_1206_3216Metric_Pad1.33x1.80mm_HandSolder -> Capacitor_SMD:C_0603_1608Metric_Pad1.08x0.95mm_HandSolder
- C37: value 10u/50V/X7R -> 1u/16V/X7R; footprint Capacitor_SMD:C_1206_3216Metric_Pad1.33x1.80mm_HandSolder -> Capacitor_SMD:C_0603_1608Metric_Pad1.08x0.95mm_HandSolder
- C38: value 4u7/50V/X7R -> 10u/50V/X7R
- R19: value 0R/5%/100mW -> 100/1%/100mW
- renumbered C35 to C39
Connections:
- net +15V_ISO is gone; now on net +14V_ISO: C36.1
- net -15V_ISO is gone; now on net +5VREF_ISO: R19.1
- net +14V_ISO: now also C37.1, C38.1, U7.2 (IN), U8.7 (V+)
- net +5VREF_ISO: now also TP5.1, C41.1, C42.1
- net -14V_ISO: now also C35.1, U8.4 (V-); no longer C39.1
- net GND_ISO: now also C35.2, C40.2, C41.2, C42.2, U7.4 (GND); no longer R18.1
- net at R18.2, R19.2: now also U8.2 (-), U8.6
- new net: C39.1, C40.1, R18.1, U7.6 (OUT), U8.3 (+)
Other:
- title: (none) -> ETH1CVOLT
- moved on the sheet: C39

Commit message: Layout
Parts:
- added J7, J8: TSW-102-23-G-S, Connector_PinHeader_2.54mm:PinHeader_1x02_P2.54mm_Vertical, symbol Connector_Generic:Conn_01x02
Connections:
- net +5VREF_ISO: now also J7.1 (Pin_1)
- net GND_ISO: now also J7.2 (Pin_2), J8.2 (Pin_2)
- net at C39.1, C40.1, R18.1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: now also J8.1 (Pin_1)
Other:
- moved on the sheet: C39, C40, U7

Commit message: Layout done
Parts:
- U7: value ADR4550 -> ADR4550CRZ
Other:
- note added: "Optional MAX6350"
Changed lines of the file:
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@@
 		(rev "01")
+	)
+	(text "Optional MAX6350"
+		(exclude_from_sim no)
+		(at 128.778 110.744 0)
+		(effects
+			(font
+				(size 1.27 1.27)
+			)
+		)
 	)
 	(junction
@@
 			)
 		)
-		(property "Value" "ADR4550"
+		(property "Value" "ADR4550CRZ"
 			(at 124.46 133.3499 0)
 			(show_name no)
