File: HARDWARE/ETH1CVOLT/Ethernet.kicad_sch (KiCad schematic)
At the start: 25 parts, among them J2 RJ45_Wuerth_7499010121A, U3 LAN8742A, Y2 NX5032GA-25

Commit message: Development
Parts:
- C17: renamed from C18; value 0.1u -> 0.1u/100V/X7R
- C18: renamed from C17; value 8p -> 8p/100V/X7R
- C19: renamed from C20; value 1u -> 1u/16V/X7R
- C20: renamed from C19; value 8p -> 8p/100V/X7R
- C21, C22: value 1u -> 1u/16V/X7R
- C23, C25, C26, C27, C28: value 0.1u -> 0.1u/100V/X7R
- C24: value 470p -> 470p/100V/X7R
- J2: value RJ45_Wuerth_7499010121A -> 7499010121A
- R10, R11: value 560 -> 560/1%/100mW
- R6, R8: value 10k -> 10k/1%/100mW
- R7: value 1k4 -> 1k4/1%/100mW
- R9: value 12k1 -> 12k1/1%/100mW
- RN1: value R_Pack04 -> EXB-V8V330JV; footprint (none) -> Resistor_SMD:R_Array_Convex_4x0603
- RN2: value R_Pack04 -> EXB-V8V103JV; footprint (none) -> Resistor_SMD:R_Array_Convex_4x0603
- RN3: value R_Pack04 -> EXB-38V510JV; footprint (none) -> Resistor_SMD:R_Array_Convex_4x0603
Other:
- moved on the sheet: C17, C18, C19, C20, C21, C22, C23, C24, C25, C26, C27, FB2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

Commit message: Development
Parts:
- Y2: footprint ETH1CVOLT_A:NX5032GA -> ETH1CVOLT:NX5032GA
Changed lines of the file:
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@@
 			)
 		)
-		(property "Footprint" "ETH1CVOLT_A:NX5032GA"
+		(property "Footprint" "ETH1CVOLT:NX5032GA"
 			(at 142.24 176.53 0)
 			(hide yes)

Commit message: Layout
Parts:
- renumbered C17 to C15, C18 to C16, C19 to C17, C20 to C18, C21 to C19, C22 to C20, C23 to C21, C24 to C22, C25 to C23, C26 to C24, C27 to C25, C28 to C26, R11 to R10, R6 to R5, R7 to R6, R8 to R7, R9 to R8, R10 to R9

Commit message: Layout and schematic
Other:
- title: (none) -> ETH1CVOLT
- moved on the sheet: R5, RN1
