File: HARDWARE/ETH1CVOLT/Range_10V.kicad_sch (KiCad schematic)
At the start: 5 parts, among them U20 OPA2196xD

Commit message: Development
Parts:
- removed U20: OPA2196xD, Package_SO:SOIC-8_3.9x4.9mm_P1.27mm, symbol Amplifier_Operational:OPA2196xD
- added C49, C50: 0.1u/100V/X7R, Capacitor_SMD:C_0603_1608Metric_Pad1.08x0.95mm_HandSolder, symbol Device:C
- added U13: OPA192IDR, Package_SO:SOIC-8_3.9x4.9mm_P1.27mm, symbol Amplifier_Operational:OPA196xD
- R42: renamed from R60; footprint Resistor_SMD:R_0603_1608Metric -> Resistor_SMD:R_0603_1608Metric_Pad0.98x0.95mm_HandSolder; now fitted
- R43: renamed from R61; footprint Resistor_SMD:R_0603_1608Metric -> Resistor_SMD:R_0603_1608Metric_Pad0.98x0.95mm_HandSolder; now fitted
- TP7: renamed from TP10; now left out of the parts list
- renumbered D7 to D3
Connections:
- net DAC_SIG: now also U13.3 (+)
- net GND_ISO: now also C49.2, C50.2
- net R10V_SIG: now also U13.6
- net -14V_ISO: now reaches D3.1 (K)
- net -14V_ISO: now also C50.1, U13.4 (V-)
- net +14V_ISO: now reaches D3.2 (A)
- net +14V_ISO: now also C49.1, U13.7 (V+)
- net at R42.2, R43.1: now also U13.2 (-)

Commit message: Development
Parts:
- renumbered TP7 to TP22
Connections:
- net R10V_SIG: now also R43.2, TP22.1
Other:
- moved on the sheet: R42
Changed lines of the file:
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@@
 	(text "+/- 10V"
 		(exclude_from_sim no)
-		(at 250.698 106.934 0)
+		(at 243.586 106.934 0)
 		(effects
 			(font
@@
 		(color 0 0 0 0)
 	)
+	(junction
+		(at 217.17 109.22)
+		(diameter 0)
+		(color 0 0 0 0)
+	)
 	(wire
 		(pts
@@
 	(wire
 		(pts
+			(xy 217.17 109.22) (xy 264.16 109.22)
+		)
+		(stroke
+			(width 0)
+			(type default)
+		)
+	)
+	(wire
+		(pts
 			(xy 217.17 134.62) (xy 208.28 134.62)
 		)
@@
 	(wire
 		(pts
+			(xy 217.17 109.22) (xy 217.17 134.62)
+		)
+		(stroke
+			(width 0)
+			(type default)
+		)
+	)
+	(wire
+		(pts
 			(xy 22.86 273.05) (xy 22.86 274.32)
 		)
@@
 	(wire
 		(pts
-			(xy 217.17 107.95) (xy 217.17 134.62)
-		)
-		(stroke
-			(width 0)
-			(type default)
-		)
-	)
-	(wire
-		(pts
-			(xy 172.72 134.62) (xy 179.07 134.62)
-		)
-		(stroke
-			(width 0)
-			(type default)
-		)
-	)
-	(wire
-		(pts
-			(xy 186.69 134.62) (xy 193.04 134.62)
+			(xy 171.45 134.62) (xy 177.8 134.62)
+		)
+		(stroke
+			(width 0)
+			(type default)
+		)
+	)
+	(wire
+		(pts
+			(xy 185.42 134.62) (xy 193.04 134.62)
+		)
+		(stroke
+			(width 0)
+			(type default)
+		)
+	)
+	(wire
+		(pts
+			(xy 217.17 107.95) (xy 217.17 109.22)
 		)
 		(stroke
@@
 	(wire
 		(pts
-			(xy 210.82 109.22) (xy 264.16 109.22)
+			(xy 210.82 109.22) (xy 217.17 109.22)
 		)
 		(stroke
@@
 		(dnp no)
 		(fields_autoplaced yes)
-		(property "Reference" "TP7"
+		(property "Reference" "TP22"
 			(at 219.71 103.3779 0)
 			(show_name no)
@@
 			(project "ETH1CVOLT"
 				(path "/8d3b546e-b30b-49b2-bc59-8e254df4c067/ea97f94c-dee1-4702-bb32-5cb010d15929/d811bb30-fa6b-4ed4-ae20-cf9a7a5d683b"
-					(reference "TP7")
+					(reference "TP22")
 					(unit 1)
 				)
@@
 	(symbol
 		(lib_id "Device:R")
-		(at 182.88 134.62 90)
+		(at 181.61 134.62 90)
 		(unit 1)
 		(body_style 1)
@@
 		(fields_autoplaced yes)
 		(property "Reference" "R42"
-			(at 182.88 128.27 90)
+			(at 181.61 128.27 90)
 			(show_name no)
 			(do_not_autoplace no)
@@
 		)
 		(property "Value" "10k/0.01%/100mW"
-			(at 182.88 130.81 90)
+			(at 181.61 130.81 90)
 			(show_name no)
 			(do_not_autoplace no)
@@
 		)
 		(property "Footprint" "Resistor_SMD:R_0603_1608Metric_Pad0.98x0.95mm_HandSolder"
-			(at 182.88 136.398 90)
+			(at 181.61 136.398 90)
 			(hide yes)
 			(show_name no)
@@
 		)
 		(property "Datasheet" ""
-			(at 182.88 134.62 0)
+			(at 181.61 134.62 0)
 			(hide yes)
 			(show_name no)
@@
 		)
 		(property "Description" "Resistor"
-			(at 182.88 134.62 0)
+			(at 181.61 134.62 0)
 			(hide yes)
 			(show_name no)
@@
 	(symbol
 		(lib_id "ETH1CVOLT_A:GND_ISO")
-		(at 172.72 134.62 270)
+		(at 171.45 134.62 270)
 		(mirror x)
 		(unit 1)
@@
 		(fields_autoplaced yes)
 		(property "Reference" "#PWR0137"
-			(at 166.37 134.62 0)
+			(at 165.1 134.62 0)
 			(hide yes)
 			(show_name no)
@@
 		)
 		(property "Value" "GND_ISO"
-			(at 168.91 134.6199 90)
+			(at 167.64 134.6199 90)
 			(show_name no)
 			(do_not_autoplace no)
@@
 		)
 		(property "Footprint" ""
-			(at 172.72 134.62 0)
+			(at 171.45 134.62 0)
 			(hide yes)
 			(show_name no)
@@
 		)
 		(property "Datasheet" ""
-			(at 172.72 134.62 0)
+			(at 171.45 134.62 0)
 			(hide yes)
 			(show_name no)
@@
 		)
 		(property "Description" "Power symbol creates a global label with name \"GND\" , ground"
-			(at 172.72 134.62 0)
-			(hide yes)
-			(show_name no)
+			(at 171.45 134.62 0)
+			(hide yes)
+			(show_name no)

Commit message: Development
Parts:
- renumbered R42 to R43, R43 to R44
Changed lines of the file:
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@@
 		(dnp no)
 		(fields_autoplaced yes)
-		(property "Reference" "R43"
+		(property "Reference" "R44"
 			(at 204.47 128.27 90)
 			(show_name no)
@@
 			(project "ETH1CVOLT"
 				(path "/8d3b546e-b30b-49b2-bc59-8e254df4c067/ea97f94c-dee1-4702-bb32-5cb010d15929/d811bb30-fa6b-4ed4-ae20-cf9a7a5d683b"
-					(reference "R43")
+					(reference "R44")
 					(unit 1)
 				)
@@
 		(dnp no)
 		(fields_autoplaced yes)
-		(property "Reference" "R42"
+		(property "Reference" "R43"
 			(at 181.61 128.27 90)
 			(show_name no)
@@
 			(project "ETH1CVOLT"
 				(path "/8d3b546e-b30b-49b2-bc59-8e254df4c067/ea97f94c-dee1-4702-bb32-5cb010d15929/d811bb30-fa6b-4ed4-ae20-cf9a7a5d683b"
-					(reference "R42")
-					(unit 1)
-				)
+					(reference "R43")
+					(unit 1)
+				)

Commit message: Layout
Parts:
- renumbered C49 to C48, C50 to C49, R43 to R42, R44 to R43
Changed lines of the file:
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@@
 		(dnp no)
 		(fields_autoplaced yes)
-		(property "Reference" "#PWR0139"
+		(property "Reference" "#PWR0138"
 			(at 200.66 113.03 0)
 			(hide yes)
@@
 			(project "ETH1CVOLT"
 				(path "/8d3b546e-b30b-49b2-bc59-8e254df4c067/ea97f94c-dee1-4702-bb32-5cb010d15929/d811bb30-fa6b-4ed4-ae20-cf9a7a5d683b"
-					(reference "#PWR0139")
+					(reference "#PWR0138")
 					(unit 1)
 				)
@@
 		(dnp no)
 		(fields_autoplaced yes)
-		(property "Reference" "#PWR0138"
+		(property "Reference" "#PWR0137"
 			(at 200.66 105.41 0)
 			(hide yes)
@@
 			(project "ETH1CVOLT"
 				(path "/8d3b546e-b30b-49b2-bc59-8e254df4c067/ea97f94c-dee1-4702-bb32-5cb010d15929/d811bb30-fa6b-4ed4-ae20-cf9a7a5d683b"
-					(reference "#PWR0138")
+					(reference "#PWR0137")
 					(unit 1)
 				)
@@
 		(dnp no)
 		(fields_autoplaced yes)
-		(property "Reference" "R44"
+		(property "Reference" "R43"
 			(at 204.47 128.27 90)
 			(show_name no)
@@
 			(project "ETH1CVOLT"
 				(path "/8d3b546e-b30b-49b2-bc59-8e254df4c067/ea97f94c-dee1-4702-bb32-5cb010d15929/d811bb30-fa6b-4ed4-ae20-cf9a7a5d683b"
-					(reference "R44")
+					(reference "R43")
 					(unit 1)
 				)
@@
 		(dnp no)
 		(fields_autoplaced yes)
-		(property "Reference" "C50"
+		(property "Reference" "C49"
 			(at 49.53 267.9699 0)
 			(show_name no)
@@
 			(project "ETH1CVOLT"
 				(path "/8d3b546e-b30b-49b2-bc59-8e254df4c067/ea97f94c-dee1-4702-bb32-5cb010d15929/d811bb30-fa6b-4ed4-ae20-cf9a7a5d683b"
-					(reference "C50")
+					(reference "C49")
 					(unit 1)
 				)
@@
 		(dnp no)
 		(fields_autoplaced yes)
-		(property "Reference" "#PWR0135"
+		(property "Reference" "#PWR0134"
 			(at 45.72 267.97 0)
 			(hide yes)
@@
 			(project "ETH1CVOLT"
 				(path "/8d3b546e-b30b-49b2-bc59-8e254df4c067/ea97f94c-dee1-4702-bb32-5cb010d15929/d811bb30-fa6b-4ed4-ae20-cf9a7a5d683b"
-					(reference "#PWR0135")
+					(reference "#PWR0134")
 					(unit 1)
 				)
@@
 		(dnp no)
 		(fields_autoplaced yes)
-		(property "Reference" "#PWR0136"
+		(property "Reference" "#PWR0135"
 			(at 45.72 280.67 0)
 			(hide yes)
@@
 			(project "ETH1CVOLT"
 				(path "/8d3b546e-b30b-49b2-bc59-8e254df4c067/ea97f94c-dee1-4702-bb32-5cb010d15929/d811bb30-fa6b-4ed4-ae20-cf9a7a5d683b"
-					(reference "#PWR0136")
+					(reference "#PWR0135")
 					(unit 1)
 				)
@@
 		(dnp no)
 		(fields_autoplaced yes)
-		(property "Reference" "R43"
+		(property "Reference" "R42"
 			(at 181.61 128.27 90)
 			(show_name no)
@@
 			(project "ETH1CVOLT"
 				(path "/8d3b546e-b30b-49b2-bc59-8e254df4c067/ea97f94c-dee1-4702-bb32-5cb010d15929/d811bb30-fa6b-4ed4-ae20-cf9a7a5d683b"
-					(reference "R43")
+					(reference "R42")
 					(unit 1)
 				)
@@
 		(dnp no)
 		(fields_autoplaced yes)
-		(property "Reference" "C49"
+		(property "Reference" "C48"
 			(at 26.67 267.9699 0)
 			(show_name no)
@@
 			(project "ETH1CVOLT"
 				(path "/8d3b546e-b30b-49b2-bc59-8e254df4c067/ea97f94c-dee1-4702-bb32-5cb010d15929/d811bb30-fa6b-4ed4-ae20-cf9a7a5d683b"
-					(reference "C49")
+					(reference "C48")
 					(unit 1)
 				)
@@
 		(dnp no)
 		(fields_autoplaced yes)
-		(property "Reference" "#PWR0134"
+		(property "Reference" "#PWR0133"
 			(at 22.86 280.67 0)
 			(hide yes)
@@
 			(project "ETH1CVOLT"
 				(path "/8d3b546e-b30b-49b2-bc59-8e254df4c067/ea97f94c-dee1-4702-bb32-5cb010d15929/d811bb30-fa6b-4ed4-ae20-cf9a7a5d683b"
-					(reference "#PWR0134")
+					(reference "#PWR0133")
 					(unit 1)
 				)
@@
 		(dnp no)
 		(fields_autoplaced yes)
-		(property "Reference" "#PWR0137"
+		(property "Reference" "#PWR0136"
 			(at 165.1 134.62 0)
 			(hide yes)
@@
 			(project "ETH1CVOLT"
 				(path "/8d3b546e-b30b-49b2-bc59-8e254df4c067/ea97f94c-dee1-4702-bb32-5cb010d15929/d811bb30-fa6b-4ed4-ae20-cf9a7a5d683b"
-					(reference "#PWR0137")
+					(reference "#PWR0136")
 					(unit 1)
 				)
@@
 		(dnp no)
 		(fields_autoplaced yes)
-		(property "Reference" "#PWR0133"
+		(property "Reference" "#PWR0132"
 			(at 22.86 267.97 0)
 			(hide yes)
@@
 			(project "ETH1CVOLT"
 				(path "/8d3b546e-b30b-49b2-bc59-8e254df4c067/ea97f94c-dee1-4702-bb32-5cb010d15929/d811bb30-fa6b-4ed4-ae20-cf9a7a5d683b"
-					(reference "#PWR0133")
+					(reference "#PWR0132")
 					(unit 1)
 				)
@@
 		(dnp no)
 		(fields_autoplaced yes)
-		(property "Reference" "#PWR0141"
+		(property "Reference" "#PWR0140"
 			(at 269.24 113.03 0)
 			(hide yes)
@@
 			(project "ETH1CVOLT"
 				(path "/8d3b546e-b30b-49b2-bc59-8e254df4c067/ea97f94c-dee1-4702-bb32-5cb010d15929/d811bb30-fa6b-4ed4-ae20-cf9a7a5d683b"
-					(reference "#PWR0141")
+					(reference "#PWR0140")
 					(unit 1)
 				)
@@
 		(dnp no)
 		(fields_autoplaced yes)
-		(property "Reference" "#PWR0140"
+		(property "Reference" "#PWR0139"
 			(at 269.24 105.41 0)
 			(hide yes)
@@
 			(project "ETH1CVOLT"
 				(path "/8d3b546e-b30b-49b2-bc59-8e254df4c067/ea97f94c-dee1-4702-bb32-5cb010d15929/d811bb30-fa6b-4ed4-ae20-cf9a7a5d683b"
-					(reference "#PWR0140")
-					(unit 1)
-				)
+					(reference "#PWR0139")
+					(unit 1)
+				)

Commit message: Layout and schematic
Parts:
- removed U13: OPA192IDR, Package_SO:SOIC-8_3.9x4.9mm_P1.27mm, symbol Amplifier_Operational:OPA196xD
- added U13: ADA4522-1ARZ, Package_SO:SOIC-8_3.9x4.9mm_P1.27mm, symbol Amplifier_Operational:ADA4522-1
- renumbered C48 to C51, C49 to C52, R42 to R28, R43 to R29, TP22 to TP19
Connections:
- net +14V_ISO: now also U13.7 (V+)
- net -14V_ISO: now also U13.4 (V-)
- net DAC_SIG: now also U13.3 (+)
- net R10V_SIG: now also U13.6
- net at R28.2, R29.1: now also U13.2 (-)
Other:
- title: (none) -> ETH1CVOLT
- moved on the sheet: TP19

Commit message: Verification
Parts:
- renumbered C51 to C52, C52 to C53
Changed lines of the file:
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@@
 		(dnp no)
 		(fields_autoplaced yes)
-		(property "Reference" "#PWR0135"
+		(property "Reference" "#PWR0137"
 			(at 200.66 113.03 0)
 			(hide yes)
@@
 			(project "ETH1CVOLT"
 				(path "/8d3b546e-b30b-49b2-bc59-8e254df4c067/ea97f94c-dee1-4702-bb32-5cb010d15929/d811bb30-fa6b-4ed4-ae20-cf9a7a5d683b"
-					(reference "#PWR0135")
+					(reference "#PWR0137")
 					(unit 1)
 				)
@@
 		(dnp no)
 		(fields_autoplaced yes)
-		(property "Reference" "#PWR0134"
+		(property "Reference" "#PWR0136"
 			(at 200.66 105.41 0)
 			(hide yes)
@@
 			(project "ETH1CVOLT"
 				(path "/8d3b546e-b30b-49b2-bc59-8e254df4c067/ea97f94c-dee1-4702-bb32-5cb010d15929/d811bb30-fa6b-4ed4-ae20-cf9a7a5d683b"
-					(reference "#PWR0134")
+					(reference "#PWR0136")
 					(unit 1)
 				)
@@
 		(dnp no)
 		(fields_autoplaced yes)
-		(property "Reference" "C52"
+		(property "Reference" "C53"
 			(at 49.53 267.9699 0)
 			(show_name no)
@@
 			(project "ETH1CVOLT"
 				(path "/8d3b546e-b30b-49b2-bc59-8e254df4c067/ea97f94c-dee1-4702-bb32-5cb010d15929/d811bb30-fa6b-4ed4-ae20-cf9a7a5d683b"
-					(reference "C52")
+					(reference "C53")
 					(unit 1)
 				)
@@
 		(dnp no)
 		(fields_autoplaced yes)
-		(property "Reference" "#PWR0131"
+		(property "Reference" "#PWR0133"
 			(at 45.72 267.97 0)
 			(hide yes)
@@
 			(project "ETH1CVOLT"
 				(path "/8d3b546e-b30b-49b2-bc59-8e254df4c067/ea97f94c-dee1-4702-bb32-5cb010d15929/d811bb30-fa6b-4ed4-ae20-cf9a7a5d683b"
-					(reference "#PWR0131")
+					(reference "#PWR0133")
 					(unit 1)
 				)
@@
 		(dnp no)
 		(fields_autoplaced yes)
-		(property "Reference" "#PWR0132"
+		(property "Reference" "#PWR0134"
 			(at 45.72 280.67 0)
 			(hide yes)
@@
 			(project "ETH1CVOLT"
 				(path "/8d3b546e-b30b-49b2-bc59-8e254df4c067/ea97f94c-dee1-4702-bb32-5cb010d15929/d811bb30-fa6b-4ed4-ae20-cf9a7a5d683b"
-					(reference "#PWR0132")
+					(reference "#PWR0134")
 					(unit 1)
 				)
@@
 		(dnp no)
 		(fields_autoplaced yes)
-		(property "Reference" "C51"
+		(property "Reference" "C52"
 			(at 26.67 267.9699 0)
 			(show_name no)
@@
 			(project "ETH1CVOLT"
 				(path "/8d3b546e-b30b-49b2-bc59-8e254df4c067/ea97f94c-dee1-4702-bb32-5cb010d15929/d811bb30-fa6b-4ed4-ae20-cf9a7a5d683b"
-					(reference "C51")
+					(reference "C52")
 					(unit 1)
 				)
@@
 		(dnp no)
 		(fields_autoplaced yes)
-		(property "Reference" "#PWR0130"
+		(property "Reference" "#PWR0132"
 			(at 22.86 280.67 0)
 			(hide yes)
@@
 			(project "ETH1CVOLT"
 				(path "/8d3b546e-b30b-49b2-bc59-8e254df4c067/ea97f94c-dee1-4702-bb32-5cb010d15929/d811bb30-fa6b-4ed4-ae20-cf9a7a5d683b"
-					(reference "#PWR0130")
+					(reference "#PWR0132")
 					(unit 1)
 				)
@@
 		(dnp no)
 		(fields_autoplaced yes)
-		(property "Reference" "#PWR0133"
+		(property "Reference" "#PWR0135"
 			(at 165.1 134.62 0)
 			(hide yes)
@@
 			(project "ETH1CVOLT"
 				(path "/8d3b546e-b30b-49b2-bc59-8e254df4c067/ea97f94c-dee1-4702-bb32-5cb010d15929/d811bb30-fa6b-4ed4-ae20-cf9a7a5d683b"
-					(reference "#PWR0133")
+					(reference "#PWR0135")
 					(unit 1)
 				)
@@
 		(dnp no)
 		(fields_autoplaced yes)
-		(property "Reference" "#PWR0129"
+		(property "Reference" "#PWR0131"
 			(at 22.86 267.97 0)
 			(hide yes)
@@
 			(project "ETH1CVOLT"
 				(path "/8d3b546e-b30b-49b2-bc59-8e254df4c067/ea97f94c-dee1-4702-bb32-5cb010d15929/d811bb30-fa6b-4ed4-ae20-cf9a7a5d683b"
-					(reference "#PWR0129")
+					(reference "#PWR0131")
 					(unit 1)
 				)
@@
 		(dnp no)
 		(fields_autoplaced yes)
-		(property "Reference" "#PWR0137"
+		(property "Reference" "#PWR0139"
 			(at 269.24 113.03 0)
 			(hide yes)
@@
 			(project "ETH1CVOLT"
 				(path "/8d3b546e-b30b-49b2-bc59-8e254df4c067/ea97f94c-dee1-4702-bb32-5cb010d15929/d811bb30-fa6b-4ed4-ae20-cf9a7a5d683b"
-					(reference "#PWR0137")
+					(reference "#PWR0139")
 					(unit 1)
 				)
@@
 		(dnp no)
 		(fields_autoplaced yes)
-		(property "Reference" "#PWR0136"
+		(property "Reference" "#PWR0138"
 			(at 269.24 105.41 0)
 			(hide yes)
@@
 			(project "ETH1CVOLT"
 				(path "/8d3b546e-b30b-49b2-bc59-8e254df4c067/ea97f94c-dee1-4702-bb32-5cb010d15929/d811bb30-fa6b-4ed4-ae20-cf9a7a5d683b"
-					(reference "#PWR0136")
-					(unit 1)
-				)
+					(reference "#PWR0138")
+					(unit 1)
+				)
