File: HARDWARE/ETH1CVOLT/Range_20V.kicad_sch (KiCad schematic)
At the start: 11 parts, among them U19 ADA4522-2

Commit message: Development
Parts:
- removed C49: 0.1u/100V/X7R, Capacitor_SMD:C_0603_1608Metric_Pad1.08x0.95mm_HandSolder, symbol Device:C
- removed R64, R65: 10k/0.01%/100mW, Resistor_SMD:R_0603_1608Metric, symbol Device:R
- removed TP12, TP13: TestPoint, TestPoint:TestPoint_Pad_D1.5mm, symbol Connector:TestPoint
- removed U19: ADA4522-2, Package_SO:SOIC-8_3.9x4.9mm_P1.27mm, symbol Amplifier_Operational:ADA4522-2
- added C51, C52: 0.1u/100V/X7R, Capacitor_SMD:C_0603_1608Metric_Pad1.08x0.95mm_HandSolder, symbol Device:C
- added U14: ADA4522-1ARZ, Package_SO:SOIC-8_3.9x4.9mm_P1.27mm, symbol Amplifier_Operational:ADA4522-1
- R44: renamed from R62; footprint Resistor_SMD:R_0603_1608Metric -> Resistor_SMD:R_0603_1608Metric_Pad0.98x0.95mm_HandSolder; now fitted
- R45: renamed from R63; footprint Resistor_SMD:R_0603_1608Metric -> Resistor_SMD:R_0603_1608Metric_Pad0.98x0.95mm_HandSolder; now fitted
- R46: renamed from R68; footprint Resistor_SMD:R_0603_1608Metric -> Resistor_SMD:R_0603_1608Metric_Pad0.98x0.95mm_HandSolder; now fitted
- R47: renamed from R69; footprint Resistor_SMD:R_0603_1608Metric -> Resistor_SMD:R_0603_1608Metric_Pad0.98x0.95mm_HandSolder; now fitted
- TP8: renamed from TP11; now left out of the parts list
Connections:
- net DAC_SIG: now also U14.3 (+)
- net GND_ISO: now also C51.2, C52.2
- net R20V_SIG: now also U14.6
- net at R44.2, R45.1: now also U14.2 (-)
- new net +22V_ISO: C51.1, U14.7 (V+)
- new net -22V_ISO: C52.1, U14.4 (V-)
Other:
- note removed: "+/- 10V"

Commit message: Development
Parts:
- renumbered TP8 to TP23
Other:
- moved on the sheet: R45, R46, R47
Changed lines of the file:
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@@
 	(wire
 		(pts
-			(xy 222.25 124.46) (xy 232.41 124.46)
+			(xy 223.52 124.46) (xy 232.41 124.46)
 		)
 		(stroke
@@
 	(wire
 		(pts
-			(xy 165.1 124.46) (xy 172.72 124.46)
+			(xy 165.1 124.46) (xy 175.26 124.46)
 		)
 		(stroke
@@
 	(wire
 		(pts
-			(xy 200.66 124.46) (xy 214.63 124.46)
+			(xy 203.2 124.46) (xy 215.9 124.46)
 		)
 		(stroke
@@
 	(wire
 		(pts
-			(xy 193.04 124.46) (xy 180.34 124.46)
+			(xy 195.58 124.46) (xy 182.88 124.46)
 		)
 		(stroke
@@
 	(symbol
 		(lib_id "Device:R")
-		(at 218.44 124.46 90)
+		(at 219.71 124.46 90)
 		(unit 1)
 		(body_style 1)
@@
 		(fields_autoplaced yes)
 		(property "Reference" "R47"
-			(at 218.44 118.11 90)
+			(at 219.71 118.11 90)
 			(show_name no)
 			(do_not_autoplace no)
@@
 		)
 		(property "Value" "10k/0.01%/100mW"
-			(at 218.44 120.65 90)
+			(at 219.71 120.65 90)
 			(show_name no)
 			(do_not_autoplace no)
@@
 		)
 		(property "Footprint" "Resistor_SMD:R_0603_1608Metric_Pad0.98x0.95mm_HandSolder"
-			(at 218.44 126.238 90)
+			(at 219.71 126.238 90)
 			(hide yes)
 			(show_name no)
@@
 		)
 		(property "Datasheet" ""
-			(at 218.44 124.46 0)
+			(at 219.71 124.46 0)
 			(hide yes)
 			(show_name no)
@@
 		)
 		(property "Description" "Resistor"
-			(at 218.44 124.46 0)
+			(at 219.71 124.46 0)
 			(hide yes)
 			(show_name no)
@@
 		(dnp no)
 		(fields_autoplaced yes)
-		(property "Reference" "TP8"
+		(property "Reference" "TP23"
 			(at 234.95 85.5979 0)
 			(show_name no)
@@
 			(project "ETH1CVOLT"
 				(path "/8d3b546e-b30b-49b2-bc59-8e254df4c067/ea97f94c-dee1-4702-bb32-5cb010d15929/4998f130-2e13-4499-8fd8-1540d762c3af"
-					(reference "TP8")
+					(reference "TP23")
 					(unit 1)
 				)
@@
 	(symbol
 		(lib_id "Device:R")
-		(at 176.53 124.46 90)
+		(at 179.07 124.46 90)
 		(unit 1)
 		(body_style 1)
@@
 		(fields_autoplaced yes)
 		(property "Reference" "R45"
-			(at 176.53 118.11 90)
+			(at 179.07 118.11 90)
 			(show_name no)
 			(do_not_autoplace no)
@@
 		)
 		(property "Value" "10k/0.01%/100mW"
-			(at 176.53 120.65 90)
+			(at 179.07 120.65 90)
 			(show_name no)
 			(do_not_autoplace no)
@@
 		)
 		(property "Footprint" "Resistor_SMD:R_0603_1608Metric_Pad0.98x0.95mm_HandSolder"
-			(at 176.53 126.238 90)
+			(at 179.07 126.238 90)
 			(hide yes)
 			(show_name no)
@@
 		)
 		(property "Datasheet" ""
-			(at 176.53 124.46 0)
+			(at 179.07 124.46 0)
 			(hide yes)
 			(show_name no)
@@
 		)
 		(property "Description" "Resistor"
-			(at 176.53 124.46 0)
+			(at 179.07 124.46 0)
 			(hide yes)
 			(show_name no)
@@
 	(symbol
 		(lib_id "Device:R")
-		(at 196.85 124.46 90)
+		(at 199.39 124.46 90)
 		(unit 1)
 		(body_style 1)
@@
 		(fields_autoplaced yes)
 		(property "Reference" "R46"
-			(at 196.85 118.11 90)
+			(at 199.39 118.11 90)
 			(show_name no)
 			(do_not_autoplace no)
@@
 		)
 		(property "Value" "10k/0.01%/100mW"
-			(at 196.85 120.65 90)
+			(at 199.39 120.65 90)
 			(show_name no)
 			(do_not_autoplace no)
@@
 		)
 		(property "Footprint" "Resistor_SMD:R_0603_1608Metric_Pad0.98x0.95mm_HandSolder"
-			(at 196.85 126.238 90)
+			(at 199.39 126.238 90)
 			(hide yes)
 			(show_name no)
@@
 		)
 		(property "Datasheet" ""
-			(at 196.85 124.46 0)
+			(at 199.39 124.46 0)
 			(hide yes)
 			(show_name no)
@@
 		)
 		(property "Description" "Resistor"
-			(at 196.85 124.46 0)
-			(hide yes)
-			(show_name no)
+			(at 199.39 124.46 0)
+			(hide yes)
+			(show_name no)

Commit message: Development
Parts:
- renumbered R44 to R45, R45 to R46, R46 to R47, R47 to R48
Changed lines of the file:
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@@
 		(dnp no)
 		(fields_autoplaced yes)
-		(property "Reference" "R44"
+		(property "Reference" "R45"
 			(at 152.4 118.11 90)
 			(show_name no)
@@
 			(project "ETH1CVOLT"
 				(path "/8d3b546e-b30b-49b2-bc59-8e254df4c067/ea97f94c-dee1-4702-bb32-5cb010d15929/4998f130-2e13-4499-8fd8-1540d762c3af"
-					(reference "R44")
+					(reference "R45")
 					(unit 1)
 				)
@@
 		(dnp no)
 		(fields_autoplaced yes)
-		(property "Reference" "R47"
+		(property "Reference" "R48"
 			(at 219.71 118.11 90)
 			(show_name no)
@@
 			(project "ETH1CVOLT"
 				(path "/8d3b546e-b30b-49b2-bc59-8e254df4c067/ea97f94c-dee1-4702-bb32-5cb010d15929/4998f130-2e13-4499-8fd8-1540d762c3af"
-					(reference "R47")
+					(reference "R48")
 					(unit 1)
 				)
@@
 		(dnp no)
 		(fields_autoplaced yes)
-		(property "Reference" "R45"
+		(property "Reference" "R46"
 			(at 179.07 118.11 90)
 			(show_name no)
@@
 			(project "ETH1CVOLT"
 				(path "/8d3b546e-b30b-49b2-bc59-8e254df4c067/ea97f94c-dee1-4702-bb32-5cb010d15929/4998f130-2e13-4499-8fd8-1540d762c3af"
-					(reference "R45")
+					(reference "R46")
 					(unit 1)
 				)
@@
 		(dnp no)
 		(fields_autoplaced yes)
-		(property "Reference" "R46"
+		(property "Reference" "R47"
 			(at 199.39 118.11 90)
 			(show_name no)
@@
 			(project "ETH1CVOLT"
 				(path "/8d3b546e-b30b-49b2-bc59-8e254df4c067/ea97f94c-dee1-4702-bb32-5cb010d15929/4998f130-2e13-4499-8fd8-1540d762c3af"
-					(reference "R46")
-					(unit 1)
-				)
+					(reference "R47")
+					(unit 1)
+				)

Commit message: Layout
Parts:
- added D10: BAV199, Package_TO_SOT_SMD:SOT-23, symbol Diode:BAV99
Connections:
- net +22V_ISO: now also D10.2 (A)
- net -22V_ISO: now also D10.1 (K)
- net R20V_SIG: now also D10.3 (K)

Commit message: Layout
Parts:
- renumbered C51 to C50, C52 to C51, D10 to D4, R45 to R44, R46 to R45, R47 to R46, R48 to R47
Changed lines of the file:
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@@
 		(dnp no)
 		(fields_autoplaced yes)
-		(property "Reference" "#PWR0144"
+		(property "Reference" "#PWR0143"
 			(at 46.99 267.97 0)
 			(hide yes)
@@
 			(project "ETH1CVOLT"
 				(path "/8d3b546e-b30b-49b2-bc59-8e254df4c067/ea97f94c-dee1-4702-bb32-5cb010d15929/4998f130-2e13-4499-8fd8-1540d762c3af"
-					(reference "#PWR0144")
+					(reference "#PWR0143")
 					(unit 1)
 				)
@@
 		(dnp no)
 		(fields_autoplaced yes)
-		(property "Reference" "#PWR0143"
+		(property "Reference" "#PWR0142"
 			(at 24.13 280.67 0)
 			(hide yes)
@@
 			(project "ETH1CVOLT"
 				(path "/8d3b546e-b30b-49b2-bc59-8e254df4c067/ea97f94c-dee1-4702-bb32-5cb010d15929/4998f130-2e13-4499-8fd8-1540d762c3af"
-					(reference "#PWR0143")
+					(reference "#PWR0142")
 					(unit 1)
 				)
@@
 		(dnp no)
 		(fields_autoplaced yes)
-		(property "Reference" "R45"
+		(property "Reference" "R44"
 			(at 152.4 118.11 90)
 			(show_name no)
@@
 			(project "ETH1CVOLT"
 				(path "/8d3b546e-b30b-49b2-bc59-8e254df4c067/ea97f94c-dee1-4702-bb32-5cb010d15929/4998f130-2e13-4499-8fd8-1540d762c3af"
-					(reference "R45")
+					(reference "R44")
 					(unit 1)
 				)
@@
 		(dnp no)
 		(fields_autoplaced yes)
-		(property "Reference" "C52"
+		(property "Reference" "C51"
 			(at 50.8 267.9699 0)
 			(show_name no)
@@
 			(project "ETH1CVOLT"
 				(path "/8d3b546e-b30b-49b2-bc59-8e254df4c067/ea97f94c-dee1-4702-bb32-5cb010d15929/4998f130-2e13-4499-8fd8-1540d762c3af"
-					(reference "C52")
+					(reference "C51")
 					(unit 1)
 				)
@@
 		(dnp no)
 		(fields_autoplaced yes)
-		(property "Reference" "R48"
+		(property "Reference" "R47"
 			(at 219.71 118.11 90)
 			(show_name no)
@@
 			(project "ETH1CVOLT"
 				(path "/8d3b546e-b30b-49b2-bc59-8e254df4c067/ea97f94c-dee1-4702-bb32-5cb010d15929/4998f130-2e13-4499-8fd8-1540d762c3af"
-					(reference "R48")
+					(reference "R47")
 					(unit 1)
 				)
@@
 		(dnp no)
 		(fields_autoplaced yes)
-		(property "Reference" "#PWR0224"
+		(property "Reference" "#PWR0149"
 			(at 255.27 96.52 0)
 			(hide yes)
@@
 			(project "ETH1CVOLT"
 				(path "/8d3b546e-b30b-49b2-bc59-8e254df4c067/ea97f94c-dee1-4702-bb32-5cb010d15929/4998f130-2e13-4499-8fd8-1540d762c3af"
-					(reference "#PWR0224")
+					(reference "#PWR0149")
 					(unit 1)
 				)
@@
 		(dnp no)
 		(fields_autoplaced yes)
-		(property "Reference" "#PWR0142"
+		(property "Reference" "#PWR0141"
 			(at 24.13 267.97 0)
 			(hide yes)
@@
 			(project "ETH1CVOLT"
 				(path "/8d3b546e-b30b-49b2-bc59-8e254df4c067/ea97f94c-dee1-4702-bb32-5cb010d15929/4998f130-2e13-4499-8fd8-1540d762c3af"
-					(reference "#PWR0142")
+					(reference "#PWR0141")
 					(unit 1)
 				)
@@
 		(dnp no)
 		(fields_autoplaced yes)
-		(property "Reference" "#PWR0147"
+		(property "Reference" "#PWR0146"
 			(at 172.72 88.9 0)
 			(hide yes)
@@
 			(project "ETH1CVOLT"
 				(path "/8d3b546e-b30b-49b2-bc59-8e254df4c067/ea97f94c-dee1-4702-bb32-5cb010d15929/4998f130-2e13-4499-8fd8-1540d762c3af"
-					(reference "#PWR0147")
+					(reference "#PWR0146")
 					(unit 1)
 				)
@@
 		(dnp no)
 		(fields_autoplaced yes)
-		(property "Reference" "R46"
+		(property "Reference" "R45"
 			(at 179.07 118.11 90)
 			(show_name no)
@@
 			(project "ETH1CVOLT"
 				(path "/8d3b546e-b30b-49b2-bc59-8e254df4c067/ea97f94c-dee1-4702-bb32-5cb010d15929/4998f130-2e13-4499-8fd8-1540d762c3af"
-					(reference "R46")
+					(reference "R45")
 					(unit 1)
 				)
@@
 		(dnp no)
 		(fields_autoplaced yes)
-		(property "Reference" "#PWR0223"
+		(property "Reference" "#PWR0148"
 			(at 255.27 88.9 0)
 			(hide yes)
@@
 			(project "ETH1CVOLT"
 				(path "/8d3b546e-b30b-49b2-bc59-8e254df4c067/ea97f94c-dee1-4702-bb32-5cb010d15929/4998f130-2e13-4499-8fd8-1540d762c3af"
-					(reference "#PWR0223")
+					(reference "#PWR0148")
 					(unit 1)
 				)
@@
 		(dnp no)
 		(fields_autoplaced yes)
-		(property "Reference" "C51"
+		(property "Reference" "C50"
 			(at 27.94 267.9699 0)
 			(show_name no)
@@
 			(project "ETH1CVOLT"
 				(path "/8d3b546e-b30b-49b2-bc59-8e254df4c067/ea97f94c-dee1-4702-bb32-5cb010d15929/4998f130-2e13-4499-8fd8-1540d762c3af"
-					(reference "C51")
+					(reference "C50")
 					(unit 1)
 				)
@@
 		(dnp no)
 		(fields_autoplaced yes)
-		(property "Reference" "#PWR0145"
+		(property "Reference" "#PWR0144"
 			(at 46.99 280.67 0)
 			(hide yes)
@@
 			(project "ETH1CVOLT"
 				(path "/8d3b546e-b30b-49b2-bc59-8e254df4c067/ea97f94c-dee1-4702-bb32-5cb010d15929/4998f130-2e13-4499-8fd8-1540d762c3af"
-					(reference "#PWR0145")
+					(reference "#PWR0144")
 					(unit 1)
 				)
@@
 		(dnp no)
 		(fields_autoplaced yes)
-		(property "Reference" "#PWR0146"
+		(property "Reference" "#PWR0145"
 			(at 135.89 124.46 0)
 			(hide yes)
@@
 			(project "ETH1CVOLT"
 				(path "/8d3b546e-b30b-49b2-bc59-8e254df4c067/ea97f94c-dee1-4702-bb32-5cb010d15929/4998f130-2e13-4499-8fd8-1540d762c3af"
-					(reference "#PWR0146")
+					(reference "#PWR0145")
 					(unit 1)
 				)
@@
 		(dnp no)
 		(fields_autoplaced yes)
-		(property "Reference" "#PWR0148"
+		(property "Reference" "#PWR0147"
 			(at 172.72 96.52 0)
 			(hide yes)
@@
 			(project "ETH1CVOLT"
 				(path "/8d3b546e-b30b-49b2-bc59-8e254df4c067/ea97f94c-dee1-4702-bb32-5cb010d15929/4998f130-2e13-4499-8fd8-1540d762c3af"
-					(reference "#PWR0148")
+					(reference "#PWR0147")
 					(unit 1)
 				)
@@
 		(dnp no)
 		(fields_autoplaced yes)
-		(property "Reference" "D10"
+		(property "Reference" "D4"
 			(at 257.81 91.4399 90)
 			(show_name no)
@@
 			(project "ETH1CVOLT"
 				(path "/8d3b546e-b30b-49b2-bc59-8e254df4c067/ea97f94c-dee1-4702-bb32-5cb010d15929/4998f130-2e13-4499-8fd8-1540d762c3af"
-					(reference "D10")
+					(reference "D4")
 					(unit 1)
 				)
@@
 		(dnp no)
 		(fields_autoplaced yes)
-		(property "Reference" "R47"
+		(property "Reference" "R46"
 			(at 199.39 118.11 90)
 			(show_name no)
@@
 			(project "ETH1CVOLT"
 				(path "/8d3b546e-b30b-49b2-bc59-8e254df4c067/ea97f94c-dee1-4702-bb32-5cb010d15929/4998f130-2e13-4499-8fd8-1540d762c3af"
-					(reference "R47")
-					(unit 1)
-				)
+					(reference "R46")
+					(unit 1)
+				)

Commit message: Layout and schematic
Parts:
- renumbered C50 to C53, C51 to C54, R44 to R30, R45 to R31, R46 to R32, R47 to R33, TP23 to TP20
Other:
- title: (none) -> ETH1CVOLT

Commit message: Verification
Parts:
- renumbered C53 to C54, C54 to C55
Changed lines of the file:
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@@
 		(dnp no)
 		(fields_autoplaced yes)
-		(property "Reference" "#PWR0140"
+		(property "Reference" "#PWR0142"
 			(at 46.99 267.97 0)
 			(hide yes)
@@
 			(project "ETH1CVOLT"
 				(path "/8d3b546e-b30b-49b2-bc59-8e254df4c067/ea97f94c-dee1-4702-bb32-5cb010d15929/4998f130-2e13-4499-8fd8-1540d762c3af"
-					(reference "#PWR0140")
+					(reference "#PWR0142")
 					(unit 1)
 				)
@@
 		(dnp no)
 		(fields_autoplaced yes)
-		(property "Reference" "#PWR0139"
+		(property "Reference" "#PWR0141"
 			(at 24.13 280.67 0)
 			(hide yes)
@@
 			(project "ETH1CVOLT"
 				(path "/8d3b546e-b30b-49b2-bc59-8e254df4c067/ea97f94c-dee1-4702-bb32-5cb010d15929/4998f130-2e13-4499-8fd8-1540d762c3af"
-					(reference "#PWR0139")
+					(reference "#PWR0141")
 					(unit 1)
 				)
@@
 		(dnp no)
 		(fields_autoplaced yes)
-		(property "Reference" "C54"
+		(property "Reference" "C55"
 			(at 50.8 267.9699 0)
 			(show_name no)
@@
 			(project "ETH1CVOLT"
 				(path "/8d3b546e-b30b-49b2-bc59-8e254df4c067/ea97f94c-dee1-4702-bb32-5cb010d15929/4998f130-2e13-4499-8fd8-1540d762c3af"
-					(reference "C54")
+					(reference "C55")
 					(unit 1)
 				)
@@
 		(dnp no)
 		(fields_autoplaced yes)
-		(property "Reference" "#PWR0146"
+		(property "Reference" "#PWR0148"
 			(at 255.27 96.52 0)
 			(hide yes)
@@
 			(project "ETH1CVOLT"
 				(path "/8d3b546e-b30b-49b2-bc59-8e254df4c067/ea97f94c-dee1-4702-bb32-5cb010d15929/4998f130-2e13-4499-8fd8-1540d762c3af"
-					(reference "#PWR0146")
+					(reference "#PWR0148")
 					(unit 1)
 				)
@@
 		(dnp no)
 		(fields_autoplaced yes)
-		(property "Reference" "#PWR0138"
+		(property "Reference" "#PWR0140"
 			(at 24.13 267.97 0)
 			(hide yes)
@@
 			(project "ETH1CVOLT"
 				(path "/8d3b546e-b30b-49b2-bc59-8e254df4c067/ea97f94c-dee1-4702-bb32-5cb010d15929/4998f130-2e13-4499-8fd8-1540d762c3af"
-					(reference "#PWR0138")
+					(reference "#PWR0140")
 					(unit 1)
 				)
@@
 		(dnp no)
 		(fields_autoplaced yes)
-		(property "Reference" "#PWR0143"
+		(property "Reference" "#PWR0145"
 			(at 172.72 88.9 0)
 			(hide yes)
@@
 			(project "ETH1CVOLT"
 				(path "/8d3b546e-b30b-49b2-bc59-8e254df4c067/ea97f94c-dee1-4702-bb32-5cb010d15929/4998f130-2e13-4499-8fd8-1540d762c3af"
-					(reference "#PWR0143")
+					(reference "#PWR0145")
 					(unit 1)
 				)
@@
 		(dnp no)
 		(fields_autoplaced yes)
-		(property "Reference" "#PWR0145"
+		(property "Reference" "#PWR0147"
 			(at 255.27 88.9 0)
 			(hide yes)
@@
 			(project "ETH1CVOLT"
 				(path "/8d3b546e-b30b-49b2-bc59-8e254df4c067/ea97f94c-dee1-4702-bb32-5cb010d15929/4998f130-2e13-4499-8fd8-1540d762c3af"
-					(reference "#PWR0145")
+					(reference "#PWR0147")
 					(unit 1)
 				)
@@
 		(dnp no)
 		(fields_autoplaced yes)
-		(property "Reference" "C53"
+		(property "Reference" "C54"
 			(at 27.94 267.9699 0)
 			(show_name no)
@@
 			(project "ETH1CVOLT"
 				(path "/8d3b546e-b30b-49b2-bc59-8e254df4c067/ea97f94c-dee1-4702-bb32-5cb010d15929/4998f130-2e13-4499-8fd8-1540d762c3af"
-					(reference "C53")
+					(reference "C54")
 					(unit 1)
 				)
@@
 		(dnp no)
 		(fields_autoplaced yes)
-		(property "Reference" "#PWR0141"
+		(property "Reference" "#PWR0143"
 			(at 46.99 280.67 0)
 			(hide yes)
@@
 			(project "ETH1CVOLT"
 				(path "/8d3b546e-b30b-49b2-bc59-8e254df4c067/ea97f94c-dee1-4702-bb32-5cb010d15929/4998f130-2e13-4499-8fd8-1540d762c3af"
-					(reference "#PWR0141")
+					(reference "#PWR0143")
 					(unit 1)
 				)
@@
 		(dnp no)
 		(fields_autoplaced yes)
-		(property "Reference" "#PWR0142"
+		(property "Reference" "#PWR0144"
 			(at 135.89 124.46 0)
 			(hide yes)
@@
 			(project "ETH1CVOLT"
 				(path "/8d3b546e-b30b-49b2-bc59-8e254df4c067/ea97f94c-dee1-4702-bb32-5cb010d15929/4998f130-2e13-4499-8fd8-1540d762c3af"
-					(reference "#PWR0142")
+					(reference "#PWR0144")
 					(unit 1)
 				)
@@
 		(dnp no)
 		(fields_autoplaced yes)
-		(property "Reference" "#PWR0144"
+		(property "Reference" "#PWR0146"
 			(at 172.72 96.52 0)
 			(hide yes)
@@
 			(project "ETH1CVOLT"
 				(path "/8d3b546e-b30b-49b2-bc59-8e254df4c067/ea97f94c-dee1-4702-bb32-5cb010d15929/4998f130-2e13-4499-8fd8-1540d762c3af"
-					(reference "#PWR0144")
-					(unit 1)
-				)
+					(reference "#PWR0146")
+					(unit 1)
+				)
