File: HARDWARE/ETH1CVOLT/DAC.kicad_sch (KiCad schematic)
At the start: 9 parts, among them U10 MAX44241AUA+, U4 MAX5719GSD+

Commit message: Development
Parts:
- added C43, C44: 0.1u/100V/X7R, Capacitor_SMD:C_0603_1608Metric_Pad1.08x0.95mm_HandSolder, symbol Device:C
- added R36, R39, R41: 0R/5%/100mW, Package_SO:TSSOP-16_4.4x5mm_P0.65mm, symbol Device:R
- renumbered C48 to C41, C34 to C42, R16 to R34, R17 to R35, R19 to R37, R18 to R38, R20 to R40, U4 to U9
Connections:
- net GND_ISO: now also C43.1, C44.1, R41.1; no longer R40.1
- net -7V_ISO: now reaches R37.1
- net at R37.2, R40.2, U10.4 (V-): now also C44.2, R41.2
- net at U10.7 (V+): now also C43.2, R36.1, R39.1
- new net +14V_ISO: R39.2
- new net +7V_ISO: R36.2
- new net -14V_ISO: R40.1
Other:
- moved on the sheet: C42, R34, R35, R37, R38, R40, U10, U9

Commit message: Development
Parts:
- R34, R35, R36, R37, R38, R39, R40, R41: footprint Package_SO:TSSOP-16_4.4x5mm_P0.65mm -> Resistor_SMD:R_0603_1608Metric_Pad0.98x0.95mm_HandSolder
Changed lines of the file:
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@@
 			)
 		)
-		(property "Footprint" "Package_SO:TSSOP-16_4.4x5mm_P0.65mm"
+		(property "Footprint" "Resistor_SMD:R_0603_1608Metric_Pad0.98x0.95mm_HandSolder"
 			(at 248.92 163.068 90)
 			(hide yes)
@@
 			)
 		)
-		(property "Footprint" "Package_SO:TSSOP-16_4.4x5mm_P0.65mm"
+		(property "Footprint" "Resistor_SMD:R_0603_1608Metric_Pad0.98x0.95mm_HandSolder"
 			(at 236.728 140.97 90)
 			(hide yes)
@@
 			)
 		)
-		(property "Footprint" "Package_SO:TSSOP-16_4.4x5mm_P0.65mm"
+		(property "Footprint" "Resistor_SMD:R_0603_1608Metric_Pad0.98x0.95mm_HandSolder"
 			(at 186.69 100.838 90)
 			(hide yes)
@@
 			)
 		)
-		(property "Footprint" "Package_SO:TSSOP-16_4.4x5mm_P0.65mm"
+		(property "Footprint" "Resistor_SMD:R_0603_1608Metric_Pad0.98x0.95mm_HandSolder"
 			(at 255.778 113.03 90)
 			(hide yes)
@@
 			)
 		)
-		(property "Footprint" "Package_SO:TSSOP-16_4.4x5mm_P0.65mm"
+		(property "Footprint" "Resistor_SMD:R_0603_1608Metric_Pad0.98x0.95mm_HandSolder"
 			(at 274.828 140.97 90)
 			(hide yes)
@@
 			)
 		)
-		(property "Footprint" "Package_SO:TSSOP-16_4.4x5mm_P0.65mm"
+		(property "Footprint" "Resistor_SMD:R_0603_1608Metric_Pad0.98x0.95mm_HandSolder"
 			(at 255.778 140.97 90)
 			(hide yes)
@@
 			)
 		)
-		(property "Footprint" "Package_SO:TSSOP-16_4.4x5mm_P0.65mm"
+		(property "Footprint" "Resistor_SMD:R_0603_1608Metric_Pad0.98x0.95mm_HandSolder"
 			(at 236.728 113.03 90)
 			(hide yes)
@@
 			)
 		)
-		(property "Footprint" "Package_SO:TSSOP-16_4.4x5mm_P0.65mm"
+		(property "Footprint" "Resistor_SMD:R_0603_1608Metric_Pad0.98x0.95mm_HandSolder"
 			(at 186.69 131.318 90)
 			(hide yes)

Commit message: Development
Parts:
- added TP9: TestPoint, TestPoint:TestPoint_Pad_D1.5mm, symbol Connector:TestPoint
- R38, R39, R40, R41: now not fitted
Connections:
- net DAC_SIG: now also TP9.1
Changed lines of the file:
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@@
 	)
 	(junction
-		(at 196.85 129.54)
+		(at 199.39 129.54)
 		(diameter 0)
 		(color 0 0 0 0)
@@
 	)
 	(junction
+		(at 280.67 127)
+		(diameter 0)
+		(color 0 0 0 0)
+	)
+	(junction
 		(at 254 118.11)
 		(diameter 0)
@@
 	(wire
 		(pts
+			(xy 280.67 127) (xy 293.37 127)
+		)
+		(stroke
+			(width 0)
+			(type default)
+		)
+	)
+	(wire
+		(pts
+			(xy 280.67 125.73) (xy 280.67 127)
+		)
+		(stroke
+			(width 0)
+			(type default)
+		)
+	)
+	(wire
+		(pts
 			(xy 146.05 119.38) (xy 146.05 116.84)
 		)
@@
 	(wire
 		(pts
-			(xy 245.11 161.29) (xy 196.85 161.29)
+			(xy 245.11 161.29) (xy 199.39 161.29)
 		)
 		(stroke
@@
 	(wire
 		(pts
-			(xy 190.5 129.54) (xy 196.85 129.54)
+			(xy 190.5 129.54) (xy 229.87 129.54)
 		)
 		(stroke
@@
 	(wire
 		(pts
-			(xy 196.85 129.54) (xy 229.87 129.54)
-		)
-		(stroke
-			(width 0)
-			(type default)
-		)
-	)
-	(wire
-		(pts
 			(xy 254 135.89) (xy 273.05 135.89)
 		)
@@
 	(wire
 		(pts
-			(xy 245.11 127) (xy 293.37 127)
-		)
-		(stroke
-			(width 0)
-			(type default)
-		)
-	)
-	(wire
-		(pts
-			(xy 196.85 161.29) (xy 196.85 129.54)
+			(xy 245.11 127) (xy 280.67 127)
+		)
+		(stroke
+			(width 0)
+			(type default)
+		)
+	)
+	(wire
+		(pts
+			(xy 199.39 161.29) (xy 199.39 129.54)
 		)
 		(stroke
@@
 	)
 	(symbol
+		(lib_id "Connector:TestPoint")
+		(at 280.67 125.73 0)
+		(mirror y)
+		(unit 1)
+		(body_style 1)
+		(exclude_from_sim no)
+		(in_bom no)
+		(on_board yes)
+		(in_pos_files yes)
+		(dnp no)
+		(property "Reference" "TP9"
+			(at 281.94 118.11 0)
+			(show_name no)
+			(do_not_autoplace no)
+			(effects
+				(font
+					(size 1.27 1.27)
+				)
+				(justify left)
+			)
+		)
+		(property "Value" "TestPoint"
+			(at 284.48 120.65 0)
+			(show_name no)
+			(do_not_autoplace no)
+			(effects
+				(font
+					(size 1.27 1.27)
+				)
+				(justify left)
+			)
+		)
+		(property "Footprint" "TestPoint:TestPoint_Pad_D1.5mm"
+			(at 275.59 125.73 0)
+			(hide yes)
+			(show_name no)
+			(do_not_autoplace no)
+			(effects
+				(font
+					(size 1.27 1.27)
+				)
+			)
+		)
+		(property "Datasheet" ""
+			(at 275.59 125.73 0)
+			(hide yes)
+			(show_name no)
+			(do_not_autoplace no)
+			(effects
+				(font
+					(size 1.27 1.27)
+				)
+			)
+		)
+		(property "Description" "test point"
+			(at 280.67 125.73 0)
+			(hide yes)
+			(show_name no)
+			(do_not_autoplace no)
+			(effects
+				(font
+					(size 1.27 1.27)
+				)
+			)
+		)
+		(pin "1"
+		)
+		(instances
+			(project "ETH1CVOLT"
+				(path "/8d3b546e-b30b-49b2-bc59-8e254df4c067/ea97f94c-dee1-4702-bb32-5cb010d15929/e2cff0f2-156b-4ebd-b442-dc8733a740cb"
+					(reference "TP9")
+					(unit 1)
+				)
+			)
+		)
+	)
+	(symbol
 		(lib_id "ETH1CVOLT_A:+5VD_ISO")
 		(at 160.02 110.49 0)
@@
 		(dnp no)
 		(fields_autoplaced yes)
-		(property "Reference" "#FLG013"
+		(property "Reference" "#FLG08"
 			(at 257.175 118.11 0)
 			(hide yes)
@@
 			(project "ETH1CVOLT"
 				(path "/8d3b546e-b30b-49b2-bc59-8e254df4c067/ea97f94c-dee1-4702-bb32-5cb010d15929/e2cff0f2-156b-4ebd-b442-dc8733a740cb"
-					(reference "#FLG013")
+					(reference "#FLG08")
 					(unit 1)
 				)
@@
 		(on_board yes)
 		(in_pos_files yes)
-		(dnp no)
+		(dnp yes)
 		(property "Reference" "R38"
 			(at 248.92 164.338 90)
@@
 		(on_board yes)
 		(in_pos_files yes)
-		(dnp no)
+		(dnp yes)
 		(property "Reference" "R39"
 			(at 262.636 112.014 0)
@@
 					(reference "R39")
 					(unit 1)
-					(variant
-						(name "A")
-						(dnp yes)
-					)
 				)
 			)
@@
 		(on_board yes)
 		(in_pos_files yes)
-		(dnp no)
+		(dnp yes)
 		(property "Reference" "R41"
 			(at 281.686 139.954 0)
@@
 					(reference "R41")
 					(unit 1)
-					(variant
-						(name "A")
-						(dnp yes)
-					)
 				)
 			)
@@
 		(on_board yes)
 		(in_pos_files yes)
-		(dnp no)
+		(dnp yes)
 		(property "Reference" "R40"
 			(at 262.636 139.954 0)
@@
 					(reference "R40")
 					(unit 1)
-					(variant
-						(name "A")
-						(dnp yes)
-					)
 				)
 			)
@@
 		(dnp no)
 		(fields_autoplaced yes)
-		(property "Reference" "#FLG014"
+		(property "Reference" "#FLG09"
 			(at 276.225 135.89 0)
 			(hide yes)
@@
 			(project "ETH1CVOLT"
 				(path "/8d3b546e-b30b-49b2-bc59-8e254df4c067/ea97f94c-dee1-4702-bb32-5cb010d15929/e2cff0f2-156b-4ebd-b442-dc8733a740cb"
-					(reference "#FLG014")
+					(reference "#FLG09")
 					(unit 1)
 				)

Commit message: Development
Parts:
- renumbered R34 to R35, R35 to R36, R36 to R37, R37 to R38, R38 to R39, R39 to R40, R40 to R41, R41 to R42
Changed lines of the file:
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@@
 		(in_pos_files yes)
 		(dnp yes)
-		(property "Reference" "R38"
+		(property "Reference" "R39"
 			(at 248.92 164.338 90)
 			(show_name no)
@@
 			(project "ETH1CVOLT"
 				(path "/8d3b546e-b30b-49b2-bc59-8e254df4c067/ea97f94c-dee1-4702-bb32-5cb010d15929/e2cff0f2-156b-4ebd-b442-dc8733a740cb"
-					(reference "R38")
+					(reference "R39")
 					(unit 1)
 				)
@@
 		(in_pos_files yes)
 		(dnp no)
-		(property "Reference" "R37"
+		(property "Reference" "R38"
 			(at 243.586 139.954 0)
 			(show_name no)
@@
 			(project "ETH1CVOLT"
 				(path "/8d3b546e-b30b-49b2-bc59-8e254df4c067/ea97f94c-dee1-4702-bb32-5cb010d15929/e2cff0f2-156b-4ebd-b442-dc8733a740cb"
-					(reference "R37")
+					(reference "R38")
 					(unit 1)
 				)
@@
 		(dnp no)
 		(fields_autoplaced yes)
-		(property "Reference" "R34"
+		(property "Reference" "R35"
 			(at 186.69 92.71 90)
 			(show_name no)
@@
 			(project "ETH1CVOLT"
 				(path "/8d3b546e-b30b-49b2-bc59-8e254df4c067/ea97f94c-dee1-4702-bb32-5cb010d15929/e2cff0f2-156b-4ebd-b442-dc8733a740cb"
-					(reference "R34")
+					(reference "R35")
 					(unit 1)
 				)
@@
 		(in_pos_files yes)
 		(dnp yes)
-		(property "Reference" "R39"
+		(property "Reference" "R40"
 			(at 262.636 112.014 0)
 			(show_name no)
@@
 			(project "ETH1CVOLT"
 				(path "/8d3b546e-b30b-49b2-bc59-8e254df4c067/ea97f94c-dee1-4702-bb32-5cb010d15929/e2cff0f2-156b-4ebd-b442-dc8733a740cb"
-					(reference "R39")
+					(reference "R40")
 					(unit 1)
 				)
@@
 		(in_pos_files yes)
 		(dnp yes)
-		(property "Reference" "R41"
+		(property "Reference" "R42"
 			(at 281.686 139.954 0)
 			(show_name no)
@@
 			(project "ETH1CVOLT"
 				(path "/8d3b546e-b30b-49b2-bc59-8e254df4c067/ea97f94c-dee1-4702-bb32-5cb010d15929/e2cff0f2-156b-4ebd-b442-dc8733a740cb"
-					(reference "R41")
+					(reference "R42")
 					(unit 1)
 				)
@@
 		(in_pos_files yes)
 		(dnp yes)
-		(property "Reference" "R40"
+		(property "Reference" "R41"
 			(at 262.636 139.954 0)
 			(show_name no)
@@
 			(project "ETH1CVOLT"
 				(path "/8d3b546e-b30b-49b2-bc59-8e254df4c067/ea97f94c-dee1-4702-bb32-5cb010d15929/e2cff0f2-156b-4ebd-b442-dc8733a740cb"
-					(reference "R40")
+					(reference "R41")
 					(unit 1)
 				)
@@
 		(in_pos_files yes)
 		(dnp no)
-		(property "Reference" "R36"
+		(property "Reference" "R37"
 			(at 243.84 111.76 0)
 			(show_name no)
@@
 			(project "ETH1CVOLT"
 				(path "/8d3b546e-b30b-49b2-bc59-8e254df4c067/ea97f94c-dee1-4702-bb32-5cb010d15929/e2cff0f2-156b-4ebd-b442-dc8733a740cb"
-					(reference "R36")
+					(reference "R37")
 					(unit 1)
 				)
@@
 		(in_pos_files yes)
 		(dnp no)
-		(property "Reference" "R35"
+		(property "Reference" "R36"
 			(at 186.69 132.588 90)
 			(show_name no)
@@
 			(project "ETH1CVOLT"
 				(path "/8d3b546e-b30b-49b2-bc59-8e254df4c067/ea97f94c-dee1-4702-bb32-5cb010d15929/e2cff0f2-156b-4ebd-b442-dc8733a740cb"
-					(reference "R35")
-					(unit 1)
-				)
+					(reference "R36")
+					(unit 1)
+				)

Commit message: Layout
Parts:
- renumbered C41 to C40, C42 to C41, C43 to C42, C44 to C43, R35 to R34, R36 to R35, R37 to R36, R38 to R37, R39 to R38, R40 to R39, R41 to R40, R42 to R41

Commit message: Layout and schematic
Parts:
- renumbered C40 to C43, C41 to C44, C42 to C45, C43 to C46, R34 to R20, R35 to R21, R36 to R22, R37 to R23, R38 to R24, R39 to R25, R40 to R26, R41 to R27, TP9 to TP6
Other:
- title: (none) -> ETH1CVOLT

Commit message: Verification
Parts:
- removed U10: MAX44241AUA+, Package_SO:VSSOP-8_3x3mm_P0.65mm, symbol ETH1CVOLT_B:MAX44241AUA+
- added U10: ADA4522-1ARZ, Package_SO:SOIC-8_3.9x4.9mm_P1.27mm, symbol Amplifier_Operational:ADA4522-1
- renumbered C43 to C44, C44 to C45, C45 to C46, C46 to C47
Connections:
- net DAC_SIG: now also U10.6
- net at C47.2, R23.2, R26.2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: now also U10.4 (V-)
- net at R21.2, R24.1: now also U10.2 (-)
- net at C46.2, R22.1, R25.1: now also U10.7 (V+)
- net at U9.2 (OUT): now also U10.3 (+)

Commit message: Modifications
Parts:
- added R63: 4k7/1%/100mW, Resistor_SMD:R_0603_1608Metric_Pad0.98x0.95mm_HandSolder, symbol Device:R
Connections:
- net +5VD_ISO: now also R63.1
- net DAC_~{LDAC}: now also R63.2
Changed lines of the file:
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@@
 		(color 0 0 0 0)
 	)
+	(junction
+		(at 115.57 151.13)
+		(diameter 0)
+		(color 0 0 0 0)
+	)
 	(wire
 		(pts
@@
 	(wire
 		(pts
+			(xy 115.57 151.13) (xy 144.78 151.13)
+		)
+		(stroke
+			(width 0)
+			(type default)
+		)
+	)
+	(wire
+		(pts
 			(xy 245.11 161.29) (xy 199.39 161.29)
 		)
@@
 	(wire
 		(pts
+			(xy 115.57 149.86) (xy 115.57 151.13)
+		)
+		(stroke
+			(width 0)
+			(type default)
+		)
+	)
+	(wire
+		(pts
 			(xy 215.9 118.11) (xy 219.71 118.11)
 		)
@@
 	(wire
 		(pts
+			(xy 144.78 151.13) (xy 144.78 132.08)
+		)
+		(stroke
+			(width 0)
+			(type default)
+		)
+	)
+	(wire
+		(pts
 			(xy 160.02 137.16) (xy 160.02 138.43)
 		)
@@
 	(wire
 		(pts
-			(xy 146.05 132.08) (xy 147.32 132.08)
+			(xy 114.3 151.13) (xy 115.57 151.13)
+		)
+		(stroke
+			(width 0)
+			(type default)
+		)
+	)
+	(wire
+		(pts
+			(xy 144.78 132.08) (xy 147.32 132.08)
 		)
 		(stroke
@@
 	(hierarchical_label "DAC_~{LDAC}"
 		(shape input)
-		(at 146.05 132.08 180)
+		(at 114.3 151.13 180)
 		(effects
 			(font
@@
 	)
 	(symbol
+		(lib_id "ETH1CVOLT_A:+5VD_ISO")
+		(at 115.57 142.24 0)
+		(unit 1)
+		(body_style 1)
+		(exclude_from_sim no)
+		(in_bom yes)
+		(on_board yes)
+		(in_pos_files yes)
+		(dnp no)
+		(fields_autoplaced yes)
+		(property "Reference" "#PWR0223"
+			(at 115.57 146.05 0)
+			(hide yes)
+			(show_name no)
+			(do_not_autoplace no)
+			(effects
+				(font
+					(size 1.27 1.27)
+				)
+			)
+		)
+		(property "Value" "+5VD_ISO"
+			(at 115.57 137.16 0)
+			(show_name no)
+			(do_not_autoplace no)
+			(effects
+				(font
+					(size 1.27 1.27)
+				)
+			)
+		)
+		(property "Footprint" "Package_SO:SOIC-8_3.9x4.9mm_P1.27mm"
+			(at 115.57 142.24 0)
+			(hide yes)
+			(show_name no)
+			(do_not_autoplace no)
+			(effects
+				(font
+					(size 1.27 1.27)
+				)
+			)
+		)
+		(property "Datasheet" ""
+			(at 115.57 142.24 0)
+			(hide yes)
+			(show_name no)
+			(do_not_autoplace no)
+			(effects
+				(font
+					(size 1.27 1.27)
+				)
+			)
+		)
+		(property "Description" "Power symbol"
+			(at 115.57 142.24 0)
+			(hide yes)
+			(show_name no)
+			(do_not_autoplace no)
+			(effects
+				(font
+					(size 1.27 1.27)
+				)
+			)
+		)
+		(pin "1"
+		)
+		(instances
+			(project "ETH1CVOLT"
+				(path "/8d3b546e-b30b-49b2-bc59-8e254df4c067/ea97f94c-dee1-4702-bb32-5cb010d15929/e2cff0f2-156b-4ebd-b442-dc8733a740cb"
+					(reference "#PWR0223")
+					(unit 1)
+				)
+			)
+		)
+	)
+	(symbol
 		(lib_id "Device:C")
 		(at 223.52 135.89 90)
@@
 					(unit 1)
 				)
+			)
+		)
+	)
+	(symbol
+		(lib_id "Device:R")
+		(at 115.57 146.05 0)
+		(unit 1)
+		(body_style 1)
+		(exclude_from_sim no)
+		(in_bom yes)
+		(on_board yes)
+		(in_pos_files yes)
+		(dnp no)
+		(fields_autoplaced yes)
+		(property "Reference" "R63"
+			(at 118.11 144.7799 0)
+			(show_name no)
+			(do_not_autoplace no)
+			(effects
+				(font
+					(size 1.27 1.27)
+				)
+				(justify left)
+			)
+		)
+		(property "Value" "4k7/1%/100mW"
+			(at 118.11 147.3199 0)
+			(show_name no)
+			(do_not_autoplace no)
+			(effects
+				(font
+					(size 1.27 1.27)
+				)
+				(justify left)
+			)
+		)
+		(property "Footprint" "Resistor_SMD:R_0603_1608Metric_Pad0.98x0.95mm_HandSolder"
+			(at 113.792 146.05 90)
+			(hide yes)
+			(show_name no)
+			(do_not_autoplace no)
+			(effects
+				(font
+					(size 1.27 1.27)
+				)
+			)
+		)
+		(property "Datasheet" ""
+			(at 115.57 146.05 0)
+			(hide yes)
+			(show_name no)
+			(do_not_autoplace no)
+			(effects
+				(font
+					(size 1.27 1.27)
+				)
+			)
+		)
+		(property "Description" "Resistor"
+			(at 115.57 146.05 0)
+			(hide yes)
+			(show_name no)
+			(do_not_autoplace no)
+			(effects
+				(font
+					(size 1.27 1.27)
+				)
+			)
+		)
+		(pin "2"
+		)
+		(pin "1"
+		)
+		(instances
+			(project "ETH1CVOLT"
+				(path "/8d3b546e-b30b-49b2-bc59-8e254df4c067/ea97f94c-dee1-4702-bb32-5cb010d15929/e2cff0f2-156b-4ebd-b442-dc8733a740cb"
+					(reference "R63")
+					(unit 1)
+				)
