File: HARDWARE/ETH1CVOLT/ETH1CVOLT.kicad_sch (KiCad schematic)
At the start: 0 parts

Commit message: Development
Changed lines of the file:
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@@
 	(paper "A3")
 	(sheet
-		(at 203.2 127)
-		(size 25.4 17.78)
+		(at 328.93 212.09)
+		(size 48.26 30.48)
 		(exclude_from_sim no)
 		(in_bom yes)
@@
 		)
 		(property "Sheetname" "BLOCK DIAGRAM"
-			(at 203.2 126.2884 0)
+			(at 328.93 211.3784 0)
 			(show_name no)
 			(do_not_autoplace no)
@@
 		)
 		(property "Sheetfile" "Block_Diagram.kicad_sch"
-			(at 203.2 145.3646 0)
+			(at 328.93 243.1546 0)
 			(show_name no)
 			(do_not_autoplace no)

Commit message: Layout and schematic
Other:
- note added: "${PROJECTNAME}${REVISION}${VARIANT}"
- title: (none) -> ETH1CVOLT
Changed lines of the file:
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@@
 	(generator_version "10.0")
 	(paper "A3")
+	(title_block
+		(title "ETH1CVOLT")
+		(date "2026-09-19")
+		(rev "01")
+	)
+	(text "${PROJECTNAME}${REVISION}${VARIANT}"
+		(exclude_from_sim no)
+		(at 209.55 44.958 0)
+		(effects
+			(font
+				(size 12.7 12.7)
+				(thickness 2.54)
+				(bold yes)
+			)
+		)
+	)
 	(sheet
 		(at 328.93 212.09)

Commit message: Modifications
Changed lines of the file:
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@@
 	)
 	(sheet
-		(at 328.93 212.09)
-		(size 48.26 30.48)
+		(at 330.2 203.2)
+		(size 38.1 38.1)
 		(exclude_from_sim no)
 		(in_bom yes)
@@
 		)
 		(property "Sheetname" "BLOCK DIAGRAM"
-			(at 328.93 211.3784 0)
+			(at 330.2 202.4884 0)
 			(show_name no)
 			(do_not_autoplace no)
@@
 		)
 		(property "Sheetfile" "Block_Diagram.kicad_sch"
-			(at 328.93 243.1546 0)
+			(at 330.2 241.8846 0)
 			(show_name no)
 			(do_not_autoplace no)
