File: HARDWARE/ETH1CVOLT/Isolated_Power.kicad_sch (KiCad schematic)
At the start: 30 parts, among them U11 ADP7142ARDZ-5.0, U16 TEC2-2419WI, U17 TMR4-2423WI, U23 ADP7142ARDZ-5.0, U24 TPS7A39

Commit message: Development
Parts:
- removed R29: 1k4, Resistor_SMD:R_0603_1608Metric_Pad0.98x0.95mm_HandSolder, symbol Device:R
- removed R30: 174k, Resistor_SMD:R_0603_1608Metric_Pad0.98x0.95mm_HandSolder, symbol Device:R
- added C100, C56, C57, C58, C59, C65, C66, C67, C68, C69, C80, C81, C99: 10u/50V/X7R, Capacitor_SMD:C_1210_3225Metric_Pad1.33x2.70mm_HandSolder, symbol Device:C
- added C60, C61, C62, C63, C64, C70, C71, C72, C73, C74, C76, C77, C78, C93, C94: 4u7/50V/X7R, Capacitor_SMD:C_1210_3225Metric_Pad1.33x2.70mm_HandSolder, symbol Device:C
- added C75, C84: C, Capacitor_SMD:C_0603_1608Metric_Pad1.08x0.95mm_HandSolder, symbol Device:C
- added L1: RLS-226, symbol Device:L
- added L2, L3: TCK-154, symbol Device:L
- added R51: 12k/1%/100mW, Resistor_SMD:R_0603_1608Metric_Pad0.98x0.95mm_HandSolder, symbol Device:R
- added R52: 140k/1%/100mW, Resistor_SMD:R_0603_1608Metric_Pad0.98x0.95mm_HandSolder, symbol Device:R
- added R53: 160k/1%/100mW, Resistor_SMD:R_0603_1608Metric_Pad0.98x0.95mm_HandSolder, symbol Device:R
- added R54: 15k/1%/100mW, Resistor_SMD:R_0603_1608Metric_Pad0.98x0.95mm_HandSolder, symbol Device:R
- added R57: 18k/1%/100mW, Resistor_SMD:R_0603_1608Metric_Pad0.98x0.95mm_HandSolder, symbol Device:R
- added R58: 105k/1%/100mW, Resistor_SMD:R_0603_1608Metric_Pad0.98x0.95mm_HandSolder, symbol Device:R
- added R65: 107k/1%/100mW, Resistor_SMD:R_0603_1608Metric_Pad0.98x0.95mm_HandSolder, symbol Device:R
- added R66: 22k1/1%/100mW, Resistor_SMD:R_0603_1608Metric_Pad0.98x0.95mm_HandSolder, symbol Device:R
- added TP10, TP11, TP12, TP13, TP14, TP15, TP16, TP9: TestPoint, TestPoint:TestPoint_Pad_D1.5mm, symbol Connector:TestPoint
- added U15: RP-2424D, ETH1CVOLT_A:RP-xxxxD, symbol ETH1CVOLT_B:RP-xxxxD
- added U18: TSR0.5-2465, Converter_DCDC:Converter_DCDC_TRACO_TSR0.5-24xx_TSR0.5-24xxx_THT, symbol Converter_DCDC:TSR0.5-2465
- added U19, U23: TPS7A3901DSCR, Package_SON:Texas_S-PVSON-N10_ThermalVias, symbol Regulator_Linear:TPS7A39
- C79: renamed from C54; now left out of the parts list
- C82: renamed from C75; value 4u7/100V -> 4u7/50V/X7R
- C83: renamed from C80; value 4u7/100V -> 4u7/50V/X7R
- C85: renamed from C76; value 10u/100V -> 10u/50V/X7R
- C86: renamed from C81; value 10u/100V -> 10u/50V/X7R
- C87: renamed from C77; footprint (none) -> Capacitor_SMD:C_0603_1608Metric_Pad1.08x0.95mm_HandSolder; now left out of the parts list
- C88: renamed from C87; footprint (none) -> Capacitor_SMD:C_0603_1608Metric_Pad1.08x0.95mm_HandSolder; now left out of the parts list
- C89: renamed from C84; value 4u7/100V -> 4u7/50V/X7R
- C90: renamed from C86; value 4u7/100V -> 4u7/50V/X7R
- C91: renamed from C78; value 4u7/100V -> 4u7/50V/X7R
- C92: renamed from C82; value 4u7/100V -> 4u7/50V/X7R
- C95: renamed from C85; value 10u/100V -> 10u/50V/X7R
- C96: renamed from C88; value 10u/100V -> 10u/50V/X7R
- C97: renamed from C79; value 10u/100V -> 10u/50V/X7R
- C98: renamed from C83; value 10u/100V -> 10u/50V/X7R
- R55: renamed from R28; value 10k -> 10k2/1%/100mW
- R56: renamed from R32; value 2k4 -> 187k/1%/100mW
- R59: renamed from R27; value 165k -> 182k/1%/100mW
- R60: renamed from R31; value 10k -> 10k5/1%/100mW
- R61: renamed from R56; footprint (none) -> Resistor_SMD:R_0603_1608Metric_Pad0.98x0.95mm_HandSolder; now left out of the parts list
- R62: renamed from R57; footprint (none) -> Resistor_SMD:R_0603_1608Metric_Pad0.98x0.95mm_HandSolder; now left out of the parts list
- R63: renamed from R66; value 0 -> 0R/5%/100mW
- R64: renamed from R67; value 0 -> 0R/5%/100mW
- U20: renamed from U24; value TPS7A39 -> TPS7A3901DSCR
- renumbered U17 to U16, U16 to U17, U11 to U21, U23 to U22
Connections:
- net +5VA_ISO: now also TP13.1
- net +5VD_ISO: now also TP14.1
- net +7V_ISO: now also C93.1, C99.1, R65.1, TP15.1, U23.10 (OUTP); no longer C82.1, C83.1, C85.1, C86.1, U21.5 (EN), U21.7 (VIN), U21.8 (VIN), U22.5 (EN), U22.7 (VIN), U22.8 (VIN)
- net GND_ISO: now also U16.7 (Com), U17.7 (-Vout), C100.1, C65.2, C66.1, C67.2, C68.1, C69.2, C70.2, C71.1, C72.2, C73.1, C74.2, C75.2, C76.2, C77.2, C78.1, C80.2, C81.1, C84.2, C93.2, C94.1, C99.2, R54.2, R66.2, U15.6 (Com), U18.2 (GND), U19.11 (GND), U19.4 (GND), U23.11 (GND), U23.4 (GND)
- net at R56.1: now also R55.2, U20.7 (FBN)
- net at R59.2: now also R60.1, U20.9 (FBP)
- net GND: now reaches U16.1 (-Vin)
- net GND: now also U17.1 (-Vin), C56.2, C57.2, C58.2, C59.2, C60.2, C61.2, C62.2, C63.2, C64.2, U15.2 (-Vin)
- net at U16.2 (+Vin): now also C63.1, L2.2
- net +15V_ISO: now reaches U16.6 (+Vout)
- net +15V_ISO: now also C67.1, C72.1, TP9.1, U19.1 (INP), U19.2 (EN), U23.1 (INP), U23.2 (EN)
- net -15V_ISO: now reaches U16.8 (-Vout)
- net -15V_ISO: now also C68.2, C73.2, TP10.1, U19.5 (INN), U23.5 (INN)
- net at U17.2 (+Vin): now also C64.1, L3.2
- net at U17.6 (+Vout): now also C69.1, C74.1, U18.1 (Vin)
- net +24V_ISO: now reaches U20.1 (INP), U20.2 (EN)
- net +24V_ISO: now also C65.1, C70.1, U15.7 (+Vout)
- net -24V_ISO: now reaches U20.5 (INN)
- net -24V_ISO: now also C66.2, C71.2, U15.5 (-Vout)
- net +21V_ISO renamed +22V_ISO
- net -21V_ISO renamed -22V_ISO
- new net: R65.2, R66.1, U23.9 (FBP)
- new net: C84.1, U23.3 (NR/SS)
- new net: R57.2, R58.1, U23.7 (FBN)
- new net: R57.1, U23.8 (BUF)
- new net: R51.1, U19.8 (BUF)
- new net: R51.2, R52.1, U19.7 (FBN)
- new net: C59.1, C62.1, L1.2, U15.1 (+Vin)
- new net: R53.2, R54.1, U19.9 (FBP)
- new net: C75.1, U19.3 (NR/SS)
- new net +14V_ISO: C77.1, C80.1, R53.1, TP11.1, U19.10 (OUTP)
- new net +24V: C56.1, C57.1, C58.1, C60.1, C61.1, L1.1, L2.1, L3.1
- new net +6V5_ISO: C76.1, C82.1, C83.1, C85.1, C86.1, U18.3 (Vout), U21.5 (EN), U21.7 (VIN), U21.8 (VIN), U22.5 (EN), U22.7 (VIN), U22.8 (VIN)
- new net -14V_ISO: C78.2, C81.2, R52.2, TP12.1, U19.6 (OUTN)
- new net -7V_ISO: C100.2, C94.2, R58.2, TP16.1, U23.6 (OUTN)
Other:
- note added: "+14V/100mA"
- note added: "+22V/100mA"
- note added: "+6V5/500mA"
- note added: "+7V/100mA"
- note added: "-14V/100mA"
- note added: "-22V/100mA"
- note added: "-7V/100mA"
- note removed: "+21V/100mA"
- note removed: "+7V/300mA"
- note removed: "-21V/100mA"
- note removed: "RP-2424D"
- moved on the sheet: C79, C89, C90, C95, C96, R55, R56, R59, R60, U16, U17, U20

Commit message: Development
Parts:
- L1: footprint (none) -> ETH1CVOLT:RLS-226
- L2, L3: value TCK-154 -> 78438366047; footprint (none) -> ETH1CVOLT:78438366047
- U15: footprint ETH1CVOLT_A:RP-xxxxD -> ETH1CVOLT:RP-xxxxD
Other:
- moved on the sheet: C100, C57, C58, C60, C61, C63, C64, C67, C68, C69, C72, C73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

Commit message: Development
Parts:
- added TP31, TP32, TP33, TP35: TestPoint, TestPoint:TestPoint_Pad_D1.5mm, symbol Connector:TestPoint
- C75, C79, C84: now not fitted
- renumbered TP9 to TP27, TP10 to TP28, TP11 to TP29, TP12 to TP30, TP16 to TP34, TP13 to TP36, TP14 to TP37, TP15 to TP38
Connections:
- net +22V_ISO: now also TP35.1
- net -22V_ISO: now also TP33.1
- net GND_ISO: now also TP31.1, TP32.1
Other:
- moved on the sheet: C69, C74, C76, TP34, U18

Commit message: Development
Parts:
- added R59, R61: 560/1%/100mW, Resistor_SMD:R_0603_1608Metric_Pad0.98x0.95mm_HandSolder, symbol Device:R
- C100, C56, C57, C58, C59, C60, C61, C62, C63, C64, C65, C66, C67, C68, C69, C70, C71, C72, C73, C74, C76, C80, C81, C82, C83, C85, C86, C89, C90, C91, C92, C93, C94, C95, C96, C97, C98, C99: footprint Capacitor_SMD:C_1210_3225Metric_Pad1.33x2.70mm_HandSolder -> Capacitor_SMD:C_1206_3216Metric_Pad1.33x1.80mm_HandSolder
- C78: renamed from C77; footprint Capacitor_SMD:C_1210_3225Metric_Pad1.33x2.70mm_HandSolder -> Capacitor_SMD:C_1206_3216Metric_Pad1.33x1.80mm_HandSolder
- C79: renamed from C78; footprint Capacitor_SMD:C_1210_3225Metric_Pad1.33x2.70mm_HandSolder -> Capacitor_SMD:C_1206_3216Metric_Pad1.33x1.80mm_HandSolder
- R56: renamed from R55; value 10k2/1%/100mW -> 10k/1%/100mW
- R60: value 10k5/1%/100mW -> 10k/1%/100mW
- renumbered C79 to C77, R51 to R52, R52 to R53, R53 to R54, R54 to R55, R56 to R57, R59 to R58, R57 to R62, R58 to R63, R61 to R64, R62 to R65, R63 to R66, R64 to R67, R65 to R68, R66 to R69, TP33 to TP31, TP31 to TP32, TP32 to TP33, TP35 to TP34, TP34 to TP35
Connections:
- net at R58.2, U20.9 (FBP): now also R59.2, R61.2; no longer R60.1
- new net: R59.1, R60.1, R61.1
Other:
- moved on the sheet: C77, R56, R57, R58, R60, TP31, TP34, U20

Commit message: Layout
Parts:
- added TP27, TP28: TestPoint, TestPoint:TestPoint_Pad_D1.5mm, symbol Connector:TestPoint
- renumbered C56 to C54, C57 to C55, C58 to C56, C59 to C57, C60 to C58, C61 to C59, C62 to C60, C63 to C61, C64 to C62, C65 to C63, C66 to C64, C67 to C65, C68 to C66, C69 to C67, C70 to C68, C71 to C69, C72 to C70, C73 to C71, C74 to C72, C75 to C73, C76 to C74, C78 to C75, C79 to C76, C80 to C78, C81 to C79, C82 to C80, C83 to C81, C84 to C82, C85 to C83, C86 to C84, C87 to C85, C88 to C86, C89 to C87, C90 to C88, C91 to C89, C92 to C90, C93 to C91, C94 to C92, C95 to C93, C96 to C94, C97 to C95, C98 to C96, C99 to C97, C100 to C98, R52 to R51, R53 to R52, R54 to R53, R55 to R54, R56 to R55, R57 to R56, R58 to R57, R59 to R58, R60 to R59, R62 to R60, R63 to R61, R61 to R62, R64 to R63, R65 to R64, R66 to R65, R67 to R66, R68 to R67, R69 to R68, TP27 to TP29, TP28 to TP30, TP29 to TP31, TP30 to TP32, TP31 to TP33, TP32 to TP34, TP33 to TP35, TP34 to TP36, TP35 to TP37, TP36 to TP38, TP37 to TP39, TP38 to TP40
Connections:
- net +24V_ISO: now also TP27.1
- net -24V_ISO: now also TP28.1

Commit message: Layout and schematic
Parts:
- renumbered C97 to C100, C98 to C101, C54 to C57, C55 to C58, C56 to C59, C57 to C60, C58 to C61, C59 to C62, C60 to C63, C61 to C64, C62 to C65, C63 to C66, C64 to C67, C65 to C68, C66 to C69, C67 to C70, C68 to C71, C69 to C72, C70 to C73, C71 to C74, C72 to C75, C73 to C76, C74 to C77, C75 to C78, C76 to C79, C77 to C80, C78 to C81, C79 to C82, C80 to C83, C81 to C84, C82 to C85, C83 to C86, C84 to C87, C85 to C88, C86 to C89, C87 to C90, C88 to C91, C89 to C92, C90 to C93, C91 to C94, C92 to C95, C93 to C96, C94 to C97, C95 to C98, C96 to C99, R51 to R37, R52 to R38, R53 to R39, R54 to R40, R55 to R41, R56 to R42, R57 to R43, R58 to R44, R59 to R45, R60 to R46, R61 to R47, R62 to R48, R63 to R49, R64 to R50, R67 to R51, R68 to R52, R65 to R53, R66 to R54, TP27 to TP24, TP28 to TP25, TP29 to TP26, TP30 to TP27, TP31 to TP28, TP32 to TP29, TP33 to TP30, TP34 to TP31, TP35 to TP32, TP36 to TP33, TP37 to TP34, TP38 to TP35, TP39 to TP36, TP40 to TP37
Other:
- note added: "+5V28/200mA"
- title: (none) -> ETH1CVOLT
- moved on the sheet: C83, C84, C86, C87, C88, C89, C92, C93, C98, C99, R49, R50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

Commit message: Verification
Parts:
- added TP42, TP43: TestPoint, TestPoint:TestPoint_Pad_D1.5mm, symbol Connector:TestPoint
- C100: renamed from C101; value 10u/50V/X7R -> 10u/35V/X7R
- C101: renamed from C98; value 10u/50V/X7R -> 10u/35V/X7R
- C102: renamed from C99; value 10u/50V/X7R -> 10u/35V/X7R
- C58: renamed from C57; value 10u/50V/X7R -> 10u/35V/X7R
- C59: renamed from C58; value 10u/50V/X7R -> 10u/35V/X7R
- C60: renamed from C59; value 10u/50V/X7R -> 10u/35V/X7R
- C61: renamed from C60; value 10u/50V/X7R -> 10u/35V/X7R
- C67: renamed from C66; value 10u/50V/X7R -> 10u/35V/X7R
- C68: renamed from C67; value 10u/50V/X7R -> 10u/35V/X7R
- C69: renamed from C68; value 10u/50V/X7R -> 10u/35V/X7R
- C70: renamed from C69; value 10u/50V/X7R -> 10u/35V/X7R
- C71: renamed from C70; value 10u/50V/X7R -> 10u/35V/X7R
- C82: renamed from C81; value 10u/50V/X7R -> 10u/35V/X7R
- C83: renamed from C82; value 10u/50V/X7R -> 10u/35V/X7R
- C87: renamed from C86; value 10u/50V/X7R -> 10u/35V/X7R
- C88: renamed from C87; value 10u/50V/X7R -> 10u/35V/X7R
- C97: renamed from C96; value 10u/50V/X7R -> 10u/35V/X7R
- C98: renamed from C97; value 10u/50V/X7R -> 10u/35V/X7R
- C99: renamed from C100; value 10u/50V/X7R -> 10u/35V/X7R
- R49: value R -> 10k/1%/100mW; now fitted
- R53: value 0R/5%/100mW -> 560/1%/100mW
- renumbered C61 to C62, C62 to C63, C63 to C64, C64 to C65, C65 to C66, C71 to C72, C72 to C73, C73 to C74, C74 to C75, C75 to C76, C76 to C77, C77 to C78, C78 to C79, C79 to C80, C80 to C81, C83 to C84, C84 to C85, C85 to C86, C88 to C89, C89 to C90, C90 to C91, C91 to C92, C92 to C93, C93 to C94, C94 to C95, C95 to C96, U23 to U21, U21 to U22, U22 to U23
Connections:
- net +6V5_ISO: now also TP43.1
- net at C71.1, C76.1, U17.6 (+Vout)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: now also TP42.1
Other:
- moved on the sheet: C78

Commit message: Modifications
Other:
- moved on the sheet: C102, C85, C88, C90, C94, R50, R54, TP32, TP36, U23
