File: HARDWARE/ETH1CVOLT/Isolated_Power.kicad_sch (KiCad schematic)
At the start: 91 parts, among them U15 RP-2424D, U16 TMR4-2423WI, U17 TEC2-2419WI, U18 TSR0.5-2465, U19 TPS7A3901DSCR, U20 TPS7A3901DSCR, U21 TPS7A3901DSCR, U22 ADP7142ARDZ-5.0, U23 ADP7142ARDZ-5.0

Commit message: HW design done
Parts:
- R50: value R -> 10k/1%/100mW; now fitted; now in the parts list
- R54: value 0R/5%/100mW -> 560/1%/100mW
Other:
- note added: "+15V/133mA"
- note added: "+24V/21mA"
- note added: "+9V/222mA"
- note added: "-15V/133mA"
- note added: "-24V/21mA"
- note removed: "+5V/200mA"
- moved on the sheet: C101, C72, C73, C74, C75, C77, C78, C79, C80, C81, C82, C83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

Commit message: Ethernet works under NetXDuo. Use MPU 0x24000000 range, never 0x30040000, like some example show. SRAM3 will not work.
Parts:
- R49: now in the parts list
Changed lines of the file:
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@@
 		(body_style 1)
 		(exclude_from_sim no)
-		(in_bom no)
+		(in_bom yes)
 		(on_board yes)
 		(in_pos_files yes)
@@
 					(variant
 						(name "A")
+						(in_bom no)
 						(field
 							(name "Value")
