File: HARDWARE/ETH1CVOLT/Output.kicad_sch (KiCad schematic)
At the start: 8 parts, among them J6 FCR7350R, J8 FCR7350B, K1 SILxx-1Cxx-51x, Q3 2N7002

Commit message: Development
Parts:
- removed R22: 1k/1%/100mW, Package_SO:TSSOP-16_4.4x5mm_P0.65mm, symbol Device:R
- added C105, C106, C107: 0.1u/100V/X7R, Capacitor_SMD:C_0603_1608Metric_Pad1.08x0.95mm_HandSolder, symbol Device:C
- added D8: 1N4148W, Diode_SMD:D_SOD-123, symbol Diode:1N4148W
- added J10, J11, J12, J13, J14, J15, J16, J17, J18, J8: 5050462-2, Connector_RJ:RJ45_Wuerth_7499010121A_Horizontal, symbol Connector:Conn_01x01_Socket
- added K2: SIL05-1C90-51D, Relay_THT:Relay_SPDT_StandexMeder_SIL_Form1C, symbol Relay:SILxx-1Cxx-51x
- added Q3: 2N7002, Package_TO_SOT_SMD:SOT-23, symbol Transistor_FET:2N7002
- added R311: 10k/1%/100mW, Resistor_SMD:R_0603_1608Metric_Pad0.98x0.95mm_HandSolder, symbol Device:R
- added R67: 100/1%/100mW, Resistor_SMD:R_0603_1608Metric_Pad0.98x0.95mm_HandSolder, symbol Device:R
- added R69, R71: 10k/0.01%/100mW, Resistor_SMD:R_0603_1608Metric_Pad0.98x0.95mm_HandSolder, symbol Device:R
- added R70: 1k/1%/100mW, Package_SO:TSSOP-16_4.4x5mm_P0.65mm, symbol Device:R
- added U25: ADA4522-2ARZ-RL, Package_SO:SOIC-8_3.9x4.9mm_P1.27mm, symbol Amplifier_Operational:ADA4522-2
- added U26: 74LV1T08GV, Package_TO_SOT_SMD:SC-74A-5_1.55x2.9mm_P0.95mm, symbol 74xx:74LV1T08GV
- K1: value SILxx-1Cxx-51x -> SIL05-1C90-51D
- renumbered D5 to D7, D6 to D9, J8 to J7, Q3 to Q2, R26 to R68
Connections:
- net +5VD_ISO: now also C107.1, D8.1 (K), K2.3, U26.5 (VCC)
- net GND_ISO: now also C105.2, C106.2, C107.2, Q3.2 (S), R311.2, R69.2, U26.3 (GND)
- net REL_RANGE_SEL: now also R311.1, U26.1 (B), U26.2 (A); no longer R68.1
- net at D9.2 (A2), J6.1 (Pin_1), K1.7: now also U25.3 (+)
- new net: R67.1, U25.6 (-), U25.7
- new net: D8.2 (A), K2.5, Q3.3 (D)
- new net: Q3.1 (G), R70.2
- new net: K2.7, U25.5 (+)
- new net +22V_ISO: C105.1, U25.8 (V+)
- new net -22V_ISO: C106.1, U25.4 (V-)
- new net MEAS_OUT: R67.2
- new net MEAS_R10V: K2.2, R71.1, U25.1, U25.2 (-)
- new net MEAS_R20V: K2.1, R69.1, R71.2
- new net REL_RNG_SEL: R68.1, R70.1, U26.4 (Y)
- no-connect marks 0 -> 10
Other:
- moved on the sheet: D7, D9, J6, J7, K1, Q2, R68

Commit message: Development
Parts:
- removed D8: 1N4148W, Diode_SMD:D_SOD-123, symbol Diode:1N4148W
- removed J10, J11, J12, J13, J14, J15, J16, J17, J18, J8: 5050462-2, Connector_RJ:RJ45_Wuerth_7499010121A_Horizontal, symbol Connector:Conn_01x01_Socket
- removed K1, K2: SIL05-1C90-51D, Relay_THT:Relay_SPDT_StandexMeder_SIL_Form1C, symbol Relay:SILxx-1Cxx-51x
- added C108: 0.1u/100V/X7R, Capacitor_SMD:C_0603_1608Metric_Pad1.08x0.95mm_HandSolder, symbol Device:C
- added D10: 1N4148W, Diode_SMD:D_SOD-123, symbol Diode:1N4148W
- added K4: G6SK-2F DC5, Relay_SMD:Relay_DPDT_Omron_G6SK-2F, symbol Relay:G6SK-2
- added R312: 10k/1%/100mW, Resistor_SMD:R_0603_1608Metric_Pad0.98x0.95mm_HandSolder, symbol Device:R
- added U27: 74LV1T08GV, Package_TO_SOT_SMD:SC-74A-5_1.55x2.9mm_P0.95mm, symbol 74xx:74LV1T08GV
- J6, J7: footprint ETH1CVOLT_A:S16N-PC -> ETH1CVOLT:S16N-PC
- R68, R70: footprint Package_SO:TSSOP-16_4.4x5mm_P0.65mm -> Resistor_SMD:R_0603_1608Metric_Pad0.98x0.95mm_HandSolder
Connections:
- net +5VD_ISO: now also C108.1, D10.1 (K), K4.1, K4.6, U27.5 (VCC)
- net GND_ISO: now also R69.1, C108.2, R312.2, U27.3 (GND); no longer R69.2
- net MEAS_R10V: now also K4.3
- net MEAS_R20V: now also R69.2, K4.5; no longer R69.1
- net R10V_SIG: now also K4.10
- net R20V_SIG: now also K4.8
- net RELAY_RESET: now reaches D7.2 (A)
- net RELAY_RESET: now also Q3.3 (D), K4.7; no longer Q2.3 (D)
- net at U25.5 (+): now also K4.4
- net at D9.2 (A2), J6.1 (Pin_1), U25.3 (+): now also K4.9
- net REL_RANGE_SEL renamed REL_SET
- net REL_RNG_SEL: no longer names the net of R68.1, U26.4 (Y)
- net REL_RNG_SEL: no longer R70.1
- new net: R70.1, U27.4 (Y)
- new net RELAY_SET: D10.2 (A), K4.12, Q2.3 (D)
- new net REL_RESET: R312.1, U27.1 (B), U27.2 (A)
- no-connect marks 10 -> 0
Other:
- note added: "OUTPUT RELAY"
- note added: "RELAY CONTROL"
- moved on the sheet: C105, C106, C107, D7, D9, J6, J7, Q2, R311, R67, R68, R69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

Commit message: Development
Parts:
- added TP40, TP41, TP42, TP43, TP44: TestPoint, TestPoint:TestPoint_Pad_D1.5mm, symbol Connector:TestPoint
- renumbered D10 to D8, J6 to J7, J7 to J8, K4 to K1, R311 to R67, R71 to R70, R67 to R71, R312 to R72, R70 to R73
Connections:
- net MEAS_R10V: now also TP42.1
- net MEAS_R20V: now also TP40.1
- net RELAY_RESET: now also TP44.1
- net RELAY_SET: now also TP41.1
- net at D9.2 (A2), J7.1 (Pin_1), K1.9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: now also TP43.1

Commit message: Development
Parts:
- D9: now not fitted
- renumbered R67 to R70, R68 to R71, R69 to R72, R70 to R73, R71 to R74, R72 to R75, R73 to R76
Other:
- moved on the sheet: R72, R73

Commit message: Layout
Parts:
- removed TP41, TP44: TestPoint, TestPoint:TestPoint_Pad_D1.5mm, symbol Connector:TestPoint
- renumbered C105 to C103, C106 to C104, C107 to C105, C108 to C106, D9 to D10, D7 to D8, D8 to D9, R70 to R69, R71 to R70, R72 to R71, R73 to R72, R74 to R73, R75 to R74, R76 to R75, TP40 to TP42, TP42 to TP43, TP43 to TP44

Commit message: Layout and schematic
Parts:
- renumbered C103 to C106, C104 to C107, C105 to C108, C106 to C109, J7 to J5, J8 to J6, R69 to R55, R70 to R56, R71 to R57, R72 to R58, R73 to R59, R74 to R60, R75 to R61, TP42 to TP39, TP43 to TP40, TP44 to TP41
Other:
- title: (none) -> ETH1CVOLT

Commit message: Verification
Parts:
- renumbered C106 to C107, C107 to C108, C108 to C109, C109 to C110, J5 to J7, J6 to J8

Commit message: Modifications
Parts:
- added C111: 0.1u/100V/X7R, Capacitor_SMD:C_0603_1608Metric_Pad1.08x0.95mm_HandSolder, symbol Device:C
- added D11: APFA3010LSEEZGKQBKC, LED_SMD:LED_Kingbright_APFA3010_3x1.5mm_Horizontal, symbol LED:APFA3010
- added R64, R65: 1k/1%/100mW, Resistor_SMD:R_0603_1608Metric_Pad0.98x0.95mm_HandSolder, symbol Device:R
- added R66: 560/1%/100mW, Resistor_SMD:R_0603_1608Metric_Pad0.98x0.95mm_HandSolder, symbol Device:R
- added U28: 74LVC2G74DP, Package_SO:TSSOP-8_3x3mm_P0.65mm, symbol 74xGxx:74LVC2G74
Connections:
- net +5VD_ISO: now also C111.1, R66.1, U28.8 (VCC)
- net GND_ISO: now also C111.2, U28.1 (C), U28.2 (D), U28.4 (GND)
- net at R56.1, U26.4 (Y): now also R64.1
- net at R61.1, U27.4 (Y): now also R65.1
- new net: D11.2 (A), R66.2
- new net: D11.4 (B), U28.3 (~{Q})
- new net: D11.1 (R), U28.5 (Q)
- new net STAT_RESET: R65.2, U28.6 (~{CLR})
- new net STAT_SET: R64.2, U28.7 (~{PRE})
- no-connect marks 0 -> 1
Other:
- note added: "RELAY STATUS LEDS"
- moved on the sheet: Q2, Q3, R55, R56, R60, R61, U26, U27
