File: HARDWARE/ETH1CVOLT/Power.kicad_sch (KiCad schematic)
At the start: 11 parts, among them J3 1715721, Q1 CSD18501Q5A

Commit message: Development
Parts:
- removed C37, C38: 2,2uF/50V/X7R, Capacitor_SMD:C_0805_2012Metric_Pad1.18x1.45mm_HandSolder, symbol Device:C
- added C54: 10u/50V/X7R, Capacitor_SMD:C_1210_3225Metric_Pad1.33x2.70mm_HandSolder, symbol Device:C
- added C55: 4u7/50V/X7R, Capacitor_SMD:C_1210_3225Metric_Pad1.33x2.70mm_HandSolder, symbol Device:C
- added J9: 1827703, symbol Connector_Generic:Conn_01x02
- C53: renamed from C36; value 10uF/50V/X7R -> 10u/50V/X7R
- D5: renamed from D2; value LED -> SML-A12UTT86
- J5: renamed from J3; value 1715721 -> 1827868; footprint TerminalBlock_Phoenix:TerminalBlock_Phoenix_MKDS-1,5-2-5.08_1x02_P5.08mm_Horizontal -> Connector_Phoenix_MC:PhoenixContact_MC_1,5_2-GF-3.81_1x02_P3.81mm_Horizontal_ThreadedFlange_MountHole
- renumbered D3 to D4, D4 to D6, R23 to R48, R24 to R49, R25 to R50
Connections:
- net +24V: now also C54.1, C55.1
- net GND: now also C54.2, C55.2
- no-connect marks 0 -> 2
Other:
- moved on the sheet: C53, D4, D5, D6, J5, Q1, R48, R49, R50

Commit message: Development
Parts:
- added TP24, TP25, TP26: TestPoint, TestPoint:TestPoint_Pad_D1.5mm, symbol Connector:TestPoint
- renumbered J9 to J5, J5 to J6
Connections:
- net +24V: now also TP25.1
- net GND: now also TP26.1
- net at J6.1 (Pin_1), Q1.5 (D): now also TP24.1

Commit message: Development
Parts:
- removed R49: 2k/1%/100mW, Resistor_SMD:R_0603_1608Metric_Pad0.98x0.95mm_HandSolder, symbol Device:R
- added R51: 2k67/1%/250mW, Resistor_SMD:R_0805_2012Metric_Pad1.20x1.40mm_HandSolder, symbol Device:R
- C53, C54, C55: footprint Capacitor_SMD:C_1210_3225Metric_Pad1.33x2.70mm_HandSolder -> Capacitor_SMD:C_1206_3216Metric_Pad1.33x1.80mm_HandSolder
- R50: value 2k/1%/100mW -> 2k67/1%/250mW; footprint Resistor_SMD:R_0603_1608Metric_Pad0.98x0.95mm_HandSolder -> Resistor_SMD:R_0805_2012Metric_Pad1.20x1.40mm_HandSolder
- renumbered R48 to R49
Connections:
- net GND: now also R51.2; no longer R50.2
- net at R50.1: now also D6.2 (A)
- new net: R50.2, R51.1

Commit message: Layout
Connections:
- net +24V: now also J6.1 (Pin_1); no longer J6.2 (Pin_2)
- net at Q1.5 (D), TP24.1: now also J6.2 (Pin_2); no longer J6.1 (Pin_1)
Other:
- moved on the sheet: J6
Changed lines of the file:
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@@
 	(symbol
 		(lib_id "Connector_Generic:Conn_01x02")
-		(at 59.69 114.3 180)
+		(at 59.69 111.76 0)
+		(mirror y)
 		(unit 1)
 		(body_style 1)
@@
 		(dnp no)
 		(property "Reference" "J6"
-			(at 56.642 111.252 0)
+			(at 56.388 111.76 0)
 			(show_name no)
 			(do_not_autoplace no)
@@
 		)
 		(property "Value" "1827868"
-			(at 56.896 114.3 0)
+			(at 56.642 114.3 0)
 			(show_name no)
 			(do_not_autoplace no)
@@
 		)
 		(property "Footprint" "Connector_Phoenix_MC:PhoenixContact_MC_1,5_2-GF-3.81_1x02_P3.81mm_Horizontal_ThreadedFlange_MountHole"
-			(at 59.69 114.3 0)
+			(at 59.69 111.76 0)
 			(hide yes)
 			(show_name no)
@@
 		)
 		(property "Datasheet" ""
-			(at 59.69 114.3 0)
+			(at 59.69 111.76 0)
 			(hide yes)
 			(show_name no)
@@
 		)
 		(property "Description" "Generic connector, single row, 01x02, script generated (kicad-library-utils/schlib/autogen/connector/)"
-			(at 59.69 114.3 0)
+			(at 59.69 111.76 0)
 			(hide yes)
 			(show_name no)

Commit message: Layout
Parts:
- removed C53: 10u/50V/X7R, Capacitor_SMD:C_1206_3216Metric_Pad1.33x1.80mm_HandSolder, symbol Device:C
- renumbered C54 to C52, C55 to C53, D4 to D5, D5 to D6, D6 to D7, R49 to R48, R50 to R49, R51 to R50

Commit message: Layout and schematic
Parts:
- renumbered C52 to C55, C53 to C56, J5 to J3, J6 to J4, R48 to R34, R49 to R35, R50 to R36, TP24 to TP21, TP25 to TP22, TP26 to TP23
Other:
- title: (none) -> ETH1CVOLT

Commit message: Verification
Parts:
- C56: renamed from C55; value 10u/50V/X7R -> 10u/35V/X7R
- renumbered C56 to C57, J3 to J5, J4 to J6
Changed lines of the file:
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@@
 		(dnp no)
 		(fields_autoplaced yes)
-		(property "Reference" "#PWR0148"
+		(property "Reference" "#PWR0150"
 			(at 181.61 149.86 0)
 			(hide yes)
@@
 			(project "ETH1CVOLT"
 				(path "/8d3b546e-b30b-49b2-bc59-8e254df4c067/ea97f94c-dee1-4702-bb32-5cb010d15929/85462291-6d94-451a-96ab-b2477caf0aa9"
-					(reference "#PWR0148")
+					(reference "#PWR0150")
 					(unit 1)
 				)
@@
 		(in_pos_files yes)
 		(dnp no)
-		(property "Reference" "J4"
+		(property "Reference" "J6"
 			(at 56.388 111.76 0)
 			(show_name no)
@@
 			(project "ETH1CVOLT"
 				(path "/8d3b546e-b30b-49b2-bc59-8e254df4c067/ea97f94c-dee1-4702-bb32-5cb010d15929/85462291-6d94-451a-96ab-b2477caf0aa9"
-					(reference "J4")
+					(reference "J6")
 					(unit 1)
 				)
@@
 		(dnp no)
 		(fields_autoplaced yes)
-		(property "Reference" "#PWR0147"
+		(property "Reference" "#PWR0149"
 			(at 181.61 113.03 0)
 			(hide yes)
@@
 			(project "ETH1CVOLT"
 				(path "/8d3b546e-b30b-49b2-bc59-8e254df4c067/ea97f94c-dee1-4702-bb32-5cb010d15929/85462291-6d94-451a-96ab-b2477caf0aa9"
-					(reference "#PWR0147")
+					(reference "#PWR0149")
 					(unit 1)
 				)
@@
 		(dnp no)
 		(fields_autoplaced yes)
-		(property "Reference" "C55"
+		(property "Reference" "C56"
 			(at 163.83 125.7299 0)
 			(show_name no)
@@
 			)
 		)
-		(property "Value" "10u/50V/X7R"
+		(property "Value" "10u/35V/X7R"
 			(at 163.83 128.2699 0)
 			(show_name no)
@@
 			(project "ETH1CVOLT"
 				(path "/8d3b546e-b30b-49b2-bc59-8e254df4c067/ea97f94c-dee1-4702-bb32-5cb010d15929/85462291-6d94-451a-96ab-b2477caf0aa9"
-					(reference "C55")
+					(reference "C56")
 					(unit 1)
 					(variant
@@
 		(dnp no)
 		(fields_autoplaced yes)
-		(property "Reference" "C56"
+		(property "Reference" "C57"
 			(at 185.42 125.7299 0)
 			(show_name no)
@@
 			(project "ETH1CVOLT"
 				(path "/8d3b546e-b30b-49b2-bc59-8e254df4c067/ea97f94c-dee1-4702-bb32-5cb010d15929/85462291-6d94-451a-96ab-b2477caf0aa9"
-					(reference "C56")
+					(reference "C57")
 					(unit 1)
 				)
@@
 		(dnp no)
 		(fields_autoplaced yes)
-		(property "Reference" "#FLG07"
+		(property "Reference" "#FLG08"
 			(at 160.02 108.585 0)
 			(hide yes)
@@
 			(project "ETH1CVOLT"
 				(path "/8d3b546e-b30b-49b2-bc59-8e254df4c067/ea97f94c-dee1-4702-bb32-5cb010d15929/85462291-6d94-451a-96ab-b2477caf0aa9"
-					(reference "#FLG07")
+					(reference "#FLG08")
 					(unit 1)
 				)
@@
 		(in_pos_files yes)
 		(dnp no)
-		(property "Reference" "J3"
+		(property "Reference" "J5"
 			(at 37.338 111.252 0)
 			(show_name no)
@@
 			(project "ETH1CVOLT"
 				(path "/8d3b546e-b30b-49b2-bc59-8e254df4c067/ea97f94c-dee1-4702-bb32-5cb010d15929/85462291-6d94-451a-96ab-b2477caf0aa9"
-					(reference "J3")
+					(reference "J5")
 					(unit 1)
 				)

Commit message: Modifications
Parts:
- removed D6: SML-A12UTT86, LED_SMD:LED_0603_1608Metric_Pad1.05x0.95mm_HandSolder, symbol Device:LED
- added D6: APFA3010LSEEZGKQBKC, LED_SMD:LED_Kingbright_APFA3010_3x1.5mm_Horizontal, symbol LED:APFA3010
Connections:
- net +24V: now also D6.2 (A)
- net at D7.1 (K): now also D6.1 (R)
- no-connect marks 2 -> 4
Other:
- moved on the sheet: C56, C57, D5, D7, Q1, R34, R35, R36, TP21, TP23
