File: HARDWARE/ETH1CVOLT/Power.kicad_sch (KiCad schematic)
At the start: 14 parts, among them J5 1827703, J6 1827868, Q1 CSD18501Q5A

Commit message: HW design done
Other:
- moved on the sheet: D7, R35
Changed lines of the file:
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@@
 	(wire
 		(pts
-			(xy 109.22 124.46) (xy 109.22 128.27)
+			(xy 109.22 124.46) (xy 109.22 125.73)
 		)
 		(stroke
@@
 	(wire
 		(pts
+			(xy 109.22 133.35) (xy 109.22 134.62)
+		)
+		(stroke
+			(width 0)
+			(type default)
+		)
+	)
+	(wire
+		(pts
 			(xy 71.12 134.62) (xy 71.12 138.43)
 		)
@@
 		(pts
 			(xy 71.12 111.76) (xy 71.12 127)
+		)
+		(stroke
+			(width 0)
+			(type default)
+		)
+	)
+	(wire
+		(pts
+			(xy 109.22 142.24) (xy 109.22 143.51)
 		)
 		(stroke
@@
 	(symbol
 		(lib_id "Device:R")
-		(at 109.22 139.7 0)
+		(at 109.22 138.43 0)
 		(unit 1)
 		(body_style 1)
@@
 		(fields_autoplaced yes)
 		(property "Reference" "R35"
-			(at 111.76 138.4299 0)
+			(at 111.76 137.1599 0)
 			(show_name no)
 			(do_not_autoplace no)
@@
 		)
 		(property "Value" "2k67/1%/250mW"
-			(at 111.76 140.9699 0)
+			(at 111.76 139.6999 0)
 			(show_name no)
 			(do_not_autoplace no)
@@
 		)
 		(property "Footprint" "Resistor_SMD:R_0805_2012Metric_Pad1.20x1.40mm_HandSolder"
-			(at 107.442 139.7 90)
+			(at 107.442 138.43 90)
 			(hide yes)
 			(show_name no)
@@
 		)
 		(property "Datasheet" ""
-			(at 109.22 139.7 0)
+			(at 109.22 138.43 0)
 			(hide yes)
 			(show_name no)
@@
 		)
 		(property "Description" "Resistor"
-			(at 109.22 139.7 0)
+			(at 109.22 138.43 0)
 			(hide yes)
 			(show_name no)
@@
 		)
 		(property "Sim.Type" ""
-			(at 109.22 139.7 0)
+			(at 109.22 138.43 0)
 			(hide yes)
 			(show_name no)
@@
 		)
 		(property "KLC_S4.5" ""
-			(at 109.22 139.7 0)
+			(at 109.22 138.43 0)
 			(hide yes)
 			(show_name no)
@@
 	(symbol
 		(lib_id "Diode:DZ2S100X0L")
-		(at 109.22 132.08 270)
+		(at 109.22 129.54 270)
 		(unit 1)
 		(body_style 1)
@@
 		(fields_autoplaced yes)
 		(property "Reference" "D7"
+			(at 111.76 128.2699 90)
+			(show_name no)
+			(do_not_autoplace no)
+			(effects
+				(font
+					(size 1.27 1.27)
+				)
+				(justify left)
+			)
+		)
+		(property "Value" "MMSZ5240C-HE3_A-08"
 			(at 111.76 130.8099 90)
 			(show_name no)
@@
 			)
 		)
-		(property "Value" "MMSZ5240C-HE3_A-08"
-			(at 111.76 133.3499 90)
-			(show_name no)
-			(do_not_autoplace no)
-			(effects
-				(font
-					(size 1.27 1.27)
-				)
-				(justify left)
-			)
-		)
 		(property "Footprint" "Diode_SMD:D_SOD-123"
-			(at 104.775 132.08 0)
+			(at 104.775 129.54 0)
 			(hide yes)
 			(show_name no)
@@
 		)
 		(property "Datasheet" "https://www.vishay.com/docs/86348/mmsz5225-g_to_mmsz5267-g.pdf"
-			(at 109.22 132.08 0)
+			(at 109.22 129.54 0)
 			(hide yes)
 			(show_name no)
@@
 		)
 		(property "Description" "Small Signal Zener Diodes"
-			(at 109.22 132.08 0)
+			(at 109.22 129.54 0)
 			(hide yes)
 			(show_name no)
@@
 		)
 		(property "Sim.Type" ""
-			(at 109.22 132.08 90)
+			(at 109.22 129.54 90)
 			(hide yes)
 			(show_name no)
@@
 		)
 		(property "KLC_S4.5" ""
-			(at 109.22 132.08 90)
-			(hide yes)
-			(show_name no)
+			(at 109.22 129.54 90)
+			(hide yes)
+			(show_name no)
