File: HARDWARE/ETH1CVOLT/ADC.kicad_sch (KiCad schematic)
At the start: 20 parts, among them U6 LTC2400CS8#TRPBF, U7 INA159AIDGKT, U8 ADG419BR, U9 DG412xUE

Commit message: Development
Parts:
- removed R33: 1k/1%/100mW, Package_SO:TSSOP-16_4.4x5mm_P0.65mm, symbol Device:R
- removed U8: ADG419BR, Package_SO:SOIC-8_3.9x4.9mm_P1.27mm, symbol Analog_Switch:ADG419BR
- added C33, C34: 0.1u/100V/X7R, Capacitor_SMD:C_0603_1608Metric_Pad1.08x0.95mm_HandSolder, symbol Device:C
- added D1: BAV199, Package_TO_SOT_SMD:SOT-23, symbol Diode:BAV99
- C35: renamed from C29; value 10u/35V/X7R -> 10u/50V/X7R; footprint Capacitor_SMD:C_0805_2012Metric_Pad1.18x1.45mm_HandSolder -> Capacitor_SMD:C_1210_3225Metric_Pad1.33x2.70mm_HandSolder
- renumbered C30 to C29, C31 to C30, C32 to C31, C33 to C32, D1 to D2, R59 to R12, R58 to R13, R21 to R15, R15 to R16, R13 to R17, R12 to R18, TP7 to TP1, TP1 to TP2, U7 to U4, U9 to U5
Connections:
- net +VD_ISO is gone; now on net +5VD_ISO: R18.1
- net GND_ISO: now also C33.2, C34.2
- net MEAS_OUT: now reaches R12.2, U4.3 (+)
- net MEAS_OUT: now also D1.3 (K)
- net +14V_ISO: now reaches U5.13 (V+)
- net +14V_ISO: now also C33.1, D1.2 (A)
- net -14V_ISO: now reaches U5.4 (V-)
- net -14V_ISO: now also C34.1, D1.1 (K)
Other:
- moved on the sheet: C35, D2, R12, R13, R14, R15, R16, R17, R18, TP1, TP2, U4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

Commit message: Development
Parts:
- R12, R13: footprint Resistor_SMD:R_0603_1608Metric -> Resistor_SMD:R_0603_1608Metric_Pad0.98x0.95mm_HandSolder
- R14, R15: footprint Package_SO:TSSOP-16_4.4x5mm_P0.65mm -> Resistor_SMD:R_0603_1608Metric_Pad0.98x0.95mm_HandSolder
Changed lines of the file:
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@@
 			)
 		)
-		(property "Footprint" "Resistor_SMD:R_0603_1608Metric"
+		(property "Footprint" "Resistor_SMD:R_0603_1608Metric_Pad0.98x0.95mm_HandSolder"
 			(at 116.332 87.63 90)
 			(hide yes)
@@
 			)
 		)
-		(property "Footprint" "Package_SO:TSSOP-16_4.4x5mm_P0.65mm"
+		(property "Footprint" "Resistor_SMD:R_0603_1608Metric_Pad0.98x0.95mm_HandSolder"
 			(at 196.85 118.618 90)
 			(hide yes)
@@
 			)
 		)
-		(property "Footprint" "Resistor_SMD:R_0603_1608Metric"
+		(property "Footprint" "Resistor_SMD:R_0603_1608Metric_Pad0.98x0.95mm_HandSolder"
 			(at 116.332 77.47 90)
 			(hide yes)
@@
 			)
 		)
-		(property "Footprint" "Package_SO:TSSOP-16_4.4x5mm_P0.65mm"
+		(property "Footprint" "Resistor_SMD:R_0603_1608Metric_Pad0.98x0.95mm_HandSolder"
 			(at 182.88 168.148 90)
 			(hide yes)

Commit message: Development
Parts:
- added TP1, TP2: TestPoint, TestPoint:TestPoint_Pad_D1.5mm, symbol Connector:TestPoint
- R15, R17: now not fitted
- renumbered TP1 to TP3, TP2 to TP4
Connections:
- net MEAS_OUT: now also TP1.1
- net at R12.1, R13.2, R15.1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: now also TP2.1
Changed lines of the file:
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@@
 	)
 	(junction
+		(at 53.34 138.43)
+		(diameter 0)
+		(color 0 0 0 0)
+	)
+	(junction
 		(at 186.69 130.81)
 		(diameter 0)
@@
 	)
 	(junction
+		(at 153.67 82.55)
+		(diameter 0)
+		(color 0 0 0 0)
+	)
+	(junction
 		(at 63.5 138.43)
 		(diameter 0)
@@
 	(wire
 		(pts
+			(xy 153.67 81.28) (xy 153.67 82.55)
+		)
+		(stroke
+			(width 0)
+			(type default)
+		)
+	)
+	(wire
+		(pts
 			(xy 204.47 130.81) (xy 215.9 130.81)
 		)
@@
 	(wire
 		(pts
+			(xy 53.34 137.16) (xy 53.34 138.43)
+		)
+		(stroke
+			(width 0)
+			(type default)
+		)
+	)
+	(wire
+		(pts
 			(xy 382.27 134.62) (xy 381 134.62)
 		)
@@
 		(in_pos_files yes)
 		(dnp no)
-		(property "Reference" "TP2"
+		(property "Reference" "TP4"
 			(at 302.26 121.92 0)
 			(show_name no)
@@
 			(project "ETH1CVOLT"
 				(path "/8d3b546e-b30b-49b2-bc59-8e254df4c067/ea97f94c-dee1-4702-bb32-5cb010d15929/1e1986d0-5f57-471e-8eff-5dbba5b60ba1"
-					(reference "TP2")
+					(reference "TP4")
 					(unit 1)
 				)
@@
 		(on_board yes)
 		(in_pos_files yes)
-		(dnp no)
+		(dnp yes)
 		(fields_autoplaced yes)
 		(property "Reference" "R15"
@@
 					(reference "R15")
 					(unit 1)
-					(variant
-						(name "A")
-						(dnp yes)
-					)
-					(variant
-						(name "B")
-						(dnp yes)
-					)
 				)
 			)
@@
 	(symbol
 		(lib_id "Connector:TestPoint")
-		(at 245.11 129.54 0)
+		(at 53.34 137.16 0)
 		(mirror y)
 		(unit 1)
@@
 		(dnp no)
 		(property "Reference" "TP1"
+			(at 54.61 129.54 0)
+			(show_name no)
+			(do_not_autoplace no)
+			(effects
+				(font
+					(size 1.27 1.27)
+				)
+				(justify left)
+			)
+		)
+		(property "Value" "TestPoint"
+			(at 57.15 132.08 0)
+			(show_name no)
+			(do_not_autoplace no)
+			(effects
+				(font
+					(size 1.27 1.27)
+				)
+				(justify left)
+			)
+		)
+		(property "Footprint" "TestPoint:TestPoint_Pad_D1.5mm"
+			(at 48.26 137.16 0)
+			(hide yes)
+			(show_name no)
+			(do_not_autoplace no)
+			(effects
+				(font
+					(size 1.27 1.27)
+				)
+			)
+		)
+		(property "Datasheet" ""
+			(at 48.26 137.16 0)
+			(hide yes)
+			(show_name no)
+			(do_not_autoplace no)
+			(effects
+				(font
+					(size 1.27 1.27)
+				)
+			)
+		)
+		(property "Description" "test point"
+			(at 53.34 137.16 0)
+			(hide yes)
+			(show_name no)
+			(do_not_autoplace no)
+			(effects
+				(font
+					(size 1.27 1.27)
+				)
+			)
+		)
+		(pin "1"
+		)
+		(instances
+			(project "ETH1CVOLT"
+				(path "/8d3b546e-b30b-49b2-bc59-8e254df4c067/ea97f94c-dee1-4702-bb32-5cb010d15929/1e1986d0-5f57-471e-8eff-5dbba5b60ba1"
+					(reference "TP1")
+					(unit 1)
+				)
+			)
+		)
+	)
+	(symbol
+		(lib_id "Connector:TestPoint")
+		(at 245.11 129.54 0)
+		(mirror y)
+		(unit 1)
+		(body_style 1)
+		(exclude_from_sim no)
+		(in_bom no)
+		(on_board yes)
+		(in_pos_files yes)
+		(dnp no)
+		(property "Reference" "TP3"
 			(at 246.38 121.92 0)
 			(show_name no)
@@
 			(project "ETH1CVOLT"
 				(path "/8d3b546e-b30b-49b2-bc59-8e254df4c067/ea97f94c-dee1-4702-bb32-5cb010d15929/1e1986d0-5f57-471e-8eff-5dbba5b60ba1"
-					(reference "TP1")
+					(reference "TP3")
 					(unit 1)
 				)
@@
 		(on_board yes)
 		(in_pos_files yes)
-		(dnp no)
+		(dnp yes)
 		(property "Reference" "R17"
 			(at 351.79 138.4299 0)
@@
 					(unit 1)
 				)
+			)
+		)
+	)
+	(symbol
+		(lib_id "Connector:TestPoint")
+		(at 153.67 81.28 0)
+		(mirror y)
+		(unit 1)
+		(body_style 1)
+		(exclude_from_sim no)
+		(in_bom no)
+		(on_board yes)
+		(in_pos_files yes)
+		(dnp no)
+		(property "Reference" "TP2"
+			(at 154.94 73.66 0)
+			(show_name no)
+			(do_not_autoplace no)
+			(effects
+				(font
+					(size 1.27 1.27)
+				)
+				(justify left)
+			)
+		)
+		(property "Value" "TestPoint"
+			(at 157.48 76.2 0)
+			(show_name no)
+			(do_not_autoplace no)
+			(effects
+				(font
+					(size 1.27 1.27)
+				)
+				(justify left)
+			)
+		)
+		(property "Footprint" "TestPoint:TestPoint_Pad_D1.5mm"
+			(at 148.59 81.28 0)
+			(hide yes)
+			(show_name no)
+			(do_not_autoplace no)
+			(effects
+				(font
+					(size 1.27 1.27)
+				)
+			)
+		)
+		(property "Datasheet" ""
+			(at 148.59 81.28 0)
+			(hide yes)
+			(show_name no)
+			(do_not_autoplace no)
+			(effects
+				(font
+					(size 1.27 1.27)
+				)
+			)
+		)
+		(property "Description" "test point"
+			(at 153.67 81.28 0)
+			(hide yes)
+			(show_name no)
+			(do_not_autoplace no)
+			(effects
+				(font
+					(size 1.27 1.27)
+				)
+			)
+		)
+		(pin "1"
+		)
+		(instances
+			(project "ETH1CVOLT"
+				(path "/8d3b546e-b30b-49b2-bc59-8e254df4c067/ea97f94c-dee1-4702-bb32-5cb010d15929/1e1986d0-5f57-471e-8eff-5dbba5b60ba1"
+					(reference "TP2")
+					(unit 1)
+				)

Commit message: Development
Parts:
- C35: footprint Capacitor_SMD:C_1210_3225Metric_Pad1.33x2.70mm_HandSolder -> Capacitor_SMD:C_1206_3216Metric_Pad1.33x1.80mm_HandSolder
- U5: value DG412xUE -> DG412CUE+
Other:
- moved on the sheet: R12, R13
Changed lines of the file:
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@@
 	(text "+0.5V - +4.5V"
 		(exclude_from_sim no)
-		(at 166.878 128.778 0)
+		(at 170.688 128.778 0)
 		(effects
 			(font
@@
 	(text_box "SETUP FOR DAC UNIPOLAR MODE"
 		(exclude_from_sim no)
-		(at 109.22 66.04 0)
+		(at 107.95 66.04 0)
 		(size 33.02 35.56)
 		(margins 0.9525 0.9525 0.9525 0.9525)
@@
 	)
 	(junction
-		(at 118.11 82.55)
+		(at 116.84 82.55)
 		(diameter 0)
 		(color 0 0 0 0)
@@
 	(wire
 		(pts
-			(xy 83.82 72.39) (xy 118.11 72.39)
+			(xy 83.82 72.39) (xy 116.84 72.39)
 		)
 		(stroke
@@
 	(wire
 		(pts
-			(xy 118.11 72.39) (xy 118.11 73.66)
+			(xy 116.84 72.39) (xy 116.84 73.66)
 		)
 		(stroke
@@
 	(wire
 		(pts
-			(xy 118.11 82.55) (xy 153.67 82.55)
+			(xy 116.84 82.55) (xy 153.67 82.55)
 		)
 		(stroke
@@
 	(wire
 		(pts
-			(xy 118.11 91.44) (xy 118.11 92.71)
+			(xy 116.84 91.44) (xy 116.84 92.71)
 		)
 		(stroke
@@
 	(wire
 		(pts
-			(xy 118.11 83.82) (xy 118.11 82.55)
+			(xy 116.84 83.82) (xy 116.84 82.55)
 		)
 		(stroke
@@
 	(wire
 		(pts
-			(xy 118.11 82.55) (xy 118.11 81.28)
+			(xy 116.84 82.55) (xy 116.84 81.28)
 		)
 		(stroke
@@
 			)
 		)
-		(property "Datasheet" "https://www.ti.com/lit/ds/symlink/ina159.pdf?ts=1789029296659&ref_url=https%253A%252F%252Fwww.ti.com%252Fproduct%252FINA159"
+		(property "Datasheet" "https://www.ti.com/lit/ds/symlink/ina159.pdf"
 			(at 124.714 133.096 0)
 			(hide yes)
@@
 	(symbol
 		(lib_id "ETH1CVOLT_A:GND_ISO")
-		(at 118.11 92.71 0)
+		(at 116.84 92.71 0)
 		(unit 1)
 		(body_style 1)
@@
 		(fields_autoplaced yes)
 		(property "Reference" "#PWR063"
-			(at 118.11 99.06 0)
+			(at 116.84 99.06 0)
 			(hide yes)
 			(show_name no)
@@
 		)
 		(property "Value" "GND_ISO"
-			(at 118.11 97.79 0)
+			(at 116.84 97.79 0)
 			(show_name no)
 			(do_not_autoplace no)
@@
 		)
 		(property "Footprint" ""
-			(at 118.11 92.71 0)
+			(at 116.84 92.71 0)
 			(hide yes)
 			(show_name no)
@@
 		)
 		(property "Datasheet" ""
-			(at 118.11 92.71 0)
+			(at 116.84 92.71 0)
 			(hide yes)
 			(show_name no)
@@
 		)
 		(property "Description" "Power symbol creates a global label with name \"GND\" , ground"
-			(at 118.11 92.71 0)
+			(at 116.84 92.71 0)
 			(hide yes)
 			(show_name no)
@@
 	(symbol
 		(lib_id "Device:R")
-		(at 118.11 87.63 0)
+		(at 116.84 87.63 0)
 		(mirror x)
 		(unit 1)
@@
 		(dnp yes)
 		(property "Reference" "R13"
-			(at 129.54 86.106 0)
+			(at 128.27 86.106 0)
 			(show_name no)
 			(do_not_autoplace no)
@@
 		)
 		(property "Value" "10k/0.01%/100mW"
-			(at 129.54 88.646 0)
+			(at 128.27 88.646 0)
 			(show_name no)
 			(do_not_autoplace no)
@@
 		)
 		(property "Footprint" "Resistor_SMD:R_0603_1608Metric_Pad0.98x0.95mm_HandSolder"
-			(at 116.332 87.63 90)
+			(at 115.062 87.63 90)
 			(hide yes)
 			(show_name no)
@@
 		)
 		(property "Datasheet" ""
-			(at 118.11 87.63 0)
+			(at 116.84 87.63 0)
 			(hide yes)
 			(show_name no)
@@
 		)
 		(property "Description" "Resistor"
-			(at 118.11 87.63 0)
+			(at 116.84 87.63 0)
 			(hide yes)
 			(show_name no)
@@
 	(symbol
 		(lib_id "Device:R")
-		(at 118.11 77.47 0)
+		(at 116.84 77.47 0)
 		(mirror x)
 		(unit 1)
@@
 		(dnp yes)
 		(property "Reference" "R12"
-			(at 129.54 76.454 0)
+			(at 128.27 76.454 0)
 			(show_name no)
 			(do_not_autoplace no)
@@
 		)
 		(property "Value" "10k/0.01%/100mW"
-			(at 129.54 78.994 0)
+			(at 128.27 78.994 0)
 			(show_name no)
 			(do_not_autoplace no)
@@
 		)
 		(property "Footprint" "Resistor_SMD:R_0603_1608Metric_Pad0.98x0.95mm_HandSolder"
-			(at 116.332 77.47 90)
+			(at 115.062 77.47 90)
 			(hide yes)
 			(show_name no)
@@
 		)
 		(property "Datasheet" ""
-			(at 118.11 77.47 0)
+			(at 116.84 77.47 0)
 			(hide yes)
 			(show_name no)
@@
 		)
 		(property "Description" "Resistor"
-			(at 118.11 77.47 0)
+			(at 116.84 77.47 0)
 			(hide yes)
 			(show_name no)
@@
 			)
 		)
-		(property "Value" "DG412xUE"
+		(property "Value" "DG412CUE+"
 			(at 196.85 125.73 0)
 			(show_name no)
@@
 			)
 		)
-		(property "Value" "DG412xUE"
+		(property "Value" "DG412CUE+"
 			(at 196.85 143.51 0)
 			(show_name no)
@@
 			)
 		)
-		(property "Value" "DG412xUE"
+		(property "Value" "DG412CUE+"
 			(at 196.85 161.29 0)
 			(show_name no)
@@
 			)
 		)
-		(property "Value" "DG412xUE"
+		(property "Value" "DG412CUE+"
 			(at 184.15 256.5399 0)
 			(show_name no)
@@
 			)
 		)
-		(property "Footprint" "Capacitor_SMD:C_1210_3225Metric_Pad1.33x2.70mm_HandSolder"
+		(property "Footprint" "Capacitor_SMD:C_1206_3216Metric_Pad1.33x1.80mm_HandSolder"
 			(at 274.0152 139.7 0)
 			(hide yes)
@@
 			)
 		)
-		(property "Value" "DG412xUE"
+		(property "Value" "DG412CUE+"
 			(at 209.55 250.19 0)
 			(show_name no)

Commit message: Layout
Parts:
- renumbered C29 to C27, C30 to C28, C31 to C29, C32 to C30, C33 to C31, C34 to C32, C35 to C33, R12 to R11, R13 to R12, R14 to R13, R15 to R14, R16 to R15, R17 to R16, R18 to R17
Connections:
- net ADC_VOLT_SCLK renamed ADC_SCLK
- net ADC_VOLT_SDO renamed ADC_SDO
- net ADC_VOLT_~{CS} renamed ADC_~{CS}

Commit message: Layout and schematic
Other:
- title: (none) -> ETH1CVOLT

Commit message: Verification
Parts:
- added C29: 10u/35V/X7R, Capacitor_SMD:C_1206_3216Metric_Pad1.33x1.80mm_HandSolder, symbol Device:C
- added R62: 100/1%/100mW, Resistor_SMD:R_0603_1608Metric_Pad0.98x0.95mm_HandSolder, symbol Device:R
- C34: renamed from C33; value 10u/50V/X7R -> 10u/35V/X7R
- renumbered C29 to C30, C30 to C31, C31 to C32, C32 to C33
Connections:
- net +5VD_ISO: now also C29.1
- net GND_ISO: now also C29.2
- net at R11.1, R12.2, TP2.1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: now also R62.2; no longer R14.1, U5.2
- new net: R14.1, R62.1, U5.2
Other:
- moved on the sheet: C30, C31, C32, C33, U5D, U5E

Commit message: HW design done
Parts:
- added R67: 1k/1%/100mW, Resistor_SMD:R_0603_1608Metric_Pad0.98x0.95mm_HandSolder, symbol Device:R
Connections:
- net +5VREF_ISO: now also R67.2; no longer U5.6
- new net: R67.1, U5.6
Other:
- moved on the sheet: R13, R16, R17
