File: HARDWARE/ETH1CVOLT/ADC.kicad_sch (KiCad schematic)
At the start: 26 parts, among them U4 INA159AIDGKT, U5 DG412CUE+, U6 LTC2400CS8#TRPBF

Commit message: Production data, cleanup.
Parts:
- added C112, C113: 0.1u/100V/X7R, Capacitor_SMD:C_0603_1608Metric_Pad1.08x0.95mm_HandSolder, symbol Device:C
- added R76: 0R/5%/100mW, Resistor_SMD:R_0603_1608Metric_Pad0.98x0.95mm_HandSolder, symbol Device:R
- added U29: ADA4522-1ARZ, Package_SO:SOIC-8_3.9x4.9mm_P1.27mm, symbol Amplifier_Operational:ADA4522-1
Connections:
- net +14V_ISO: now also C112.1, U29.7 (V+)
- net -14V_ISO: now also C113.1, U29.4 (V-)
- net GND_ISO: now also C112.2, C113.2
- net MEAS_OUT: now also R76.1, U29.3 (+); no longer D1.3 (K), R11.2, U4.3 (+)
- new net: D1.3 (K), R11.2, R76.2, U29.2 (-), U29.6, U4.3 (+)
Other:
- moved on the sheet: C34, D1, D2, R11, R12, R13, R14, R15, R16, R17, R62, R67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
