File: HARDWARE/ETH1CVOLT/Isolation_Digital.kicad_sch (KiCad schematic)
At the start: 6 parts, among them U22 ISO7761FDBQ, U5 ISO7760DBQ

Commit message: Development
Parts:
- removed U5: ISO7760DBQ, Package_SO:SSOP-16_3.9x4.9mm_P0.635mm, symbol Isolator:ISO7760DBQ
- added U12: ISO7761FDBQ, Package_SO:SSOP-16_3.9x4.9mm_P0.635mm, symbol Isolator:ISO7761FDBQ
- renumbered C44 to C45, C45 to C46, C46 to C47, C47 to C48, U22 to U11
Connections:
- net +3.3V: now also U12.1 (Vcc1)
- net +5VD_ISO: now also U12.16 (Vcc2)
- net DAC_DIN: now also U12.14 (OUTB)
- net DAC_SCLK: now also U12.13 (OUTC)
- net DAC_~{CS}: now also U12.15 (OUTA)
- net DAC_~{LDAC}: now also U12.12 (OUTD)
- net GND: now also U12.8 (GND1)
- net GND_ISO: now also U12.9 (GND2)
- net MCU_DAC_DIN: now also U12.3 (INB)
- net MCU_DAC_SCLK: now also U12.4 (INC)
- net MCU_DAC_~{CS}: now also U12.2 (INA)
- net MCU_DAC_~{LDAC}: now also U12.5 (IND)
- net MCU_REL_RANGE_SEL: now also U12.6 (INE)
- net REL_RANGE_SEL: now also U12.11 (OUTE)
- no-connect marks 0 -> 2
Other:
- moved on the sheet: C47, C48

Commit message: Development
Parts:
- removed U12: ISO7761FDBQ, Package_SO:SSOP-16_3.9x4.9mm_P0.635mm, symbol Isolator:ISO7761FDBQ
- added U28: ISO7760DBQ, Package_SO:SSOP-16_3.9x4.9mm_P0.635mm, symbol Isolator:ISO7760DBQ
Connections:
- net +3.3V: now also U28.1 (Vcc1)
- net +5VD_ISO: now also U28.16 (Vcc2)
- net DAC_DIN: now also U28.14 (OUTB)
- net DAC_SCLK: now also U28.13 (OUTC)
- net DAC_~{CS}: now also U28.15 (OUTA)
- net DAC_~{LDAC}: now also U28.12 (OUTD)
- net GND: now also U28.8 (GND1)
- net GND_ISO: now also U28.9 (GND2)
- net MCU_DAC_DIN: now also U28.3 (INB)
- net MCU_DAC_SCLK: now also U28.4 (INC)
- net MCU_DAC_~{CS}: now also U28.2 (INA)
- net MCU_DAC_~{LDAC}: now also U28.5 (IND)
- new net MCU_REL_RESET: U28.7 (INF)
- new net MCU_REL_SET: U28.6 (INE)
- new net REL_RESET: U28.10 (OUTF)
- new net REL_SET: U28.11 (OUTE)
- no-connect marks 2 -> 0
Changed lines of the file:
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@@
 	(generator_version "10.0")
 	(paper "A3")
-	(no_connect
-		(at 196.85 177.8)
-	)
-	(no_connect
-		(at 217.17 177.8)
-	)
 	(wire
 		(pts
@@
 	(wire
 		(pts
+			(xy 194.31 177.8) (xy 196.85 177.8)
+		)
+		(stroke
+			(width 0)
+			(type default)
+		)
+	)
+	(wire
+		(pts
 			(xy 201.93 187.96) (xy 201.93 189.23)
 		)
@@
 		(pts
 			(xy 194.31 165.1) (xy 196.85 165.1)
+		)
+		(stroke
+			(width 0)
+			(type default)
+		)
+	)
+	(wire
+		(pts
+			(xy 217.17 177.8) (xy 219.71 177.8)
 		)
 		(stroke
@@
 		)
 	)
+	(hierarchical_label "MCU_REL_RESET"
+		(shape input)
+		(at 194.31 177.8 180)
+		(effects
+			(font
+				(size 1.27 1.27)
+			)
+			(justify right)
+		)
+	)
 	(hierarchical_label "MCU_DAC_~{LDAC}"
 		(shape input)
@@
 		)
 	)
+	(hierarchical_label "REL_RESET"
+		(shape output)
+		(at 219.71 177.8 0)
+		(effects
+			(font
+				(size 1.27 1.27)
+			)
+			(justify left)
+		)
+	)
 	(hierarchical_label "DAC_DIN"
 		(shape output)
@@
 		)
 	)
-	(hierarchical_label "MCU_REL_RANGE_SEL"
+	(hierarchical_label "MCU_REL_SET"
 		(shape input)
 		(at 194.31 175.26 180)
@@
 		)
 	)
-	(hierarchical_label "REL_RANGE_SEL"
+	(hierarchical_label "REL_SET"
 		(shape output)
 		(at 219.71 175.26 0)
@@
 	)
 	(symbol
-		(lib_id "Isolator:ISO7761FDBQ")
-		(at 207.01 172.72 0)
-		(unit 1)
-		(body_style 1)
-		(exclude_from_sim no)
-		(in_bom yes)
-		(on_board yes)
-		(in_pos_files yes)
-		(dnp no)
-		(fields_autoplaced yes)
-		(property "Reference" "U12"
-			(at 214.2333 152.4 0)
-			(show_name no)
-			(do_not_autoplace no)
-			(effects
-				(font
-					(size 1.27 1.27)
-				)
-				(justify left)
-			)
-		)
-		(property "Value" "ISO7761FDBQ"
-			(at 214.2333 154.94 0)
-			(show_name no)
-			(do_not_autoplace no)
-			(effects
-				(font
-					(size 1.27 1.27)
-				)
-				(justify left)
-			)
-		)
-		(property "Footprint" "Package_SO:SSOP-16_3.9x4.9mm_P0.635mm"
-			(at 212.725 186.69 0)
-			(hide yes)
-			(show_name no)
-			(do_not_autoplace no)
-			(effects
-				(font
-					(size 1.27 1.27)
-				)
-				(justify left)
-			)
-		)
-		(property "Datasheet" "https://www.ti.com/lit/ds/symlink/iso7763.pdf?ts=1596905577895"
-			(at 217.17 175.26 0)
-			(hide yes)
-			(show_name no)
-			(do_not_autoplace no)
-			(effects
-				(font
-					(size 1.27 1.27)
-				)
-			)
-		)
-		(property "Description" "Default low, High-speed, robust EMC, reinforced, six-channel, digital, isolator, SSOP-16"
-			(at 207.01 172.72 0)
-			(hide yes)
-			(show_name no)
-			(do_not_autoplace no)
-			(effects
-				(font
-					(size 1.27 1.27)
-				)
-			)
-		)
-		(pin "1"
-		)
-		(pin "16"
-		)
-		(pin "8"
-		)
-		(pin "15"
-		)
-		(pin "2"
-		)
-		(pin "3"
-		)
-		(pin "7"
-		)
-		(pin "11"
-		)
-		(pin "10"
-		)
-		(pin "13"
-		)
-		(pin "5"
-		)
-		(pin "9"
-		)
-		(pin "12"
-		)
-		(pin "6"
-		)
-		(pin "14"
-		)
-		(pin "4"
-		)
-		(instances
-			(project "ETH1CVOLT"
-				(path "/8d3b546e-b30b-49b2-bc59-8e254df4c067/ea97f94c-dee1-4702-bb32-5cb010d15929/2cbb7ee0-d677-45ec-ab6c-39870dae0fe6"
-					(reference "U12")
-					(unit 1)
-				)
-			)
-		)
-	)
-	(symbol
 		(lib_id "Device:C")
 		(at 25.4 262.89 0)
@@
 					(unit 1)
 				)
+			)
+		)
+	)
+	(symbol
+		(lib_id "Isolator:ISO7760DBQ")
+		(at 207.01 172.72 0)
+		(unit 1)
+		(body_style 1)
+		(exclude_from_sim no)
+		(in_bom yes)
+		(on_board yes)
+		(in_pos_files yes)
+		(dnp no)
+		(fields_autoplaced yes)
+		(property "Reference" "U28"
+			(at 214.2333 152.4 0)
+			(show_name no)
+			(do_not_autoplace no)
+			(effects
+				(font
+					(size 1.27 1.27)
+				)
+				(justify left)
+			)
+		)
+		(property "Value" "ISO7760DBQ"
+			(at 214.2333 154.94 0)
+			(show_name no)
+			(do_not_autoplace no)
+			(effects
+				(font
+					(size 1.27 1.27)
+				)
+				(justify left)
+			)
+		)
+		(property "Footprint" "Package_SO:SSOP-16_3.9x4.9mm_P0.635mm"
+			(at 212.725 186.69 0)
+			(hide yes)
+			(show_name no)
+			(do_not_autoplace no)
+			(effects
+				(font
+					(size 1.27 1.27)
+				)
+				(justify left)
+			)
+		)
+		(property "Datasheet" "https://www.ti.com/lit/ds/symlink/iso7763.pdf"
+			(at 217.17 175.26 0)
+			(hide yes)
+			(show_name no)
+			(do_not_autoplace no)
+			(effects
+				(font
+					(size 1.27 1.27)
+				)
+			)
+		)
+		(property "Description" "Default high, High-speed, robust EMC, reinforced, six-channel, digital, isolator, SSOP-16"
+			(at 207.01 172.72 0)
+			(hide yes)
+			(show_name no)
+			(do_not_autoplace no)
+			(effects
+				(font
+					(size 1.27 1.27)
+				)
+			)
+		)
+		(pin "5"
+		)
+		(pin "9"
+		)
+		(pin "1"
+		)
+		(pin "12"
+		)
+		(pin "15"
+		)
+		(pin "8"
+		)
+		(pin "11"
+		)
+		(pin "3"
+		)
+		(pin "7"
+		)
+		(pin "4"
+		)
+		(pin "10"
+		)
+		(pin "13"
+		)
+		(pin "2"
+		)
+		(pin "14"
+		)
+		(pin "16"
+		)
+		(pin "6"
+		)
+		(instances
+			(project "ETH1CVOLT"
+				(path "/8d3b546e-b30b-49b2-bc59-8e254df4c067/ea97f94c-dee1-4702-bb32-5cb010d15929/2cbb7ee0-d677-45ec-ab6c-39870dae0fe6"
+					(reference "U28")
+					(unit 1)
+				)

Commit message: Development
Parts:
- added TP10, TP11, TP12, TP13, TP14, TP15, TP16, TP17, TP18, TP19, TP20, TP21: TestPoint, TestPoint:TestPoint_Pad_D1.5mm, symbol Connector:TestPoint
- renumbered U28 to U12
Connections:
- net ADC_SW1: now also TP10.1
- net ADC_SW2: now also TP14.1
- net ADC_SW3: now also TP18.1
- net ADC_VOLT_SCLK: now also TP11.1
- net ADC_VOLT_SDO: now also TP19.1
- net ADC_VOLT_~{CS}: now also TP15.1
- net DAC_DIN: now also TP16.1
- net DAC_SCLK: now also TP20.1
- net DAC_~{CS}: now also TP12.1
- net DAC_~{LDAC}: now also TP13.1
- net REL_RESET: now also TP21.1
- net REL_SET: now also TP17.1
Other:
- moved on the sheet: U11

Commit message: Layout
Parts:
- TP10, TP11, TP12, TP15, TP16, TP20: footprint TestPoint:TestPoint_Pad_D1.5mm -> TestPoint:TestPoint_Pad_D1.0mm
- TP13: renamed from TP18; footprint TestPoint:TestPoint_Pad_D1.5mm -> TestPoint:TestPoint_Pad_D1.0mm
- TP14: renamed from TP17; footprint TestPoint:TestPoint_Pad_D1.5mm -> TestPoint:TestPoint_Pad_D1.0mm
- TP17: renamed from TP14; footprint TestPoint:TestPoint_Pad_D1.5mm -> TestPoint:TestPoint_Pad_D1.0mm
- TP18: renamed from TP21; footprint TestPoint:TestPoint_Pad_D1.5mm -> TestPoint:TestPoint_Pad_D1.0mm
- TP19: renamed from TP13; footprint TestPoint:TestPoint_Pad_D1.5mm -> TestPoint:TestPoint_Pad_D1.0mm
- TP21: renamed from TP19; footprint TestPoint:TestPoint_Pad_D1.5mm -> TestPoint:TestPoint_Pad_D1.0mm
- renumbered C45 to C44, C46 to C45, C47 to C46, C48 to C47
Connections:
- net ADC_VOLT_SCLK is gone; now on net ADC_SW2: TP11.1, U11.12 (OUTD)
- net ADC_VOLT_~{CS} is gone; now on net ADC_SW1: TP15.1, U11.11 (OUTE)
- net MCU_ADC_VOLT_SCLK is gone; now on net MCU_ADC_SW2: U11.5 (IND)
- net MCU_ADC_VOLT_~{CS} is gone; now on net MCU_ADC_SW1: U11.6 (INE)
- net ADC_SW1: no longer TP10.1, U11.15 (OUTA)
- net ADC_SW2: no longer TP17.1, U11.14 (OUTB)
- net ADC_SW3: now also TP18.1; no longer TP13.1
- net DAC_DIN: now also TP21.1, U12.10 (OUTF); no longer TP16.1, U12.14 (OUTB)
- net DAC_SCLK: now also TP13.1, U12.12 (OUTD); no longer TP20.1, U12.13 (OUTC)
- net DAC_~{CS}: now also TP17.1, U12.11 (OUTE); no longer TP12.1, U12.15 (OUTA)
- net DAC_~{LDAC}: now also TP20.1, U12.13 (OUTC); no longer TP19.1, U12.12 (OUTD)
- net MCU_ADC_SW1: no longer U11.2 (INA)
- net MCU_ADC_SW2: no longer U11.3 (INB)
- net MCU_DAC_DIN: now also U12.7 (INF); no longer U12.3 (INB)
- net MCU_DAC_SCLK: now also U12.5 (IND); no longer U12.4 (INC)
- net MCU_DAC_~{CS}: now also U12.6 (INE); no longer U12.2 (INA)
- net MCU_DAC_~{LDAC}: now also U12.4 (INC); no longer U12.5 (IND)
- net MCU_REL_RESET: now also U11.3 (INB); no longer U12.7 (INF)
- net MCU_REL_SET: now also U11.2 (INA); no longer U12.6 (INE)
- net REL_RESET: now also TP14.1, U11.14 (OUTB); no longer TP18.1, U12.10 (OUTF)
- net REL_SET: now also TP10.1, U11.15 (OUTA); no longer TP14.1, U12.11 (OUTE)
- net ADC_VOLT_SDO renamed ADC_SDO
- net ADC_SDO: now also TP19.1; no longer TP21.1
- net MCU_ADC_VOLT_SDO renamed MCU_ADC_SDO
- new net ADC_SCLK: TP16.1, U12.14 (OUTB)
- new net ADC_~{CS}: TP12.1, U12.15 (OUTA)
- new net MCU_ADC_SCLK: U12.3 (INB)
- new net MCU_ADC_~{CS}: U12.2 (INA)
Other:
- moved on the sheet: TP10, TP11, TP12, TP13, TP14, TP15, TP16, TP17, TP18, TP19, TP20, TP21

Commit message: Layout and schematic
Parts:
- renumbered C44 to C47, C45 to C48, C46 to C49, C47 to C50, TP13 to TP10, TP14 to TP11, TP15 to TP12, TP16 to TP13, TP17 to TP14, TP18 to TP15, TP19 to TP16, TP20 to TP17, TP21 to TP18, TP10 to TP7, TP11 to TP8, TP12 to TP9
Other:
- title: (none) -> ETH1CVOLT

Commit message: Verification
Parts:
- renumbered C47 to C48, C48 to C49, C49 to C50, C50 to C51
Changed lines of the file:
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@@
 		(dnp no)
 		(fields_autoplaced yes)
-		(property "Reference" "C49"
+		(property "Reference" "C50"
 			(at 231.14 261.6199 0)
 			(show_name no)
@@
 			(project "ETH1CVOLT"
 				(path "/8d3b546e-b30b-49b2-bc59-8e254df4c067/ea97f94c-dee1-4702-bb32-5cb010d15929/2cbb7ee0-d677-45ec-ab6c-39870dae0fe6"
-					(reference "C49")
+					(reference "C50")
 					(unit 1)
 				)
@@
 		(dnp no)
 		(fields_autoplaced yes)
-		(property "Reference" "#PWR0128"
+		(property "Reference" "#PWR0130"
 			(at 251.46 274.32 0)
 			(hide yes)
@@
 			(project "ETH1CVOLT"
 				(path "/8d3b546e-b30b-49b2-bc59-8e254df4c067/ea97f94c-dee1-4702-bb32-5cb010d15929/2cbb7ee0-d677-45ec-ab6c-39870dae0fe6"
-					(reference "#PWR0128")
+					(reference "#PWR0130")
 					(unit 1)
 				)
@@
 		(dnp no)
 		(fields_autoplaced yes)
-		(property "Reference" "#PWR0123"
+		(property "Reference" "#PWR0125"
 			(at 214.63 153.67 0)
 			(hide yes)
@@
 			(project "ETH1CVOLT"
 				(path "/8d3b546e-b30b-49b2-bc59-8e254df4c067/ea97f94c-dee1-4702-bb32-5cb010d15929/2cbb7ee0-d677-45ec-ab6c-39870dae0fe6"
-					(reference "#PWR0123")
+					(reference "#PWR0125")
 					(unit 1)
 				)
@@
 		(dnp no)
 		(fields_autoplaced yes)
-		(property "Reference" "#PWR0119"
+		(property "Reference" "#PWR0121"
 			(at 199.39 153.67 0)
 			(hide yes)
@@
 			(project "ETH1CVOLT"
 				(path "/8d3b546e-b30b-49b2-bc59-8e254df4c067/ea97f94c-dee1-4702-bb32-5cb010d15929/2cbb7ee0-d677-45ec-ab6c-39870dae0fe6"
-					(reference "#PWR0119")
+					(reference "#PWR0121")
 					(unit 1)
 				)
@@
 		(dnp no)
 		(fields_autoplaced yes)
-		(property "Reference" "#PWR0120"
+		(property "Reference" "#PWR0122"
 			(at 199.39 196.85 0)
 			(hide yes)
@@
 			(project "ETH1CVOLT"
 				(path "/8d3b546e-b30b-49b2-bc59-8e254df4c067/ea97f94c-dee1-4702-bb32-5cb010d15929/2cbb7ee0-d677-45ec-ab6c-39870dae0fe6"
-					(reference "#PWR0120")
+					(reference "#PWR0122")
 					(unit 1)
 				)
@@
 		(dnp no)
 		(fields_autoplaced yes)
-		(property "Reference" "#PWR0113"
+		(property "Reference" "#PWR0115"
 			(at 25.4 261.62 0)
 			(hide yes)
@@
 			(project "ETH1CVOLT"
 				(path "/8d3b546e-b30b-49b2-bc59-8e254df4c067/ea97f94c-dee1-4702-bb32-5cb010d15929/2cbb7ee0-d677-45ec-ab6c-39870dae0fe6"
-					(reference "#PWR0113")
+					(reference "#PWR0115")
 					(unit 1)
 				)
@@
 		(dnp no)
 		(fields_autoplaced yes)
-		(property "Reference" "#PWR0117"
+		(property "Reference" "#PWR0119"
 			(at 199.39 68.58 0)
 			(hide yes)
@@
 			(project "ETH1CVOLT"
 				(path "/8d3b546e-b30b-49b2-bc59-8e254df4c067/ea97f94c-dee1-4702-bb32-5cb010d15929/2cbb7ee0-d677-45ec-ab6c-39870dae0fe6"
-					(reference "#PWR0117")
+					(reference "#PWR0119")
 					(unit 1)
 				)
@@
 		(dnp no)
 		(fields_autoplaced yes)
-		(property "Reference" "C50"
+		(property "Reference" "C51"
 			(at 255.27 261.6199 0)
 			(show_name no)
@@
 			(project "ETH1CVOLT"
 				(path "/8d3b546e-b30b-49b2-bc59-8e254df4c067/ea97f94c-dee1-4702-bb32-5cb010d15929/2cbb7ee0-d677-45ec-ab6c-39870dae0fe6"
-					(reference "C50")
+					(reference "C51")
 					(unit 1)
 				)
@@
 		(dnp no)
 		(fields_autoplaced yes)
-		(property "Reference" "#PWR0116"
+		(property "Reference" "#PWR0118"
 			(at 49.53 274.32 0)
 			(hide yes)
@@
 			(project "ETH1CVOLT"
 				(path "/8d3b546e-b30b-49b2-bc59-8e254df4c067/ea97f94c-dee1-4702-bb32-5cb010d15929/2cbb7ee0-d677-45ec-ab6c-39870dae0fe6"
-					(reference "#PWR0116")
+					(reference "#PWR0118")
 					(unit 1)
 				)
@@
 		(dnp no)
 		(fields_autoplaced yes)
-		(property "Reference" "#PWR0121"
+		(property "Reference" "#PWR0123"
 			(at 214.63 68.58 0)
 			(hide yes)
@@
 			(project "ETH1CVOLT"
 				(path "/8d3b546e-b30b-49b2-bc59-8e254df4c067/ea97f94c-dee1-4702-bb32-5cb010d15929/2cbb7ee0-d677-45ec-ab6c-39870dae0fe6"
-					(reference "#PWR0121")
+					(reference "#PWR0123")
 					(unit 1)
 				)
@@
 		(dnp no)
 		(fields_autoplaced yes)
-		(property "Reference" "#PWR0122"
+		(property "Reference" "#PWR0124"
 			(at 214.63 111.76 0)
 			(hide yes)
@@
 			(project "ETH1CVOLT"
 				(path "/8d3b546e-b30b-49b2-bc59-8e254df4c067/ea97f94c-dee1-4702-bb32-5cb010d15929/2cbb7ee0-d677-45ec-ab6c-39870dae0fe6"
-					(reference "#PWR0122")
+					(reference "#PWR0124")
 					(unit 1)
 				)
@@
 		(dnp no)
 		(fields_autoplaced yes)
-		(property "Reference" "#PWR0118"
+		(property "Reference" "#PWR0120"
 			(at 199.39 111.76 0)
 			(hide yes)
@@
 			(project "ETH1CVOLT"
 				(path "/8d3b546e-b30b-49b2-bc59-8e254df4c067/ea97f94c-dee1-4702-bb32-5cb010d15929/2cbb7ee0-d677-45ec-ab6c-39870dae0fe6"
-					(reference "#PWR0118")
+					(reference "#PWR0120")
 					(unit 1)
 				)
@@
 		(dnp no)
 		(fields_autoplaced yes)
-		(property "Reference" "#PWR0126"
+		(property "Reference" "#PWR0128"
 			(at 227.33 274.32 0)
 			(hide yes)
@@
 			(project "ETH1CVOLT"
 				(path "/8d3b546e-b30b-49b2-bc59-8e254df4c067/ea97f94c-dee1-4702-bb32-5cb010d15929/2cbb7ee0-d677-45ec-ab6c-39870dae0fe6"
-					(reference "#PWR0126")
+					(reference "#PWR0128")
 					(unit 1)
 				)
@@
 		(dnp no)
 		(fields_autoplaced yes)
-		(property "Reference" "#PWR0115"
+		(property "Reference" "#PWR0117"
 			(at 49.53 261.62 0)
 			(hide yes)
@@
 			(project "ETH1CVOLT"
 				(path "/8d3b546e-b30b-49b2-bc59-8e254df4c067/ea97f94c-dee1-4702-bb32-5cb010d15929/2cbb7ee0-d677-45ec-ab6c-39870dae0fe6"
-					(reference "#PWR0115")
+					(reference "#PWR0117")
 					(unit 1)
 				)
@@
 		(dnp no)
 		(fields_autoplaced yes)
-		(property "Reference" "#PWR0124"
+		(property "Reference" "#PWR0126"
 			(at 214.63 196.85 0)
 			(hide yes)
@@
 			(project "ETH1CVOLT"
 				(path "/8d3b546e-b30b-49b2-bc59-8e254df4c067/ea97f94c-dee1-4702-bb32-5cb010d15929/2cbb7ee0-d677-45ec-ab6c-39870dae0fe6"
-					(reference "#PWR0124")
+					(reference "#PWR0126")
 					(unit 1)
 				)
@@
 		(dnp no)
 		(fields_autoplaced yes)
-		(property "Reference" "C47"
+		(property "Reference" "C48"
 			(at 29.21 261.6199 0)
 			(show_name no)
@@
 			(project "ETH1CVOLT"
 				(path "/8d3b546e-b30b-49b2-bc59-8e254df4c067/ea97f94c-dee1-4702-bb32-5cb010d15929/2cbb7ee0-d677-45ec-ab6c-39870dae0fe6"
-					(reference "C47")
+					(reference "C48")
 					(unit 1)
 				)
@@
 		(dnp no)
 		(fields_autoplaced yes)
-		(property "Reference" "#PWR0127"
+		(property "Reference" "#PWR0129"
 			(at 251.46 261.62 0)
 			(hide yes)
@@
 			(project "ETH1CVOLT"
 				(path "/8d3b546e-b30b-49b2-bc59-8e254df4c067/ea97f94c-dee1-4702-bb32-5cb010d15929/2cbb7ee0-d677-45ec-ab6c-39870dae0fe6"
-					(reference "#PWR0127")
+					(reference "#PWR0129")
 					(unit 1)
 				)
@@
 		(dnp no)
 		(fields_autoplaced yes)
-		(property "Reference" "C48"
+		(property "Reference" "C49"
 			(at 53.34 261.6199 0)
 			(show_name no)
@@
 			(project "ETH1CVOLT"
 				(path "/8d3b546e-b30b-49b2-bc59-8e254df4c067/ea97f94c-dee1-4702-bb32-5cb010d15929/2cbb7ee0-d677-45ec-ab6c-39870dae0fe6"
-					(reference "C48")
+					(reference "C49")
 					(unit 1)
 				)
@@
 		(dnp no)
 		(fields_autoplaced yes)
-		(property "Reference" "#PWR0125"
+		(property "Reference" "#PWR0127"
 			(at 227.33 261.62 0)
 			(hide yes)
@@
 			(project "ETH1CVOLT"
 				(path "/8d3b546e-b30b-49b2-bc59-8e254df4c067/ea97f94c-dee1-4702-bb32-5cb010d15929/2cbb7ee0-d677-45ec-ab6c-39870dae0fe6"
-					(reference "#PWR0125")
+					(reference "#PWR0127")
 					(unit 1)
 				)
@@
 		(dnp no)
 		(fields_autoplaced yes)
-		(property "Reference" "#PWR0114"
+		(property "Reference" "#PWR0116"
 			(at 25.4 274.32 0)
 			(hide yes)
@@
 			(project "ETH1CVOLT"
 				(path "/8d3b546e-b30b-49b2-bc59-8e254df4c067/ea97f94c-dee1-4702-bb32-5cb010d15929/2cbb7ee0-d677-45ec-ab6c-39870dae0fe6"
-					(reference "#PWR0114")
+					(reference "#PWR0116")
 					(unit 1)
 				)

Commit message: Modifications
Parts:
- U11: value ISO7761FDBQ -> ISO7761DBQR
Changed lines of the file:
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@@
 			)
 		)
-		(property "Value" "ISO7761FDBQ"
+		(property "Value" "ISO7761DBQR"
 			(at 214.2333 69.85 0)
 			(show_name no)

Commit message: HW design done
Parts:
- added R71, R72: 4k7/1%/100mW, Resistor_SMD:R_0603_1608Metric_Pad0.98x0.95mm_HandSolder, symbol Device:R
Connections:
- net GND: now also R71.2, R72.2
- net MCU_REL_RESET: now also R71.1
- net MCU_REL_SET: now also R72.1
