File: HARDWARE/ETH1CVOLT/MCU.kicad_sch (KiCad schematic)
At the start: 27 parts, among them J1 20021111-00010T4LF, U1 STM32H743VITx, U2 24LC08B-E/MS, Y1 NX5032GA-16

Commit message: Development
Parts:
- removed JP1: Open, Jumper:SolderJumper-2_P1.3mm_Open_Pad1.0x1.5mm, symbol Jumper:SolderJumper_2_Open
- added JP8: SolderJumper_2_Open, Jumper:SolderJumper-2_P1.3mm_Open_Pad1.0x1.5mm, symbol Jumper:SolderJumper_2_Open
- C1, C16, C2, C3, C4, C5: value 0.1u -> 0.1u/100V/X7R
- C10: renamed from C13; value 2u2 -> 2u2/16V/X7R
- C11: renamed from C7; value 1u -> 1u/16V/X7R
- C12: renamed from C15; value 2u2 -> 2u2/16V/X7R
- C13: renamed from C8; value 1u -> 1u/16V/X7R
- C14: renamed from C12; value 10u -> 10u/16V/X7R; footprint Capacitor_SMD:C_0603_1608Metric_Pad1.08x0.95mm_HandSolder -> Capacitor_SMD:C_0805_2012Metric_Pad1.18x1.45mm_HandSolder
- C15: renamed from C14; value 0.1u -> 0.1u/100V/X7R
- C6: renamed from C10; value 8p -> 8p/100V/X7R
- C7: renamed from C6; value 0.1u -> 0.1u/100V/X7R
- C8: renamed from C9; value 0.1u -> 0.1u/100V/X7R
- C9: renamed from C11; value 8p -> 8p/100V/X7R
- R1, R3: value 10k -> 10k/1%/100mW
- R2: value 0 -> 0R/5%/100mW
- R4, R5: value 4k7 -> 4k7/1%/100mW
Connections:
- net GND: now also JP8.1 (A)
- net MCU_DEF: now also JP8.2 (B)
- net MCU_ADC_CURR_SCLK: no longer names the net of U1.1 (PE2)
- no-connect marks 48 -> 63
Other:
- moved on the sheet: C10, C12, C13, C15, C16, C6, C9, R2, R3, R5, Y1

Commit message: Development
Parts:
- Y1: footprint ETH1CVOLT_A:NX5032GA -> ETH1CVOLT:NX5032GA
Changed lines of the file:
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@@
 	(hierarchical_label "MCU_ADC_SW2"
 		(shape output)
-		(at 326.39 45.72 180)
+		(at 323.85 55.88 0)
+		(effects
+			(font
+				(size 1.27 1.27)
+			)
+			(justify left)
+		)
+	)
+	(hierarchical_label "MCU_ADC_VOLT_~{CS}"
+		(shape output)
+		(at 323.85 63.5 0)
+		(effects
+			(font
+				(size 1.27 1.27)
+			)
+			(justify left)
+		)
+	)
+	(hierarchical_label "MCU_ADC_CURR_SDI"
+		(shape output)
+		(at 189.23 99.06 180)
 		(effects
 			(font
@@
 		)
 	)
-	(hierarchical_label "MCU_ADC_VOLT_~{CS}"
-		(shape output)
-		(at 326.39 53.34 180)
-		(effects
-			(font
-				(size 1.27 1.27)
-			)
-			(justify right)
-		)
-	)
-	(hierarchical_label "MCU_ADC_CURR_SDI"
-		(shape output)
-		(at 189.23 99.06 180)
-		(effects
-			(font
-				(size 1.27 1.27)
-			)
-			(justify right)
-		)
-	)
 	(hierarchical_label "MCU_ADC_SW3"
 		(shape output)
-		(at 326.39 48.26 180)
-		(effects
-			(font
-				(size 1.27 1.27)
-			)
-			(justify right)
+		(at 323.85 58.42 0)
+		(effects
+			(font
+				(size 1.27 1.27)
+			)
+			(justify left)
 		)
 	)
@@
 	(hierarchical_label "MCU_DAC_SCLK"
 		(shape output)
-		(at 326.39 107.95 180)
-		(effects
-			(font
-				(size 1.27 1.27)
-			)
-			(justify right)
+		(at 326.39 105.41 0)
+		(effects
+			(font
+				(size 1.27 1.27)
+			)
+			(justify left)
 		)
 	)
 	(hierarchical_label "MCU_ADC_VOLT_SDO"
 		(shape input)
-		(at 326.39 55.88 180)
-		(effects
-			(font
-				(size 1.27 1.27)
-			)
-			(justify right)
+		(at 323.85 66.04 0)
+		(effects
+			(font
+				(size 1.27 1.27)
+			)
+			(justify left)
 		)
 	)
@@
 		(shape bidirectional)
 		(at 237.49 63.5 0)
+		(effects
+			(font
+				(size 1.27 1.27)
+			)
+			(justify left)
+		)
+	)
+	(hierarchical_label "MCU_REL_SET"
+		(shape output)
+		(at 325.12 91.44 0)
 		(effects
 			(font
@@
 	(hierarchical_label "MCU_ADC_SW1"
 		(shape output)
-		(at 326.39 43.18 180)
-		(effects
-			(font
-				(size 1.27 1.27)
-			)
-			(justify right)
+		(at 323.85 53.34 0)
+		(effects
+			(font
+				(size 1.27 1.27)
+			)
+			(justify left)
 		)
 	)
@@
 		)
 	)
+	(hierarchical_label "MCU_REL_RESET"
+		(shape output)
+		(at 325.12 93.98 0)
+		(effects
+			(font
+				(size 1.27 1.27)
+			)
+			(justify left)
+		)
+	)
 	(hierarchical_label "MCU_ADC_VOLT_SCLK"
 		(shape output)
-		(at 326.39 50.8 180)
+		(at 323.85 60.96 0)
+		(effects
+			(font
+				(size 1.27 1.27)
+			)
+			(justify left)
+		)
+	)
+	(hierarchical_label "MCU_DAC_DIN"
+		(shape output)
+		(at 326.39 102.87 0)
+		(effects
+			(font
+				(size 1.27 1.27)
+			)
+			(justify left)
+		)
+	)
+	(hierarchical_label "ADC_VOLT_~{CS}"
+		(shape output)
+		(at 237.49 71.12 0)
+		(effects
+			(font
+				(size 1.27 1.27)
+			)
+			(justify left)
+		)
+	)
+	(hierarchical_label "MCU_ADC_CURR_~{CS}"
+		(shape output)
+		(at 189.23 93.98 180)
 		(effects
 			(font
@@
 		)
 	)
-	(hierarchical_label "MCU_DAC_DIN"
-		(shape output)
-		(at 326.39 105.41 180)
-		(effects
-			(font
-				(size 1.27 1.27)
-			)
-			(justify right)
-		)
-	)
-	(hierarchical_label "ADC_VOLT_~{CS}"
-		(shape output)
-		(at 237.49 71.12 0)
-		(effects
-			(font
-				(size 1.27 1.27)
-			)
-			(justify left)
-		)
-	)
-	(hierarchical_label "MCU_REL_RANGE_SEL"
-		(shape output)
-		(at 326.39 113.03 180)
-		(effects
-			(font
-				(size 1.27 1.27)
-			)
-			(justify right)
-		)
-	)
-	(hierarchical_label "MCU_ADC_CURR_~{CS}"
-		(shape output)
-		(at 189.23 93.98 180)
-		(effects
-			(font
-				(size 1.27 1.27)
-			)
-			(justify right)
-		)
-	)
 	(hierarchical_label "RMII_RXD0"
 		(shape bidirectional)
@@
 	(hierarchical_label "MCU_DAC_~{CS}"
 		(shape output)
-		(at 326.39 102.87 180)
-		(effects
-			(font
-				(size 1.27 1.27)
-			)
-			(justify right)
+		(at 326.39 100.33 0)
+		(effects
+			(font
+				(size 1.27 1.27)
+			)
+			(justify left)
 		)
 	)
 	(hierarchical_label "MCU_DAC_~{LDAC}"
 		(shape output)
-		(at 326.39 110.49 180)
-		(effects
-			(font
-				(size 1.27 1.27)
-			)
-			(justify right)
+		(at 326.39 107.95 0)
+		(effects
+			(font
+				(size 1.27 1.27)
+			)
+			(justify left)
 		)
 	)
@@
 			)
 		)
-		(property "Footprint" "ETH1CVOLT_A:NX5032GA"
+		(property "Footprint" "ETH1CVOLT:NX5032GA"
 			(at 147.32 81.28 0)
 			(hide yes)

Commit message: Development
Parts:
- renumbered JP8 to JP1
Changed lines of the file:
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@@
 		(dnp no)
 		(fields_autoplaced yes)
-		(property "Reference" "JP8"
+		(property "Reference" "JP1"
 			(at 269.24 267.9699 90)
 			(show_name no)
@@
 			(project "ETH1CVOLT"
 				(path "/8d3b546e-b30b-49b2-bc59-8e254df4c067/ea97f94c-dee1-4702-bb32-5cb010d15929/9ecb7694-9b5a-4e75-86d6-fbc3af4f394e"
-					(reference "JP8")
+					(reference "JP1")
 					(unit 1)
 				)

Commit message: Layout
Parts:
- removed C11: 1u/16V/X7R, Capacitor_SMD:C_0603_1608Metric_Pad1.08x0.95mm_HandSolder, symbol Device:C
- removed C7: 0.1u/100V/X7R, Capacitor_SMD:C_0603_1608Metric_Pad1.08x0.95mm_HandSolder, symbol Device:C
- removed R2: 0R/5%/100mW, Resistor_SMD:R_0603_1608Metric_Pad0.98x0.95mm_HandSolder, symbol Device:R
- renumbered C14 to C11, C15 to C13, C16 to C14, C13 to C7, R3 to R2, R4 to R3, R5 to R4
Connections:
- net EEPROM_nWP: now also U1.68 (PA9); no longer U1.91 (PB5)
- net GND: now also U1.94 (BOOT0)
- net I2C1_SCL: now also U1.67 (PA8); no longer U1.92 (PB6)
- net I2C1_SDA: now also U1.66 (PC9); no longer U1.93 (PB7)
- net MCU_ADC_SW1: now also U1.93 (PB7)
- net MCU_ADC_SW2: now also U1.95 (PB8)
- net MCU_ADC_SW3: now also U1.96 (PB9)
- net MCU_DAC_DIN: now also U1.80 (PC12)
- net MCU_DAC_SCLK: now also U1.78 (PC10)
- net MCU_DAC_~{CS}: now also U1.77 (PA15)
- net MCU_DAC_~{LDAC}: now also U1.81 (PD0)
- net MCU_DEF: now also U1.1 (PE2); no longer U1.98 (PE1)
- net MCU_REL_RESET: now also U1.97 (PE0)
- net MCU_REL_SET: now also U1.98 (PE1)
- net MCU_ADC_SCLK: now reaches U1.89 (PB3)
- net MCU_ADC_SDO: now reaches U1.90 (PB4)
- net ADC_VOLT_SCLK: no longer names the net of U1.29 (PA5)
- net ADC_VOLT_SDO: no longer names the net of U1.30 (PA6)
- net ADC_VOLT_~{CS} renamed MCU_ADC_~{CS}
- net MCU_ADC_CURR_SDI: no longer names the net of U1.5 (PE6)
- net MCU_ADC_CURR_SDO: no longer names the net of U1.4 (PE5)
- net MCU_ADC_CURR_~{CS}: no longer names the net of U1.3 (PE4)
- no-connect marks 63 -> 57
Other:
- moved on the sheet: C11, C13, C6, C7, C9, FB1, JP1, R2, Y1

Commit message: Layout and schematic
Other:
- title: (none) -> ETH1CVOLT

Commit message: Modifications
Connections:
- net I2C1_SCL renamed I2C3_SCL
- net I2C1_SDA renamed I2C3_SDA
Changed lines of the file:
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@@
 		)
 	)
-	(label "I2C1_SDA"
+	(label "I2C3_SDA"
 		(at 260.35 170.18 180)
 		(effects
@@
 		)
 	)
-	(label "I2C1_SDA"
+	(label "I2C3_SDA"
 		(at 320.04 151.13 180)
 		(effects
@@
 		)
 	)
-	(label "I2C1_SCL"
+	(label "I2C3_SCL"
 		(at 320.04 153.67 180)
 		(effects
@@
 		)
 	)
-	(label "I2C1_SCL"
+	(label "I2C3_SCL"
 		(at 260.35 81.28 180)
 		(effects

Commit message: HW design done
Parts:
- added R68, R69, R70, R73, R74, R75: 4k7/1%/100mW, Resistor_SMD:R_0603_1608Metric_Pad0.98x0.95mm_HandSolder, symbol Device:R
Connections:
- net +3.3V: now also R73.1, R74.1, R75.1
- net GND: now also R68.2, R69.2, R70.2
- net MCU_ADC_SW1: now also R70.1
- net MCU_ADC_SW2: now also R69.1
- net MCU_ADC_SW3: now also R68.1
- net MCU_ADC_~{CS}: now also R75.2
- net MCU_DAC_~{CS}: now also R74.2
- net MCU_DAC_~{LDAC}: now also R73.2
Other:
- note added: "EEPROM"
- note added: "MCU"
- note added: "PROGRAMMING INTERFACE"
- moved on the sheet: C10, C12, C14, C6, C8, C9, J1, R1, R3, R4, U1, U2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
