File: HARDWARE/ETH1CVOLT/Block_Diagram.kicad_sch (KiCad schematic)
At the start: 0 parts

Commit message: Development
Parts:
- added N1: BOX3-1455N-SV, symbol Mechanical:Housing
Other:
- sheet ADC ports: added MEAS_OUT; removed MEAS_R10V, MEAS_R20V, RANGE_SEL
- sheet ISO DIG ports: added none; removed MCU_RANGE_SEL, RANGE_SEL
- sheet MCU ports: added none; removed MCU_RANGE_SEL
- sheet OUTPUT ports: added MEAS_OUT; removed none
- sheet RANGE 10V ports: added none; removed MEAS_R10V
- sheet RANGE 20V ports: added none; removed MEAS_R20V
Changed lines of the file:
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@@
+	(wire
+		(pts
+			(xy 250.19 119.38) (xy 306.07 119.38)
+		)
+		(stroke
+			(width 0)
+			(type default)
+		)
+	)
 	(wire
 		(pts
@@
 	(wire
 		(pts
-			(xy 198.12 111.76) (xy 207.01 111.76)
-		)
-		(stroke
-			(width 0)
-			(type default)
-		)
-	)
-	(wire
-		(pts
-			(xy 250.19 107.95) (xy 259.08 107.95)
-		)
-		(stroke
-			(width 0)
-			(type default)
-		)
-	)
-	(wire
-		(pts
 			(xy 198.12 101.6) (xy 207.01 101.6)
 		)
@@
 	(wire
 		(pts
-			(xy 259.08 85.09) (xy 252.73 85.09)
-		)
-		(stroke
-			(width 0)
-			(type default)
-		)
-	)
-	(wire
-		(pts
-			(xy 146.05 111.76) (xy 154.94 111.76)
-		)
-		(stroke
-			(width 0)
-			(type default)
-		)
-	)
-	(wire
-		(pts
 			(xy 198.12 87.63) (xy 207.01 87.63)
 		)
@@
 	(wire
 		(pts
-			(xy 252.73 85.09) (xy 252.73 102.87)
-		)
-		(stroke
-			(width 0)
-			(type default)
-		)
-	)
-	(wire
-		(pts
 			(xy 93.98 88.9) (xy 102.87 88.9)
 		)
@@
 	(wire
 		(pts
-			(xy 252.73 102.87) (xy 250.19 102.87)
-		)
-		(stroke
-			(width 0)
-			(type default)
-		)
-	)
-	(wire
-		(pts
 			(xy 198.12 130.81) (xy 306.07 130.81)
 		)
@@
 			(width 0)
 			(type default)
+		)
+	)
+	(symbol
+		(lib_id "Mechanical:Housing")
+		(at 68.58 264.16 0)
+		(unit 1)
+		(body_style 1)
+		(exclude_from_sim no)
+		(in_bom yes)
+		(on_board no)
+		(in_pos_files yes)
+		(dnp no)
+		(fields_autoplaced yes)
+		(property "Reference" "N1"
+			(at 72.39 263.2074 0)
+			(show_name no)
+			(do_not_autoplace no)
+			(effects
+				(font
+					(size 1.27 1.27)
+				)
+				(justify left)
+			)
+		)
+		(property "Value" "BOX3-1455N-SV"
+			(at 72.39 265.7474 0)
+			(show_name no)
+			(do_not_autoplace no)
+			(effects
+				(font
+					(size 1.27 1.27)
+				)
+				(justify left)
+			)
+		)
+		(property "Footprint" ""
+			(at 69.85 262.89 0)
+			(hide yes)
+			(show_name no)
+			(do_not_autoplace no)
+			(effects
+				(font
+					(size 1.27 1.27)
+				)
+			)
+		)
+		(property "Datasheet" ""
+			(at 69.85 262.89 0)
+			(hide yes)
+			(show_name no)
+			(do_not_autoplace no)
+			(effects
+				(font
+					(size 1.27 1.27)
+				)
+			)
+		)
+		(property "Description" "Housing"
+			(at 68.58 264.16 0)
+			(hide yes)
+			(show_name no)
+			(do_not_autoplace no)
+			(effects
+				(font
+					(size 1.27 1.27)
+				)
+			)
+		)
+		(instances
+			(project "ETH1CVOLT"
+				(path "/8d3b546e-b30b-49b2-bc59-8e254df4c067/ea97f94c-dee1-4702-bb32-5cb010d15929"
+					(reference "N1")
+					(unit 1)
+				)
+			)
 		)
 	)
@@
 			)
 		)
-		(pin "MEAS_R20V" input
-			(at 250.19 107.95 0)
-			(effects
-				(font
-					(size 1.27 1.27)
-				)
-				(justify right)
-			)
-		)
 		(pin "ADC_SW3" input
 			(at 207.01 119.38 180)
@@
 			)
 		)
-		(pin "RANGE_SEL" input
-			(at 207.01 111.76 180)
-			(effects
-				(font
-					(size 1.27 1.27)
-				)
-				(justify left)
-			)
-		)
-		(pin "MEAS_R10V" input
-			(at 250.19 102.87 0)
+		(pin "MEAS_OUT" input
+			(at 250.19 119.38 0)
 			(effects
 				(font
@@
 			)
 		)
-		(pin "RANGE_SEL" output
-			(at 198.12 111.76 0)
-			(effects
-				(font
-					(size 1.27 1.27)
-				)
-				(justify right)
-			)
-		)
 		(pin "DAC_~{CS}" output
 			(at 198.12 80.01 0)
@@
 				)
 				(justify right)
-			)
-		)
-		(pin "MCU_RANGE_SEL" input
-			(at 154.94 111.76 180)
-			(effects
-				(font
-					(size 1.27 1.27)
-				)
-				(justify left)
 			)
 		)
@@
 			)
 		)
-		(pin "MEAS_R20V" output
-			(at 259.08 107.95 180)
-			(effects
-				(font
-					(size 1.27 1.27)
-				)
-				(justify left)
-			)
-		)
 		(instances
 			(project "ETH1CVOLT"
@@
 			)
 		)
+		(pin "MEAS_OUT" output
+			(at 306.07 119.38 180)
+			(effects
+				(font
+					(size 1.27 1.27)
+				)
+				(justify left)
+			)
+		)
 		(instances
 			(project "ETH1CVOLT"
@@
 			)
 		)
-		(pin "MCU_RANGE_SEL" output
-			(at 146.05 111.76 0)
-			(effects
-				(font
-					(size 1.27 1.27)
-				)
-				(justify right)
-			)
-		)
 		(pin "MCU_DAC_SCLK" output
 			(at 146.05 85.09 0)
@@
 	)
 	(sheet
-		(at 307.34 153.67)
-		(size 36.83 38.1)
+		(at 306.07 153.67)
+		(size 38.1 38.1)
 		(exclude_from_sim no)
 		(in_bom yes)
@@
 		)
 		(property "Sheetname" "VOLTAGE REFERENCE"
-			(at 307.34 152.9584 0)
+			(at 306.07 152.9584 0)
 			(show_name no)
 			(do_not_autoplace no)
@@
 		)
 		(property "Sheetfile" "Voltage_Reference.kicad_sch"
-			(at 307.34 192.3546 0)
+			(at 306.07 192.3546 0)
 			(show_name no)
 			(do_not_autoplace no)
@@
 			)
 		)
-		(pin "MEAS_R10V" output
-			(at 259.08 85.09 180)
-			(effects
-				(font
-					(size 1.27 1.27)
-				)
-				(justify left)
-			)
-		)

Commit message: Development
Other:
- sheet ISO DIG ports: added MCU_REL_RESET, MCU_REL_SET, REL_RESET, REL_SET; removed MCU_REL_RANGE_SEL, REL_RANGE_SEL
- sheet MCU ports: added MCU_REL_RESET, MCU_REL_SET; removed MCU_REL_RANGE_SEL
- sheet OUTPUT ports: added REL_RESET, REL_SET; removed REL_RANGE_SEL
Changed lines of the file:
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@@
+	(wire
+		(pts
+			(xy 198.12 128.27) (xy 306.07 128.27)
+		)
+		(stroke
+			(width 0)
+			(type default)
+		)
+	)
 	(wire
 		(pts
@@
 		(pts
 			(xy 146.05 80.01) (xy 154.94 80.01)
+		)
+		(stroke
+			(width 0)
+			(type default)
+		)
+	)
+	(wire
+		(pts
+			(xy 146.05 128.27) (xy 154.94 128.27)
 		)
 		(stroke
@@
 			)
 		)
-		(pin "REL_RANGE_SEL" output
+		(pin "REL_SET" output
 			(at 198.12 130.81 0)
 			(effects
@@
 			)
 		)
-		(pin "MCU_REL_RANGE_SEL" input
+		(pin "MCU_REL_SET" input
 			(at 154.94 130.81 180)
 			(effects
@@
 		(pin "MCU_ADC_VOLT_SCLK" input
 			(at 154.94 101.6 180)
+			(effects
+				(font
+					(size 1.27 1.27)
+				)
+				(justify left)
+			)
+		)
+		(pin "REL_RESET" output
+			(at 198.12 128.27 0)
+			(effects
+				(font
+					(size 1.27 1.27)
+				)
+				(justify right)
+			)
+		)
+		(pin "MCU_REL_RESET" input
+			(at 154.94 128.27 180)
 			(effects
 				(font
@@
 			)
 		)
-		(pin "REL_RANGE_SEL" input
-			(at 306.07 130.81 180)
-			(effects
-				(font
-					(size 1.27 1.27)
-				)
-				(justify left)
-			)
-		)
 		(pin "R20V_SIG" input
 			(at 306.07 102.87 180)
@@
 		(pin "MEAS_OUT" output
 			(at 306.07 119.38 180)
+			(effects
+				(font
+					(size 1.27 1.27)
+				)
+				(justify left)
+			)
+		)
+		(pin "REL_SET" input
+			(at 306.07 130.81 180)
+			(effects
+				(font
+					(size 1.27 1.27)
+				)
+				(justify left)
+			)
+		)
+		(pin "REL_RESET" input
+			(at 306.07 128.27 180)
 			(effects
 				(font
@@
 			)
 		)
-		(pin "MCU_REL_RANGE_SEL" output
-			(at 146.05 130.81 0)
-			(effects
-				(font
-					(size 1.27 1.27)
-				)
-				(justify right)
-			)
-		)
 		(pin "MCU_DAC_~{CS}" output
 			(at 146.05 80.01 0)
@@
 			(effects
 				(font
+					(size 1.27 1.27)
+				)
+				(justify right)
+			)
+		)
+		(pin "MCU_REL_SET" output
+			(at 146.05 130.81 0)
+			(effects
+				(font
+					(size 1.27 1.27)
+				)
+				(justify right)
+			)
+		)
+		(pin "MCU_REL_RESET" output
+			(at 146.05 128.27 0)
+			(effects
+				(font

Commit message: Development
Parts:
- N1: footprint (none) -> ETH1CVOLT:BOX3-1455N
Changed lines of the file:
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@@
 			)
 		)
-		(property "Footprint" ""
+		(property "Footprint" "ETH1CVOLT:BOX3-1455N"
 			(at 69.85 262.89 0)
 			(hide yes)
@@
 			)
 		)
-		(property "Datasheet" ""
+		(property "Datasheet" "https://www.busboard.com/documents/datasheets/BPS-DAT-(BOX3-1455N)-Datasheet.pdf"
 			(at 69.85 262.89 0)
 			(hide yes)

Commit message: Layout
Parts:
- added FID1, FID2, FID3, FID4, FID5, FID6: Fiducial, Fiducial:Fiducial_1.5mm_Mask3mm, symbol Mechanical:Fiducial
Other:
- sheet ADC ports: added ADC_SCLK, ADC_SDO, ADC_~{CS}; removed ADC_VOLT_SCLK, ADC_VOLT_SDO, ADC_VOLT_~{CS}
- sheet ISO DIG ports: added ADC_SCLK, ADC_SDO, ADC_~{CS}, MCU_ADC_SCLK, MCU_ADC_SDO, MCU_ADC_~{CS}; removed ADC_VOLT_SCLK, ADC_VOLT_SDO, ADC_VOLT_~{CS}, MCU_ADC_VOLT_SCLK, MCU_ADC_VOLT_SDO, MCU_ADC_VOLT_~{CS}
- sheet MCU ports: added MCU_ADC_SCLK, MCU_ADC_SDO, MCU_ADC_~{CS}; removed MCU_ADC_VOLT_SCLK, MCU_ADC_VOLT_SDO, MCU_ADC_VOLT_~{CS}

Commit message: Layout and schematic
Other:
- title: (none) -> ETH1CVOLT
Changed lines of the file:
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@@
 	(generator_version "10.0")
 	(paper "A3")
+	(title_block
+		(title "ETH1CVOLT")
+		(rev "01")
+	)
 	(junction
 		(at 256.54 80.01)
@@
 			)
 		)
+		(property "Sim.Type" ""
+			(at 152.4 264.16 0)
+			(hide yes)
+			(show_name no)
+			(do_not_autoplace no)
+			(effects
+				(font
+					(size 1.27 1.27)
+				)
+			)
+		)
+		(property "KLC_S4.5" ""
+			(at 152.4 264.16 0)
+			(hide yes)
+			(show_name no)
+			(do_not_autoplace no)
+			(effects
+				(font
+					(size 1.27 1.27)
+				)
+			)
+		)
 		(instances
 			(project "ETH1CVOLT"
@@
 			)
 		)
+		(property "Sim.Type" ""
+			(at 111.76 264.16 0)
+			(hide yes)
+			(show_name no)
+			(do_not_autoplace no)
+			(effects
+				(font
+					(size 1.27 1.27)
+				)
+			)
+		)
+		(property "KLC_S4.5" ""
+			(at 111.76 264.16 0)
+			(hide yes)
+			(show_name no)
+			(do_not_autoplace no)
+			(effects
+				(font
+					(size 1.27 1.27)
+				)
+			)
+		)
 		(instances
 			(project "ETH1CVOLT"
@@
 			)
 		)
+		(property "Sim.Type" ""
+			(at 97.79 264.16 0)
+			(hide yes)
+			(show_name no)
+			(do_not_autoplace no)
+			(effects
+				(font
+					(size 1.27 1.27)
+				)
+			)
+		)
+		(property "KLC_S4.5" ""
+			(at 97.79 264.16 0)
+			(hide yes)
+			(show_name no)
+			(do_not_autoplace no)
+			(effects
+				(font
+					(size 1.27 1.27)
+				)
+			)
+		)
 		(instances
 			(project "ETH1CVOLT"
@@
 			)
 		)
+		(property "Sim.Type" ""
+			(at 124.46 264.16 0)
+			(hide yes)
+			(show_name no)
+			(do_not_autoplace no)
+			(effects
+				(font
+					(size 1.27 1.27)
+				)
+			)
+		)
+		(property "KLC_S4.5" ""
+			(at 124.46 264.16 0)
+			(hide yes)
+			(show_name no)
+			(do_not_autoplace no)
+			(effects
+				(font
+					(size 1.27 1.27)
+				)
+			)
+		)
 		(instances
 			(project "ETH1CVOLT"
@@
 			)
 		)
+		(property "Sim.Type" ""
+			(at 165.1 264.16 0)
+			(hide yes)
+			(show_name no)
+			(do_not_autoplace no)
+			(effects
+				(font
+					(size 1.27 1.27)
+				)
+			)
+		)
+		(property "KLC_S4.5" ""
+			(at 165.1 264.16 0)
+			(hide yes)
+			(show_name no)
+			(do_not_autoplace no)
+			(effects
+				(font
+					(size 1.27 1.27)
+				)
+			)
+		)
 		(instances
 			(project "ETH1CVOLT"
@@
 			)
 		)
+		(property "Sim.Type" ""
+			(at 138.43 264.16 0)
+			(hide yes)
+			(show_name no)
+			(do_not_autoplace no)
+			(effects
+				(font
+					(size 1.27 1.27)
+				)
+			)
+		)
+		(property "KLC_S4.5" ""
+			(at 138.43 264.16 0)
+			(hide yes)
+			(show_name no)
+			(do_not_autoplace no)
+			(effects
+				(font
+					(size 1.27 1.27)
+				)
+			)
+		)
 		(instances
 			(project "ETH1CVOLT"
@@
 			(at 68.58 264.16 0)
 			(hide yes)
+			(show_name no)
+			(do_not_autoplace no)
+			(effects
+				(font
+					(size 1.27 1.27)
+				)
+			)
+		)
+		(property "Sim.Type" ""
+			(at 68.58 264.16 0)
+			(hide yes)
+			(show_name no)
+			(do_not_autoplace no)
+			(effects
+				(font
+					(size 1.27 1.27)
+				)
+			)
+		)
+		(property "KLC_S4.5" ""
+			(at 68.58 264.16 0)
+			(hide yes)

Commit message: Production data, cleanup.
Parts:
- added H1, H2, H3, H4: MountingHole, MountingHole:MountingHole_3.2mm_M3, symbol Mechanical:MountingHole
